File: Hardware/power.sch (KiCad schematic (older format))
At the start: 87 parts

Commit message: pcb: import footprints; finishing schematics
Parts:
- removed R?: 365K/1%, Resistor_SMD:R_0603_1608Metric, symbol Device:R
- added C43, C44: 2.2uF, Capacitor_SMD:C_0402_1005Metric, symbol Device:C
- added C45, C46: 10nF, Capacitor_SMD:C_0402_1005Metric, symbol Device:C
- added C47, C48: 10uF, Capacitor_SMD:C_0402_1005Metric, symbol Device:C
- added R25, R?: 49.9K/1%, Resistor_SMD:R_0402_1005Metric, symbol Device:R
- added R26: 115K/1%, Resistor_SMD:R_0402_1005Metric, symbol Device:R
- added R27: 464K/1%, Resistor_SMD:R_0402_1005Metric, symbol Device:R
- added R28: 243K/1%, Resistor_SMD:R_0402_1005Metric, symbol Device:R
- added R?: 316K/1%, Resistor_SMD:R_0402_1005Metric, symbol Device:R
- added R?: 20K/1%, Resistor_SMD:R_0402_1005Metric, symbol Device:R
- added U10, U11: LT1964-BYP, Package_TO_SOT_SMD:TSOT-23-5, symbol Regulator_Linear:LT1964-BYP
- D1: renamed from D?; footprint (none) -> LED_SMD:LED_0603_1608Metric
- R1: renamed from R?; value 324K -> 316K/1%; footprint Resistor_SMD:R_0603_1608Metric -> Resistor_SMD:R_0402_1005Metric
- R10: renamed from R?; value 487K/1% -> 464K/1%; footprint Resistor_SMD:R_0603_1608Metric -> Resistor_SMD:R_0402_1005Metric
- R11, R13, R14, R19, R20, R6, R8, R9: renamed from R?; footprint Resistor_SMD:R_0603_1608Metric -> Resistor_SMD:R_0402_1005Metric
- R15: renamed from R?; value 50K -> 49.9K/1%; footprint (none) -> Resistor_SMD:R_0402_1005Metric
- R16: renamed from R?; value 11K/1% -> 10K/1%; footprint (none) -> Resistor_SMD:R_0402_1005Metric
- R17: renamed from R?; value 23.7K/1% -> 49.9K/1%; footprint Resistor_SMD:R_0603_1608Metric -> Resistor_SMD:R_0402_1005Metric
- R18, R24: renamed from R?; value 150K/1% -> 200K/1%; footprint Resistor_SMD:R_0603_1608Metric -> Resistor_SMD:R_0402_1005Metric
- R2: value 324K -> 316K/1%; footprint Resistor_SMD:R_0603_1608Metric -> Resistor_SMD:R_0402_1005Metric
- R21: renamed from R?; value 127K/1% -> 115K/1%; footprint Resistor_SMD:R_0603_1608Metric -> Resistor_SMD:R_0402_1005Metric
- R22: renamed from R?; value 11K/1% -> 10K/1%; footprint Resistor_SMD:R_0603_1608Metric -> Resistor_SMD:R_0402_1005Metric
- R23: renamed from R?; value 68.1K/1% -> 150K/1%; footprint Resistor_SMD:R_0603_1608Metric -> Resistor_SMD:R_0402_1005Metric
- R3: value 105K -> 100K/1%; footprint Resistor_SMD:R_0603_1608Metric -> Resistor_SMD:R_0402_1005Metric
- R5: renamed from R?; value 75K -> 60.4K/1%; footprint Resistor_SMD:R_0603_1608Metric -> Resistor_SMD:R_0402_1005Metric
- RV1: renamed from RV?; footprint (none) -> Resistor_SMD:R_0402_1005Metric
- gave numbers to parts that had none: 52
Connections:
- net +19V: now also U7.7 (~SHDN1), U7.9 (~SHDN2)
- net -8V: now also C43.1, C44.1, U10.2 (VIN), U11.2 (VIN)
- net -9V: now also R?.1
- net GND: now also C43.2, C44.2, C47.2, C48.2, R25.1, R27.1, U10.1 (GND), U11.1 (GND)
- net at C25.2, U4.6 (FBN): now also R?.2; no longer R10.2
- net at R1.1, R5.2, U5.3 (~SHDN)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: now also U8.7 (~SHDN1), U8.9 (~SHDN2)
- net at C27.2, U6.6 (FBN): now also R?.2
- net PMIC_ON_REQ renamed ON
- new net: R10.2, R?.1
- new net: C45.1, U10.3 (BYP)
- new net: R25.2, R26.1, U10.4 (ADJ)
- new net: C46.1, U11.3 (BYP)
- new net: R27.2, R28.1, U11.4 (ADJ)
- new net: R?.1, R?.2
- new net -3V5: C46.2, C48.1, R28.2, U11.5 (VOUT)
- new net -4V: C45.2, C47.1, R26.2, U10.5 (VOUT)
Other:
- moved on the sheet: BT1, C2, C3, C33, C38, C6, C7, C8, C9, D1, L1, L11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
