File: Hardware/sdram.sch (KiCad schematic (older format))
At the start: 20 parts, among them U200 MT48LC32M16A2B4, U201 MT48LC32M16A2B4

Commit message: pcb: import footprints; finishing schematics
Parts:
- added C317: 22uF, Capacitor_SMD:C_0805_2012Metric, symbol Device:C
- added L301: 120R, Inductor_SMD:L_0603_1608Metric, symbol Device:L
- C300: renamed from C201; footprint (none) -> Capacitor_SMD:C_0402_1005Metric
- C301: renamed from C202; footprint (none) -> Capacitor_SMD:C_0402_1005Metric
- C302: renamed from C203; footprint (none) -> Capacitor_SMD:C_0402_1005Metric
- C303: renamed from C204; footprint (none) -> Capacitor_SMD:C_0402_1005Metric
- C304: renamed from C205; footprint (none) -> Capacitor_SMD:C_0402_1005Metric
- C305: renamed from C206; footprint (none) -> Capacitor_SMD:C_0402_1005Metric
- C306: renamed from C207; footprint (none) -> Capacitor_SMD:C_0402_1005Metric
- C307: renamed from C215; footprint (none) -> Capacitor_SMD:C_0805_2012Metric
- C308: renamed from C208; footprint (none) -> Capacitor_SMD:C_0402_1005Metric
- C309: renamed from C209; footprint (none) -> Capacitor_SMD:C_0402_1005Metric
- C310: renamed from C210; footprint (none) -> Capacitor_SMD:C_0402_1005Metric
- C311: renamed from C211; footprint (none) -> Capacitor_SMD:C_0402_1005Metric
- C312: renamed from C212; footprint (none) -> Capacitor_SMD:C_0402_1005Metric
- C313: renamed from C213; footprint (none) -> Capacitor_SMD:C_0402_1005Metric
- C314: renamed from C214; footprint (none) -> Capacitor_SMD:C_0402_1005Metric
- C315: renamed from C216; footprint (none) -> Capacitor_SMD:C_0805_2012Metric
- C316: renamed from C217; footprint (none) -> Capacitor_SMD:C_0805_2012Metric
- L300: renamed from L200; footprint (none) -> Inductor_SMD:L_0603_1608Metric
- renumbered U200 to U300, U201 to U301
Connections:
- net +3V3: now also L301.2
- net GND: now also C317.2
- net at C300.1, C301.1, C302.1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: no longer C308.1, C309.1, C310.1, C311.1, C312.1, C313.1, C314.1, C315.1, U301.A7 (VDDQ), U301.A9 (VDD), U301.B3 (VDDQ), U301.C7 (VDDQ), U301.D3 (VDDQ), U301.E7 (VDD), U301.J9 (VDD)
- new net: C308.1, C309.1, C310.1, C311.1, C312.1, C313.1, C314.1, C315.1, C317.1, L301.1, U301.A7 (VDDQ), U301.A9 (VDD), U301.B3 (VDDQ), U301.C7 (VDDQ), U301.D3 (VDDQ), U301.E7 (VDD), U301.J9 (VDD)
Other:
- moved on the sheet: C300, C301, C302, C303, C304, C305, C306, C307, C308, C309, C310, C311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
