File: Hardware/usb.sch (KiCad schematic (older format))
At the start: 7 parts, among them J700 USB_B_Micro, U700 USBLC6-2SC6

Commit message: pcb: import footprints; finishing schematics
Parts:
- L500: renamed from L?; value L_Coupled_Small_1243 -> 90R; footprint (none) -> Inductor_SMD:L_CommonModeChoke_Coilcraft_0805USB
- renumbered C700 to C500, C701 to C501, D700 to D500, J700 to J500, R701 to R501, U700 to U500
Changed lines of the file:
@@
 $EndDescr
 $Comp
-L Connector:USB_B_Micro J700
+L Connector:USB_B_Micro J500
 U 1 1 5C995A78
 P 7600 4300
-F 0 "J700" H 7655 4767 50  0000 C CNN
+F 0 "J500" H 7655 4767 50  0000 C CNN
 F 1 "USB_B_Micro" H 7655 4676 50  0000 C CNN
 F 2 "Connector_USB:USB_Micro-B_Amphenol_10103594-0001LF_Horizontal" H 7750 4250 50  0001 C CNN
@@
 $EndComp
 $Comp
-L Power_Protection:USBLC6-2SC6 U700
+L Power_Protection:USBLC6-2SC6 U500
 U 1 1 5C995C17
 P 6500 3300
-F 0 "U700" H 6500 3978 50  0000 C CNN
+F 0 "U500" H 6500 3978 50  0000 C CNN
 F 1 "USBLC6-2SC6" H 6500 3887 50  0000 C CNN
 F 2 "Package_TO_SOT_SMD:SOT-23-6" H 5750 3700 50  0001 C CNN
@@
 $EndComp
 $Comp
-L Device:D_TVS D700
+L Device:D_TVS D500
 U 1 1 5C995E54
 P 6700 4850
-F 0 "D700" V 6654 4929 50  0000 L CNN
+F 0 "D500" V 6654 4929 50  0000 L CNN
 F 1 "B72590D0050H160" V 6900 4850 50  0000 L CNN
 F 2 "Diode_SMD:D_0402_1005Metric" H 6700 4850 50  0001 C CNN
@@
 $EndComp
 $Comp
-L Device:R R701
+L Device:R R501
 U 1 1 5C995E96
 P 7700 5050
-F 0 "R701" H 7770 5096 50  0000 L CNN
+F 0 "R501" H 7770 5096 50  0000 L CNN
 F 1 "0" H 7770 5005 50  0000 L CNN
 F 2 "Resistor_SMD:R_0805_2012Metric" V 7630 5050 50  0001 C CNN
@@
 $EndComp
 $Comp
-L Device:C C701
+L Device:C C501
 U 1 1 5C995EF6
 P 7400 5050
-F 0 "C701" H 7515 5096 50  0000 L CNN
+F 0 "C501" H 7515 5096 50  0000 L CNN
 F 1 "100nF" H 7515 5005 50  0000 L CNN
 F 2 "Capacitor_SMD:C_0805_2012Metric" H 7438 4900 50  0001 C CNN
@@
 $EndComp
 $Comp
-L Device:C C700
+L Device:C C500
 U 1 1 5C9960AD
 P 5300 3350
-F 0 "C700" H 5415 3396 50  0000 L CNN
+F 0 "C500" H 5415 3396 50  0000 L CNN
 F 1 "10uF" H 5415 3305 50  0000 L CNN
 F 2 "Capacitor_SMD:C_0603_1608Metric" H 5338 3200 50  0001 C CNN
@@
 	5800 3200 5800 4100
 $Comp
-L Device:L_Coupled_Small_1243 L?
+L Device:L_Coupled_Small_1243 L500
 U 1 1 5F80E98E
 P 5600 4350
-F 0 "L?" H 5600 4581 50  0000 C CNN
-F 1 "L_Coupled_Small_1243" H 5600 4490 50  0000 C CNN
-F 2 "" H 5600 4350 50  0001 C CNN
+F 0 "L500" H 5600 4581 50  0000 C CNN
+F 1 "90R" H 5600 4490 50  0000 C CNN
+F 2 "Inductor_SMD:L_CommonModeChoke_Coilcraft_0805USB" H 5600 4350 50  0001 C CNN
 F 3 "~" H 5600 4350 50  0001 C CNN
 	1    5600 4350
