File: Hardware/vsub.sch (KiCad schematic (older format))
At the start: 0 parts

Commit message: pcb: working on h-driver schematics
Parts:
- added C? (x3): 1uF/25V, symbol Device:C
- added C? (x2): 10nF, symbol Device:C
- added C?: 4.7uF/25V, symbol Device:C
- added C? (x3): 100nF/25V, symbol Device:C
- added C? (x2): 100nF, symbol Device:C
- added D? (x2): HSMS-2805, symbol Device:D_Schottky
- added Q? (x2): BC847BPN, Package_TO_SOT_SMD:SOT-363_SC-70-6, symbol Transistor_BJT:BC847BPN
- added R? (x2): 100K, symbol Device:R
- added R?: 15K/1%, symbol Device:R
- added R?: 196K, symbol Device:R
- added R?: 9.09K, symbol Device:R
- added R?: 63.4K, symbol Device:R
- added R? (x3): 10K/1%, symbol Device:R
- added U?: LT3050MSE, Package_SO:MSOP-12-1EP_3x4mm_P0.65mm_EP1.65x2.85mm_ThermalVias, symbol Sitina:LT3050MSE
- added U?: NC7SZ08, Package_TO_SOT_SMD:SOT-23-5, symbol Sitina:NC7SZ08
Connections:
- new net: C?.2, U?.1 (REF/BYP)
- new net: C?.2, R?.1, U?.11 (Imax)
- new net: R?.2, U?.1, U?.3 (~FAULT)
- new net: R?.1, R?.2, R?.2, U?.9 (ADJ)
- new net: C?.2, C?.2, U?.4
- new net: C?.1, Q?.5 (B2), R?.2
- new net: C?.1, D?.1 (K), Q?.2 (B1), R?.1
- new net: C?.2, Q?.3 (C2), Q?.6 (C1)
- new net +16V: C?.2, C?.2, Q?.4 (E2), R?.1, U?.5 (IN), U?.6 (IN)
- new net +3V3: R?.1, U?.5
- new net -12V: C?.1, D?.2 (A), Q?.1 (E1)
- new net GND: C?.1, C?.1, C?.1, C?.1, C?.1, C?.1, C?.2, R?.2, R?.2, R?.2, R?.2, R?.2, U?.10 (GND), U?.12 (Imon), U?.13 (EP), U?.3
- new net STROBE_AB: U?.2
- new net SUBCK: C?.2
- new net VAB: C?.2, C?.2, D?.2 (A), R?.1, U?.7 (OUT), U?.8 (OUT)
- new net VAB_ADJ: R?.1
- new net VAB_EN: R?.1, U?.4 (~SHDN)
- new net VSUB: C?.1, C?.1, D?.1 (K), R?.1
- no-connect marks 0 -> 1

Commit message: pcb: working on h-driver and v-driver
Parts:
- added R?: 0, symbol Device:R
Connections:
- net -12V: now also R?.2; no longer Q?.1 (E1)
- new net: Q?.1 (E1), R?.1
Other:
- note added: "TODO: Pulse voltage of 28V might not be sufficient over the whole VAB range. Optimal value should be 31V."
Changed lines of the file:
@@
 $Descr A4 11693 8268
 encoding utf-8
-Sheet 5 7
+Sheet 5 8
 Title ""
 Date ""
@@
 P 6300 5750
 F 0 "D?" V 6254 5830 50  0000 L CNN
-F 1 "HSMS-2805" V 6345 5830 50  0000 L CNN
+F 1 "HSMS-2805" V 6500 5500 50  0000 L CNN
 F 2 "" H 6300 5750 50  0001 C CNN
 F 3 "~" H 6300 5750 50  0001 C CNN
@@
 Wire Wire Line
 	6600 5900 6600 6000
-Wire Wire Line
-	6600 5600 6600 5900
 Connection ~ 6600 5900
 Wire Wire Line
@@
 Text HLabel 8100 5100 2    50   Output ~ 0
 VSUB
+$Comp
+L Device:R R?
+U 1 1 5F507730
+P 6600 5750
+F 0 "R?" H 6670 5796 50  0000 L CNN
+F 1 "0" H 6670 5705 50  0000 L CNN
+F 2 "" V 6530 5750 50  0001 C CNN
+F 3 "~" H 6600 5750 50  0001 C CNN
+	1    6600 5750
+	1    0    0    -1
+$EndComp
+Text Notes 4250 6450 0    50   ~ 0
+TODO: Pulse voltage of 28V might not be sufficient over the whole VAB range. Optimal value should be 31V.
 $EndSCHEMATC

Commit message: pcb: working on power supply
Parts:
- removed R?: 100K, symbol Device:R
- removed R?: 196K, symbol Device:R
- removed R?: 9.09K, symbol Device:R
- removed R?: 63.4K, symbol Device:R
Connections:
- net VAB_EN is gone; now on net +19V: U?.4 (~SHDN)
- net +16V renamed +19V
Other:
- note added: "Pulse Voltage: 31V"
- note added: "VAB range: 6.2V - 17.4V (Target range: 8V - 17V)"
- note added: "Voltage range: 39V - 48V"
- note removed: "TODO: Pulse voltage of 28V might not be sufficient over the whole VAB range. Optimal value should be 31V."
Changed lines of the file:
@@
 $Descr A4 11693 8268
 encoding utf-8
-Sheet 4 9
-Title ""
+Sheet 4 14
+Title "Sitina Ne"
 Date ""
-Rev ""
-Comp ""
+Rev "R0P2"
+Comp "ZephRay"
 Comment1 ""
 Comment2 ""
@@
 	-1   0    0    1
 $EndComp
-$Comp
-L Device:R R?
-U 1 1 5F4F080C
-P 3600 2450
-F 0 "R?" H 3670 2496 50  0000 L CNN
-F 1 "100K" H 3670 2405 50  0000 L CNN
-F 2 "" V 3530 2450 50  0001 C CNN
-F 3 "~" H 3600 2450 50  0001 C CNN
-	1    3600 2450
-	1    0    0    -1
-$EndComp
-Text HLabel 3300 1400 0    50   Input ~ 0
-VAB_ADJ
-Text HLabel 3300 2200 0    50   Input ~ 0
-VAB_EN
-$Comp
-L Sitina:+16V #PWR?
-U 1 1 5F4F26C2
-P 4000 1900
-F 0 "#PWR?" H 4000 1750 50  0001 C CNN
-F 1 "+16V" H 4015 2073 50  0000 C CNN
-F 2 "" H 4000 1900 50  0001 C CNN
-F 3 "" H 4000 1900 50  0001 C CNN
-	1    4000 1900
-	1    0    0    -1
-$EndComp
 Wire Wire Line
 	5200 2000 5100 2000
@@
 	1    0    0    -1
 $EndComp
-$Comp
-L power:GND #PWR?
-U 1 1 5F4F3A88
-P 3600 2600
-F 0 "#PWR?" H 3600 2350 50  0001 C CNN
-F 1 "GND" H 3605 2427 50  0000 C CNN
-F 2 "" H 3600 2600 50  0001 C CNN
-F 3 "" H 3600 2600 50  0001 C CNN
-	1    3600 2600
-	1    0    0    -1
-$EndComp
-Wire Wire Line
-	3600 2300 3600 2200
-Wire Wire Line
-	3300 2200 3600 2200
 $Comp
 L Device:C C?
@@
 	1    0    0    -1
 $EndComp
-Connection ~ 3600 2200
-Wire Wire Line
-	3600 2200 5200 2200
 Wire Wire Line
 	4400 2600 4800 2600
@@
 Wire Wire Line
 	4000 1900 5100 1900
-Connection ~ 4000 1900
-$Comp
-L Device:R R?
-U 1 1 5F4F925A
-P 6600 2150
-F 0 "R?" H 6670 2196 50  0000 L CNN
-F 1 "196K" H 6670 2105 50  0000 L CNN
-F 2 "" V 6530 2150 50  0001 C CNN
-F 3 "~" H 6600 2150 50  0001 C CNN
-	1    6600 2150
-	1    0    0    -1
-$EndComp
-$Comp
-L Device:R R?
-U 1 1 5F4FA025
-P 6600 2650
-F 0 "R?" H 6670 2696 50  0000 L CNN
-F 1 "9.09K" H 6670 2605 50  0000 L CNN
-F 2 "" V 6530 2650 50  0001 C CNN
-F 3 "~" H 6600 2650 50  0001 C CNN
-	1    6600 2650
-	1    0    0    -1
-$EndComp
-$Comp
-L power:GND #PWR?
-U 1 1 5F4FA02B
-P 6600 2800
-F 0 "#PWR?" H 6600 2550 50  0001 C CNN
-F 1 "GND" H 6605 2627 50  0000 C CNN
-F 2 "" H 6600 2800 50  0001 C CNN
-F 3 "" H 6600 2800 50  0001 C CNN
-	1    6600 2800
-	1    0    0    -1
-$EndComp
 $Comp
 L Device:C C?
@@
 $EndComp
 Wire Wire Line
-	6600 2400 6600 2500
-Wire Wire Line
-	6600 2300 6600 2400
-Connection ~ 6600 2400
-Wire Wire Line
 	6200 1900 6300 1900
 Wire Wire Line
@@
 	6300 2000 6300 1900
 Connection ~ 6300 1900
-Wire Wire Line
-	6600 2000 6600 1900
-Wire Wire Line
-	6300 1900 6600 1900
-Wire Wire Line
-	6200 2600 6500 2600
-Wire Wire Line
-	6500 2600 6500 3200
 $Comp
 L power:GND #PWR?
 U 1 1 5F4FCD6D
-P 6500 3200
-F 0 "#PWR?" H 6500 2950 50  0001 C CNN
-F 1 "GND" H 6505 3027 50  0000 C CNN
-F 2 "" H 6500 3200 50  0001 C CNN
-F 3 "" H 6500 3200 50  0001 C CNN
-	1    6500 3200
+P 6400 3200
+F 0 "#PWR?" H 6400 2950 50  0001 C CNN
+F 1 "GND" H 6405 3027 50  0000 C CNN
+F 2 "" H 6400 3200 50  0001 C CNN
+F 3 "" H 6400 3200 50  0001 C CNN
+	1    6400 3200
 	1    0    0    -1
 $EndComp
@@
 	1    0    0    -1
 $EndComp
-$Comp
-L Device:R R?
-U 1 1 5F4FF519
-P 6950 2400
-F 0 "R?" V 6743 2400 50  0000 C CNN
-F 1 "63.4K" V 6834 2400 50  0000 C CNN
-F 2 "" V 6880 2400 50  0001 C CNN
-F 3 "~" H 6950 2400 50  0001 C CNN
-	1    6950 2400
-	0    1    1    0
-$EndComp
-Wire Wire Line
-	6800 2400 6600 2400
-Wire Wire Line
-	7100 2400 7200 2400
 $Comp
 L Device:C C?
@@
 Wire Wire Line
 	5900 4800 6300 4800
-$Comp
-L Sitina:+16V #PWR?
-U 1 1 5F52A4FF
-P 5900 4300
-F 0 "#PWR?" H 5900 4150 50  0001 C CNN
-F 1 "+16V" H 5915 4473 50  0000 C CNN
-F 2 "" H 5900 4300 50  0001 C CNN
-F 3 "" H 5900 4300 50  0001 C CNN
-	1    5900 4300
-	1    0    0    -1
-$EndComp
 Wire Wire Line
 	5900 4400 5900 4300
 Wire Wire Line
-	5900 4300 6600 4300
-Wire Wire Line
 	6600 4300 6600 4600
-Connection ~ 5900 4300
 $Comp
 L Device:C C?
@@
 Wire Wire Line
 	6600 4300 7000 4300
-Connection ~ 6600 4300
 $Comp
 L power:GND #PWR?
@@
 Wire Wire Line
 	6200 2800 6200 2900
-Wire Wire Line
-	6200 2400 6600 2400
-Connection ~ 6600 1900
-Wire Wire Line
-	7200 2400 7200 1400
-Wire Wire Line
-	7200 1400 3300 1400
 Connection ~ 8200 1900
 Wire Wire Line
 	8200 1900 8800 1900
-Wire Wire Line
-	6600 1900 7800 1900
 Wire Wire Line
 	7800 4600 7800 1900
@@
 	1    0    0    -1
 $EndComp
-Text Notes 4250 6450 0    50   ~ 0
-TODO: Pulse voltage of 28V might not be sufficient over the whole VAB range. Optimal value should be 31V.
+Wire Wire Line
+	6600 4300 5900 4300
+Connection ~ 6600 4300
+Wire Wire Line
+	5200 2200 5100 2200
+Wire Wire Line
+	5100 2200 5100 2000
+Connection ~ 5100 2000
+Wire Wire Line
+	6200 2600 6300 2600
+Wire Wire Line
+	6300 2600 6300 3200
+Wire Wire Line
+	6300 3200 6400 3200
+Text Notes 6350 1800 0    50   ~ 0
+VAB range: 6.2V - 17.4V (Target range: 8V - 17V)
+Text Notes 5700 4200 0    50   ~ 0
+Pulse Voltage: 31V
+Text Notes 8050 5250 0    50   ~ 0
+Voltage range: 39V - 48V
+$Comp
+L Sitina:+19V #PWR?
+U 1 1 60B20E91
+P 5100 1900
+F 0 "#PWR?" H 5100 1750 50  0001 C CNN
+F 1 "+19V" H 5115 2073 50  0000 C CNN
+F 2 "" H 5100 1900 50  0001 C CNN
+F 3 "" H 5100 1900 50  0001 C CNN
+	1    5100 1900
+	1    0    0    -1
+$EndComp
+$Comp
+L Sitina:+19V #PWR?
+U 1 1 60B21704
+P 6600 4300
+F 0 "#PWR?" H 6600 4150 50  0001 C CNN
+F 1 "+19V" H 6615 4473 50  0000 C CNN
+F 2 "" H 6600 4300 50  0001 C CNN
+F 3 "" H 6600 4300 50  0001 C CNN
+	1    6600 4300
+	1    0    0    -1
+$EndComp
+Wire Wire Line
+	6300 1900 7800 1900
 $EndSCHEMATC

Commit message: pcb: import footprints; finishing schematics
Parts:
- removed C?: 1uF/25V, symbol Device:C
- removed C? (x2): 10nF, symbol Device:C
- removed C?: 4.7uF/25V, symbol Device:C
- removed C?: 100nF/25V, symbol Device:C
- removed R?: 15K/1%, symbol Device:R
- removed R?: 100K, symbol Device:R
- removed U?: LT3050MSE, Package_SO:MSOP-12-1EP_3x4mm_P0.65mm_EP1.65x2.85mm_ThermalVias, symbol Sitina:LT3050MSE
- removed U?: NC7SZ08, Package_TO_SOT_SMD:SOT-23-5, symbol Sitina:NC7SZ08
- C1100, C1101: renamed from C?; footprint (none) -> Capacitor_SMD:C_0402_1005Metric
- C1102, C1104: renamed from C?; footprint (none) -> Capacitor_SMD:C_0603_1608Metric
- C1103, C1105: renamed from C?; footprint (none) -> Capacitor_SMD:C_0805_2012Metric
- D1100, D1101: renamed from D?; value HSMS-2805 -> B0540W; footprint (none) -> Diode_SMD:D_SOD-123
- R1100, R1101, R1102, R1103: renamed from R?; footprint (none) -> Resistor_SMD:R_0402_1005Metric
- gave numbers to parts that had none: 1
Connections:
- net STROBE_AB: now also C1100.2, C1101.2
- no-connect marks 1 -> 0
Other:
- note removed: "VAB range: 6.2V - 17.4V (Target range: 8V - 17V)"
- moved on the sheet: C1100, C1101, C1102, C1103, C1104, C1105, D1100, D1101, Q1100A, Q1100B, R1100, R1101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
