File: Hardware/afe.sch (KiCad schematic (older format))
At the start: 26 parts, among them U300 AD9990

Commit message: pcb: working on h-driver schematics
Parts:
- removed C324: 100nF, symbol Device:C
- added C? (x6): 100nF/25V, symbol Device:C
- added C?: 100nF, symbol Device:C
- added C? (x2): 18pF, Capacitor_SMD:C_0603_1608Metric, symbol Device:C
- added R? (x4): 49.9K, symbol Device:R
- added U? (x2): ADA4800, Package_DFN_QFN:DFN-6-1EP_2x1.8mm_P0.5mm_EP1.2x1.6mm, symbol Sitina:ADA4800
- added Y?: 25MHz, Crystal:Crystal_SMD_3225-4Pin_3.2x2.5mm, symbol Device:Crystal_GND24
Connections:
- net AFE_H1_A: now also U300.E1 (H1A); no longer U300.D2 (H4A)
- net AFE_H1_B: now also U300.E11 (H1B); no longer U300.D10 (H4B)
- net AFE_H2_A: now also U300.E2 (H2A); no longer U300.C1 (HL_A)
- net AFE_H2_B: now also U300.E10 (H2B); no longer U300.C11 (HL_B)
- net AFE_H3_A: now also U300.D1 (H3A); no longer U300.B11 (RG_B)
- net AFE_H3_B: now also U300.D11 (H3B)
- net AFE_H4_A: now also U300.D2 (H4A); no longer U300.E11 (H1B)
- net AFE_H4_B: now also U300.D10 (H4B); no longer U300.F4 (SUBCK)
- net AFE_HL_A: now also U300.C1 (HL_A); no longer U300.E10 (H2B)
- net AFE_HL_B: now also U300.C11 (HL_B); no longer U300.F3 (XV1)
- net AFE_RG_A: now also U300.B1 (RG_A); no longer U300.D1 (H3A)
- net AFE_RG_B: now also U300.B11 (RG_B); no longer U300.D11 (H3B)
- net AFE_SUBCK: now also U300.F4 (SUBCK); no longer U300.F1 (XV3)
- net AFE_XV1: now also U300.F3 (XV1); no longer U300.G4 (XV4)
- net AFE_XV10: now also U300.H3 (XV10); no longer U300.K1 (XV13)
- net AFE_XV11: now also U300.H4 (XV11); no longer U300.L2 (XV14)
- net AFE_XV12: now also U300.J1 (XV12); no longer U300.K2 (XV15)
- net AFE_XV13: now also U300.K1 (XV13); no longer U300.J2 (XV16)
- net AFE_XV14: now also U300.L2 (XV14); no longer U300.J3 (XV17)
- net AFE_XV15: now also U300.K2 (XV15); no longer U300.K3 (XV18)
- net AFE_XV16: now also U300.J2 (XV16); no longer U300.L3 (XV19)
- net AFE_XV2: now also U300.F2 (XV2); no longer U300.G3 (XV5)
- net AFE_XV3: now also U300.F1 (XV3); no longer U300.G2 (XV6)
- net AFE_XV4: now also U300.G4 (XV4); no longer U300.G1 (XV7)
- net AFE_XV5: now also U300.G3 (XV5); no longer U300.H1 (XV8)
- net AFE_XV6: now also U300.G2 (XV6); no longer U300.H2 (XV9)
- net AFE_XV7: now also U300.G1 (XV7); no longer U300.H3 (XV10)
- net AFE_XV8: now also U300.H1 (XV8); no longer U300.H4 (XV11)
- net AFE_XV9: now also U300.H2 (XV9); no longer U300.J1 (XV12)
- net CCDIN_A: now also U?.1 (IN); no longer C323.2
- net CCDIN_B: now also U?.1 (IN)
- net GND: now also C?.1, C?.1, C?.2, C?.2, C?.2, C?.2, C?.2, C?.2, U?.2 (VEE), U?.2 (VEE), U?.7 (EPAD), U?.7 (EPAD), Y?.2, Y?.4
- net at U300.A10 (CCDIN_B): now also C?.1
- net at U300.B5 (CLI): now also C?.2, Y?.1
- net at U300.B6 (CLO): now also C?.2, Y?.3
- new net: C323.2, U?.3 (OUT)
- new net: C?.1, R?.2, U?.4 (IDRV) (x2)
- new net: C?.1, R?.2, U?.6 (ISF) (x2)
- new net: C?.2, U?.3 (OUT)
- new net +15V: C?.1, C?.1, R?.1, R?.1, R?.1, R?.1, U?.5 (VCC), U?.5 (VCC)
Other:
- moved on the sheet: C300, C301, C302, C303, C304, C305, C306, C307, C308, C309, C310, C311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

Commit message: pcb: cleanup schematics; working on lcd
Connections:
- net GPO1_STROBE: now reaches U300.G11 (GPO1)
- net AFE_H3_A: no longer names the net of U300.D1 (H3A)
- net AFE_H3_B: no longer names the net of U300.D11 (H3B)
- net AFE_H4_A: no longer names the net of U300.D2 (H4A)
- net AFE_H4_B: no longer names the net of U300.D10 (H4B)
- net AFE_XV1 renamed AFE_V1
- net AFE_XV10: no longer names the net of U300.H3 (XV10)
- net AFE_XV11: no longer names the net of U300.H4 (XV11)
- net AFE_XV12: no longer names the net of U300.J1 (XV12)
- net AFE_XV13: no longer names the net of U300.K1 (XV13)
- net AFE_XV14: no longer names the net of U300.L2 (XV14)
- net AFE_XV15: no longer names the net of U300.K2 (XV15)
- net AFE_XV16: no longer names the net of U300.J2 (XV16)
- net AFE_XV2 renamed AFE_V2
- net AFE_XV3 renamed AFE_V2_3rd
- net AFE_XV4 renamed AFE_FDG
- net AFE_XV5: no longer names the net of U300.G3 (XV5)
- net AFE_XV6: no longer names the net of U300.G2 (XV6)
- net AFE_XV7: no longer names the net of U300.G1 (XV7)
- net AFE_XV8: no longer names the net of U300.H1 (XV8)
- net AFE_XV9: no longer names the net of U300.H2 (XV9)
- no-connect marks 0 -> 31
Changed lines of the file:
@@
 $Descr A4 11693 8268
 encoding utf-8
-Sheet 4 8
+Sheet 8 9
 Title ""
 Date ""
@@
 AFE_SL
 Text HLabel 6500 4700 2    50   Output ~ 0
-AFE_D[0..13]
+CSI_D[0..13]
 Wire Wire Line
 	5900 4800 6500 4800
@@
 Text HLabel 4200 2100 0    50   Output ~ 0
 AFE_H2_A
-Text HLabel 4200 2200 0    50   Output ~ 0
-AFE_H3_A
-Text HLabel 4200 2300 0    50   Output ~ 0
-AFE_H4_A
 Text HLabel 4200 2400 0    50   Output ~ 0
 AFE_HL_A
@@
 Text HLabel 4200 2700 0    50   Output ~ 0
 AFE_H2_B
-Text HLabel 4200 2800 0    50   Output ~ 0
-AFE_H3_B
-Text HLabel 4200 2900 0    50   Output ~ 0
-AFE_H4_B
 Text HLabel 4200 3000 0    50   Output ~ 0
 AFE_HL_B
@@
 AFE_SUBCK
 Text HLabel 4200 3300 0    50   Output ~ 0
-AFE_XV1
+AFE_V1
 Text HLabel 4200 3400 0    50   Output ~ 0
-AFE_XV2
+AFE_V2
 Text HLabel 4200 3500 0    50   Output ~ 0
-AFE_XV3
-Text HLabel 4200 3600 0    50   Output ~ 0
-AFE_XV4
-Text HLabel 4200 3700 0    50   Output ~ 0
-AFE_XV5
-Text HLabel 4200 3800 0    50   Output ~ 0
-AFE_XV6
-Text HLabel 4200 3900 0    50   Output ~ 0
-AFE_XV7
-Text HLabel 4200 4000 0    50   Output ~ 0
-AFE_XV8
-Text HLabel 4200 4100 0    50   Output ~ 0
-AFE_XV9
-Text HLabel 4200 4200 0    50   Output ~ 0
-AFE_XV10
-Text HLabel 4200 4300 0    50   Output ~ 0
-AFE_XV11
-Text HLabel 4200 4400 0    50   Output ~ 0
-AFE_XV12
-Text HLabel 4200 4500 0    50   Output ~ 0
-AFE_XV13
-Text HLabel 4200 4600 0    50   Output ~ 0
-AFE_XV14
-Text HLabel 4200 4700 0    50   Output ~ 0
-AFE_XV15
-Text HLabel 4200 4800 0    50   Output ~ 0
-AFE_XV16
+AFE_V2_3rd
 Wire Wire Line
 	4200 1900 4400 1900
@@
 	4200 2100 4400 2100
 Wire Wire Line
-	4200 2200 4400 2200
-Wire Wire Line
-	4200 2300 4400 2300
-Wire Wire Line
 	4200 2400 4400 2400
 Wire Wire Line
@@
 	4200 2700 4400 2700
 Wire Wire Line
-	4200 2800 4400 2800
-Wire Wire Line
-	4200 2900 4400 2900
-Wire Wire Line
 	4200 3000 4400 3000
 Wire Wire Line
@@
 Wire Wire Line
 	4200 3500 4400 3500
-Wire Wire Line
-	4200 3600 4400 3600
-Wire Wire Line
-	4200 3700 4400 3700
-Wire Wire Line
-	4200 3800 4400 3800
-Wire Wire Line
-	4200 3900 4400 3900
-Wire Wire Line
-	4200 4000 4400 4000
-Wire Wire Line
-	4200 4100 4400 4100
-Wire Wire Line
-	4200 4200 4400 4200
-Wire Wire Line
-	4200 4300 4400 4300
-Wire Wire Line
-	4200 4400 4400 4400
-Wire Wire Line
-	4200 4500 4400 4500
-Wire Wire Line
-	4200 4600 4400 4600
-Wire Wire Line
-	4200 4700 4400 4700
-Wire Wire Line
-	4200 4800 4400 4800
 $Comp
 L Sitina:ADA4800 U?
@@
 	3700 6200 2400 6200
 Wire Wire Line
+	4200 3600 4400 3600
+Text HLabel 4200 3600 0    50   Output ~ 0
+AFE_FDG
+NoConn ~ 4400 3700
+NoConn ~ 4400 3800
+NoConn ~ 4400 3900
+NoConn ~ 4400 4000
+NoConn ~ 4400 4100
+NoConn ~ 4400 4200
+NoConn ~ 4400 4300
+NoConn ~ 4400 4400
+NoConn ~ 4400 4500
+NoConn ~ 4400 4600
+NoConn ~ 4400 4700
+NoConn ~ 4400 4800
+NoConn ~ 4400 4900
+NoConn ~ 4400 5000
+NoConn ~ 4400 5100
+NoConn ~ 4400 5200
+NoConn ~ 4400 5300
+NoConn ~ 4400 5400
+NoConn ~ 4400 5500
+NoConn ~ 4400 5600
+NoConn ~ 4400 2800
+NoConn ~ 4400 2900
+NoConn ~ 4400 2200
+NoConn ~ 4400 2300
+Text HLabel 4200 5800 0    50   Output ~ 0
+GPO1_STROBE
+Wire Wire Line
+	4200 5800 4400 5800
+NoConn ~ 4400 5900
+NoConn ~ 4400 6000
+NoConn ~ 4400 6100
+NoConn ~ 4400 6200
+NoConn ~ 4400 6300
+NoConn ~ 4400 6400
+NoConn ~ 4400 6500
+Wire Wire Line
 	5900 5400 6500 5400

Commit message: pcb: working on power supply
Parts:
- Y?: value 25MHz -> 30MHz
Changed lines of the file:
@@
 $Descr A4 11693 8268
 encoding utf-8
-Sheet 8 9
-Title ""
+Sheet 8 14
+Title "Sitina Ne"
 Date ""
-Rev ""
-Comp ""
+Rev "R0P2"
+Comp "ZephRay"
 Comment1 ""
 Comment2 ""
@@
 AFE_SL
 Text HLabel 6500 4700 2    50   Output ~ 0
-CSI_D[0..13]
+CSI_D[13..0]
 Wire Wire Line
 	5900 4800 6500 4800
@@
 AR Path="/5D0B94DA/5F88A2CB" Ref="Y?"  Part="1"
 F 0 "Y?" H 2894 6546 50  0000 L CNN
-F 1 "25MHz" H 2850 6400 50  0000 L CNN
+F 1 "30MHz" H 2850 6400 50  0000 L CNN
 F 2 "Crystal:Crystal_SMD_3225-4Pin_3.2x2.5mm" H 2700 6500 50  0001 C CNN
 F 3 "~" H 2700 6500 50  0001 C CNN

Commit message: pcb: import footprints; finishing schematics
Parts:
- added TP1, TP2: TestPoint, Connector_Pin:Pin_D1.0mm_L10.0mm, symbol Connector:TestPoint
- C800: renamed from C300; footprint (none) -> Capacitor_SMD:C_0402_1005Metric
- C801: renamed from C301; footprint (none) -> Capacitor_SMD:C_0805_2012Metric
- C802: renamed from C302; footprint (none) -> Capacitor_SMD:C_0402_1005Metric
- C803: renamed from C303; footprint (none) -> Capacitor_SMD:C_0402_1005Metric
- C804: renamed from C304; footprint (none) -> Capacitor_SMD:C_0805_2012Metric
- C805: renamed from C305; footprint (none) -> Capacitor_SMD:C_0402_1005Metric
- C806: renamed from C306; footprint (none) -> Capacitor_SMD:C_0402_1005Metric
- C807: renamed from C307; footprint (none) -> Capacitor_SMD:C_0402_1005Metric
- C808: renamed from C308; footprint (none) -> Capacitor_SMD:C_0402_1005Metric
- C809: renamed from C309; footprint (none) -> Capacitor_SMD:C_0402_1005Metric
- C810: renamed from C310; footprint (none) -> Capacitor_SMD:C_0805_2012Metric
- C811: renamed from C311; footprint (none) -> Capacitor_SMD:C_0402_1005Metric
- C812: renamed from C312; footprint (none) -> Capacitor_SMD:C_0805_2012Metric
- C813: renamed from C313; footprint (none) -> Capacitor_SMD:C_0402_1005Metric
- C814: renamed from C314; footprint (none) -> Capacitor_SMD:C_0402_1005Metric
- C815: renamed from C315; footprint (none) -> Capacitor_SMD:C_0402_1005Metric
- C816: renamed from C316; footprint (none) -> Capacitor_SMD:C_0805_2012Metric
- C817: renamed from C317; footprint (none) -> Capacitor_SMD:C_0402_1005Metric
- C818: renamed from C318; footprint (none) -> Capacitor_SMD:C_0805_2012Metric
- C819: renamed from C319; footprint (none) -> Capacitor_SMD:C_0402_1005Metric
- C820: renamed from C320; footprint (none) -> Capacitor_SMD:C_0402_1005Metric
- C821: renamed from C321; footprint (none) -> Capacitor_SMD:C_0402_1005Metric
- C822: renamed from C322; footprint (none) -> Capacitor_SMD:C_0402_1005Metric
- C823: renamed from C323; footprint (none) -> Capacitor_SMD:C_0402_1005Metric
- C824, C825, C826, C827, C828, C829: renamed from C?; footprint (none) -> Capacitor_SMD:C_0603_1608Metric
- C830: renamed from C?; footprint (none) -> Capacitor_SMD:C_0402_1005Metric
- R800, R801, R802, R803: renamed from R?; value 49.9K -> 49.9K/1%; footprint (none) -> Resistor_SMD:R_0402_1005Metric
- gave numbers to parts that had none: 5
- renumbered U300 to U800
Connections:
- net CSI_HSYNC: now also TP2.1
- net CSI_VSYNC: now also TP1.1
- net PWR_EN: now reaches U800.G10 (GPO2)
- no-connect marks 31 -> 30
Other:
- moved on the sheet: C800, C801, C802, C803, C804, C805, C806, C807, C808, C809, C810, C811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

Commit message: pcb: finishing overall design
Parts:
- U800: footprint (none) -> Footprints:BGA-112_11x11_8.0x8.0mm
Changed lines of the file:
@@
 F 0 "U800" H 5650 4215 50  0000 C CNN
 F 1 "AD9990" H 5650 4124 50  0000 C CNN
-F 2 "" H 5600 2500 50  0001 C CNN
+F 2 "Footprints:BGA-112_11x11_8.0x8.0mm" H 5600 2500 50  0001 C CNN
 F 3 "" H 5600 2500 50  0001 C CNN
 	1    5600 2500
