File: Hardware/debug.sch (KiCad schematic (older format))
At the start: 8 parts, among them J100 Conn_02x05_Odd_Even

Commit message: pcb: import footprints; finishing schematics
Parts:
- R200, R201, R202, R203: renamed from R?; footprint (none) -> Resistor_SMD:R_0402_1005Metric
- R204: renamed from R108; footprint Resistor_SMD:R_0603_1608Metric -> Resistor_SMD:R_0402_1005Metric
- gave numbers to parts that had none: 1
- renumbered D100 to D200, J100 to J200
Changed lines of the file:
@@
 $EndDescr
 $Comp
-L Connector_Generic:Conn_02x05_Odd_Even J100
+L Connector_Generic:Conn_02x05_Odd_Even J200
 U 1 1 5D31C612
 P 6500 4300
-F 0 "J100" H 6550 4717 50  0000 C CNN
+F 0 "J200" H 6550 4717 50  0000 C CNN
 F 1 "Conn_02x05_Odd_Even" H 6550 4626 50  0000 C CNN
 F 2 "Connector_PinHeader_1.27mm:PinHeader_2x05_P1.27mm_Vertical_SMD" H 6500 4300 50  0001 C CNN
@@
 $EndComp
 $Comp
-L Device:R R108
+L Device:R R204
 U 1 1 5D32601B
 P 6900 3750
-F 0 "R108" H 6970 3796 50  0000 L CNN
+F 0 "R204" H 6970 3796 50  0000 L CNN
 F 1 "10K" H 6970 3705 50  0000 L CNN
-F 2 "Resistor_SMD:R_0603_1608Metric" V 6830 3750 50  0001 C CNN
+F 2 "Resistor_SMD:R_0402_1005Metric" V 6830 3750 50  0001 C CNN
 F 3 "~" H 6900 3750 50  0001 C CNN
 	1    6900 3750
@@
 NoConn ~ 6300 4400
 $Comp
-L Device:D_Schottky D100
+L Device:D_Schottky D200
 U 1 1 5D37EF0D
 P 7150 4500
-F 0 "D100" H 6950 4550 50  0000 C CNN
+F 0 "D200" H 6950 4550 50  0000 C CNN
 F 1 "1N5819" H 7400 4550 50  0000 C CNN
 F 2 "Diode_SMD:D_SOD-123" H 7150 4500 50  0001 C CNN
@@
 	7500 4400 6800 4400
 $Comp
-L Switch:SW_DIP_x02 SW?
+L Switch:SW_DIP_x02 SW200
 U 1 1 60A7F175
 P 4900 4200
-F 0 "SW?" V 4946 4070 50  0000 R CNN
+F 0 "SW200" V 4946 4070 50  0000 R CNN
 F 1 "SW_DIP_x02" V 4855 4070 50  0000 R CNN
 F 2 "" H 4900 4200 50  0001 C CNN
@@
 AR Path="/5F5596FF/60A81364" Ref="R?"  Part="1"
 AR Path="/5FE3519F/60A81364" Ref="R?"  Part="1"
-AR Path="/5F6B6546/60A81364" Ref="R?"  Part="1"
-F 0 "R?" V 4143 4700 50  0000 C CNN
+AR Path="/5F6B6546/60A81364" Ref="R202"  Part="1"
+F 0 "R202" V 4143 4700 50  0000 C CNN
 F 1 "10K" V 4234 4700 50  0000 C CNN
-F 2 "" V 4280 4700 50  0001 C CNN
+F 2 "Resistor_SMD:R_0402_1005Metric" V 4280 4700 50  0001 C CNN
 F 3 "~" H 4350 4700 50  0001 C CNN
 	1    4350 4700
@@
 AR Path="/5F5596FF/60A81854" Ref="R?"  Part="1"
 AR Path="/5FE3519F/60A81854" Ref="R?"  Part="1"
-AR Path="/5F6B6546/60A81854" Ref="R?"  Part="1"
-F 0 "R?" V 4143 5000 50  0000 C CNN
+AR Path="/5F6B6546/60A81854" Ref="R203"  Part="1"
+F 0 "R203" V 4143 5000 50  0000 C CNN
 F 1 "10K" V 4234 5000 50  0000 C CNN
-F 2 "" V 4280 5000 50  0001 C CNN
+F 2 "Resistor_SMD:R_0402_1005Metric" V 4280 5000 50  0001 C CNN
 F 3 "~" H 4350 5000 50  0001 C CNN
 	1    4350 5000
@@
 AR Path="/5F5596FF/60A82BB6" Ref="R?"  Part="1"
 AR Path="/5FE3519F/60A82BB6" Ref="R?"  Part="1"
-AR Path="/5F6B6546/60A82BB6" Ref="R?"  Part="1"
-F 0 "R?" H 4900 3600 50  0000 L CNN
+AR Path="/5F6B6546/60A82BB6" Ref="R200"  Part="1"
+F 0 "R200" H 4900 3600 50  0000 L CNN
 F 1 "1K" H 4900 3700 50  0000 L CNN
-F 2 "" V 4730 3650 50  0001 C CNN
+F 2 "Resistor_SMD:R_0402_1005Metric" V 4730 3650 50  0001 C CNN
 F 3 "~" H 4800 3650 50  0001 C CNN
 	1    4800 3650
@@
 AR Path="/5F5596FF/60A830D3" Ref="R?"  Part="1"
 AR Path="/5FE3519F/60A830D3" Ref="R?"  Part="1"
-AR Path="/5F6B6546/60A830D3" Ref="R?"  Part="1"
-F 0 "R?" H 4970 3696 50  0000 L CNN
-F 1 "1K" H 4970 3605 50  0000 L CNN
-F 2 "" V 4830 3650 50  0001 C CNN
+AR Path="/5F6B6546/60A830D3" Ref="R201"  Part="1"
+F 0 "R201" H 5000 3700 50  0000 L CNN
+F 1 "1K" H 5000 3600 50  0000 L CNN
+F 2 "Resistor_SMD:R_0402_1005Metric" V 4830 3650 50  0001 C CNN
 F 3 "~" H 4900 3650 50  0001 C CNN
 	1    4900 3650
@@
 $EndComp
 $Comp
-L power:GND #PWR?
+L power:GND #PWR0300
 U 1 1 60A84403
 P 4000 5100
-F 0 "#PWR?" H 4000 4850 50  0001 C CNN
+F 0 "#PWR0300" H 4000 4850 50  0001 C CNN
 F 1 "GND" H 4005 4927 50  0000 C CNN
 F 2 "" H 4000 5100 50  0001 C CNN
@@
 	4800 3500 4800 3400
 $Comp
-L power:+3V3 #PWR?
+L power:+3V3 #PWR0301
 U 1 1 60A86541
 P 4800 3400
-F 0 "#PWR?" H 4800 3250 50  0001 C CNN
+F 0 "#PWR0301" H 4800 3250 50  0001 C CNN
 F 1 "+3V3" H 4815 3573 50  0000 C CNN
 F 2 "" H 4800 3400 50  0001 C CNN

Commit message: pcb: finishing overall design
Parts:
- SW200: footprint (none) -> Button_Switch_SMD:SW_DIP_SPSTx02_Slide_Copal_CHS-02B_W7.62mm_P1.27mm
Changed lines of the file:
@@
 F 0 "SW200" V 4946 4070 50  0000 R CNN
 F 1 "SW_DIP_x02" V 4855 4070 50  0000 R CNN
-F 2 "" H 4900 4200 50  0001 C CNN
+F 2 "Button_Switch_SMD:SW_DIP_SPSTx02_Slide_Copal_CHS-02B_W7.62mm_P1.27mm" H 4900 4200 50  0001 C CNN
 F 3 "~" H 4900 4200 50  0001 C CNN
 	1    4900 4200
