File: Hardware/hdriver.sch (KiCad schematic (older format))
At the start: 36 parts

Commit message: pcb: working on h-driver and v-driver
Parts:
- removed C? (x2): 100nF/25V, symbol Device:C
- removed D? (x2): HSMS-2805, symbol Device:D_Schottky
- removed R? (x2): 200K/1%, symbol Device:R
- added C?: 100nF/25V, symbol Device:C
- added U?: 74LCX541BQX, symbol 74xx:74LS541
Connections:
- net labels added: +1V5, +2V, -3V5, -4V
- net labels removed: -VH, -VRESET
- wire segments 212 -> 215
- no-connect marks 0 -> 9
Other:
- moved on the sheet: C?, D?, R?

Commit message: pcb: import footprints; finishing schematics
Parts:
- C900, C901, C902, C903, C904, C905, C906, C907, C908, C909, C910, C911: renamed from C?; footprint (none) -> Capacitor_SMD:C_0603_1608Metric
- D900, D901, D902, D903, D904, D905, D906, D907: renamed from D?; value HSMS-2805 -> B0540W; footprint (none) -> Diode_SMD:D_SOD-123
- R900, R901, R902, R903, R904, R905, R906, R907: renamed from R?; footprint (none) -> Resistor_SMD:R_0402_1005Metric
- gave numbers to parts that had none: 4

Commit message: pcb: finishing overall design
Parts:
- U900, U901, U902, U903: footprint (none) -> Package_SO:SSOP-20_4.4x6.5mm_P0.65mm
Changed lines of the file:
@@
 F 0 "U900" H 6400 2700 50  0000 C CNN
 F 1 "74LCX541BQX" H 6500 2600 50  0000 C CNN
-F 2 "" H 6200 1900 50  0001 C CNN
+F 2 "Package_SO:SSOP-20_4.4x6.5mm_P0.65mm" H 6200 1900 50  0001 C CNN
 F 3 "http://www.ti.com/lit/gpn/sn74LS541" H 6200 1900 50  0001 C CNN
 	1    6200 1900
@@
 F 0 "U901" H 6400 4900 50  0000 C CNN
 F 1 "74LCX541BQX" H 6500 4800 50  0000 C CNN
-F 2 "" H 6200 4100 50  0001 C CNN
+F 2 "Package_SO:SSOP-20_4.4x6.5mm_P0.65mm" H 6200 4100 50  0001 C CNN
 F 3 "http://www.ti.com/lit/gpn/sn74LS541" H 6200 4100 50  0001 C CNN
 	1    6200 4100
@@
 F 0 "U902" H 6400 7100 50  0000 C CNN
 F 1 "74LCX541BQX" H 6500 7000 50  0000 C CNN
-F 2 "" H 6200 6300 50  0001 C CNN
+F 2 "Package_SO:SSOP-20_4.4x6.5mm_P0.65mm" H 6200 6300 50  0001 C CNN
 F 3 "http://www.ti.com/lit/gpn/sn74LS541" H 6200 6300 50  0001 C CNN
 	1    6200 6300
@@
 F 0 "U903" H 9300 4900 50  0000 C CNN
 F 1 "74LCX541BQX" H 9400 4800 50  0000 C CNN
-F 2 "" H 9100 4100 50  0001 C CNN
+F 2 "Package_SO:SSOP-20_4.4x6.5mm_P0.65mm" H 9100 4100 50  0001 C CNN
 F 3 "http://www.ti.com/lit/gpn/sn74LS541" H 9100 4100 50  0001 C CNN
 	1    9100 4100
