File: Hardware/mcu.sch (KiCad schematic (older format))
At the start: 40 parts, among them U100 IMXRT1050

Commit message: pcb: cleanup schematics; working on lcd
Connections:
- net labels added: WAKEUP
- net labels removed: ARM_NMI, CSI_MCLK
- wire segments 286 -> 284
Other:
- moved on the sheet: C100, C101, C102, C103, C104, C105, C106, C107, C108, C109, C110, C111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

Commit message: pcb: working on power supply
Parts:
- added C? (x4): 18pF, Capacitor_SMD:C_0402_1005Metric, symbol Device:C
- added R? (x2): 10K, symbol Device:R
- added Y?: 24MHz, Oscillator:Oscillator_SMD_Abracon_ASE-4Pin_3.2x2.5mm, symbol Device:Crystal_GND24
- added Y?: Crystal, Crystal:Crystal_SMD_TXC_9HT11-2Pin_2.0x1.2mm_HandSoldering, symbol Device:Crystal
Connections:
- net +1V8 is gone; now on net +3V3: C115.1, C116.1, U100.K5 (NVCC_SD1)
- net +3V3: now also R?.1
- net GND: now also U100.K6 (TESTMODE), C?.1, C?.1, C?.2, C?.2, R?.2, Y?.2, Y?.4
- net JTAG_MOD: now also R?.1
- net JTAG_TRSTB: now also R?.2
- net LCD_EN: now also U100.M3 (GPIO_SD_B1_02); no longer U100.E7 (GPIO_B0_01)
- net LCD_CS: now reaches U100.B14 (GPIO_B1_15)
- net ONOFF: now reaches U100.M6 (ONOFF)
- net LCD_RST: now reaches U100.M7 (POR_B)
- net at U100.N11 (XTALO): now also C?.1, Y?.3
- net at U100.N9 (RTC_XTALI): now also C?.2, Y?.1
- net at U100.P11 (XTALI): now also C?.1, Y?.1
- net at U100.P9 (RTC_XTALO): now also C?.2, Y?.2
- net KO0: now reaches U100.H14 (GPIO_AD_B0_14)
- net KI2: now reaches U100.J12 (GPIO_AD_B1_06)
- net KI3: now reaches U100.K10 (GPIO_AD_B1_07)
- net KI1: now reaches U100.K12 (GPIO_AD_B1_05)
- net KO1: now reaches U100.L10 (GPIO_AD_B0_15)
- net KI0: now reaches U100.L12 (GPIO_AD_B1_04)
- net SD_PWR_EN: now reaches U100.M12 (GPIO_AD_B1_03)
- net SD_WP renamed KO2
- net SPI_MOSI renamed LCD_DI
- net SPI_SCK renamed LCD_SCK
- net USB_VBUS renamed VBUS
- new net LCD_DE: U100.E7 (GPIO_B0_01)
- no-connect marks 3 -> 13
Other:
- moved on the sheet: C115, C116, C117, C118, C119, C120, C121, C122, C123, C124, C125, L100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

Commit message: pcb: import footprints; finishing schematics
Parts:
- added R100: 10K, Resistor_SMD:R_0402_1005Metric, symbol Device:R
- C100, C101, C102, C103, C104, C105, C106, C107, C110, C120, C121, C122: footprint (none) -> Capacitor_SMD:C_0402_1005Metric
- C108, C109, C119, C124: footprint (none) -> Capacitor_SMD:C_0805_2012Metric
- C123: value 0.1uF -> 100nF; footprint (none) -> Capacitor_SMD:C_0402_1005Metric
- C125, C144: renamed from C115; footprint (none) -> Capacitor_SMD:C_0402_1005Metric
- C126: renamed from C116; footprint (none) -> Capacitor_SMD:C_0805_2012Metric
- C127: renamed from C117; footprint (none) -> Capacitor_SMD:C_0402_1005Metric
- C128, C141: renamed from C118; footprint (none) -> Capacitor_SMD:C_0402_1005Metric
- C129: renamed from C111; footprint (none) -> Capacitor_SMD:C_0402_1005Metric
- C130: renamed from C112; footprint (none) -> Capacitor_SMD:C_0805_2012Metric
- C131: renamed from C113; footprint (none) -> Capacitor_SMD:C_0402_1005Metric
- C132: renamed from C114; footprint (none) -> Capacitor_SMD:C_0805_2012Metric
- C133: renamed from C122; footprint (none) -> Capacitor_SMD:C_0805_2012Metric
- C134: renamed from C123; value 0.1uF -> 100nF; footprint (none) -> Capacitor_SMD:C_0402_1005Metric
- C135: renamed from C124; value 0.1uF -> 100nF; footprint (none) -> Capacitor_SMD:C_0402_1005Metric
- C136: renamed from C125; value 0.1uF -> 100nF; footprint (none) -> Capacitor_SMD:C_0402_1005Metric
- C137: renamed from C119; footprint (none) -> Capacitor_SMD:C_0805_2012Metric
- C138: renamed from C120; value 0.1uF -> 100nF; footprint (none) -> Capacitor_SMD:C_0402_1005Metric
- C139: renamed from C121; value 0.1uF -> 100nF; footprint (none) -> Capacitor_SMD:C_0402_1005Metric
- C140: renamed from C117; value 33uF -> 47uF; footprint (none) -> Capacitor_SMD:C_0805_2012Metric
- C142: renamed from C113; footprint (none) -> Capacitor_SMD:C_0805_2012Metric
- C143: renamed from C114; footprint (none) -> Capacitor_SMD:C_0402_1005Metric
- C145: renamed from C116; footprint (none) -> Capacitor_SMD:C_0402_1005Metric
- L100: footprint (none) -> Inductor_SMD:L_Vishay_IHLP-1212
- R101, R102: renamed from R?; footprint (none) -> Resistor_SMD:R_0402_1005Metric
- Y101: renamed from Y?; value Crystal -> 32.768K
- gave numbers to parts that had none: 5
Connections:
- net +3V3: now also R100.1
- net AFE_RST: now reaches U100.G14 (GPIO_AD_B0_05)
- net AFE_SYNC: now reaches U100.L5 (GPIO_SD_B1_00)
- net LCD_RST renamed POR
- net POR: now also R100.2
- net PMIC_ON_REQ renamed ON
- net PMIC_STBY_REQ: no longer names the net of U100.L7 (PMIC_STBY_REQ)
- net WAKEUP: no longer names the net of U100.L6 (WAKEUP)

Commit message: pcb: finishing overall design
Parts:
- U100: footprint (none) -> Footprints:BGA-196_14x14_12.0x12.0mm
Changed lines of the file:
@@
 F 0 "U100" H 1700 7450 50  0000 L CNN
 F 1 "IMXRT1050" H 1550 7350 50  0000 L CNN
-F 2 "" H 2500 6500 50  0001 C CNN
+F 2 "Footprints:BGA-196_14x14_12.0x12.0mm" H 2500 6500 50  0001 C CNN
 F 3 "" H 2500 6500 50  0001 C CNN
 	2    2500 5800
@@
 F 0 "U100" H 6550 4200 50  0000 L CNN
 F 1 "IMXRT1050" H 6550 4100 50  0000 L CNN
-F 2 "" H 7000 3100 50  0001 C CNN
+F 2 "Footprints:BGA-196_14x14_12.0x12.0mm" H 7000 3100 50  0001 C CNN
 F 3 "" H 7000 3100 50  0001 C CNN
 	4    7000 2400
@@
 F 0 "U100" H 2050 4200 50  0000 L CNN
 F 1 "IMXRT1050" H 2050 4100 50  0000 L CNN
-F 2 "" H 2500 3100 50  0001 C CNN
+F 2 "Footprints:BGA-196_14x14_12.0x12.0mm" H 2500 3100 50  0001 C CNN
 F 3 "" H 2500 3100 50  0001 C CNN
 	1    2500 2400
@@
 F 0 "U100" H 4250 4200 50  0000 L CNN
 F 1 "IMXRT1050" H 4250 4100 50  0000 L CNN
-F 2 "" H 4700 3100 50  0001 C CNN
+F 2 "Footprints:BGA-196_14x14_12.0x12.0mm" H 4700 3100 50  0001 C CNN
 F 3 "" H 4700 3100 50  0001 C CNN
 	5    4700 2400
@@
 F 0 "U100" H 4750 6600 50  0000 L CNN
 F 1 "IMXRT1050" H 4750 6500 50  0000 L CNN
-F 2 "" H 5200 5500 50  0001 C CNN
+F 2 "Footprints:BGA-196_14x14_12.0x12.0mm" H 5200 5500 50  0001 C CNN
 F 3 "" H 5200 5500 50  0001 C CNN
 	3    5200 4800
@@
 F 0 "U100" H 10050 5100 50  0000 C CNN
 F 1 "IMXRT1050" H 10150 5000 50  0000 C CNN
-F 2 "" H 10400 4000 50  0001 C CNN
+F 2 "Footprints:BGA-196_14x14_12.0x12.0mm" H 10400 4000 50  0001 C CNN
 F 3 "" H 10400 4000 50  0001 C CNN
 	6    10400 3300
