File: Hardware/ProcessingBoard/connector.sch (KiCad schematic (older format))
At the start: 1 part

Commit message: pcb: change footprint assignments
Parts:
- gave numbers to parts that had none: 1
Changed lines of the file:
@@
 CSI_PCLK
 $Comp
-L Connector_Generic_MountingPin:Conn_01x30_MountingPin J?
+L Connector_Generic_MountingPin:Conn_01x30_MountingPin J1
 U 1 1 5F7F691E
 P 6400 3900
-F 0 "J?" H 6488 3814 50  0000 L CNN
+F 0 "J1" H 6488 3814 50  0000 L CNN
 F 1 "Conn_01x30_MountingPin" H 6488 3723 50  0000 L CNN
 F 2 "" H 6400 3900 50  0001 C CNN
@@
 AFE_SYNC
 $Comp
-L power:+3V3 #PWR?
+L power:+3V3 #PWR0150
 U 1 1 5F8052CF
 P 6000 5200
-F 0 "#PWR?" H 6000 5050 50  0001 C CNN
+F 0 "#PWR0150" H 6000 5050 50  0001 C CNN
 F 1 "+3V3" V 6015 5328 50  0000 L CNN
 F 2 "" H 6000 5200 50  0001 C CNN
@@
 $EndComp
 $Comp
-L Sitina:+SYS #PWR?
+L Sitina:+SYS #PWR0152
 U 1 1 5F80574E
 P 6000 5300
-F 0 "#PWR?" H 6000 5150 50  0001 C CNN
+F 0 "#PWR0152" H 6000 5150 50  0001 C CNN
 F 1 "+SYS" V 6015 5428 50  0000 L CNN
 F 2 "" H 6000 5300 50  0001 C CNN
@@
 	6100 5100 6100 5600
 $Comp
-L power:GND #PWR?
+L power:GND #PWR0153
 U 1 1 5F80D4CA
 P 6400 5700
-F 0 "#PWR?" H 6400 5450 50  0001 C CNN
+F 0 "#PWR0153" H 6400 5450 50  0001 C CNN
 F 1 "GND" H 6405 5527 50  0000 C CNN
 F 2 "" H 6400 5700 50  0001 C CNN

Commit message: pcb: start initial layouting
Parts:
- J1: footprint (none) -> Connector_FFC-FPC:TE_3-84952-0_1x30-1MP_P1.0mm_Horizontal
Changed lines of the file:
@@
 F 0 "J1" H 6488 3814 50  0000 L CNN
 F 1 "Conn_01x30_MountingPin" H 6488 3723 50  0000 L CNN
-F 2 "" H 6400 3900 50  0001 C CNN
+F 2 "Connector_FFC-FPC:TE_3-84952-0_1x30-1MP_P1.0mm_Horizontal" H 6400 3900 50  0001 C CNN
 F 3 "~" H 6400 3900 50  0001 C CNN
 	1    6400 3900
