File: Hardware/ProcessingBoard/storage.sch (KiCad schematic (older format))
At the start: 21 parts, among them Q400 2N7002, U400 ADP163, U401 W25Q32JVZP

Commit message: pcb: start initial layouting
Parts:
- MICRO_SD400: footprint footprint:TFC-WPAPR-08 -> Footprints:TFC-WPAPR-08
Changed lines of the file:
@@
 $Descr A4 11693 8268
 encoding utf-8
-Sheet 10 10
+Sheet 4 10
 Title "Sitina Ne"
 Date ""
@@
 F 0 "MICRO_SD400" H 8828 4503 60  0000 L CNN
 F 1 "MICRO_SD(TFC-WPAPR-08)" H 8828 4397 60  0000 L CNN
-F 2 "footprint:TFC-WPAPR-08" H 8750 4400 60  0001 C CNN
+F 2 "Footprints:TFC-WPAPR-08" H 8750 4400 60  0001 C CNN
 F 3 "" H 8750 4400 60  0001 C CNN
 	1    8500 4400
@@
 $EndComp
 Connection ~ 8000 1800
-Wire Bus Line
-	5000 4800 5000 5300
-Wire Bus Line
-	6100 4000 6100 4400
 $Comp
 L power:+3V3 #PWR0239
@@
 	1    0    0    -1
 $EndComp
+Wire Bus Line
+	5000 4800 5000 5300
+Wire Bus Line
+	6100 4000 6100 4400
 $EndSCHEMATC
