File: Hardware/ProcessingBoard/Sitina.kicad_pcb (KiCad board)
At the start: 2 copper layers, 162 parts, among them J1 Conn_01x30_MountingPin, J200 Conn_02x05_Odd_Even, J500 USB_B_Micro, Q400 2N7002, SW200 SW_DIP_x02, SW600 SW_Push, SW601 SW_Push, SW602 SW_Push, SW603 SW_Push, SW610 SW_Push, SW611 SW_Push, SW612 SW_Push, SW613 SW_Push, SW620 SW_Push, SW621 SW_Push, SW622 SW_Push, SW623 SW_Push, U100 IMXRT1050, U3 LN2401, U300 MT48LC16M16A2BG, U301 MT48LC16M16A2BG, U400 ADP163, U401 W25Q32JVZP, U500 USBLC6-2SC6, U9 LTC3567, Y100 24MHz, Y101 32.768K

Commit message: PBr0p2, CBr0p1, submitted for prototype production
Parts:
- removed C3, C6: 1uF, Capacitor_SMD:C_0402_1005Metric
- removed C308, C309, C310, C311, C312, C313, C314: 100nF, Capacitor_SMD:C_0402_1005Metric
- removed C315: 4.7uF, Capacitor_SMD:C_0805_2012Metric
- removed C317: 22uF, Capacitor_SMD:C_0805_2012Metric
- removed C501: 100nF, Capacitor_SMD:C_0805_2012Metric
- removed C704: 220nF, Capacitor_SMD:C_0402_1005Metric
- removed L300, L301: 120R, Inductor_SMD:L_0603_1608Metric
- removed LCD700: TM032PDZ17, Footprints:Hirose_FH23-51S-0.3SHW_2Rows-51Pins-1MP-P0.60mm_Horizontal
- removed R4, R7: 0/0R05, Resistor_SMD:R_0805_2012Metric
- removed R501: 0, Resistor_SMD:R_0805_2012Metric
- removed SW613, SW620, SW621, SW622, SW623: SW_Push, Footprints:contact
- removed TP700, TP701, TP702, TP703, TP704: TestPoint, Connector_Pin:Pin_D1.0mm_L10.0mm
- removed U3: LN2401, Package_TO_SOT_SMD:SOT-23-5
- removed U301: MT48LC16M16A2BG, Footprints:BGA-54_9x9_8.0x14.0mm
- added D700: MBR0530, Diode_SMD:D_SOD-123, F.Cu at (137.6, 112.0)
- added J700: TXW280064B0, Connector_FFC-FPC:Hirose_FH12-40S-0.5SH_1x40-1MP_P0.50mm_Horizontal, F.Cu at (141.9, 129.0)
- added U700: CAT4139, Package_TO_SOT_SMD:SOT-23-5, F.Cu at (140.8, 108.5)
- BT1, C100, C101, C102, C103, C104, C123, C131, C139, C143, C144, C302, C303, C304, C305, C403, C404, C405, C500, D500, J1, J500, L500, MICRO_SD400, R404, R405, R406, U500: moved to B.Cu
- C701, C702: footprint Capacitor_SMD:C_0805_2012Metric -> Capacitor_SMD:C_0402_1005Metric
- C703: value 100nF/25V -> 100nF; footprint Capacitor_SMD:C_0603_1608Metric -> Capacitor_SMD:C_0402_1005Metric
- C705: value 220nF -> 1uF/35V; footprint Capacitor_SMD:C_0402_1005Metric -> Capacitor_SMD:C_0603_1608Metric
- R702: value 100K -> 10K
- R703: value 4.7K -> 1K
- R704: value 1.62R -> 15R
- SW612: value SW_Push -> TM-4175-B-B; footprint Footprints:contact -> Footprints:TM4175
- moved R13 109.4 mm to (83.9, 149.7)
- moved D1 103.0 mm to (84.2, 133.2)
- moved R14 100.8 mm to (84.7, 134.8)
- moved TH1 99.3 mm to (84.5, 151.1)
- moved J1 97.7 mm to (177.8, 127.0), turned to 90 degrees
- moved C33 90.3 mm to (102.3, 149.1), turned to -90 degrees
- moved BT1 89.5 mm to (86.4, 141.5), turned to 90 degrees
- moved C38 88.2 mm to (108.6, 152.4), turned to -90 degrees
- moved R3 87.7 mm to (112.0, 152.4), turned to -90 degrees
- moved SW612 86.2 mm to (167.0, 96.0), turned to 90 degrees
- moved R19 85.4 mm to (109.0, 154.5), turned to 90 degrees
- moved R2 85.1 mm to (109.8, 152.4), turned to -90 degrees
- moved C8 84.8 mm to (110.9, 152.4), turned to 90 degrees
- moved C9 83.7 mm to (107.5, 152.4), turned to 90 degrees
- moved L1 81.4 mm to (114.7, 148.7), turned to -90 degrees
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Connections:
- net /MCU/AFE_RST renamed /connector/AFE_RST
- net /MCU/SDRAM_CAS renamed /SDRAM/SDRAM_CAS
- net /MCU/SDRAM_RAS renamed /SDRAM/SDRAM_RAS
- net /MCU/SDRAM_WE renamed /SDRAM/SDRAM_WE
- net /MCU/SD_CMD renamed /storage/SD_CMD
- net /connector/AFE_SCK renamed /MCU/LCD_SCK
- net /connector/AFE_SDATA renamed /MCU/LCD_DI
- net /connector/AFE_SL renamed /MCU/SPI_CS
- net /storage/QSPI_CLK renamed /MCU/QSPI_SCK
- net /storage/QSPI_CS renamed /MCU/QSPI_SS_B
- net /storage/SD_CD renamed /MCU/SD_CD_B
- C300 pad 1: Net-(C300-Pad1) -> +3V3
- C301 pad 1: Net-(C300-Pad1) -> +3V3
- C302 pad 1: Net-(C300-Pad1) -> +3V3
- C303 pad 1: Net-(C300-Pad1) -> +3V3
- C304 pad 1: Net-(C300-Pad1) -> +3V3
- C305 pad 1: Net-(C300-Pad1) -> +3V3
- C306 pad 1: Net-(C300-Pad1) -> +3V3
- C307 pad 1: Net-(C300-Pad1) -> +3V3
- C316 pad 1: Net-(C300-Pad1) -> +3V3
- C703 pad 1: +SYS -> GND
- C703 pad 2: GND -> +SYS
- J500 pad 5: Net-(C501-Pad1) -> GND
- J500 pad 6: Net-(C501-Pad1) -> GND
- L3 pad 2: Net-(C6-Pad1) -> +SYS
- L500 pad 1: /MCU/USB_DP -> Net-(J500-Pad3)
- L500 pad 2: Net-(J500-Pad3) -> /MCU/USB_DP
- L500 pad 3: Net-(J500-Pad2) -> /usb/USB_DM
- L500 pad 4: /usb/USB_DM -> Net-(J500-Pad2)
- L700 pad 1: Net-(L700-Pad1) -> +SYS
- L700 pad 2: /lcd/LEDA -> Net-(L700-Pad2)
- R2 pad 2: Net-(C3-Pad1) -> +3V3
- SW612 pad 1: /MCU/KO1 -> /MCU/KI0
- SW612 pad 2: /MCU/KI2 -> (no net)
- U100 pad A7: (no net) -> /MCU/AFE_SYNC
- U100 pad B7: (no net) -> /MCU/LCD_PWM
- U100 pad C1: (no net) -> /MCU/SDRAM_BA0
- U100 pad C7: /MCU/SDRAM_CS0 -> /MCU/LCD_EN
- U100 pad D12: /MCU/LCD_D17 -> (no net)
- U100 pad E1: /MCU/SDRAM_CS0 -> /SDRAM/SDRAM_CS0
- U100 pad E12: /MCU/LCD_D16 -> (no net)
- U100 pad E3: (no net) -> /MCU/SDRAM_D0
- U100 pad F1: (no net) -> /MCU/SDRAM_BA1
- U100 pad L5: /MCU/AFE_SYNC -> (no net)
- U100 pad M3: /MCU/LCD_EN -> (no net)
- U100 pad M5: /MCU/LCD_PWM -> (no net)
- U300 pad A7: Net-(C300-Pad1) -> +3V3
- U300 pad A8: GND -> /MCU/SDRAM_D0
- U300 pad A9: Net-(C300-Pad1) -> +3V3
- U300 pad B3: Net-(C300-Pad1) -> +3V3
- U300 pad C7: Net-(C300-Pad1) -> +3V3
- U300 pad D3: Net-(C300-Pad1) -> +3V3
- U300 pad E7: Net-(C300-Pad1) -> +3V3
- U300 pad G7: /SDRAM/SDRAM_BA0 -> /MCU/SDRAM_BA0
- U300 pad G8: /SDRAM/SDRAM_BA1 -> /MCU/SDRAM_BA1
- U300 pad G9: /MCU/SDRAM_CS0 -> /SDRAM/SDRAM_CS0
- U300 pad J9: Net-(C300-Pad1) -> +3V3
- U9 pad 10: Net-(C3-Pad1) -> +3V3
- U9 pad 20: Net-(C6-Pad1) -> +SYS
Routing:
- net GND: track 0.00 -> 165.0 mm, vias 0 -> 126
- net /MCU/KI0: track 0.00 -> 163.3 mm, vias 0 -> 5
- net +SYS: track 0.00 -> 152.3 mm, vias 0 -> 4
- net /MCU/KI1: track 0.00 -> 148.5 mm, vias 0 -> 5
- net /MCU/KI3: track 0.00 -> 144.7 mm, vias 0 -> 5
- net /MCU/KI2: track 0.00 -> 142.9 mm, vias 0 -> 4
- net /MCU/KO2: track 0.00 -> 139.8 mm, vias 0 -> 4
- net /MCU/LCD_SCK: track 0.00 -> 129.8 mm, vias 0 -> 2
- net /connector/AFE_RST: track 0.00 -> 116.7 mm, vias 0 -> 4
- net /MCU/KO0: track 0.00 -> 100.0 mm, vias 0 -> 2
- net VBUS: track 0.00 -> 99.0 mm, vias 0 -> 4
- net /MCU/SPI_CS: track 0.00 -> 93.4 mm, vias 0 -> 3
- net /MCU/POR: track 0.00 -> 81.5 mm, vias 0 -> 2
- net +3V3: track 0.00 -> 78.1 mm, vias 0 -> 35
- net /MCU/LCD_DI: track 0.00 -> 74.1 mm, vias 0 -> 3
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- added copper zone on In1.Cu, net +1V0
- added copper zone on In1.Cu, net +3V3
- added copper zone on B.Cu, net GND
- added copper zone on F.Cu, net GND
- added copper zone on In2.Cu, net GND
Other:
- board outline added: 100 x 68 mm
- copper layers 2 -> 4
- net class Default removed
- rule pad_to_mask_clearance: 0.05 -> 0
- board text added: "Capture Board"
- board text added: "Copyright 2021 Wenting Z."
- board text added: "Image Area"
- board text added: "SNE-PB r0.1"
- board text added: "Sitina"
- board text added: "ne"

Commit message: Bug fixes and changes for PB r0p2
Parts:
- removed C400: 10uF, Capacitor_SMD:C_0805_2012Metric
- removed C401: 100nF, Capacitor_SMD:C_0402_1005Metric
- removed Q400: 2N7002, Package_TO_SOT_SMD:SOT-23
- removed R101: 10K, Resistor_SMD:R_0402_1005Metric
- removed R201: 1K, Resistor_SMD:R_0402_1005Metric
- removed R400: 464K/1%, Resistor_SMD:R_0402_1005Metric
- removed R401, R402: 200K/1%, Resistor_SMD:R_0402_1005Metric
- removed R403: 243K/1%, Resistor_SMD:R_0402_1005Metric
- removed U400: ADP163, Package_TO_SOT_SMD:TSOT-23-5
- added C1: 0.22uF, Capacitor_SMD:C_0402_1005Metric, F.Cu at (169.6, 139.4)
- added C3: 10uF, Capacitor_SMD:C_0603_1608Metric, F.Cu at (178.2, 81.1)
- added C4: 100nF, Capacitor_SMD:C_0402_1005Metric, F.Cu at (177.8, 82.7)
- added C5: 10uF, Capacitor_SMD:C_0603_1608Metric, F.Cu at (182.5, 84.3)
- added C707: 10uF, Capacitor_SMD:C_0603_1608Metric, F.Cu at (108.8, 125.0)
- added D201: 1N5819, Diode_SMD:D_SOD-123, F.Cu at (175.8, 76.8)
- added J701: Conn_01x09, Footprints:FPC_9, B.Cu at (133.4, 117.5)
- added Q1: 2N7002, Package_TO_SOT_SMD:SOT-23, F.Cu at (180.0, 88.8)
- added R1: 30K, Resistor_SMD:R_0402_1005Metric, F.Cu at (167.6, 139.4)
- added R4: 464K/1%, Resistor_SMD:R_0402_1005Metric, F.Cu at (181.9, 86.0)
- added R5: 200K/1%, Resistor_SMD:R_0402_1005Metric, F.Cu at (177.3, 88.0)
- added R6: 200K/1%, Resistor_SMD:R_0402_1005Metric, F.Cu at (180.8, 91.2)
- added R7: 243K/1%, Resistor_SMD:R_0402_1005Metric, F.Cu at (182.5, 88.4)
- added RN700: 33R, Resistor_SMD:R_Array_Convex_4x0402, B.Cu at (166.5, 111.0)
- added RN701: 33R, Resistor_SMD:R_Array_Convex_4x0402, B.Cu at (166.5, 113.5)
- added RN702: 33R, Resistor_SMD:R_Array_Convex_4x0402, B.Cu at (166.5, 116.0)
- added RN703: 33R, Resistor_SMD:R_Array_Convex_4x0402, B.Cu at (166.5, 118.5)
- added RN704: 33R, Resistor_SMD:R_Array_Convex_4x0402, B.Cu at (166.5, 121.0)
- added SW620: TM-4175-B-B, Footprints:TM4175, F.Cu at (167.0, 70.0)
- added TP1: TestPoint_Small, TestPoint:TestPoint_Pad_D1.0mm, B.Cu at (140.0, 126.3)
- added TP2: TestPoint_Small, TestPoint:TestPoint_Pad_D1.0mm, B.Cu at (140.0, 129.5)
- added TP3: TestPoint_Small, TestPoint:TestPoint_Pad_D1.0mm, B.Cu at (143.0, 126.3)
- added TP4: TestPoint_Small, TestPoint:TestPoint_Pad_D1.0mm, B.Cu at (143.0, 129.5)
- added U1: ADP163, Package_TO_SOT_SMD:TSOT-23-5, F.Cu at (178.9, 85.2)
- C108, C316, C402, C700: footprint Capacitor_SMD:C_0805_2012Metric -> Capacitor_SMD:C_0603_1608Metric; moved to B.Cu
- C109, C119, C124, C126, C130, C132, C133, C137, C140, C142, C2, C307, C7: footprint Capacitor_SMD:C_0805_2012Metric -> Capacitor_SMD:C_0603_1608Metric
- C301, C701, C702, D1, R14, R704: moved to B.Cu
- C404, C405: value 18pF -> DNP
- J700: value TXW280064B0 -> TXW280064B0-R; moved to B.Cu
- L700: value 2.2uH -> 22uH
- SW200: value SW_DIP_x02 -> DNP; footprint Button_Switch_SMD:SW_DIP_SPSTx02_Slide_Copal_CHS-02B_W7.62mm_P1.27mm -> Button_Switch_SMD:SW_SPST_CK_RS282G05A3
- SW600, SW601, SW602, SW603, SW610, SW611: footprint Footprints:contact -> Button_Switch_SMD:SW_SPST_SKQG_WithStem
- SW612: value TM-4175-B-B -> SW_Push; footprint Footprints:TM4175 -> Button_Switch_SMD:SW_SPST_SKQG_WithStem
- U300: footprint Footprints:BGA-54_9x9_8.0x14.0mm -> Footprints:BGA-54_9x9_8.0x8.0mm
- moved J200 83.4 mm to (180.1, 69.0), turned to -90 degrees
- moved R204 81.0 mm to (182.7, 74.8), turned to 90 degrees
- moved SW612 77.8 mm to (94.0, 123.0), turned to 0 degrees
- moved R202 75.8 mm to (182.2, 106.0), turned to -90 degrees
- moved R200 74.9 mm to (181.0, 92.9), turned to 90 degrees
- moved SW200 74.8 mm to (181.6, 99.4), turned to 90 degrees
- moved R203 74.1 mm to (181.0, 106.0), turned to -90 degrees
- moved D200 73.6 mm to (178.4, 76.8), turned to -90 degrees
- moved C147 69.7 mm to (183.2, 139.6), turned to -90 degrees
- moved Y100 68.7 mm to (180.9, 138.8), turned to -90 degrees
- moved C122 68.3 mm to (176.1, 140.6), turned to 0 degrees
- moved C119 68.1 mm to (183.4, 136.3)
- moved C130 66.4 mm to (178.1, 139.1), turned to -90 degrees
- moved C128 66.3 mm to (183.1, 134.2), turned to 0 degrees
- moved C146 65.8 mm to (180.5, 136.1), turned to 0 degrees
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Connections:
- net /MCU/AFE_SYNC renamed /cb_interface/AFE_SYNC
- net /MCU/CSI_D0 renamed /cb_interface/CSI_D0
- net /MCU/CSI_D1 renamed /cb_interface/CSI_D1
- net /MCU/CSI_D10 renamed /cb_interface/CSI_D10
- net /MCU/CSI_D11 renamed /cb_interface/CSI_D11
- net /MCU/CSI_D12 renamed /cb_interface/CSI_D12
- net /MCU/CSI_D13 renamed /cb_interface/CSI_D13
- net /MCU/CSI_D2 renamed /cb_interface/CSI_D2
- net /MCU/CSI_D3 renamed /cb_interface/CSI_D3
- net /MCU/CSI_D4 renamed /cb_interface/CSI_D4
- net /MCU/CSI_D5 renamed /cb_interface/CSI_D5
- net /MCU/CSI_D6 renamed /cb_interface/CSI_D6
- net /MCU/CSI_D7 renamed /cb_interface/CSI_D7
- net /MCU/CSI_D8 renamed /cb_interface/CSI_D8
- net /MCU/CSI_D9 renamed /cb_interface/CSI_D9
- net /MCU/CSI_HSYNC renamed /cb_interface/CSI_HSYNC
- net /MCU/CSI_PCLK renamed /cb_interface/CSI_PCLK
- net /MCU/CSI_VSYNC renamed /cb_interface/CSI_VSYNC
- net /MCU/JTAG_MOD renamed /mcu/JTAG_MOD
- net /MCU/JTAG_TCK renamed /debug/JTAG_TCK
- net /MCU/JTAG_TMS renamed /debug/JTAG_TMS
- net /MCU/KO0 renamed /key/KO0
- net /MCU/LCD_EN renamed /lcd/LCD_EN
- net /MCU/ON renamed /mcu/ON
- net /MCU/POR renamed /debug/SYS_RST
- net /MCU/QSPI_D0 renamed /mcu/QSPI_D0
- net /MCU/QSPI_D1 renamed /mcu/QSPI_D1
- net /MCU/QSPI_D2 renamed /mcu/QSPI_D2
- net /MCU/QSPI_D3 renamed /mcu/QSPI_D3
- net /MCU/QSPI_SCK renamed /mcu/QSPI_SCK
- net /MCU/QSPI_SS_B renamed /mcu/QSPI_SS_B
- net /MCU/SDRAM_A0 renamed /mcu/SDRAM_A0
- net /MCU/SDRAM_A1 renamed /mcu/SDRAM_A1
- net /MCU/SDRAM_A10 renamed /mcu/SDRAM_A10
- net /MCU/SDRAM_A11 renamed /mcu/SDRAM_A11
- net /MCU/SDRAM_A12 renamed /mcu/SDRAM_A12
- net /MCU/SDRAM_A2 renamed /mcu/SDRAM_A2
- net /MCU/SDRAM_A3 renamed /mcu/SDRAM_A3
- net /MCU/SDRAM_A4 renamed /mcu/SDRAM_A4
- net /MCU/SDRAM_A5 renamed /mcu/SDRAM_A5
- net /MCU/SDRAM_A6 renamed /mcu/SDRAM_A6
- net /MCU/SDRAM_A7 renamed /mcu/SDRAM_A7
- net /MCU/SDRAM_A8 renamed /mcu/SDRAM_A8
- net /MCU/SDRAM_A9 renamed /mcu/SDRAM_A9
- net /MCU/SDRAM_BA0 renamed /mcu/SDRAM_BA0
- net /MCU/SDRAM_BA1 renamed /mcu/SDRAM_BA1
- net /MCU/SDRAM_CKE renamed /sdram/SDRAM_CKE
- net /MCU/SDRAM_CLK renamed /sdram/SDRAM_CLK
- net /MCU/SDRAM_D0 renamed /mcu/SDRAM_D0
- net /MCU/SDRAM_D1 renamed /mcu/SDRAM_D1
- net /MCU/SDRAM_D10 renamed /mcu/SDRAM_D10
- net /MCU/SDRAM_D11 renamed /mcu/SDRAM_D11
- net /MCU/SDRAM_D12 renamed /mcu/SDRAM_D12
- net /MCU/SDRAM_D13 renamed /mcu/SDRAM_D13
- net /MCU/SDRAM_D14 renamed /mcu/SDRAM_D14
- net /MCU/SDRAM_D15 renamed /mcu/SDRAM_D15
- net /MCU/SDRAM_D2 renamed /mcu/SDRAM_D2
- net /MCU/SDRAM_D3 renamed /mcu/SDRAM_D3
- net /MCU/SDRAM_D4 renamed /mcu/SDRAM_D4
- net /MCU/SDRAM_D5 renamed /mcu/SDRAM_D5
- net /MCU/SDRAM_D6 renamed /mcu/SDRAM_D6
- net /MCU/SDRAM_D7 renamed /mcu/SDRAM_D7
- net /MCU/SDRAM_D8 renamed /mcu/SDRAM_D8
- net /MCU/SDRAM_D9 renamed /mcu/SDRAM_D9
- net /MCU/SDRAM_DM0 renamed /mcu/SDRAM_DM0
- net /MCU/SDRAM_DM1 renamed /mcu/SDRAM_DM1
- net /MCU/SD_CD_B renamed /mcu/SD_CD_B
- net /MCU/SD_CLK renamed /mcu/SD_CLK
- net /MCU/SD_D0 renamed /mcu/SD_D0
- net /MCU/SD_D1 renamed /mcu/SD_D1
- net /MCU/SD_D2 renamed /mcu/SD_D2
- net /MCU/SD_D3 renamed /mcu/SD_D3
- net /MCU/USB_DP renamed /mcu/USB_DP
- net /SDRAM/SDRAM_CAS renamed /sdram/SDRAM_CAS
- net /SDRAM/SDRAM_CS0 renamed /sdram/SDRAM_CS0
- net /SDRAM/SDRAM_RAS renamed /sdram/SDRAM_RAS
- net /SDRAM/SDRAM_WE renamed /sdram/SDRAM_WE
- net /storage/SD_CMD renamed /mcu/SD_CMD
- net /usb/USB_DM renamed /mcu/USB_DN
- C402 pad 1: +VSD -> +3V3
- C403 pad 1: +VSD -> +3V3
- J1 pad 22: /MCU/SPI_CS -> /cb_interface/AFE_SL
- J1 pad 23: /MCU/LCD_DI -> /cb_interface/AFE_SDATA
- J1 pad 24: /MCU/LCD_SCK -> /cb_interface/AFE_SCK
- J1 pad 25: /connector/AFE_RST -> /cb_interface/AFE_RST
- J200 pad 1: +3V3 -> Net-(D201-Pad2)
- J200 pad 6: /MCU/JTAG_TDO -> (no net)
- J200 pad 8: /MCU/JTAG_TDI -> (no net)
- J700 pad 1: /lcd/LEDA -> GND
- J700 pad 10: GND -> /lcd/D_D13
- J700 pad 11: GND -> /lcd/D_D12
- J700 pad 12: GND -> /lcd/D_D11
- J700 pad 13: GND -> /lcd/D_D10
- J700 pad 14: /MCU/LCD_VSYNC -> /lcd/D_D9
- J700 pad 15: /MCU/LCD_HSYNC -> /lcd/D_D8
- J700 pad 16: /MCU/LCD_CLK -> /lcd/D_D7
- J700 pad 17: /MCU/LCD_DE -> /lcd/D_D6
- J700 pad 18: /MCU/LCD_D0 -> /lcd/D_D5
- J700 pad 19: /MCU/LCD_D1 -> /lcd/D_D4
- J700 pad 2: /lcd/LEDK -> +3V3
- J700 pad 20: /MCU/LCD_D2 -> /lcd/D_D3
- J700 pad 21: /MCU/LCD_D3 -> /lcd/D_D2
- J700 pad 22: /MCU/LCD_D4 -> /lcd/D_D1
- J700 pad 23: /MCU/LCD_D5 -> /lcd/D_D0
- J700 pad 24: /MCU/LCD_D6 -> /lcd/D_DE
- J700 pad 25: /MCU/LCD_D7 -> /lcd/D_DCLK
- J700 pad 26: /MCU/LCD_D8 -> /lcd/D_HSYNC
- J700 pad 27: /MCU/LCD_D9 -> /lcd/D_VSYNC
- J700 pad 28: /MCU/LCD_D10 -> GND
- J700 pad 29: /MCU/LCD_D11 -> GND
- J700 pad 3: +3V3 -> GND
- J700 pad 30: /MCU/LCD_D12 -> GND
- J700 pad 31: /MCU/LCD_D13 -> GND
- J700 pad 32: /MCU/LCD_D14 -> GND
- J700 pad 33: /MCU/LCD_D15 -> GND
- J700 pad 34: /connector/AFE_RST -> GND
- J700 pad 35: /MCU/LCD_CS -> GND
- J700 pad 36: /MCU/LCD_SCK -> GND
- J700 pad 37: /MCU/LCD_DI -> GND
- J700 pad 38: GND -> +3V3
- J700 pad 39: +3V3 -> /lcd/LEDK
- J700 pad 4: GND -> /cb_interface/AFE_SDATA
- J700 pad 40: GND -> /lcd/LEDA
- J700 pad 5: GND -> /cb_interface/AFE_SCK
- J700 pad 6: GND -> /lcd/LCD_CSN
- J700 pad 7: GND -> /cb_interface/AFE_RST
- J700 pad 8: GND -> /lcd/D_D15
- J700 pad 9: GND -> /lcd/D_D14
- MICRO_SD400 pad 4: +VSD -> +3V3
- R100 pad 1: +3V3 -> +VRTC
- R13 pad 1: Net-(R13-Pad1) -> VBUS
- R202 pad 1: /MCU/BOOT0 -> /debug/BOOT0
- R203 pad 1: /MCU/BOOT1 -> /debug/BOOT1
- R405 pad 1: +VSD -> +3V3
- R406 pad 1: +VSD -> +3V3
- R701 pad 2: /MCU/LCD_PWM -> /lcd/LCD_PWM
- SW200 pad 1: /MCU/BOOT1 -> /debug/BOOT0
- SW200 pad 2: /MCU/BOOT0 -> Net-(R200-Pad1)
- SW600 pad 2: /MCU/KI0 -> /key/KI0
- SW601 pad 2: /MCU/KI1 -> /key/KI1
- SW602 pad 2: /MCU/KI2 -> /key/KI2
- SW603 pad 2: /MCU/KI3 -> /key/KI3
- SW610 pad 1: /MCU/KO1 -> /key/KO1
- SW610 pad 2: /MCU/KI0 -> /key/KI0
- SW611 pad 1: /MCU/KO1 -> /key/KO1
- SW611 pad 2: /MCU/KI1 -> /key/KI1
- SW612 pad 1: /MCU/KI0 -> /key/KO1
- SW612 pad 2: (no net) -> /key/KI2
- TH1 pad 1: Net-(R13-Pad1) -> VBUS
- U100 pad A10: /MCU/LCD_D7 -> /lcd/LCD_D7
- U100 pad A11: /MCU/LCD_D12 -> /lcd/LCD_D12
- U100 pad A8: /MCU/LCD_D2 -> /lcd/LCD_D2
- U100 pad A9: /MCU/LCD_D3 -> /lcd/LCD_D3
- U100 pad B11: /MCU/LCD_D13 -> /lcd/LCD_D13
- U100 pad B14: /MCU/LCD_CS -> /lcd/LCD_CSN
- U100 pad B7: /MCU/LCD_PWM -> (no net)
- U100 pad B8: /MCU/LCD_D1 -> /lcd/LCD_D1
- U100 pad B9: /MCU/LCD_D4 -> /lcd/LCD_D4
- U100 pad C10: /MCU/LCD_D8 -> /lcd/LCD_D8
- U100 pad C11: /MCU/LCD_D14 -> /lcd/LCD_D14
- U100 pad C8: /MCU/LCD_D0 -> /lcd/LCD_D0
- U100 pad C9: /MCU/LCD_D5 -> /lcd/LCD_D5
- U100 pad D10: /MCU/LCD_D9 -> /lcd/LCD_D9
- U100 pad D11: /MCU/LCD_D15 -> /lcd/LCD_D15
- U100 pad D7: /MCU/LCD_CLK -> /lcd/LCD_CLK
- U100 pad D8: /MCU/LCD_VSYNC -> /lcd/LCD_VSYNC
- U100 pad D9: /MCU/LCD_D6 -> /lcd/LCD_D6
- U100 pad E10: /MCU/LCD_D10 -> /lcd/LCD_D10
- U100 pad E11: /MCU/LCD_D11 -> /lcd/LCD_D11
- U100 pad E7: /MCU/LCD_DE -> /lcd/LCD_DE
- U100 pad E8: /MCU/LCD_HSYNC -> /lcd/LCD_HSYNC
- U100 pad F11: /MCU/BOOT1 -> /debug/BOOT0
- U100 pad F14: /MCU/JTAG_TDI -> /grip_interface/USER1
- U100 pad G10: /MCU/JTAG_TRSTB -> (no net)
- U100 pad G11: /MCU/BOOT0 -> /cb_interface/AFE_RST
- U100 pad G13: /MCU/JTAG_TDO -> /grip_interface/USER2
- U100 pad G14: /connector/AFE_RST -> /debug/BOOT1
- U100 pad H10: /MCU/LCD_DI -> /cb_interface/AFE_SDATA
- U100 pad J11: /MCU/KO2 -> /key/KO2
- U100 pad J12: /MCU/KI2 -> /key/KI2
- U100 pad K10: /MCU/KI3 -> /key/KI3
- U100 pad K11: /MCU/SD_VSELECT -> /mcu/SD_VSELECT
- U100 pad K12: /MCU/KI1 -> /key/KI1
- U100 pad K14: (no net) -> /cb_interface/AFE_SL
- U100 pad K3: +3V3 -> Net-(C1-Pad1)
- U100 pad L10: /MCU/KO1 -> /key/KO1
- U100 pad L12: /MCU/KI0 -> /key/KI0
- U100 pad L14: (no net) -> /lcd/LCD2_CS
- U100 pad M11: /MCU/SPI_CS -> /lcd/LCD2_RS
- U100 pad M12: /MCU/SD_PWR_EN -> /grip_interface/SHUTTER
- U100 pad M14: /MCU/LCD_SCK -> /cb_interface/AFE_SCK
- U100 pad M3: (no net) -> /mcu/I2C_SCL
- U100 pad M5: (no net) -> /lcd/LCD_PWM
- U100 pad M6: (no net) -> /grip_interface/ONOFF
- U100 pad N3: /MCU/I2C_SDA -> (no net)
- U100 pad P2: /MCU/I2C_SCL -> /mcu/I2C_SDA
- U9 pad 13: /MCU/I2C_SCL -> /mcu/I2C_SCL
- U9 pad 14: /MCU/I2C_SDA -> /mcu/I2C_SDA
- U9 pad 3: Net-(R13-Pad1) -> VBUS
Routing:
- net /key/KI3: track 0.00 -> 203.8 mm, vias 0 -> 5
- net /key/KI0: track 0.00 -> 170.5 mm, vias 0 -> 4
- net /cb_interface/AFE_SDATA: track 0.00 -> 168.3 mm, vias 0 -> 6
- net /MCU/KI0: track 163.3 -> 0.00 mm, vias 5 -> 0
- net /key/KI1: track 0.00 -> 161.1 mm, vias 0 -> 5
- net /MCU/KI1: track 148.5 -> 0.00 mm, vias 5 -> 0
- net /key/KO2: track 0.00 -> 148.3 mm, vias 0 -> 4
- net /key/KI2: track 0.00 -> 148.0 mm, vias 0 -> 4
- net /MCU/KI3: track 144.7 -> 0.00 mm, vias 5 -> 0
- net /MCU/KI2: track 142.9 -> 0.00 mm, vias 4 -> 0
- net /MCU/KO2: track 139.8 -> 0.00 mm, vias 4 -> 0
- net /cb_interface/AFE_SCK: track 0.00 -> 131.0 mm, vias 0 -> 5
- net /MCU/LCD_SCK: track 129.8 -> 0.00 mm, vias 2 -> 0
- net /cb_interface/AFE_RST: track 0.00 -> 129.1 mm, vias 0 -> 3
- net /connector/AFE_RST: track 116.7 -> 0.00 mm, vias 4 -> 0
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Other:
- board size 100 x 68 mm -> 97 x 79.5 mm
- board text added: "SNE Processor Board r0.2"
- board text removed: "SNE-PB r0.1"

Commit message: pcb: switch to ad9978 wip
Parts:
- moved C3 96.1 mm to (102.5, 140.2), turned to 90 degrees
- moved C4 93.8 mm to (104.1, 140.6), turned to 90 degrees
- moved C5 92.5 mm to (105.7, 135.9), turned to 90 degrees
- moved U1 90.5 mm to (106.6, 139.5), turned to 90 degrees
- moved R4 90.1 mm to (107.4, 136.5), turned to 0 degrees
- moved R7 86.8 mm to (109.8, 135.9), turned to 0 degrees
- moved R5 86.2 mm to (109.5, 141.1), turned to 0 degrees
- moved Q1 85.6 mm to (110.2, 138.5), turned to -90 degrees
- moved R6 82.5 mm to (112.6, 137.6), turned to -90 degrees
- moved C402 62.9 mm to (105.4, 81.6)
- moved R13 11.4 mm to (91.2, 138.9)
- moved TH1 11.4 mm to (91.7, 140.3)
- moved C8 5.56 mm to (94.4, 129.1)
- moved R3 5.56 mm to (93.3, 129.1)
- moved R2 5.56 mm to (95.5, 129.1)
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Connections:
- net /mcu/SD_CLK renamed /storage/SD_CLK
- net /sdram/SDRAM_CAS renamed /mcu/SDRAM_CAS
- net /sdram/SDRAM_CKE renamed /mcu/SDRAM_CKE
- net /sdram/SDRAM_CS0 renamed /mcu/SDRAM_CS0
- J1 pad 25: /cb_interface/AFE_RST -> (no net)
- J1 pad 26: /cb_interface/AFE_SYNC -> (no net)
- J700 pad 7: /cb_interface/AFE_RST -> /lcd/LCD_RST
- J701 pad 2: /cb_interface/AFE_RST -> /lcd/LCD_RST
- R13 pad 1: VBUS -> Net-(R13-Pad1)
- SW620 pad 2: unconnected-(SW620-Pad2) -> /key/KO1
- TH1 pad 1: VBUS -> Net-(R13-Pad1)
- U100 pad A7: /cb_interface/AFE_SYNC -> (no net)
- U100 pad G11: /cb_interface/AFE_RST -> /lcd/LCD_RST
- U9 pad 3: VBUS -> Net-(R13-Pad1)
Routing:
- net /cb_interface/AFE_RST: track 129.1 -> 0.00 mm, vias 3 -> 0
- net /lcd/LCD_RST: track 0.00 -> 108.0 mm, vias 0 -> 3
- net /grip_interface/USER2: track 82.7 -> 182.3 mm, vias 1 -> 3
- net /grip_interface/USER1: track 66.1 -> 164.2 mm, vias 1 -> 3
- net /key/KO1: track 106.0 -> 202.5 mm, vias 2 -> 5
- net /grip_interface/SHUTTER: track 1.96 -> 72.8 mm, vias 0 -> 3
- net +VSD: track 22.1 -> 86.0 mm
- net /debug/JTAG_TCK: track 9.30 -> 58.0 mm, vias 1 -> 2
- net /lcd/LEDA: track 3.05 -> 49.8 mm, vias 0 -> 1
- net Net-(C706-Pad2): track 3.68 -> 49.9 mm
- net /cb_interface/AFE_SYNC: track 44.6 -> 0.00 mm, vias 1 -> 0
- net /lcd/LEDK: track 0.87 -> 45.5 mm, vias 0 -> 1
- net /grip_interface/ONOFF: track 36.3 -> 50.8 mm, vias 1 -> 3
- net Net-(D201-Pad2): track 0.00 -> 14.1 mm
- net GND: track 128.1 -> 116.1 mm
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Other:
- board text added: "Length-match the SD card traces!!!!"

Commit message: pcb: finish routing PB 0.2
Parts:
- moved R14 1.69 mm to (91.7, 107.0), turned to 0 degrees
- moved C402 0.98 mm to (106.4, 81.6)
- moved R13 0.18 mm to (91.1, 138.7)
- moved TH1 0.18 mm to (91.7, 140.1)
- moved R4 0.12 mm to (107.5, 136.5)
- turned D1 to 0 degrees
Routing:
- net +VRTC: track 49.9 -> 135.4 mm, vias 2 -> 6
- net +SYS: track 90.1 -> 168.4 mm, vias 2 -> 5
- net /lcd/LCD_EN: track 1.65 -> 77.1 mm, vias 0 -> 2
- net /debug/SYS_RST: track 8.95 -> 83.2 mm, vias 2 -> 4
- net /key/KI2: track 148.0 -> 222.1 mm, vias 4 -> 5
- net /key/KO2: track 148.3 -> 83.7 mm, vias 4 -> 2
- net /mcu/I2C_SDA: track 24.3 -> 83.5 mm, vias 2 -> 4
- net /mcu/I2C_SCL: track 27.2 -> 85.0 mm, vias 2 -> 4
- net /mcu/ON: track 44.3 -> 98.5 mm
- net /key/KI1: track 161.2 -> 209.9 mm
- net /key/KO1: track 202.5 -> 245.8 mm
- net /key/KO0: track 161.2 -> 203.0 mm
- net /key/KI0: track 170.6 -> 207.4 mm, vias 4 -> 5
- net VBUS: track 130.4 -> 166.8 mm, vias 3 -> 5
- net Net-(D1-Pad1): track 0.85 -> 36.2 mm, vias 0 -> 1
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Other:
- board text removed: "Length-match the SD card traces!!!!"

Commit message: pcb: PB r0p2 and CB r0p3 freeze
Connections:
- net /mcu/SDRAM_CAS renamed /sdram/SDRAM_CAS
- net /mcu/SDRAM_CKE renamed /sdram/SDRAM_CKE
- net /mcu/SDRAM_CS0 renamed /sdram/SDRAM_CS0
- net /mcu/SD_CMD renamed /storage/SD_CMD
- net /mcu/USB_DN renamed /usb/USB_DM
- net /mcu/USB_DP renamed /usb/USB_DP
- J1 pad 17: /cb_interface/CSI_VSYNC -> /cb_interface/CSI_PCLK
- J1 pad 18: /cb_interface/CSI_HSYNC -> GND
- J1 pad 19: GND -> /cb_interface/CSI_VSYNC
- J1 pad 20: /cb_interface/CSI_PCLK -> /cb_interface/CSI_HSYNC
- J1 pad 23: /cb_interface/AFE_SDATA -> /cb_interface/AFE_SCK
- J1 pad 24: /cb_interface/AFE_SCK -> /cb_interface/AFE_RST
- J1 pad 25: (no net) -> unconnected-(J1-Pad25)
- J1 pad 26: (no net) -> /cb_interface/AFE_SDATA
- J200 pad 6: (no net) -> unconnected-(J200-Pad6)
- J200 pad 7: (no net) -> unconnected-(J200-Pad7)
- J200 pad 8: (no net) -> unconnected-(J200-Pad8)
- J200 pad 9: (no net) -> unconnected-(J200-Pad9)
- J500 pad 4: (no net) -> unconnected-(J500-Pad4)
- J700 pad 7: /lcd/LCD_RST -> /cb_interface/AFE_RST
- J701 pad 2: /lcd/LCD_RST -> /cb_interface/AFE_RST
- J701 pad 8: (no net) -> unconnected-(J701-Pad8)
- J701 pad 9: (no net) -> unconnected-(J701-Pad9)
- U100 pad A7: (no net) -> unconnected-(U100-PadA7)
- U100 pad B7: (no net) -> /mcu/SDRAM_DQS
- U100 pad D12: (no net) -> /lcd/LCD_D17
- U100 pad E12: (no net) -> /lcd/LCD_D16
- U100 pad G10: (no net) -> /mcu/JTAG_TRSTB
- U100 pad G11: /lcd/LCD_RST -> /cb_interface/AFE_RST
- U100 pad L5: (no net) -> unconnected-(U100-PadL5)
- U100 pad L6: (no net) -> unconnected-(U100-PadL6)
- U100 pad L7: (no net) -> unconnected-(U100-PadL7)
- U100 pad M4: (no net) -> unconnected-(U100-PadM4)
- U100 pad N10: (no net) -> unconnected-(U100-PadN10)
- U100 pad N12: (no net) -> unconnected-(U100-PadN12)
- U100 pad N13: (no net) -> unconnected-(U100-PadN13)
- U100 pad N3: (no net) -> /mcu/QSPI_DQS
- U100 pad N7: (no net) -> unconnected-(U100-PadN7)
- U100 pad P13: (no net) -> unconnected-(U100-PadP13)
- U100 pad P6: (no net) -> unconnected-(U100-PadP6)
- U100 pad P7: (no net) -> unconnected-(U100-PadP7)
- U300 pad E2: (no net) -> unconnected-(U300-PadE2)
- U500 pad 5: (no net) -> unconnected-(U500-Pad5)
- U9 pad 18: (no net) -> unconnected-(U9-Pad18)
- U9 pad 23: (no net) -> unconnected-(U9-Pad23)
Routing:
- net /cb_interface/AFE_RST: track 0.00 -> 137.2 mm, vias 0 -> 5
- net /lcd/LCD_RST: track 108.0 -> 0.00 mm, vias 3 -> 0
- net +SYS: track 168.4 -> 162.4 mm
- net /cb_interface/CSI_PCLK: track 37.2 -> 34.4 mm
- net /cb_interface/CSI_VSYNC: track 33.8 -> 36.2 mm
- net /mcu/ON: track 98.5 -> 100.8 mm
- net /lcd/LCD_EN: track 77.1 -> 75.0 mm
- net /cb_interface/CSI_HSYNC: track 34.3 -> 35.9 mm
- net /cb_interface/AFE_SDATA: track 167.8 -> 166.6 mm
- net /lcd/LCD_CSN: track 82.4 -> 81.5 mm
- net /cb_interface/AFE_SCK: track 131.4 -> 130.5 mm
- net /key/KI2: track 222.1 -> 221.4 mm
- net +VRTC: track 135.4 -> 136.1 mm
- net /cb_interface/CSI_D2: track 24.1 -> 23.6 mm
- net /debug/JTAG_TCK: track 58.0 -> 58.5 mm
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