File: Hardware/ProcessingBoard/Sitina.kicad_sch (KiCad schematic)
At the start: 0 parts

Commit message: pcb: bug fixes for PB r0.2
Other:
- note added: "Changelog: r0.1: 1. Initial version r0.2: 1. Add R/C delay for DCDC PSWITCH 2. Fix boot mode selection pin 3. Remove incorrect pull-up for RESET line 4. Move LCD_PWM from EMC_39 to SD_B1_01 EMC_39 is now reserved for SEMC DQS 5. Move I2C_SDA from SD_B1_04 to SD_B1_02 6. Move I2C_SCL from SD_B1_05 to SD_B1_03 SD_B1_05 is now reserved for SPI DQS Forced to use software I2C"
Changed lines of the file:
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@@
+    (effects (font (size 1.27 1.27)) (justify left bottom))
+  )
+  (text "Changelog:\nr0.1:\n1. Initial version\nr0.2:\n1. Add R/C delay for DCDC PSWITCH\n2. Fix boot mode selection pin\n3. Remove incorrect pull-up for RESET line\n4. Move LCD_PWM from EMC_39 to SD_B1_01\n   EMC_39 is now reserved for SEMC DQS\n5. Move I2C_SDA from SD_B1_04 to SD_B1_02\n6. Move I2C_SCL from SD_B1_05 to SD_B1_03\n   SD_B1_05 is now reserved for SPI DQS\n   Forced to use software I2C"
+    (at 213.36 53.34 0)
     (effects (font (size 1.27 1.27)) (justify left bottom))
   )
@@
       (reference "#PWR0149") (unit 1) (value "+3V3") (footprint "")
     )
+    (path "/00000000-0000-0000-0000-00005d0408df/4bac5e56-63ee-4fe4-aac0-11875615cfd5"
+      (reference "#PWR?") (unit 1) (value "+3V3") (footprint "")
+    )
+    (path "/00000000-0000-0000-0000-00005d0408df/f578e944-931e-4904-a84a-99b6a9a0b8a3"
+      (reference "#PWR?") (unit 1) (value "GND") (footprint "")
+    )
     (path "/00000000-0000-0000-0000-00005d0408df/00000000-0000-0000-0000-00005d2d9f87"
       (reference "C100") (unit 1) (value "0.22uF") (footprint "Capacitor_SMD:C_0402_1005Metric")
@@
       (reference "C149") (unit 1) (value "18pF") (footprint "Capacitor_SMD:C_0402_1005Metric")
     )
+    (path "/00000000-0000-0000-0000-00005d0408df/d97e3bae-6bed-4d11-98c7-f39778284ece"
+      (reference "C?") (unit 1) (value "0.22uF") (footprint "Capacitor_SMD:C_0402_1005Metric")
+    )
     (path "/00000000-0000-0000-0000-00005d0408df/00000000-0000-0000-0000-00005d5d3b8f"
       (reference "L100") (unit 1) (value "4.7uH") (footprint "Inductor_SMD:L_Vishay_IHLP-1212")
@@
       (reference "R102") (unit 1) (value "10K") (footprint "Resistor_SMD:R_0402_1005Metric")
     )
+    (path "/00000000-0000-0000-0000-00005d0408df/5b9ee988-070f-486d-80f3-e7b79475c248"
+      (reference "R?") (unit 1) (value "30K") (footprint "Resistor_SMD:R_0402_1005Metric")
+    )
+    (path "/00000000-0000-0000-0000-00005d0408df/44a47b70-f6f6-475d-abbb-f42848cdf26b"
+      (reference "TP?") (unit 1) (value "TestPoint_Small") (footprint "")
+    )
+    (path "/00000000-0000-0000-0000-00005d0408df/bc65f4f9-cb45-49aa-973b-51008514c06b"
+      (reference "TP?") (unit 1) (value "TestPoint_Small") (footprint "")
+    )
     (path "/00000000-0000-0000-0000-00005d0408df/00000000-0000-0000-0000-00005d5d6758"

Commit message: Bug fixes and changes for PB r0p2
Other:
- sheet MCU renamed mcu
- sheet SDRAM renamed sdram
- sheet connector renamed cb_interface
- added sheet grip_interface (grip_interface.kicad_sch)
- sheet cb_interface: file connector.kicad_sch -> cb_interface.kicad_sch
- sheet debug ports: added none; removed JTAG_TDI, JTAG_TDO
- sheet lcd ports: added LCD2_CS, LCD2_RS; removed none
- sheet mcu ports: added LCD2_CS, LCD2_RS, SHUTTER, USER1, USER2; removed JTAG_TDI, JTAG_TDO, POR, SD_PWR_EN
- sheet power ports: added SD_VSELECT; removed none
- sheet storage ports: added none; removed SD_PWR_EN, SD_VSELECT
- note added: "Changelog: r0.1: 1. Initial version r0.2: 1. Add R/C delay for DCDC PSWITCH 2. Fix boot mode selection pin 3. Fix incorrect pull-up for RESET line 4. Move LCD_PWM from EMC_39 to SD_B1_01 EMC_39 is now reserved for SEMC DQS 5. Move I2C_SDA from SD_B1_04 to SD_B1_02 6. Move I2C_SCL from SD_B1_05 to SD_B1_03 SD_B1_05 is now reserved for SPI DQS Forced to use software I2C 7. Fix incorrect SD power su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"
- note removed: "Changelog: r0.1: 1. Initial version r0.2: 1. Add R/C delay for DCDC PSWITCH 2. Fix boot mode selection pin 3. Remove incorrect pull-up for RESET line 4. Move LCD_PWM from EMC_39 to SD_B1_01 EMC_39 is now reserved for SEMC DQS 5. Move I2C_SDA from SD_B1_04 to SD_B1_02 6. Move I2C_SCL from SD_B1_05 to SD_B1_03 SD_B1_05 is now reserved for SPI DQS Forced to use software I2C"
- company: ZephRay -> Wenting
- title: Sitina Ne -> SitinaNe

Commit message: pcb: switch to ad9978 wip
Other:
- sheet cb_interface ports: added none; removed AFE_RST, AFE_SYNC
- sheet mcu ports: added none; removed AFE_RST, AFE_SYNC

Commit message: pcb: PB r0p2 and CB r0p3 freeze
Other:
- sheet cb_interface ports: added AFE_RST; removed none
- sheet mcu ports: added AFE_RST, POR; removed none
