File: Hardware/ProcessingBoard/cb_interface.kicad_sch (KiCad schematic)
At the start: 1 part, among them J1 Conn_01x30_MountingPin

Commit message: Bug fixes and changes for PB r0p2
Other:
- company: (none) -> Wenting
- title: (none) -> SitinaNe
Changed lines of the file:
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@@
 (kicad_sch (version 20210126) (generator eeschema)
   (paper "A4")
+  (title_block
+    (title "SitinaNe")
+    (rev "R0.2")
+    (company "Wenting")
+  )
   (junction (at 152.4 134.62) (diameter 0.9144) (color 0 0 0 0))
   (junction (at 154.94 101.6) (diameter 0.9144) (color 0 0 0 0))
@@
     (stroke (width 0) (type solid) (color 0 0 0 0))
   )
-  (bus (pts (xy 139.7 60.96) (xy 139.7 96.52))
-    (stroke (width 0) (type solid) (color 0 0 0 0))
-  )
+  (bus (pts (xy 139.7 60.96) (xy 139.7 63.5))
+    (stroke (width 0) (type solid) (color 0 0 0 0))
+  )
+  (bus (pts (xy 139.7 63.5) (xy 139.7 66.04))
+    (stroke (width 0) (type solid) (color 0 0 0 0))
+  )
+  (bus (pts (xy 139.7 66.04) (xy 139.7 68.58))
+    (stroke (width 0) (type solid) (color 0 0 0 0))
+  )
+  (bus (pts (xy 139.7 68.58) (xy 139.7 71.12))
+    (stroke (width 0) (type solid) (color 0 0 0 0))
+  )
+  (bus (pts (xy 139.7 71.12) (xy 139.7 73.66))
+    (stroke (width 0) (type solid) (color 0 0 0 0))
+  )
+  (bus (pts (xy 139.7 73.66) (xy 139.7 76.2))
+    (stroke (width 0) (type solid) (color 0 0 0 0))
+  )
+  (bus (pts (xy 139.7 76.2) (xy 139.7 78.74))
+    (stroke (width 0) (type solid) (color 0 0 0 0))
+  )
+  (bus (pts (xy 139.7 78.74) (xy 139.7 81.28))
+    (stroke (width 0) (type solid) (color 0 0 0 0))
+  )
+  (bus (pts (xy 139.7 81.28) (xy 139.7 83.82))
+    (stroke (width 0) (type solid) (color 0 0 0 0))
+  )
+  (bus (pts (xy 139.7 83.82) (xy 139.7 86.36))
+    (stroke (width 0) (type solid) (color 0 0 0 0))
+  )
+  (bus (pts (xy 139.7 86.36) (xy 139.7 88.9))
+    (stroke (width 0) (type solid) (color 0 0 0 0))
+  )
+  (bus (pts (xy 139.7 88.9) (xy 139.7 91.44))
+    (stroke (width 0) (type solid) (color 0 0 0 0))
+  )
+  (bus (pts (xy 139.7 91.44) (xy 139.7 93.98))
+    (stroke (width 0) (type solid) (color 0 0 0 0))
+  )
+  (bus (pts (xy 139.7 93.98) (xy 139.7 96.52))
+    (stroke (width 0) (type solid) (color 0 0 0 0))
+  )

Commit message: pcb: switch to ad9978 wip
Connections:
- net AFE_RST: no longer names the net of J1.25 (Pin_25)
- net AFE_SYNC: no longer names the net of J1.26 (Pin_26)
- no-connect marks 0 -> 2
Changed lines of the file:
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@@
-(kicad_sch (version 20210126) (generator eeschema)
+(kicad_sch (version 20210621) (generator eeschema)
   (paper "A4")
   (title_block
@@
   (junction (at 154.94 129.54) (diameter 0.9144) (color 0 0 0 0))
   (junction (at 162.56 142.24) (diameter 0.9144) (color 0 0 0 0))
+  (no_connect (at 157.48 124.46))
+  (no_connect (at 157.48 127))
   (bus_entry (at 139.7 63.5) (size 2.54 2.54)
     (stroke (width 0.1524) (type solid) (color 0 0 0 0))
@@
     (stroke (width 0) (type solid) (color 0 0 0 0))
   )
-  (wire (pts (xy 137.16 124.46) (xy 157.48 124.46))
-    (stroke (width 0) (type solid) (color 0 0 0 0))
-  )
-  (wire (pts (xy 137.16 127) (xy 157.48 127))
-    (stroke (width 0) (type solid) (color 0 0 0 0))
-  )
   (wire (pts (xy 142.24 66.04) (xy 157.48 66.04))
     (stroke (width 0) (type solid) (color 0 0 0 0))
@@
     (stroke (width 0) (type solid) (color 0 0 0 0))
   )
-  (bus (pts (xy 139.7 60.96) (xy 139.7 63.5))
-    (stroke (width 0) (type solid) (color 0 0 0 0))
-  )
-  (bus (pts (xy 139.7 63.5) (xy 139.7 66.04))
-    (stroke (width 0) (type solid) (color 0 0 0 0))
-  )
-  (bus (pts (xy 139.7 66.04) (xy 139.7 68.58))
-    (stroke (width 0) (type solid) (color 0 0 0 0))
-  )
-  (bus (pts (xy 139.7 68.58) (xy 139.7 71.12))
-    (stroke (width 0) (type solid) (color 0 0 0 0))
-  )
-  (bus (pts (xy 139.7 71.12) (xy 139.7 73.66))
-    (stroke (width 0) (type solid) (color 0 0 0 0))
-  )
-  (bus (pts (xy 139.7 73.66) (xy 139.7 76.2))
-    (stroke (width 0) (type solid) (color 0 0 0 0))
-  )
-  (bus (pts (xy 139.7 76.2) (xy 139.7 78.74))
-    (stroke (width 0) (type solid) (color 0 0 0 0))
-  )
-  (bus (pts (xy 139.7 78.74) (xy 139.7 81.28))
-    (stroke (width 0) (type solid) (color 0 0 0 0))
-  )
-  (bus (pts (xy 139.7 81.28) (xy 139.7 83.82))
-    (stroke (width 0) (type solid) (color 0 0 0 0))
-  )
-  (bus (pts (xy 139.7 83.82) (xy 139.7 86.36))
-    (stroke (width 0) (type solid) (color 0 0 0 0))
-  )
-  (bus (pts (xy 139.7 86.36) (xy 139.7 88.9))
-    (stroke (width 0) (type solid) (color 0 0 0 0))
-  )
-  (bus (pts (xy 139.7 88.9) (xy 139.7 91.44))
-    (stroke (width 0) (type solid) (color 0 0 0 0))
-  )
-  (bus (pts (xy 139.7 91.44) (xy 139.7 93.98))
-    (stroke (width 0) (type solid) (color 0 0 0 0))
-  )
-  (bus (pts (xy 139.7 93.98) (xy 139.7 96.52))
+  (bus (pts (xy 139.7 60.96) (xy 139.7 96.52))
     (stroke (width 0) (type solid) (color 0 0 0 0))
   )
@@
     (effects (font (size 1.27 1.27)) (justify left bottom))
   )
-  (label "AFE_RST" (at 142.24 124.46 0)
-    (effects (font (size 1.27 1.27)) (justify left bottom))
-  )
-  (label "AFE_SYNC" (at 142.24 127 0)
-    (effects (font (size 1.27 1.27)) (justify left bottom))
-  )
   (hierarchical_label "CSI_D[13..0]" (shape output) (at 137.16 60.96 180)
     (effects (font (size 1.27 1.27)) (justify right))
@@
     (effects (font (size 1.27 1.27)) (justify right))
   )
-  (hierarchical_label "AFE_RST" (shape input) (at 137.16 124.46 180)
-    (effects (font (size 1.27 1.27)) (justify right))
-  )
-  (hierarchical_label "AFE_SYNC" (shape input) (at 137.16 127 180)
-    (effects (font (size 1.27 1.27)) (justify right))
-  )

Commit message: pcb: PB r0p2 and CB r0p3 freeze
Connections:
- net AFE_SCK: now also J1.23 (Pin_23); no longer J1.24 (Pin_24)
- net AFE_SDATA: now also J1.26 (Pin_26); no longer J1.23 (Pin_23)
- net CSI_HSYNC: now also J1.20 (Pin_20); no longer J1.18 (Pin_18)
- net CSI_PCLK: now also J1.17 (Pin_17); no longer J1.20 (Pin_20)
- net CSI_VSYNC: now also J1.19 (Pin_19); no longer J1.17 (Pin_17)
- net GND: now also J1.18 (Pin_18); no longer J1.19 (Pin_19)
- new net AFE_RST: J1.24 (Pin_24)
- no-connect marks 2 -> 1
