File: Hardware/ProcessingBoard/lcd.kicad_sch (KiCad schematic)
At the start: 15 parts, among them J700 TXW280064B0, U700 CAT4139

Commit message: Update License to match source code; test and fix USB, SEMC, and XIP on actual hardware
Changed lines of the file:
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@@
     (stroke (width 0) (type solid) (color 0 0 0 0))
   )
-  (bus (pts (xy 86.36 86.36) (xy 86.36 88.9))
+  (bus (pts (xy 86.36 86.36) (xy 86.36 127))
     (stroke (width 0) (type solid) (color 0 0 0 0))
   )
-  (bus (pts (xy 86.36 88.9) (xy 86.36 91.44))
-    (stroke (width 0) (type solid) (color 0 0 0 0))
-  )
-  (bus (pts (xy 86.36 91.44) (xy 86.36 93.98))
-    (stroke (width 0) (type solid) (color 0 0 0 0))
-  )
-  (bus (pts (xy 86.36 93.98) (xy 86.36 96.52))
-    (stroke (width 0) (type solid) (color 0 0 0 0))
-  )
-  (bus (pts (xy 86.36 96.52) (xy 86.36 99.06))
-    (stroke (width 0) (type solid) (color 0 0 0 0))
-  )
-  (bus (pts (xy 86.36 99.06) (xy 86.36 101.6))
-    (stroke (width 0) (type solid) (color 0 0 0 0))
-  )
-  (bus (pts (xy 86.36 101.6) (xy 86.36 104.14))
-    (stroke (width 0) (type solid) (color 0 0 0 0))
-  )
-  (bus (pts (xy 86.36 104.14) (xy 86.36 106.68))
-    (stroke (width 0) (type solid) (color 0 0 0 0))
-  )
-  (bus (pts (xy 86.36 106.68) (xy 86.36 109.22))
-    (stroke (width 0) (type solid) (color 0 0 0 0))
-  )
-  (bus (pts (xy 86.36 109.22) (xy 86.36 111.76))
-    (stroke (width 0) (type solid) (color 0 0 0 0))
-  )
-  (bus (pts (xy 86.36 111.76) (xy 86.36 114.3))
-    (stroke (width 0) (type solid) (color 0 0 0 0))
-  )
-  (bus (pts (xy 86.36 114.3) (xy 86.36 116.84))
-    (stroke (width 0) (type solid) (color 0 0 0 0))
-  )
-  (bus (pts (xy 86.36 116.84) (xy 86.36 119.38))
-    (stroke (width 0) (type solid) (color 0 0 0 0))
-  )
-  (bus (pts (xy 86.36 119.38) (xy 86.36 121.92))
-    (stroke (width 0) (type solid) (color 0 0 0 0))
-  )
-  (bus (pts (xy 86.36 121.92) (xy 86.36 124.46))
-    (stroke (width 0) (type solid) (color 0 0 0 0))
-  )
-  (bus (pts (xy 86.36 124.46) (xy 86.36 127))
-    (stroke (width 0) (type solid) (color 0 0 0 0))
-  )

Commit message: Bug fixes and changes for PB r0p2
Parts:
- removed J700: TXW280064B0, Connector_FFC-FPC:Hirose_FH12-40S-0.5SH_1x40-1MP_P0.50mm_Horizontal, symbol Sitina:TXW280064B0
- added C707: 10uF, Capacitor_SMD:C_0603_1608Metric, symbol Device:C
- added J700: TXW280064B0-R, Connector_FFC-FPC:Hirose_FH12-40S-0.5SH_1x40-1MP_P0.50mm_Horizontal, symbol Sitina:TXW280064B0-R
- added J701: Conn_01x09, Footprints:FPC_9, symbol Connector_Generic:Conn_01x09
- added RN700, RN701, RN702, RN703, RN704: 33R, Resistor_SMD:R_Array_Convex_4x0402, symbol Device:R_Pack04
- C700: footprint Capacitor_SMD:C_0805_2012Metric -> Capacitor_SMD:C_0603_1608Metric
- L700: value 2.2uH -> 22uH
Connections:
- net +3V3: now also J700.2 (VCC), J700.38 (VCC)
- net +SYS: now also C707.2
- net GND: now also C707.1, J700.1 (GND), J700.28 (GND), J700.29 (GND), J700.3 (GND), J700.30 (GND), J700.31 (GND), J700.32 (GND), J700.33 (GND), J700.34 (GND), J700.35 (GND), J700.36 (GND), J700.37 (GND), J701.7 (Pin_7)
- net LCD_CLK: now also RN704.2 (R2.1)
- net LCD_CSN: now also J700.6 (CS)
- net LCD_D0: now also RN704.3 (R3.1)
- net LCD_D1: now also RN701.2 (R2.1)
- net LCD_D10: now also RN702.2 (R2.1)
- net LCD_D11: now also RN701.4 (R4.1)
- net LCD_D12: now also RN700.2 (R2.1)
- net LCD_D13: now also RN700.1 (R1.1)
- net LCD_D14: now also RN702.4 (R4.1)
- net LCD_D15: now also RN702.1 (R1.1)
- net LCD_D2: now also RN701.3 (R3.1)
- net LCD_D3: now also RN701.1 (R1.1)
- net LCD_D4: now also RN700.3 (R3.1)
- net LCD_D5: now also RN704.1 (R1.1)
- net LCD_D6: now also RN703.2 (R2.1)
- net LCD_D7: now also RN700.4 (R4.1)
- net LCD_D8: now also RN702.3 (R3.1)
- net LCD_D9: now also RN703.1 (R1.1)
- net LCD_DE: now also RN704.4 (R4.1)
- net LCD_DI: now also J700.4 (SDA), J701.5 (Pin_5)
- net LCD_HSYNC: now also RN703.3 (R3.1)
- net LCD_RST: now also J700.7 (RESET), J701.2 (Pin_2)
- net LCD_SCK: now also J700.5 (SCL), J701.4 (Pin_4)
- net LCD_VSYNC: now also RN703.4 (R4.1)
- net LEDA: now also J700.40 (LEDA)
- net LEDK: now also J700.39 (LEDK)
- new net +VRTC: J701.6 (Pin_6)
- new net D_D0: J700.23 (DB0), RN704.6 (R3.2)
- new net D_D1: J700.22 (DB1), RN701.7 (R2.2)
- new net D_D10: J700.13 (DB10), RN702.7 (R2.2)
- new net D_D11: J700.12 (DB11), RN701.5 (R4.2)
- new net D_D12: J700.11 (DB12), RN700.7 (R2.2)
- new net D_D13: J700.10 (DB13), RN700.8 (R1.2)
- new net D_D14: J700.9 (DB14), RN702.5 (R4.2)
- new net D_D15: J700.8 (DB15), RN702.8 (R1.2)
- new net D_D2: J700.21 (DB2), RN701.6 (R3.2)
- new net D_D3: J700.20 (DB3), RN701.8 (R1.2)
- new net D_D4: J700.19 (DB4), RN700.6 (R3.2)
- new net D_D5: J700.18 (DB5), RN704.8 (R1.2)
- new net D_D6: J700.17 (DB6), RN703.7 (R2.2)
- new net D_D7: J700.16 (DB7), RN700.5 (R4.2)
- new net D_D8: J700.15 (DB8), RN702.6 (R3.2)
- new net D_D9: J700.14 (DB9), RN703.8 (R1.2)
- new net D_DCLK: J700.25 (DOTCLK), RN704.7 (R2.2)
- new net D_DE: J700.24 (DE), RN704.5 (R4.2)
- new net D_HSYNC: J700.26 (HSYNC), RN703.6 (R3.2)
- new net D_VSYNC: J700.27 (VSYNC), RN703.5 (R4.2)
- new net LCD2_CS: J701.1 (Pin_1)
- new net LCD2_RS: J701.3 (Pin_3)
- no-connect marks 0 -> 2
Other:
- note added: "Termination resistors connections based on layout"
- company: ZephRay -> Wenting
- title: Sitina Ne -> SitinaNe
- moved on the sheet: C703, C705, C706, D700, L700, R700, R701, R702, R703, R704, U700
