File: Hardware/ProcessingBoard/storage.kicad_sch (KiCad schematic)
At the start: 21 parts, among them Q400 2N7002, U400 ADP163, U401 W25Q32JVZP

Commit message: Update License to match source code; test and fix USB, SEMC, and XIP on actual hardware
Changed lines of the file:
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@@
     (stroke (width 0) (type solid) (color 0 0 0 0))
   )
-  (bus (pts (xy 127 121.92) (xy 127 124.46))
+  (bus (pts (xy 127 121.92) (xy 127 134.62))
     (stroke (width 0) (type solid) (color 0 0 0 0))
   )
@@
     (stroke (width 0) (type solid) (color 0 0 0 0))
   )
-  (bus (pts (xy 127 124.46) (xy 127 127))
-    (stroke (width 0) (type solid) (color 0 0 0 0))
-  )
-  (bus (pts (xy 127 127) (xy 127 132.08))
-    (stroke (width 0) (type solid) (color 0 0 0 0))
-  )
-  (bus (pts (xy 127 132.08) (xy 127 134.62))
-    (stroke (width 0) (type solid) (color 0 0 0 0))
-  )
   (bus (pts (xy 154.94 101.6) (xy 152.4 101.6))
     (stroke (width 0) (type solid) (color 0 0 0 0))
   )
-  (bus (pts (xy 154.94 101.6) (xy 154.94 104.14))
+  (bus (pts (xy 154.94 101.6) (xy 154.94 111.76))
     (stroke (width 0) (type solid) (color 0 0 0 0))
   )
-  (bus (pts (xy 154.94 104.14) (xy 154.94 106.68))
-    (stroke (width 0) (type solid) (color 0 0 0 0))
-  )
-  (bus (pts (xy 154.94 106.68) (xy 154.94 109.22))
-    (stroke (width 0) (type solid) (color 0 0 0 0))
-  )
-  (bus (pts (xy 154.94 109.22) (xy 154.94 111.76))
-    (stroke (width 0) (type solid) (color 0 0 0 0))
-  )

Commit message: Bug fixes and changes for PB r0p2
Parts:
- removed C400: 10uF, Capacitor_SMD:C_0805_2012Metric, symbol Device:C
- removed C401: 100nF, Capacitor_SMD:C_0402_1005Metric, symbol Device:C
- removed Q400: 2N7002, Package_TO_SOT_SMD:SOT-23, symbol Transistor_FET:2N7002
- removed R400: 464K/1%, Resistor_SMD:R_0402_1005Metric, symbol Device:R
- removed R401, R402: 200K/1%, Resistor_SMD:R_0402_1005Metric, symbol Device:R
- removed R403: 243K/1%, Resistor_SMD:R_0402_1005Metric, symbol Device:R
- removed U400: ADP163, Package_TO_SOT_SMD:TSOT-23-5, symbol Regulator_Linear:ADP7142AUJZ
- C402: footprint Capacitor_SMD:C_0805_2012Metric -> Capacitor_SMD:C_0603_1608Metric
- C404, C405: value 18pF -> DNP
Connections:
- net +VSD is gone; now on net +3V3: C402.1, C403.1, MICRO_SD400.4 (VDD), R405.1, R406.1
Other:
- note removed: "47uF is required to comply with SD 3.0 spec"
- company: ZephRay -> Wenting
- title: Sitina Ne -> SitinaNe

Commit message: pcb: switch to ad9978 wip
Changed lines of the file:
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@@
-(kicad_sch (version 20210126) (generator eeschema)
+(kicad_sch (version 20210621) (generator eeschema)
   (paper "A4")
   (title_block
@@
     (stroke (width 0) (type solid) (color 0 0 0 0))
   )
-  (bus (pts (xy 127 121.92) (xy 127 124.46))
+  (bus (pts (xy 127 121.92) (xy 127 134.62))
     (stroke (width 0) (type solid) (color 0 0 0 0))
   )
@@
     (stroke (width 0) (type solid) (color 0 0 0 0))
   )
-  (bus (pts (xy 127 124.46) (xy 127 127))
-    (stroke (width 0) (type solid) (color 0 0 0 0))
-  )
-  (bus (pts (xy 127 127) (xy 127 132.08))
-    (stroke (width 0) (type solid) (color 0 0 0 0))
-  )
-  (bus (pts (xy 127 132.08) (xy 127 134.62))
-    (stroke (width 0) (type solid) (color 0 0 0 0))
-  )
   (bus (pts (xy 154.94 101.6) (xy 152.4 101.6))
     (stroke (width 0) (type solid) (color 0 0 0 0))
   )
-  (bus (pts (xy 154.94 101.6) (xy 154.94 104.14))
-    (stroke (width 0) (type solid) (color 0 0 0 0))
-  )
-  (bus (pts (xy 154.94 104.14) (xy 154.94 106.68))
-    (stroke (width 0) (type solid) (color 0 0 0 0))
-  )
-  (bus (pts (xy 154.94 106.68) (xy 154.94 109.22))
-    (stroke (width 0) (type solid) (color 0 0 0 0))
-  )
-  (bus (pts (xy 154.94 109.22) (xy 154.94 111.76))
-    (stroke (width 0) (type solid) (color 0 0 0 0))
-  )
+  (bus (pts (xy 154.94 101.6) (xy 154.94 111.76))
+    (stroke (width 0) (type solid) (color 0 0 0 0))
+  )
