File: Hardware/CaptureBoard/vsub.sch (KiCad schematic (older format))
At the start: 13 parts, among them Q1100 BC847BPN

Commit message: pcb: working on layout
Parts:
- D1100, D1101: footprint Diode_SMD:D_SOD-123 -> Diode_SMD:D_SOD-323
Changed lines of the file:
@@
 $Descr A4 11693 8268
 encoding utf-8
-Sheet 4 8
+Sheet 2 8
 Title "Sitina Ne"
 Date ""
@@
 F 0 "D1100" V 5554 4730 50  0000 L CNN
 F 1 "B0540W" V 5800 4400 50  0000 L CNN
-F 2 "Diode_SMD:D_SOD-123" H 5600 4650 50  0001 C CNN
+F 2 "Diode_SMD:D_SOD-323" H 5600 4650 50  0001 C CNN
 F 3 "~" H 5600 4650 50  0001 C CNN
 	1    5600 4650
@@
 F 0 "D1101" V 7146 3570 50  0000 R CNN
 F 1 "B0540W" V 7055 3570 50  0000 R CNN
-F 2 "Diode_SMD:D_SOD-123" H 7100 3650 50  0001 C CNN
+F 2 "Diode_SMD:D_SOD-323" H 7100 3650 50  0001 C CNN
 F 3 "~" H 7100 3650 50  0001 C CNN
 	1    7100 3650
