File: Hardware/CaptureBoard/afe.sch (KiCad schematic (older format))
At the start: 43 parts, among them U1 ADA4800, U2 ADA4800, U800 AD9990, Y800 30MHz

Commit message: pcb: start initial layouting
Parts:
- removed TP1, TP2: TestPoint, Connector_Pin:Pin_D1.0mm_L10.0mm, symbol Connector:TestPoint
Changed lines of the file:
@@
 	1    0    0    -1
 $EndComp
-$Comp
-L Connector:TestPoint TP?
-U 1 1 61979555
-P 8300 5300
-AR Path="/5FE3519F/61979555" Ref="TP?"  Part="1"
-AR Path="/5D0B94DA/61979555" Ref="TP1"  Part="1"
-F 0 "TP1" V 8358 5374 50  0000 L CNN
-F 1 "TestPoint" H 8358 5329 50  0001 L CNN
-F 2 "Connector_Pin:Pin_D1.0mm_L10.0mm" H 8500 5300 50  0001 C CNN
-F 3 "~" H 8500 5300 50  0001 C CNN
-	1    8300 5300
-	0    -1   -1   0
-$EndComp
-$Comp
-L Connector:TestPoint TP?
-U 1 1 6197955B
-P 8300 5500
-AR Path="/5FE3519F/6197955B" Ref="TP?"  Part="1"
-AR Path="/5D0B94DA/6197955B" Ref="TP2"  Part="1"
-F 0 "TP2" V 8358 5574 50  0000 L CNN
-F 1 "TestPoint" H 8358 5529 50  0001 L CNN
-F 2 "Connector_Pin:Pin_D1.0mm_L10.0mm" H 8500 5500 50  0001 C CNN
-F 3 "~" H 8500 5500 50  0001 C CNN
-	1    8300 5500
-	0    -1   -1   0
-$EndComp
-Wire Wire Line
-	8300 5500 8500 5500
-Wire Wire Line
-	8300 5300 8500 5300
-Text HLabel 8500 5500 2    50   Output ~ 0
-CSI_HSYNC
-Text HLabel 8500 5300 2    50   Output ~ 0
-CSI_VSYNC
 Text HLabel 4700 5900 0    50   Output ~ 0
 PWR_EN

Commit message: pcb: working on layout
Connections:
- net at U800.A10 (CCDIN_B): now also C823.1; no longer C830.1
- net at U800.A2 (CCDIN_A): now also C830.1; no longer C823.1
Changed lines of the file:
@@
 	3600 2200 3800 2200
 Wire Wire Line
-	3800 2200 3800 1600
+	3800 2200 3800 1700
 Wire Wire Line
 	3600 4200 3900 4200
-Wire Wire Line
-	3900 4200 3900 1700
 $Comp
 L power:GND #PWR0222
@@
 	6500 2900 6400 2900
 Wire Wire Line
-	3800 1600 4900 1600
-Wire Wire Line
 	6500 2700 6400 2700
-Wire Wire Line
-	3900 1700 4900 1700
 Wire Wire Line
 	6400 2600 6500 2600
@@
 	6500 6900 6400 6900
 Wire Wire Line
+	4900 1700 3800 1700
+Wire Wire Line
+	4900 1600 3900 1600
+Wire Wire Line
+	3900 1600 3900 4200
+Wire Wire Line
 	6400 5400 7000 5400

Commit message: pcb: wip
Connections:
- net at U800.A10 (CCDIN_B): now also C830.1; no longer C823.1
- net at U800.A2 (CCDIN_A): now also C823.1; no longer C830.1
Changed lines of the file:
@@
 	3600 2200 3800 2200
-Wire Wire Line
-	3800 2200 3800 1700
 Wire Wire Line
 	3600 4200 3900 4200
@@
 	6500 6900 6400 6900
 Wire Wire Line
-	4900 1700 3800 1700
-Wire Wire Line
-	4900 1600 3900 1600
-Wire Wire Line
-	3900 1600 3900 4200
+	3800 1600 4900 1600
+Wire Wire Line
+	3800 1600 3800 2200
+Wire Wire Line
+	4900 1700 3900 1700
+Wire Wire Line
+	3900 1700 3900 4200
 Wire Wire Line
 	6400 5400 7000 5400
