File: Hardware/CaptureBoard/ccd.sch (KiCad schematic (older format))
At the start: 7 parts, among them U1200 KAI-1100x

Commit message: pcb: working on layout
Connections:
- net GND: no longer U1200.25 (V1), U1200.37 (V1)
- net -8V: now reaches U1200.27 (ESD)
- new net V1: U1200.25 (V1), U1200.37 (V1)
Changed lines of the file:
@@
 $Descr A4 11693 8268
 encoding utf-8
-Sheet 7 8
+Sheet 5 8
 Title "Sitina Ne"
 Date ""
@@
 	5000 3100 5000 2700
 Wire Wire Line
-	6300 2600 6300 3000
-Wire Wire Line
 	6400 2500 6400 3100
 Wire Wire Line
@@
 	6000 3000 6200 3000
 Connection ~ 6000 3000
-Connection ~ 6300 3000
-Wire Wire Line
-	6300 3000 6300 3100
-Wire Wire Line
-	6300 3000 7000 3000
 Connection ~ 6200 3000
-Wire Wire Line
-	6200 3000 6300 3000
 Wire Wire Line
 	6100 3100 6100 2400
@@
 	-1   0    0    1
 $EndComp
+$Comp
+L power:-8V #PWR?
+U 1 1 5F8D2B35
+P 6100 2400
+F 0 "#PWR?" H 6100 2500 50  0001 C CNN
+F 1 "-8V" V 6115 2528 50  0000 L CNN
+F 2 "" H 6100 2400 50  0001 C CNN
+F 3 "" H 6100 2400 50  0001 C CNN
+	1    6100 2400
+	1    0    0    -1
+$EndComp
+Wire Wire Line
+	6300 2600 6300 3100
+Wire Wire Line
+	6200 3000 7000 3000
 $EndSCHEMATC

Commit message: pcb: wip
Parts:
- R1201: value 20K/1% -> 51K/1%
- R1202: value 60.4K/1% -> 100K/1%
- R1203: value 200K/1% -> 154K/1%
Connections:
- net +15V: no longer R1202.1
- net GND: now also C1200.1
- net VOD: now also C1200.2; no longer C1200.1
- net -4V renamed -9V
- net -9V: no longer C1200.2
- new net +19V: R1202.1
Other:
- moved on the sheet: C1200
Changed lines of the file:
@@
 P 3700 2950
 F 0 "R1203" H 3770 2996 50  0000 L CNN
-F 1 "200K/1%" H 3770 2905 50  0000 L CNN
+F 1 "154K/1%" H 3770 2905 50  0000 L CNN
 F 2 "Resistor_SMD:R_0402_1005Metric" V 3630 2950 50  0001 C CNN
 F 3 "~" H 3700 2950 50  0001 C CNN
@@
 P 3700 2450
 F 0 "R1202" H 3770 2496 50  0000 L CNN
-F 1 "60.4K/1%" H 3770 2405 50  0000 L CNN
+F 1 "100K/1%" H 3770 2405 50  0000 L CNN
 F 2 "Resistor_SMD:R_0402_1005Metric" V 3630 2450 50  0001 C CNN
 F 3 "~" H 3700 2450 50  0001 C CNN
@@
 	3700 3200 3700 3100
 Connection ~ 3700 3100
-$Comp
-L power:+15V #PWR0198
-U 1 1 5F54BB49
-P 3700 2200
-F 0 "#PWR0198" H 3700 2050 50  0001 C CNN
-F 1 "+15V" H 3715 2373 50  0000 C CNN
-F 2 "" H 3700 2200 50  0001 C CNN
-F 3 "" H 3700 2200 50  0001 C CNN
-	1    3700 2200
-	1    0    0    -1
-$EndComp
 Wire Wire Line
 	3700 2700 4100 2700
@@
 L Device:C C1200
 U 1 1 5F566DE0
-P 4500 2050
-F 0 "C1200" H 4615 2096 50  0000 L CNN
-F 1 "100nF/25V" H 4615 2005 50  0000 L CNN
-F 2 "Capacitor_SMD:C_0603_1608Metric" H 4538 1900 50  0001 C CNN
-F 3 "~" H 4500 2050 50  0001 C CNN
-	1    4500 2050
+P 4500 1550
+F 0 "C1200" H 4615 1596 50  0000 L CNN
+F 1 "100nF/25V" H 4615 1505 50  0000 L CNN
+F 2 "Capacitor_SMD:C_0603_1608Metric" H 4538 1400 50  0001 C CNN
+F 3 "~" H 4500 1550 50  0001 C CNN
+	1    4500 1550
 	1    0    0    -1
 $EndComp
@@
 P 4100 2050
 F 0 "R1201" H 4170 2096 50  0000 L CNN
-F 1 "20K/1%" H 4170 2005 50  0000 L CNN
+F 1 "51K/1%" H 4170 2005 50  0000 L CNN
 F 2 "Resistor_SMD:R_0402_1005Metric" V 4030 2050 50  0001 C CNN
 F 3 "~" H 4100 2050 50  0001 C CNN
@@
 $EndComp
 Wire Wire Line
-	4500 2200 4100 2200
-Wire Wire Line
 	4100 2300 4100 2200
-Connection ~ 4100 2200
-Wire Wire Line
-	4100 1800 4500 1800
-Wire Wire Line
-	4500 1900 4500 1800
 Wire Wire Line
 	4100 1900 4100 1800
@@
 	4100 1300 4100 1400
 Wire Wire Line
-	4500 1800 4800 1800
-Wire Wire Line
 	4800 1800 4800 2900
-Connection ~ 4500 1800
 Text Label 4500 1800 0    50   ~ 0
 VOD
@@
 	6100 3100 6100 2400
 $Comp
-L Sitina:-4V #PWR0203
-U 1 1 61BFCFC1
-P 4100 2300
-F 0 "#PWR0203" H 4100 2150 50  0001 C CNN
-F 1 "-4V" H 4115 2473 50  0000 C CNN
-F 2 "" H 4100 2300 50  0001 C CNN
-F 3 "" H 4100 2300 50  0001 C CNN
-	1    4100 2300
-	-1   0    0    1
-$EndComp
-$Comp
 L power:-8V #PWR0105
 U 1 1 5F8D2B35
@@
 Wire Wire Line
 	6200 3000 7000 3000
+$Comp
+L Sitina:+19V #PWR0124
+U 1 1 5FBCB818
+P 3700 2200
+F 0 "#PWR0124" H 3700 2050 50  0001 C CNN
+F 1 "+19V" H 3715 2373 50  0000 C CNN
+F 2 "" H 3700 2200 50  0001 C CNN
+F 3 "" H 3700 2200 50  0001 C CNN
+	1    3700 2200
+	1    0    0    -1
+$EndComp
+$Comp
+L power:-9V #PWR01
+U 1 1 5FBE904B
+P 4100 2300
+F 0 "#PWR01" H 4100 2175 50  0001 C CNN
+F 1 "-9V" H 4115 2473 50  0000 C CNN
+F 2 "" H 4100 2300 50  0001 C CNN
+F 3 "" H 4100 2300 50  0001 C CNN
+	1    4100 2300
+	-1   0    0    1
+$EndComp
+Wire Wire Line
+	4100 1800 4500 1800
+Wire Wire Line
+	4500 1700 4500 1800
+Connection ~ 4500 1800
+Wire Wire Line
+	4500 1800 4800 1800
+Wire Wire Line
+	4500 1400 4500 1300
+Wire Wire Line
+	4500 1300 4100 1300
+Connection ~ 4100 1300
 $EndSCHEMATC
