File: Hardware/CaptureBoard/power.sch (KiCad schematic (older format))
At the start: 79 parts, among them U10 LT1964-BYP, U11 LT1964-BYP, U4 LT3472, U5 LT3472, U6 LT3472, U7 LT3023, U8 LT3023

Commit message: pcb: start initial layouting
Parts:
- RV1: footprint Resistor_SMD:R_0402_1005Metric -> Potentiometer_SMD:Potentiometer_Vishay_TS53YL_Vertical
- gave numbers to parts that had none: 3
Changed lines of the file:
@@
 F 0 "RV1" H 6330 2854 50  0000 R CNN
 F 1 "100K" H 6330 2945 50  0000 R CNN
-F 2 "Resistor_SMD:R_0402_1005Metric" H 6400 2900 50  0001 C CNN
+F 2 "Potentiometer_SMD:Potentiometer_Vishay_TS53YL_Vertical" H 6400 2900 50  0001 C CNN
 F 3 "~" H 6400 2900 50  0001 C CNN
 	1    6400 2900
@@
 CCD_PWR_EN
 $Comp
-L Device:R R?
+L Device:R R3
 U 1 1 61C3D1E0
 P 3750 6300
-F 0 "R?" V 3550 6300 50  0000 C CNN
+F 0 "R3" V 3550 6300 50  0000 C CNN
 F 1 "316K/1%" V 3650 6300 50  0000 C CNN
 F 2 "Resistor_SMD:R_0402_1005Metric" V 3680 6300 50  0001 C CNN
@@
 Connection ~ 3600 6300
 $Comp
-L Device:R R?
+L Device:R R4
 U 1 1 61C4D25E
 P 4050 6300
-F 0 "R?" V 3850 6300 50  0000 C CNN
+F 0 "R4" V 3850 6300 50  0000 C CNN
 F 1 "49.9K/1%" V 3950 6300 50  0000 C CNN
 F 2 "Resistor_SMD:R_0402_1005Metric" V 3980 6300 50  0001 C CNN
@@
 	6000 1800 6800 1800
 $Comp
-L Device:R R?
+L Device:R R2
 U 1 1 61CCD1D7
 P 3750 2300
-F 0 "R?" V 3550 2300 50  0000 C CNN
+F 0 "R2" V 3550 2300 50  0000 C CNN
 F 1 "20K/1%" V 3650 2300 50  0000 C CNN
 F 2 "Resistor_SMD:R_0402_1005Metric" V 3680 2300 50  0001 C CNN

Commit message: pcb: move stuff around, add more capacitors
Parts:
- added C49, C50, C54: 6.3V/100uF, Capacitor_SMD:CP_Elec_5x4.5, symbol Device:CP
- added C51, C52, C55, C56, C57: 16V/47uF, Capacitor_SMD:CP_Elec_5x4.5, symbol Device:CP
- added C53: 25V/33uF, Capacitor_SMD:CP_Elec_5x4.5, symbol Device:CP
Connections:
- net +19V: now also C53.1
- net +3V3: now also C54.1
- net +5V: now also C51.1
- net +8V: now also C52.1
- net +SYS: now also C49.1, C50.1
- net -12V: now also C57.2
- net -8V: now also C56.2
- net -9V: now also C55.2
- net GND: now also C49.2, C50.2, C51.2, C52.2, C53.2, C54.2, C55.1, C56.1, C57.1

Commit message: pcb: wip
Parts:
- added D1, D10, D11, D12, D13, D14, D2, D3, D4, D5, D6, D7, D8, D9: LED, Diode_SMD:D_0603_1608Metric, symbol Device:LED
- added R12, R31, R35, R7: 3.3K, Resistor_SMD:R_0402_1005Metric, symbol Device:R
- added R13, R20, R29, R32: 4.7K, Resistor_SMD:R_0402_1005Metric, symbol Device:R
- added R14, R33: 10K, Resistor_SMD:R_0402_1005Metric, symbol Device:R
- added R19, R34, R36: 2K, Resistor_SMD:R_0402_1005Metric, symbol Device:R
- added R30: 7.5K, Resistor_SMD:R_0402_1005Metric, symbol Device:R
Connections:
- net +15V: now also R31.2
- net +19V: now also R14.2
- net +1V5: now also R34.2
- net +2V: now also R33.2
- net +3V3: now also R19.2
- net +5V: now also R12.2
- net +8V: now also R13.2
- net +SYS: now also R7.2
- net -12V: now also D8.1 (K)
- net -3V5: now also D14.1 (K)
- net -4V: now also D13.1 (K)
- net -8V: now also D7.1 (K)
- net -9V: now also D6.1 (K)
- net GND: now also D1.1 (K), D10.1 (K), D11.1 (K), D12.1 (K), D2.1 (K), D3.1 (K), D4.1 (K), D5.1 (K), D9.1 (K), R20.2, R29.2, R30.2, R35.2, R36.2
- net VAB: now also R32.2
- new net: D1.2 (A), R7.1
- new net: D2.2 (A), R12.1
- new net: D3.2 (A), R13.1
- new net: D4.2 (A), R14.1
- new net: D5.2 (A), R19.1
- new net: D6.2 (A), R20.1
- new net: D7.2 (A), R29.1
- new net: D8.2 (A), R30.1
- new net: D13.2 (A), R35.1
- new net: D14.2 (A), R36.1
- new net: D9.2 (A), R31.1
- new net: D10.2 (A), R32.1
- new net: D11.2 (A), R33.1
- new net: D12.2 (A), R34.1
Other:
- moved on the sheet: C43, C44, C45, C46, C47, C48, R25, R26, R27, R28, U10, U11
