File: Hardware/CaptureBoard/Sitina.kicad_pcb (KiCad board)
At the start: 2 copper layers, 202 parts, among them J100 Conn_01x30_MountingPin, Q1000 DMC3071LVT, Q1001 DMC3071LVT, Q1002 DMC3071LVT, Q1003 DMC3071LVT, Q1100 BC847BPN, U1 ADA4800, U10 LT1964-BYP, U11 LT1964-BYP, U1200 KAI-1100x, U2 ADA4800, U4 LT3472, U5 LT3472, U6 LT3472, U7 LT3023, U8 LT3023, U800 AD9990, U900 74LCX541BQX, U901 74LCX541BQX, U902 74LCX541BQX, U903 74LCX541BQX, Y800 30MHz

Commit message: pcb: working on layout
Parts:
- D1100, D1101, D900, D901, D902, D903, D904, D905, D906, D907: footprint Diode_SMD:D_SOD-123 -> Diode_SMD:D_SOD-323
- moved R1006 120.1 mm to (122.8, 87.3), turned to 180 degrees
- moved C1105 115.3 mm to (133.4, 97.6), turned to 180 degrees
- moved R800 113.4 mm to (124.7, 119.0), turned to 180 degrees
- moved R1007 113.2 mm to (122.8, 92.0), turned to 180 degrees
- moved C824 112.3 mm to (122.1, 117.3), turned to 180 degrees
- moved C1009 112.2 mm to (128.3, 87.3)
- moved C1012 111.0 mm to (125.3, 89.6), turned to 90 degrees
- moved C1100 110.8 mm to (147.8, 69.2)
- moved C1104 110.8 mm to (142.7, 67.5)
- moved Q1100 110.8 mm to (138.4, 71.1)
- moved R1103 110.8 mm to (144.9, 69.7)
- moved C1101 110.8 mm to (143.3, 72.1)
- moved C1102 110.8 mm to (136.9, 74.3)
- moved D1100 110.8 mm to (133.4, 71.2)
- moved R1100 110.8 mm to (142.0, 70.2)
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Connections:
- C1006 pad 1: GND -> /ccd/V1
- C1007 pad 2: GND -> /ccd/V1
- C902 pad 2: GND -> +2V
- Q1002 pad 4: GND -> /ccd/V1
- Q1002 pad 6: GND -> /ccd/V1
- U1200 pad 25: GND -> /ccd/V1
- U1200 pad 27: (no net) -> -8V
- U1200 pad 37: GND -> /ccd/V1
- U800 pad A10: Net-(C830-Pad1) -> Net-(C823-Pad1)
- U800 pad A2: Net-(C823-Pad1) -> Net-(C830-Pad1)
Routing:
- net Net-(C830-Pad2): track 0.00 -> 24.2 mm
- net Net-(C823-Pad2): track 0.00 -> 17.1 mm
- net /afe/CCDIN_B: track 0.00 -> 12.7 mm
- net /afe/CCDIN_A: track 0.00 -> 6.49 mm
- net +1V8A: track 12.5 -> 16.2 mm, vias 1 -> 2
- net Net-(C831-Pad2): track 5.79 -> 9.21 mm
- net +3V3: track 19.5 -> 16.8 mm
- net Net-(C821-Pad1): track 5.09 -> 3.06 mm
- net Net-(C820-Pad1): track 4.29 -> 2.54 mm
- net Net-(C822-Pad1): track 4.27 -> 2.58 mm
- net Net-(C830-Pad1): track 2.23 -> 3.82 mm
- net GND: track 21.4 -> 20.1 mm
- net Net-(C832-Pad2): track 5.21 -> 6.40 mm
- net Net-(C819-Pad1): track 5.10 -> 3.94 mm
Other:
- board outline added: 67 x 39 mm

Commit message: pcb: move stuff around, add more capacitors
Parts:
- added C49: 6.3V/100uF, Capacitor_SMD:CP_Elec_5x4.5, F.Cu at (134.4, 132.6)
- added C50: 6.3V/100uF, Capacitor_SMD:CP_Elec_5x4.5, F.Cu at (134.4, 139.4)
- added C51: 16V/47uF, Capacitor_SMD:CP_Elec_5x4.5, F.Cu at (143.3, 132.6)
- added C52: 16V/47uF, Capacitor_SMD:CP_Elec_5x4.5, F.Cu at (134.4, 146.3)
- added C53: 25V/33uF, Capacitor_SMD:CP_Elec_5x4.5, F.Cu at (143.3, 139.4)
- added C54: 6.3V/100uF, Capacitor_SMD:CP_Elec_5x4.5, F.Cu at (152.3, 132.6)
- added C55: 16V/47uF, Capacitor_SMD:CP_Elec_5x4.5, F.Cu at (143.3, 146.3)
- added C56: 16V/47uF, Capacitor_SMD:CP_Elec_5x4.5, F.Cu at (152.3, 139.4)
- added C57: 16V/47uF, Capacitor_SMD:CP_Elec_5x4.5, F.Cu at (161.2, 132.6)
- C800, C801, C802, C803, C804, C805, C806, C807, C808, C809, C810, C811, C812, C813, C814, C815, C816, C817, C818, C819, C820, C821, C822, C823, C824, C825, C826, C827, C828, C829, C830, C831, C832, R800, R801, R802, R803, U1, U2, U800, Y800: moved to B.Cu
- moved C5 94.3 mm to (138.2, 100.5)
- moved C46 91.3 mm to (132.1, 97.7), turned to 270 degrees
- moved C43 87.4 mm to (138.8, 95.8), turned to 90 degrees
- moved R17 86.0 mm to (145.9, 94.0), turned to 180 degrees
- moved R28 85.9 mm to (137.8, 97.8), turned to 90 degrees
- moved C44 85.1 mm to (132.1, 95.7), turned to 90 degrees
- moved R18 83.1 mm to (145.9, 95.0), turned to 180 degrees
- moved R24 82.7 mm to (152.3, 97.3)
- moved C47 81.9 mm to (144.4, 95.8), turned to 270 degrees
- moved R27 81.4 mm to (136.2, 98.4)
- moved R4 80.2 mm to (154.7, 93.8), turned to 180 degrees
- moved C42 79.6 mm to (152.3, 93.3)
- moved R11 79.6 mm to (158.8, 111.3), turned to 90 degrees
- moved R26 78.9 mm to (144.4, 97.8), turned to 90 degrees
- moved R25 77.7 mm to (142.9, 98.5)
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Routing:
- net Net-(C830-Pad2): track 24.2 -> 1.57 mm
- net /afe/CCDIN_B: track 12.7 -> 2.94 mm
- net /afe/CCDIN_A: track 6.49 -> 1.71 mm
Other:
- board text added: "Copyright 2020 Wenting Zhang"
- board text added: "SitinaNe Capture Board R0.1"

Commit message: pcb: wip
Parts:
- J100: moved to B.Cu
- moved C55 66.8 mm to (172.0, 86.0)
- moved C57 59.7 mm to (118.0, 91.5)
- moved C53 59.6 mm to (118.0, 85.5)
- moved C52 56.6 mm to (172.0, 104.0)
- moved R6 55.7 mm to (115.5, 95.0), turned to 180 degrees
- moved C49 55.3 mm to (172.0, 92.0)
- moved R2 54.7 mm to (117.5, 95.0), turned to 180 degrees
- moved C1 54.2 mm to (115.4, 99.2)
- moved C10 54.2 mm to (117.0, 97.2)
- moved C16 54.2 mm to (116.0, 97.2)
- moved C19 54.2 mm to (118.0, 97.2)
- moved C22 54.2 mm to (120.1, 101.5)
- moved C25 54.2 mm to (119.0, 97.2)
- moved R1 54.2 mm to (114.3, 99.2)
- moved U4 54.2 mm to (117.7, 100.4)
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Connections:
- U800 pad A10: Net-(C823-Pad1) -> Net-(C830-Pad1)
- U800 pad A2: Net-(C830-Pad1) -> Net-(C823-Pad1)
Routing:
- net Net-(C823-Pad2): track 17.1 -> 1.14 mm
- net /afe/CSI_D0: track 5.90 -> 1.21 mm
- net /afe/CSI_D7: track 5.52 -> 1.23 mm
- net Net-(C830-Pad1): track 3.82 -> 0.00 mm
- net /afe/CSI_D6: track 5.14 -> 1.43 mm
- net /afe/AFE_SL: track 4.67 -> 1.26 mm
- net /afe/AFE_RST: track 4.20 -> 0.90 mm
- net /afe/AFE_SCK: track 4.13 -> 0.88 mm
- net Net-(C823-Pad1): track 3.00 -> 0.00 mm
- net /afe/CCDIN_B: track 2.94 -> 0.00 mm
- net /afe/CCDIN_A: track 1.71 -> 3.46 mm
- net Net-(C830-Pad2): track 1.57 -> 0.00 mm
Other:
- board size 67 x 39 mm -> 64 x 38 mm
- board text added: "Copyright 2020 W.Z."
- board text removed: "Copyright 2020 Wenting Zhang"

Commit message: pcb: wip
Parts:
- moved C903 3.15 mm to (156.6, 114.2)
- moved C904 2.58 mm to (155.0, 102.0)
- moved C905 2.58 mm to (151.5, 102.0)
- moved D900 2.58 mm to (156.8, 103.1)
- moved D901 2.58 mm to (153.2, 103.2)
- moved R900 2.58 mm to (155.2, 104.5)
- moved R901 2.58 mm to (151.7, 104.5)
- moved U903 2.58 mm to (154.1, 109.5)
- moved C43 1.83 mm to (140.8, 93.9)
- moved C44 1.83 mm to (134.1, 93.8)
- moved C45 1.83 mm to (140.8, 95.9)
- moved C46 1.83 mm to (134.1, 95.9)
- moved C47 1.83 mm to (146.4, 93.9)
- moved C48 1.83 mm to (139.8, 93.9)
- moved R25 1.83 mm to (144.9, 96.6)
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Connections:
- J100 pad 17: /afe/CSI_VSYNC -> /afe/CSI_PCLK
- J100 pad 18: /afe/CSI_HSYNC -> GND
- J100 pad 19: GND -> /afe/CSI_VSYNC
- J100 pad 20: /afe/CSI_PCLK -> /afe/CSI_HSYNC
- U901 pad 11: /ccd/H2SL -> /ccd/H2SR
- U901 pad 12: /ccd/H2SL -> /ccd/H2SR
- U901 pad 13: /ccd/H2SR -> /ccd/H1SR
- U901 pad 14: /ccd/H2SR -> /ccd/H1SR
- U901 pad 15: /ccd/H1SR -> /ccd/H1BR
- U901 pad 16: /ccd/H1SR -> /ccd/H1BR
- U901 pad 17: /ccd/H1BR -> /ccd/H2SL
- U901 pad 18: /ccd/H1BR -> /ccd/H2SL
- U901 pad 2: Net-(C908-Pad1) -> Net-(C910-Pad1)
- U901 pad 3: Net-(C908-Pad1) -> Net-(C910-Pad1)
- U901 pad 4: Net-(C909-Pad1) -> Net-(C908-Pad1)
- U901 pad 5: Net-(C909-Pad1) -> Net-(C908-Pad1)
- U901 pad 6: Net-(C910-Pad1) -> Net-(C909-Pad1)
- U901 pad 7: Net-(C910-Pad1) -> Net-(C909-Pad1)
- U902 pad 13: /ccd/H2BL -> /ccd/H1SL
- U902 pad 14: /ccd/H2BL -> /ccd/H1SL
- U902 pad 17: /ccd/H1SL -> /ccd/H2BL
- U902 pad 18: /ccd/H1SL -> /ccd/H2BL
- U902 pad 2: Net-(C909-Pad1) -> Net-(C910-Pad1)
- U902 pad 3: Net-(C909-Pad1) -> Net-(C910-Pad1)
- U902 pad 6: Net-(C910-Pad1) -> Net-(C909-Pad1)
- U902 pad 7: Net-(C910-Pad1) -> Net-(C909-Pad1)
- U903 pad 15: /ccd/RL -> /ccd/RR
- U903 pad 16: /ccd/RL -> /ccd/RR
- U903 pad 17: /ccd/RR -> /ccd/RL
- U903 pad 18: /ccd/RR -> /ccd/RL
- U903 pad 2: Net-(C904-Pad1) -> Net-(C905-Pad1)
- U903 pad 3: Net-(C904-Pad1) -> Net-(C905-Pad1)
- U903 pad 4: Net-(C905-Pad1) -> Net-(C904-Pad1)
- U903 pad 5: Net-(C905-Pad1) -> Net-(C904-Pad1)
Routing:
- net /afe/GPO1_STROBE: track 1.62 -> 59.3 mm, vias 0 -> 1
- net /afe/AFE_RST: track 0.90 -> 57.5 mm, vias 1 -> 2
- net /afe/AFE_SCK: track 0.88 -> 57.2 mm, vias 1 -> 2
- net /afe/AFE_SYNC: track 3.01 -> 56.4 mm
- net /ccd/RL: track 0.00 -> 49.9 mm, vias 0 -> 1
- net /power/CCD_PWR_EN: track 2.60 -> 52.4 mm
- net /afe/AFE_SDATA: track 3.03 -> 50.8 mm
- net /afe/CSI_HSYNC: track 1.54 -> 45.2 mm
- net /afe/CSI_VSYNC: track 2.05 -> 45.6 mm
- net /afe/CSI_D0: track 1.21 -> 41.1 mm, vias 1 -> 2
- net /afe/CSI_D7: track 1.23 -> 38.0 mm, vias 1 -> 2
- net /afe/CSI_D6: track 1.43 -> 37.9 mm, vias 1 -> 2
- net /afe/CSI_D1: track 3.06 -> 37.9 mm
- net /afe/CSI_D2: track 2.10 -> 36.6 mm
- net /afe/CSI_D3: track 1.31 -> 35.3 mm
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
Commit message: pcb: wip
Parts:
- added D1: LED, Diode_SMD:D_0603_1608Metric, B.Cu at (175.2, 90.8)
- added D10: LED, Diode_SMD:D_0603_1608Metric, B.Cu at (156.2, 106.6)
- added D11: LED, Diode_SMD:D_0603_1608Metric, B.Cu at (153.6, 107.9)
- added D12: LED, Diode_SMD:D_0603_1608Metric, B.Cu at (156.2, 103.5)
- added D13: LED, Diode_SMD:D_0603_1608Metric, B.Cu at (130.8, 107.0)
- added D14: LED, Diode_SMD:D_0603_1608Metric, B.Cu at (148.4, 112.4)
- added D2: LED, Diode_SMD:D_0603_1608Metric, B.Cu at (175.2, 96.8)
- added D3: LED, Diode_SMD:D_0603_1608Metric, B.Cu at (175.2, 102.8)
- added D4: LED, Diode_SMD:D_0603_1608Metric, B.Cu at (114.8, 84.2)
- added D5: LED, Diode_SMD:D_0603_1608Metric, B.Cu at (114.7, 115.3)
- added D6: LED, Diode_SMD:D_0603_1608Metric, B.Cu at (175.2, 84.8)
- added D7: LED, Diode_SMD:D_0603_1608Metric, B.Cu at (175.2, 108.8)
- added D8: LED, Diode_SMD:D_0603_1608Metric, B.Cu at (114.7, 90.3)
- added D9: LED, Diode_SMD:D_0603_1608Metric, B.Cu at (169.5, 116.0)
- added R12: 3.3K, Resistor_SMD:R_0402_1005Metric, B.Cu at (175.4, 99.4)
- added R13: 4.7K, Resistor_SMD:R_0402_1005Metric, B.Cu at (175.4, 105.4)
- added R14: 10K, Resistor_SMD:R_0402_1005Metric, B.Cu at (114.6, 86.8)
- added R19: 2K, Resistor_SMD:R_0402_1005Metric, B.Cu at (114.5, 117.9)
- added R20: 4.7K, Resistor_SMD:R_0402_1005Metric, B.Cu at (175.4, 87.4)
- added R29: 4.7K, Resistor_SMD:R_0402_1005Metric, B.Cu at (175.4, 111.4)
- added R30: 7.5K, Resistor_SMD:R_0402_1005Metric, B.Cu at (114.5, 92.9)
- added R31: 3.3K, Resistor_SMD:R_0402_1005Metric, B.Cu at (169.0, 114.5)
- added R32: 4.7K, Resistor_SMD:R_0402_1005Metric, B.Cu at (157.5, 106.5)
- added R33: 10K, Resistor_SMD:R_0402_1005Metric, B.Cu at (153.7, 105.3)
- added R34: 2K, Resistor_SMD:R_0402_1005Metric, B.Cu at (157.5, 103.4)
- added R35: 3.3K, Resistor_SMD:R_0402_1005Metric, B.Cu at (132.3, 107.0)
- added R36: 2K, Resistor_SMD:R_0402_1005Metric, B.Cu at (148.8, 114.5)
- added R7: 3.3K, Resistor_SMD:R_0402_1005Metric, B.Cu at (175.4, 93.4)
- R1201: value 20K/1% -> 51K/1%
- R1202: value 60.4K/1% -> 100K/1%
- R1203: value 200K/1% -> 154K/1%
- moved C5 18.1 mm to (158.2, 100.2), turned to 270 degrees
- moved C831 5.95 mm to (146.3, 112.3), turned to 270 degrees
- moved C832 5.95 mm to (140.4, 112.3), turned to 90 degrees
- moved R5 4.04 mm to (114.3, 101.3), turned to 90 degrees
- moved C817 3.72 mm to (138.8, 97.3)
- moved C905 3.60 mm to (155.1, 102.0)
- moved D901 3.60 mm to (156.8, 103.2)
- moved R901 3.60 mm to (155.3, 104.5)
- moved C909 3.55 mm to (131.2, 101.8)
- moved D905 3.55 mm to (132.9, 103.2)
- moved R905 3.55 mm to (131.4, 104.3)
- moved C904 3.50 mm to (151.5, 102.1)
- moved D900 3.50 mm to (153.3, 103.2)
- moved R900 3.50 mm to (151.7, 104.6)
- moved D906 3.40 mm to (136.4, 103.3)
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Connections:
- C1200 pad 1: /ccd/VOD -> GND
- C1200 pad 2: -4V -> /ccd/VOD
- J100 pad 23: /afe/AFE_SDATA -> /afe/AFE_SCK
- J100 pad 24: /afe/AFE_SCK -> /afe/AFE_RST
- J100 pad 25: /afe/AFE_RST -> /afe/AFE_SYNC
- J100 pad 26: /afe/AFE_SYNC -> /afe/AFE_SDATA
- R1201 pad 2: -4V -> -9V
- R1202 pad 1: +15V -> +19V
Routing:
- net GND: track 20.5 -> 185.7 mm, vias 10 -> 88
- net +SYS: track 0.00 -> 123.2 mm, vias 0 -> 6
- net -4V: track 0.00 -> 122.3 mm, vias 0 -> 4
- net /afe/AFE_V2: track 1.74 -> 120.2 mm, vias 0 -> 1
- net +19V: track 0.00 -> 105.8 mm, vias 0 -> 3
- net /afe/AFE_V2_3rd: track 0.70 -> 104.6 mm, vias 0 -> 1
- net Net-(R1-Pad1): track 0.00 -> 101.4 mm, vias 0 -> 7
- net -8V: track 0.00 -> 100.9 mm, vias 0 -> 4
- net /afe/AFE_V1: track 2.85 -> 97.6 mm, vias 0 -> 1
- net +15V: track 0.00 -> 89.0 mm, vias 0 -> 3
- net -3V5: track 0.00 -> 76.3 mm, vias 0 -> 1
- net -9V: track 0.00 -> 71.6 mm, vias 0 -> 4
- net /afe/AFE_FDG: track 4.72 -> 76.3 mm, vias 0 -> 1
- net +2V: track 0.00 -> 68.8 mm, vias 0 -> 6
- net VAB: track 0.00 -> 68.2 mm, vias 0 -> 3
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- added copper zone on In1.Cu, net +3V3
- added copper zone on B.Cu, net GND
- added copper zone on F.Cu, net GND
- added copper zone on In2.Cu, net GND
Other:
- board size 64 x 38 mm -> 64 x 40 mm
- copper layers 2 -> 4

Commit message: Migrate to KiCAD 6, capture board layout changes
Parts:
- moved R30 13.6 mm to (124.0, 83.2), turned to 180 degrees
- moved R14 13.2 mm to (127.2, 83.2), turned to 0 degrees
- moved D4 13.0 mm to (127.5, 81.8), turned to 180 degrees
- moved D8 12.9 mm to (124.5, 81.8), turned to 0 degrees
- moved D5 11.8 mm to (125.5, 120.0), turned to 180 degrees
- moved R19 8.61 mm to (122.8, 120.0), turned to 180 degrees
- moved C1200 1.11 mm to (164.8, 83.8)
- moved R1200 1.08 mm to (164.1, 85.3)
- moved R1201 1.08 mm to (166.1, 85.3)
- moved C1201 0.90 mm to (125.4, 83.8)
- moved R1202 0.70 mm to (124.0, 85.3)
- moved R1203 0.70 mm to (126.0, 85.3)
Routing:
- net -12V: track 28.2 -> 40.2 mm
- net GND: track 185.7 -> 192.0 mm, vias 88 -> 91
- net +3V3: track 55.7 -> 60.5 mm
- net +19V: track 105.8 -> 110.5 mm
- net -9V: track 71.6 -> 72.8 mm
- net /ccd/VRD: track 41.9 -> 41.4 mm
- net /ccd/VOD: track 43.0 -> 42.5 mm
Other:
- net class Default removed
- board text added: "Copyright 2021 Wenting"
- board text removed: "Copyright 2020 W.Z."

Commit message: PBr0p2, CBr0p1, submitted for prototype production
Parts:
- moved R19 2.05 mm to (124.3, 118.6)
Routing:
- net +3V3: track 60.5 -> 62.6 mm
- net GND: vias 91 -> 115
Other:
- board text added: "SNE-CB r0.2"
- board text removed: "SitinaNe Capture Board R0.1"

Commit message: pcb: switch to ad9978 wip
Parts:
- removed C1105: 1uF/25V, Capacitor_SMD:C_0805_2012Metric
- removed D12: LED, Diode_SMD:D_0603_1608Metric
- removed U1, U2: ADA4800, Package_DFN_QFN:DFN-6-1EP_2x1.8mm_P0.5mm_EP1.2x1.6mm
- removed Y800: 30MHz, Crystal:Crystal_SMD_3225-4Pin_3.2x2.5mm
- added C833: 100nF, Capacitor_SMD:C_0402_1005Metric, B.Cu at (147.0, 137.9)
- added C834: 100nF, Capacitor_SMD:C_0402_1005Metric, B.Cu at (144.5, 133.3)
- added C835: 100nF, Capacitor_SMD:C_0402_1005Metric, B.Cu at (161.0, 149.1)
- added C836: 100nF, Capacitor_SMD:C_0402_1005Metric, B.Cu at (156.0, 145.3)
- added C837: 100nF, Capacitor_SMD:C_0402_1005Metric, B.Cu at (147.0, 135.9)
- added C838: 100nF, Capacitor_SMD:C_0402_1005Metric, B.Cu at (158.1, 147.3)
- added C839: 470nF, Capacitor_SMD:C_0402_1005Metric, B.Cu at (149.9, 138.8)
- added D801: LED, Diode_SMD:D_0603_1608Metric, B.Cu at (147.9, 133.6)
- added D802: 1N5819, Diode_SMD:D_SOD-123, B.Cu at (161.0, 142.4)
- added J801: Conn_02x05_Odd_Even, Connector_PinHeader_1.27mm:PinHeader_2x05_P1.27mm_Vertical_SMD, B.Cu at (159.1, 136.5)
- added R804: 2K, Resistor_SMD:R_0402_1005Metric, B.Cu at (152.8, 138.8)
- added R805: 100, Resistor_SMD:R_0402_1005Metric, B.Cu at (139.8, 102.8)
- added R806: 100, Resistor_SMD:R_0402_1005Metric, B.Cu at (141.2, 102.0)
- added R807: 100, Resistor_SMD:R_0402_1005Metric, B.Cu at (139.8, 100.8)
- added R808: 100, Resistor_SMD:R_0402_1005Metric, B.Cu at (141.2, 99.8)
- added R809: 100, Resistor_SMD:R_0402_1005Metric, B.Cu at (139.8, 98.8)
- added R810: 100K, Resistor_SMD:R_0402_1005Metric, B.Cu at (161.8, 145.1)
- added R811: 100K, Resistor_SMD:R_0402_1005Metric, B.Cu at (166.8, 149.8)
- added R812: 100K, Resistor_SMD:R_0402_1005Metric, B.Cu at (163.9, 149.8)
- added R813: 33R, Capacitor_SMD:C_0402_1005Metric, B.Cu at (152.4, 142.8)
- added R814: 10K, Capacitor_SMD:C_0402_1005Metric, B.Cu at (149.5, 140.8)
- added U801: ICE40HX4K-BG121, Package_BGA:BGA-121_9.0x9.0mm_Layout11x11_P0.8mm_Ball0.4mm_Pad0.35mm_NSMD, B.Cu at (133.4, 100.5)
- added U802: W25Q32JVZP, Package_SON:WSON-8-1EP_6x5mm_P1.27mm_EP3.4x4.3mm, B.Cu at (137.4, 127.5)
- added U803: ADA4800, Package_DFN_QFN:DFN-6-1EP_2x2mm_P0.5mm_EP0.6x1.37mm, B.Cu at (152.1, 134.1)
- added U804: ADA4800, Package_DFN_QFN:DFN-6-1EP_2x2mm_P0.5mm_EP0.6x1.37mm, B.Cu at (156.0, 142.5)
- added X801: 33.33MHz, Oscillator:Oscillator_SMD_Abracon_ASE-4Pin_3.2x2.5mm, B.Cu at (165.7, 146.6)
- C819, C820, C822: value 1uF -> 100nF
- C821: value 1uF -> 220nF
- C831, C832: value 18pF -> 100nF; footprint Capacitor_SMD:C_0603_1608Metric -> Capacitor_SMD:C_0402_1005Metric
- R34: value 2K -> 10K
- U800: value AD9990 -> AD9978; footprint Footprints:BGA-112_11x11_8.0x8.0mm -> Package_DFN_QFN:QFN-40-1EP_6x6mm_P0.5mm_EP4.6x4.6mm
- moved C800 64.7 mm to (212.6, 127.2)
- moved C803 64.7 mm to (212.6, 119.5)
- moved C805 64.7 mm to (212.6, 120.5)
- moved C831 64.7 mm to (207.8, 132.5)
- moved C832 64.7 mm to (201.9, 132.4)
- moved R33 64.7 mm to (215.2, 125.5)
- moved C801 64.7 mm to (214.4, 131.8)
- moved C802 64.7 mm to (200.2, 129.3)
- moved C804 64.7 mm to (199.3, 127.3)
- moved C806 64.7 mm to (205.8, 129.3)
- moved C810 64.7 mm to (213.2, 118.0)
- moved C812 64.7 mm to (199.8, 123.0)
- moved C816 64.7 mm to (212.4, 129.8)
- moved C818 64.7 mm to (203.1, 117.8)
- moved C819 64.7 mm to (203.2, 129.3)
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Connections:
- C1100 pad 2: /afe/GPO1_STROBE -> /afe/SUB_STROBE
- C1101 pad 2: /afe/GPO1_STROBE -> /afe/SUB_STROBE
- C801 pad 2: +3V3 -> +1V2
- C804 pad 2: +3V3 -> +1V2
- C806 pad 2: +3V3 -> +1V8A
- C807 pad 1: GND -> +1V8A
- C807 pad 2: +3V3 -> GND
- C808 pad 1: GND -> +1V8A
- C808 pad 2: +3V3 -> GND
- C809 pad 1: GND -> +3V3
- C809 pad 2: +3V3 -> GND
- C810 pad 1: GND -> +3V3
- C810 pad 2: +3V3 -> GND
- C811 pad 1: GND -> +3V3
- C811 pad 2: +3V3 -> GND
- C812 pad 1: GND -> +3V3
- C812 pad 2: +3V3 -> GND
- C813 pad 1: GND -> +3V3
- C813 pad 2: +1V8A -> GND
- C814 pad 1: GND -> +1V8A
- C814 pad 2: +1V8A -> GND
- C815 pad 1: GND -> +1V8A
- C815 pad 2: +1V8A -> GND
- C816 pad 1: GND -> +1V8A
- C816 pad 2: +1V8A -> GND
- C817 pad 1: GND -> +1V8A
- C817 pad 2: +1V8A -> GND
- C818 pad 1: GND -> +1V8A
- C818 pad 2: +1V8A -> GND
- C819 pad 1: Net-(C819-Pad1) -> GND
- C819 pad 2: GND -> +3V3
- C820 pad 1: Net-(C820-Pad1) -> GND
- C820 pad 2: GND -> +3V3
- C821 pad 1: Net-(C821-Pad1) -> GND
- C821 pad 2: GND -> +3V3
- C822 pad 1: Net-(C822-Pad1) -> GND
- C822 pad 2: GND -> +1V8A
- C831 pad 2: Net-(C831-Pad2) -> +1V2
- C832 pad 2: Net-(C832-Pad2) -> +1V2
- J100 pad 17: /afe/CSI_PCLK -> /afe/CSI_VSYNC
- J100 pad 18: GND -> /afe/CSI_HSYNC
- J100 pad 19: /afe/CSI_VSYNC -> GND
- J100 pad 20: /afe/CSI_HSYNC -> /afe/CSI_PCLK
- J100 pad 22: /afe/AFE_SL -> /afe/FPGA_CS
- J100 pad 23: /afe/AFE_SCK -> /afe/FPGA_MOSI
- J100 pad 24: /afe/AFE_RST -> /afe/FPGA_SCK
- J100 pad 25: /afe/AFE_SYNC -> (no net)
- J100 pad 26: /afe/AFE_SDATA -> (no net)
- R34 pad 1: Net-(D12-Pad2) -> GND
- R34 pad 2: +1V5 -> /afe/PWR_EN
- U4 pad 3: /power/CCD_PWR_EN -> /afe/PWR_EN
Routing:
- net /afe/AFE_V2: track 120.1 -> 5.03 mm
- net /afe/AFE_V2_3rd: track 104.5 -> 5.03 mm
- net /afe/AFE_V1: track 97.5 -> 7.28 mm
- net -4V: track 122.3 -> 39.4 mm, vias 4 -> 3
- net /power/CCD_PWR_EN: track 70.4 -> 0.00 mm, vias 3 -> 0
- net +1V8A: track 66.6 -> 0.00 mm, vias 6 -> 0
- net /afe/AFE_FDG: track 76.3 -> 9.95 mm
- net /afe/AFE_SDATA: track 54.3 -> 0.00 mm
- net /afe/AFE_RST: track 53.4 -> 0.00 mm, vias 2 -> 0
- net /afe/AFE_SCK: track 53.2 -> 0.00 mm, vias 2 -> 0
- net /afe/AFE_SL: track 53.1 -> 0.00 mm, vias 2 -> 0
- net /afe/AFE_SYNC: track 52.3 -> 0.00 mm
- net +3V3: track 62.6 -> 15.2 mm, vias 11 -> 7
- net GND: track 192.0 -> 145.8 mm, vias 115 -> 86
- net /afe/GPO1_STROBE: track 45.3 -> 0.00 mm, vias 1 -> 0
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