File: Hardware/CaptureBoard/afe.kicad_sch (KiCad schematic)
At the start: 41 parts, among them U1 ADA4800, U2 ADA4800, U800 AD9990, Y800 24MHz

Commit message: pcb: CB r0p4
Parts:
- added J800: Conn_02x15_Odd_Even, Connector_PinHeader_2.00mm:PinHeader_2x15_P2.00mm_Vertical, symbol Connector_Generic:Conn_02x15_Odd_Even
- C800, C802, C803, C805, C806, C807, C808, C809, C811, C813, C814, C815, C817, C823, C830: value 100nF -> 100nF/25V
- C801, C804, C810, C812, C816, C818: value 4.7uF -> 10uF/6.3V; footprint Capacitor_SMD:C_0805_2012Metric -> Capacitor_SMD:C_0402_1005Metric
- C824, C825, C826, C827, C828, C829, C831, C832: footprint Capacitor_SMD:C_0603_1608Metric -> Capacitor_SMD:C_0402_1005Metric
- U1, U2: footprint Package_DFN_QFN:DFN-6-1EP_2x1.8mm_P0.5mm_EP1.2x1.6mm -> Footprints:DFN-6-1EP_1.6x1.6mm_P0.5mm_EP0.5x1.05mm
Connections:
- net AFE_FDG: now also J800.28 (Pin_28); no longer U800.G4 (XV4)
- net AFE_H1_A: now also J800.4 (Pin_4); no longer U800.E1 (H1A)
- net AFE_H1_B: now also J800.12 (Pin_12); no longer U800.E11 (H1B)
- net AFE_H2_A: now also J800.6 (Pin_6); no longer U800.E2 (H2A)
- net AFE_H2_B: now also J800.14 (Pin_14); no longer U800.E10 (H2B)
- net AFE_HL_A: now also J800.8 (Pin_8); no longer U800.C1 (HL_A)
- net AFE_HL_B: now also J800.16 (Pin_16); no longer U800.C11 (HL_B)
- net AFE_RG_A: now also J800.2 (Pin_2); no longer U800.B1 (RG_A)
- net AFE_RG_B: now also J800.10 (Pin_10); no longer U800.B11 (RG_B)
- net AFE_V1: now also J800.22 (Pin_22); no longer U800.F3 (XV1)
- net AFE_V2: now also J800.24 (Pin_24); no longer U800.F2 (XV2)
- net AFE_V2_3rd: now also J800.26 (Pin_26); no longer U800.F1 (XV3)
- net GPO1_STROBE: now also J800.18 (Pin_18), J800.20 (Pin_20); no longer U800.G11 (GPO1)
- net PWR_EN: now also J800.30 (Pin_30); no longer U800.G10 (GPO2)
- net CLI: now reaches C832.2, U800.B5 (CLI), Y800.1
- net CLO: now reaches C831.2, U800.B6 (CLO), Y800.3
- net AFE_SUBCK renamed SUB
- net SUB: now also J800.19 (Pin_19)
- new net FDG: J800.27 (Pin_27), U800.G4 (XV4)
- new net H1A: J800.3 (Pin_3), U800.E1 (H1A)
- new net H1B: J800.11 (Pin_11), U800.E11 (H1B)
- new net H2A: J800.5 (Pin_5), U800.E2 (H2A)
- new net H2B: J800.13 (Pin_13), U800.E10 (H2B)
- new net HLA: J800.7 (Pin_7), U800.C1 (HL_A)
- new net HLB: J800.15 (Pin_15), U800.C11 (HL_B)
- new net PEN: J800.29 (Pin_29), U800.G10 (GPO2)
- new net RGA: J800.1 (Pin_1), U800.B1 (RG_A)
- new net RGB: J800.9 (Pin_9), U800.B11 (RG_B)
- new net STB: J800.17 (Pin_17), U800.G11 (GPO1)
- new net V1: J800.21 (Pin_21), U800.F3 (XV1)
- new net V2: J800.23 (Pin_23), U800.F2 (XV2)
- new net V23: J800.25 (Pin_25), U800.F1 (XV3)
Other:
- title: Sitina Ne -> SitinaNe
