File: Hardware/CaptureBoard/vdriver.kicad_sch (KiCad schematic)
At the start: 29 parts, among them Q1000 DMC3071LVT, Q1001 DMC3071LVT, Q1002 DMC3071LVT, Q1003 DMC3071LVT

Commit message: pcb: CB r0p4
Parts:
- removed C1000, C1006, C1007, C1009, C1010: 1nF, Capacitor_SMD:C_0402_1005Metric, symbol Device:C
- removed C1008, C1011, C1012: 100nF/25V, Capacitor_SMD:C_0603_1608Metric, symbol Device:C
- removed D1000, D1001, D1002, D1003: BAT54S, Package_TO_SOT_SMD:SOT-23, symbol Diode:BAT54S
- removed Q1000, Q1001, Q1002, Q1003: DMC3071LVT, Package_TO_SOT_SMD:TSOT-23-6, symbol Transistor_FET:DMC3071LVT
- removed R1000, R1001, R1006: 220, Resistor_SMD:R_0402_1005Metric, symbol Device:R
- removed R1002, R1003, R1004, R1005: 100, Resistor_SMD:R_0402_1005Metric, symbol Device:R
- removed R1007: 200, Resistor_SMD:R_0402_1005Metric, symbol Device:R
- added R1028, R1029, R1035: 330K/1%, Resistor_SMD:R_0402_1005Metric, symbol Device:R
- added R1030, R1031, R1036: 316K/1%, Resistor_SMD:R_0402_1005Metric, symbol Device:R
- added R1032, R1033, R1034, R1037: 0.1, Resistor_SMD:R_0603_1608Metric, symbol Device:R
- added U1001, U1002, U1003, U1004: UCC27517A, Package_TO_SOT_SMD:SOT-23-5, symbol Sitina:UCC27517A
- C1001: value 1nF -> 10nF
- C1002, C1005: footprint Capacitor_SMD:C_0603_1608Metric -> Capacitor_SMD:C_0402_1005Metric
- C1003, C1004: value 1nF -> 100nF/25V
Connections:
- net +5V: now also C1005.2, U1004.1 (VDD)
- net +8V: now also U1001.1 (VDD)
- net -9V: now also C1003.2, C1004.2, U1002.2 (GND), U1002.4 (IN-), U1003.2 (GND), U1003.4 (IN-), U1004.2 (GND), U1004.4 (IN-)
- net FDG: now also R1037.1
- net FDG_CD_AFE: now also R1035.1
- net GND: now also C1001.1, C1003.1, C1004.1, U1001.2 (GND), U1001.4 (IN-), U1003.1 (VDD); no longer C1005.2
- net V1: now also R1034.1
- net V1_AFE: now also R1029.1
- net V2: now also R1033.1; no longer C1003.1, C1004.2
- net V2_3rd_AFE: now also U1001.3 (IN+)
- net V2_AFE: now also R1028.1
- net at C1001.2: now also R1032.1, U1002.1 (VDD)
- new net: R1035.2, R1036.1, U1004.3 (IN+)
- new net: R1028.2, R1030.1, U1002.3 (IN+)
- new net: R1033.2, U1002.5 (OUT)
- new net: R1037.2, U1004.5 (OUT)
- new net: R1029.2, R1031.1, U1003.3 (IN+)
- new net: R1032.2, U1001.5 (OUT)
- new net: R1034.2, U1003.5 (OUT)
- new net -16V: R1030.2, R1031.2, R1036.2
Other:
- title: Sitina Ne -> SitinaNe
- moved on the sheet: C1002
