File: Hardware/CaptureBoard/vsub.kicad_sch (KiCad schematic)
At the start: 13 parts, among them Q1100 BC847BPN

Commit message: pcb: switch to ad9978 wip
Parts:
- removed C1105: 1uF/25V, Capacitor_SMD:C_0805_2012Metric, symbol Device:C
Changed lines of the file:
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@@
-(kicad_sch (version 20210126) (generator eeschema)
+(kicad_sch (version 20210621) (generator eeschema)
   (paper "A4")
   (title_block
@@
   (junction (at 149.86 101.6) (diameter 0.9144) (color 0 0 0 0))
   (junction (at 149.86 121.92) (diameter 0.9144) (color 0 0 0 0))
-  (junction (at 172.72 101.6) (diameter 0.9144) (color 0 0 0 0))
   (junction (at 180.34 101.6) (diameter 0.9144) (color 0 0 0 0))
   (wire (pts (xy 106.68 101.6) (xy 119.38 101.6))
     (stroke (width 0) (type solid) (color 0 0 0 0))
   )
-  (wire (pts (xy 106.68 132.08) (xy 111.76 132.08))
-    (stroke (width 0) (type solid) (color 0 0 0 0))
-  )
   (wire (pts (xy 119.38 93.98) (xy 119.38 101.6))
     (stroke (width 0) (type solid) (color 0 0 0 0))
@@
     (stroke (width 0) (type solid) (color 0 0 0 0))
   )
-  (wire (pts (xy 119.38 132.08) (xy 172.72 132.08))
-    (stroke (width 0) (type solid) (color 0 0 0 0))
-  )
   (wire (pts (xy 121.92 93.98) (xy 119.38 93.98))
     (stroke (width 0) (type solid) (color 0 0 0 0))
@@
     (stroke (width 0) (type solid) (color 0 0 0 0))
   )
-  (wire (pts (xy 165.1 101.6) (xy 172.72 101.6))
-    (stroke (width 0) (type solid) (color 0 0 0 0))
-  )
-  (wire (pts (xy 172.72 101.6) (xy 180.34 101.6))
-    (stroke (width 0) (type solid) (color 0 0 0 0))
-  )
-  (wire (pts (xy 172.72 132.08) (xy 172.72 101.6))
+  (wire (pts (xy 165.1 101.6) (xy 180.34 101.6))
     (stroke (width 0) (type solid) (color 0 0 0 0))
   )
@@
     (effects (font (size 1.27 1.27)) (justify right))
   )
-  (hierarchical_label "SUBCK" (shape input) (at 106.68 132.08 180)
-    (effects (font (size 1.27 1.27)) (justify right))
-  )
   (hierarchical_label "VSUB" (shape output) (at 187.96 101.6 0)
     (effects (font (size 1.27 1.27)) (justify left))
@@
       (effects (font (size 1.27 1.27)) hide)
     )
-    (pin "1")
-    (pin "2")
-  )
-  (symbol (lib_id "Device:C") (at 115.57 132.08 270) (unit 1)
-    (in_bom yes) (on_board yes)
-    (property "Reference" "C1105" (id 0) (at 115.57 125.6792 90))
-    (property "Value" "1uF/25V" (id 1) (at 115.57 127.9906 90))
-    (property "Footprint" "Capacitor_SMD:C_0805_2012Metric" (id 2) (at 111.76 133.0452 0)
-      (effects (font (size 1.27 1.27)) hide)
-    )
-    (property "Datasheet" "~" (id 3) (at 115.57 132.08 0)
-      (effects (font (size 1.27 1.27)) hide)
-    )

Commit message: pcb: PB r0p2 and CB r0p3 freeze
Parts:
- added C1105: 1uF/25V, Capacitor_SMD:C_0805_2012Metric, symbol Device:C
Connections:
- net VSUB: now also C1105.1
- new net SUBCK: C1105.2

Commit message: pcb: CB r0p4
Parts:
- removed C1105: 1uF/25V, Capacitor_SMD:C_0805_2012Metric, symbol Device:C
- C1100, C1101: value 100nF -> 100nF/25V
- C1102, C1104: footprint Capacitor_SMD:C_0603_1608Metric -> Capacitor_SMD:C_0402_1005Metric
- C1103: footprint Capacitor_SMD:C_0805_2012Metric -> Capacitor_SMD:C_0603_1608Metric
Connections:
- net +19V renamed +15V
- net -12V renamed -16V
Other:
- title: Sitina Ne -> SitinaNe
Changed lines of the file:
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@@
-(kicad_sch (version 20210621) (generator eeschema)
+(kicad_sch (version 20211123) (generator eeschema)
   (paper "A4")
   (title_block
-    (title "Sitina Ne")
-    (rev "R0P2")
+    (title "SitinaNe")
+    (rev "R0.3")
     (company "ZephRay")
   )
-  (junction (at 149.86 101.6) (diameter 0.9144) (color 0 0 0 0))
-  (junction (at 142.24 109.22) (diameter 0.9144) (color 0 0 0 0))
-  (junction (at 132.08 93.98) (diameter 0.9144) (color 0 0 0 0))
-  (junction (at 180.34 101.6) (diameter 0.9144) (color 0 0 0 0))
-  (junction (at 149.86 121.92) (diameter 0.9144) (color 0 0 0 0))
-  (junction (at 119.38 101.6) (diameter 0.9144) (color 0 0 0 0))
-  (junction (at 149.86 81.28) (diameter 0.9144) (color 0 0 0 0))
-  (junction (at 172.72 101.6) (diameter 0.9144) (color 0 0 0 0))
-  (junction (at 132.08 109.22) (diameter 0.9144) (color 0 0 0 0))
+  (junction (at 142.24 109.22) (diameter 0.9144) (color 0 0 0 0)
+  )
+  (junction (at 119.38 101.6) (diameter 0.9144) (color 0 0 0 0)
+  )
+  (junction (at 149.86 81.28) (diameter 0.9144) (color 0 0 0 0)
+  )
+  (junction (at 180.34 101.6) (diameter 0.9144) (color 0 0 0 0)
+  )
+  (junction (at 132.08 93.98) (diameter 0.9144) (color 0 0 0 0)
+  )
+  (junction (at 132.08 109.22) (diameter 0.9144) (color 0 0 0 0)
+  )
+  (junction (at 149.86 101.6) (diameter 0.9144) (color 0 0 0 0)
+  )
+  (junction (at 149.86 121.92) (diameter 0.9144) (color 0 0 0 0)
+  )
   (wire (pts (xy 129.54 109.22) (xy 132.08 109.22))
     (stroke (width 0) (type solid) (color 0 0 0 0))
@@
     (stroke (width 0) (type solid) (color 0 0 0 0))
   )
-  (wire (pts (xy 165.1 101.6) (xy 172.72 101.6))
+  (wire (pts (xy 165.1 101.6) (xy 180.34 101.6))
     (stroke (width 0) (type solid) (color 0 0 0 0))
   )
@@
     (stroke (width 0) (type solid) (color 0 0 0 0))
   )
-  (wire (pts (xy 172.72 132.08) (xy 172.72 101.6))
-    (stroke (width 0) (type solid) (color 0 0 0 0))
-  )
-  (wire (pts (xy 106.68 132.08) (xy 111.76 132.08))
-    (stroke (width 0) (type solid) (color 0 0 0 0))
-  )
   (wire (pts (xy 119.38 93.98) (xy 119.38 101.6))
     (stroke (width 0) (type solid) (color 0 0 0 0))
@@
     (stroke (width 0) (type solid) (color 0 0 0 0))
   )
-  (wire (pts (xy 172.72 101.6) (xy 180.34 101.6))
-    (stroke (width 0) (type solid) (color 0 0 0 0))
-  )
   (wire (pts (xy 149.86 99.06) (xy 149.86 101.6))
     (stroke (width 0) (type solid) (color 0 0 0 0))
   )
   (wire (pts (xy 106.68 101.6) (xy 119.38 101.6))
-    (stroke (width 0) (type solid) (color 0 0 0 0))
-  )
-  (wire (pts (xy 119.38 132.08) (xy 172.72 132.08))
     (stroke (width 0) (type solid) (color 0 0 0 0))
   )
@@
     (effects (font (size 1.27 1.27)) (justify left))
   )
-  (hierarchical_label "SUBCK" (shape input) (at 106.68 132.08 180)
-    (effects (font (size 1.27 1.27)) (justify right))
-  )
   (symbol (lib_id "Device:R") (at 149.86 118.11 0) (unit 1)
     (in_bom yes) (on_board yes)
@@
     (in_bom yes) (on_board yes)
     (property "Reference" "C1100" (id 0) (at 125.73 87.5792 90))
-    (property "Value" "100nF" (id 1) (at 125.73 89.8906 90))
+    (property "Value" "100nF/25V" (id 1) (at 125.73 89.8906 90))
     (property "Footprint" "Capacitor_SMD:C_0402_1005Metric" (id 2) (at 121.92 94.9452 0)
       (effects (font (size 1.27 1.27)) hide)
@@
     (in_bom yes) (on_board yes)
     (property "Reference" "C1101" (id 0) (at 125.73 102.8192 90))
-    (property "Value" "100nF" (id 1) (at 125.73 105.1306 90))
+    (property "Value" "100nF/25V" (id 1) (at 125.73 105.1306 90))
     (property "Footprint" "Capacitor_SMD:C_0402_1005Metric" (id 2) (at 121.92 110.1852 0)
       (effects (font (size 1.27 1.27)) hide)
@@
       (effects (font (size 1.27 1.27)) (justify right))
     )
-    (property "Footprint" "Capacitor_SMD:C_0603_1608Metric" (id 2) (at 159.0548 81.28 0)
+    (property "Footprint" "Capacitor_SMD:C_0402_1005Metric" (id 2) (at 159.0548 81.28 0)
       (effects (font (size 1.27 1.27)) hide)
     )
@@
     (pin "1")
   )
-  (symbol (lib_id "power:-12V") (at 149.86 124.46 180) (unit 1)
-    (in_bom yes) (on_board yes)
-    (property "Reference" "#PWR0153" (id 0) (at 149.86 127 0)
-      (effects (font (size 1.27 1.27)) hide)
-    )
-    (property "Value" "-12V" (id 1) (at 149.479 128.8542 0))
-    (property "Footprint" "" (id 2) (at 149.86 124.46 0)
-      (effects (font (size 1.27 1.27)) hide)
-    )
-    (property "Datasheet" "" (id 3) (at 149.86 124.46 0)
-      (effects (font (size 1.27 1.27)) hide)
-    )
-    (pin "1")
-  )
   (symbol (lib_id "Device:C") (at 160.02 118.11 180) (unit 1)
     (in_bom yes) (on_board yes)
@@
       (effects (font (size 1.27 1.27)) (justify right))
     )
-    (property "Footprint" "Capacitor_SMD:C_0603_1608Metric" (id 2) (at 159.0548 114.3 0)
+    (property "Footprint" "Capacitor_SMD:C_0402_1005Metric" (id 2) (at 159.0548 114.3 0)
       (effects (font (size 1.27 1.27)) hide)
     )
@@
     (property "Reference" "C1103" (id 0) (at 161.29 95.1992 90))
     (property "Value" "1uF/25V" (id 1) (at 161.29 97.5106 90))
-    (property "Footprint" "Capacitor_SMD:C_0805_2012Metric" (id 2) (at 157.48 102.5652 0)
+    (property "Footprint" "Capacitor_SMD:C_0603_1608Metric" (id 2) (at 157.48 102.5652 0)
       (effects (font (size 1.27 1.27)) hide)
     )
     (property "Datasheet" "~" (id 3) (at 161.29 101.6 0)
-      (effects (font (size 1.27 1.27)) hide)
-    )
-    (pin "1")
-    (pin "2")
-  )
-  (symbol (lib_id "Device:C") (at 115.57 132.08 270) (unit 1)
-    (in_bom yes) (on_board yes)
-    (property "Reference" "C1105" (id 0) (at 115.57 125.6792 90))
-    (property "Value" "1uF/25V" (id 1) (at 115.57 127.9906 90))
-    (property "Footprint" "Capacitor_SMD:C_0805_2012Metric" (id 2) (at 111.76 133.0452 0)
-      (effects (font (size 1.27 1.27)) hide)
-    )
-    (property "Datasheet" "~" (id 3) (at 115.57 132.08 0)
       (effects (font (size 1.27 1.27)) hide)
     )
@@
     (pin "2")
   )
-  (symbol (lib_id "Sitina:+19V") (at 149.86 81.28 0) (unit 1)
-    (in_bom yes) (on_board yes)
-    (property "Reference" "#PWR0157" (id 0) (at 149.86 85.09 0)
-      (effects (font (size 1.27 1.27)) hide)
-    )
-    (property "Value" "+19V" (id 1) (at 150.241 76.8858 0))
+  (symbol (lib_id "power:+15V") (at 149.86 81.28 0) (unit 1)
+    (in_bom yes) (on_board yes)
+    (property "Reference" "#PWR0134" (id 0) (at 149.86 85.09 0)
+      (effects (font (size 1.27 1.27)) hide)
+    )
+    (property "Value" "+15V" (id 1) (at 149.86 77.47 0))
     (property "Footprint" "" (id 2) (at 149.86 81.28 0)
       (effects (font (size 1.27 1.27)) hide)
@@
       (effects (font (size 1.27 1.27)) hide)
     )
+    (pin "1")
+  )
+  (symbol (lib_id "Sitina:-16V") (at 149.86 124.46 180) (unit 1)
+    (in_bom yes) (on_board yes)
+    (property "Reference" "#PWR0132" (id 0) (at 149.86 127 0)
+      (effects (font (size 1.27 1.27)) hide)
+    )
+    (property "Value" "-16V" (id 1) (at 149.86 128.27 0))
+    (property "Footprint" "" (id 2) (at 149.86 124.46 0)
+      (effects (font (size 1.27 1.27)) hide)
+    )
+    (property "Datasheet" "" (id 3) (at 149.86 124.46 0)
+      (effects (font (size 1.27 1.27)) hide)
+    )
