File: Hardware/mainboard/ccd.kicad_sch (KiCad schematic)
At the start: 14 parts, among them J901 AudioJack2, J902 Conn_01x10_MountingPin, SW901 DNP, U901 KAI-1100x

Commit message: New PCB rev
Parts:
- removed J902: Conn_01x10_MountingPin, Connector_FFC-FPC:Hirose_FH12-10S-0.5SH_1x10-1MP_P0.50mm_Horizontal, symbol Connector_Generic_MountingPin:Conn_01x10_MountingPin
- R905: value 6.8 -> 7.5
- SW901: footprint footprints:MXOnly-1U-NoLED -> Connector_PinSocket_2.54mm:PinSocket_1x02_P2.54mm_Vertical
Other:
- moved on the sheet: J901, SW901

Commit message: Update PCB files to rev 0.6 used for production
Parts:
- C901: value 22uF/25V -> 22uF 25V
- R901: value 82K/1% -> 82K 1%
- R902: value 270K/1% -> 270K 1%
- R903: value 200K/1% -> 200K 1%
- R904: value 120K/1% -> 120K 1%
Other:
- company: Copyright 2022 Wenting Zhang -> Copyright 2023 Wenting Zhang
Changed lines of the file:
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@@
   (title_block
     (title "Sitina 1 Mainboard")
-    (date "2022-04-28")
-    (rev "R0.1")
-    (company "Copyright 2022 Wenting Zhang")
+    (date "2023-03-16")
+    (rev "R0.6")
+    (company "Copyright 2023 Wenting Zhang")
     (comment 2 "MERCHANTABILITY, SATISFACTORY QUALITY AND FITNESS FOR A PARTICULAR PURPOSE.")
     (comment 3 "This source is distributed WITHOUT ANY EXPRESS OR IMPLIED WARRANTY, INCLUDING OF")
@@
       (effects (font (size 1.27 1.27)) (justify left))
     )
-    (property "Value" "82K/1%" (at 98.298 65.913 0)
+    (property "Value" "82K 1%" (at 98.298 65.913 0)
       (effects (font (size 1.27 1.27)) (justify left))
     )
@@
       (effects (font (size 1.27 1.27)) (justify left))
     )
-    (property "Value" "200K/1%" (at 110.998 43.053 0)
+    (property "Value" "200K 1%" (at 110.998 43.053 0)
       (effects (font (size 1.27 1.27)) (justify left))
     )
@@
       (effects (font (size 1.27 1.27)) (justify left))
     )
-    (property "Value" "120K/1%" (at 110.998 55.753 0)
+    (property "Value" "120K 1%" (at 110.998 55.753 0)
       (effects (font (size 1.27 1.27)) (justify left))
     )
@@
       (effects (font (size 1.27 1.27)) (justify left))
     )
-    (property "Value" "270K/1%" (at 98.298 78.613 0)
+    (property "Value" "270K 1%" (at 98.298 78.613 0)
       (effects (font (size 1.27 1.27)) (justify left))
     )
@@
       (effects (font (size 1.27 1.27)) (justify left))
     )
-    (property "Value" "22uF/25V" (at 99.441 139.573 0)
-      (effects (font (size 1.27 1.27)) (justify left))
-    )
+    (property "Value" "22uF 25V" (at 99.441 139.573 0)
+      (effects (font (size 1.27 1.27)) (justify left))
+    )
