File: Hardware/mainboard/ccd_power.kicad_sch (KiCad schematic)
At the start: 97 parts, among them U1201 TPS65130RGE, U1202 TPS65130RGE, U1203 LT1964-BYP, U1204 TPS65130RGE, U1205 AP2127K-ADJTRG1, U1206 AP2127K-ADJTRG1

Commit message: New PCB rev
Parts:
- removed C1234: 47uF/16V, Capacitor_SMD:CP_Elec_5x4.5, symbol Sitina-rescue:CP-Device
- removed U1205, U1206: AP2127K-ADJTRG1, Package_TO_SOT_SMD:TSOT-23-5, symbol Regulator_Linear:ADP7142AUJZ
- added C1240: DNP, Capacitor_SMD:C_0402_1005Metric, symbol Device:C
- added C1241: 22uF/25V, Capacitor_SMD:C_0805_2012Metric, symbol Device:C
- added D1216: LED, Diode_SMD:D_0603_1608Metric, symbol Device:LED
- added R1231: 10K, Resistor_SMD:R_0402_1005Metric, symbol Device:R
- added TP1201: TestPoint, TestPoint:TestPoint_Pad_D1.0mm, symbol Connector:TestPoint
- added U1205: LT3023, Package_DFN_QFN:DFN-10-1EP_3x3mm_P0.5mm_EP1.65x2.38mm_ThermalVias, symbol Sitina:LT3023
- C1201, C1202, C1220: footprint Capacitor_SMD:C_0603_1608Metric -> Capacitor_SMD:C_0402_1005Metric
- C1211, C1212, C1214, C1215, C1228: value 30pF -> 22pF
- C1221, C1222: value 10uF -> 220nF; footprint Capacitor_SMD:C_0603_1608Metric -> Capacitor_SMD:C_0402_1005Metric
- C1223: value 100nF -> 2.2uF/25V; footprint Capacitor_SMD:C_0402_1005Metric -> Capacitor_SMD:C_0603_1608Metric
- C1224: value 100nF -> 220nF
- C1229, C1230: value 10uF -> 10nF; footprint Capacitor_SMD:C_0603_1608Metric -> Capacitor_SMD:C_0402_1005Metric
- C1231: value 30pF -> 10uF/25V; footprint Capacitor_SMD:C_0402_1005Metric -> Capacitor_SMD:C_0805_2012Metric
- C1232: value 22uF/25V -> 10uF/25V
- R1203: value 68K/1% -> 36K/1%
- R1204: value 24K/1% -> 68K/1%
- R1210: value 24K/1% -> 22K/1%
- R1214: value 36K/1% -> 49.9K/1%
- R1215: value 24K/1% -> 10K/1%
- R1216: value 24K/1% -> 270K/1%
- R1217: value 27K/1% -> 24K/1%
- R1220: value 49.9K/1% -> 68K/1%
- R1221: value 10K -> 22K/1%
- R1230: value 5.1K/1% -> 10K
Connections:
- net +15V: now also C1229.1, C1231.1, R1216.2, U1205.6 (OUT1); no longer C1211.1, C1216.1, C1236.1, D1201.1 (K), R1209.1, U1201.23 (VPOS)
- net +3V3: no longer C1221.1, C1222.1, C1223.1, C1224.1
- net -4V: now also C1240.2; no longer C1231.2
- net CCD_POWEREN: now also TP1201.1
- net GND: now also C1231.2, R1217.1, C1241.2, D1216.1 (K), U1205.11 (EP), U1205.3 (GND); no longer C1229.2, C1230.2, R1217.2
- net IPSOUT: no longer R1226.2
- net VAB: now also C1230.1, R1214.1, U1205.10 (OUT2); no longer C1228.1, D1205.1 (K), R1220.1, U1204.23 (VPOS)
- net at R1202.1, U1202.11 (PSN), U1202.4 (VIN)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: now also C1222.1
- net at C1228.2, R1221.1, U1204.22 (FBP): now also R1220.2; no longer RV1201.1, RV1201.2
- net at R1215.1: now also RV1201.1, RV1201.2, U1205.2 (ADJ2); no longer R1214.2
- net at RV1201.3: now also R1214.2; no longer R1220.2
- net at R1218.2, R1219.1, U1204.16 (FBN): now also C1240.1; no longer C1231.1
- net at R1213.1, U1204.11 (PSN), U1204.4 (VIN)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: now also C1224.1
- net at R1201.1, U1201.11 (PSN), U1201.4 (VIN)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: now also C1221.1
- net +1V5: no longer names the net of R1216.1
- net +1V5: now also R1217.2, U1205.4 (ADJ1); no longer C1230.1
- removed net +2V: C1229.1, R1214.1
- new net: D1216.2 (A), R1231.1
- new net: C1230.2, U1205.1 (BYP2)
- new net: C1229.2, U1205.5 (BYP1)
- new net +16V: C1211.1, C1216.1, C1223.1, C1236.1, D1201.1 (K), R1209.1, R1231.2, U1201.23 (VPOS), U1205.7 (~{SHDN1}), U1205.8 (IN), U1205.9 (~{SHDN2})
- new net +5V: C1228.1, C1241.1, D1205.1 (K), R1220.1, R1226.2, U1204.23 (VPOS)
Other:
- moved on the sheet: D1215, R1230

Commit message: Update PCB files to rev 0.6 used for production
Parts:
- C1216, C1217, C1218, C1219, C1241: value 22uF/25V -> 22uF 25V
- C1223: value 2.2uF/25V -> 2.2uF 25V
- C1231, C1232: value 10uF/25V -> 10uF 25V
- C1235, C1238, C1239: value 47uF/16V -> 47uF 16V
- C1236: value 33uF/25V -> 33uF 25V
- C1237: value 100uF/6.3V -> 100uF 6.3V
- R1203, R1212: value 36K/1% -> 36K 1%
- R1204, R1220: value 68K/1% -> 68K 1%
- R1205, R1210, R1221: value 22K/1% -> 22K 1%
- R1206, R1209, R1216, R1219: value 270K/1% -> 270K 1%
- R1207: value 27K/1% -> 27K 1%
- R1208, R1211: value 200K/1% -> 200K 1%
- R1214: value 49.9K/1% -> 49.9K 1%
- R1215: value 10K/1% -> 10K 1%
- R1217: value 24K/1% -> 24K 1%
- R1218: value 82K/1% -> 82K 1%
- R1222, R1227: value 5.1K/1% -> 5.1K 1%
Other:
- company: Copyright 2022 Wenting Zhang -> Copyright 2023 Wenting Zhang
Changed lines of the file:
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@@
   (title_block
     (title "Sitina 1 Mainboard")
-    (date "2022-04-28")
-    (rev "R0.1")
-    (company "Copyright 2022 Wenting Zhang")
+    (date "2023-03-16")
+    (rev "R0.6")
+    (company "Copyright 2023 Wenting Zhang")
     (comment 2 "MERCHANTABILITY, SATISFACTORY QUALITY AND FITNESS FOR A PARTICULAR PURPOSE.")
     (comment 3 "This source is distributed WITHOUT ANY EXPRESS OR IMPLIED WARRANTY, INCLUDING OF")
@@
       (effects (font (size 1.27 1.27)) (justify left))
     )
-    (property "Value" "22K/1%" (at 203.708 50.673 0)
+    (property "Value" "22K 1%" (at 203.708 50.673 0)
       (effects (font (size 1.27 1.27)) (justify left))
     )
@@
       (effects (font (size 1.27 1.27)) (justify left))
     )
-    (property "Value" "200K/1%" (at 88.138 116.713 0)
+    (property "Value" "200K 1%" (at 88.138 116.713 0)
       (effects (font (size 1.27 1.27)) (justify left))
     )
@@
       (effects (font (size 1.27 1.27)) (justify left))
     )
-    (property "Value" "22K/1%" (at 98.298 37.973 0)
+    (property "Value" "22K 1%" (at 98.298 37.973 0)
       (effects (font (size 1.27 1.27)) (justify left))
     )
@@
       (effects (font (size 1.27 1.27)) (justify left))
     )
-    (property "Value" "100uF/6.3V" (at 279.4 127 90)
+    (property "Value" "100uF 6.3V" (at 279.4 127 90)
       (effects (font (size 1.27 1.27)) (justify left))
     )
@@
       (effects (font (size 1.27 1.27)) (justify left))
     )
-    (property "Value" "68K/1%" (at 203.708 43.053 0)
+    (property "Value" "68K 1%" (at 203.708 43.053 0)
       (effects (font (size 1.27 1.27)) (justify left))
     )
@@
       (effects (font (size 1.27 1.27)) (justify left))
     )
-    (property "Value" "200K/1%" (at 98.298 98.933 0)
+    (property "Value" "200K 1%" (at 98.298 98.933 0)
       (effects (font (size 1.27 1.27)) (justify left))
     )
@@
       (effects (font (size 1.27 1.27)) (justify left))
     )
-    (property "Value" "22uF/25V" (at 215.011 43.053 0)
+    (property "Value" "22uF 25V" (at 215.011 43.053 0)
       (effects (font (size 1.27 1.27)) (justify left))
     )
@@
       (effects (font (size 1.27 1.27)) (justify left))
     )
-    (property "Value" "10K/1%" (at 179.578 142.113 0)
+    (property "Value" "10K 1%" (at 179.578 142.113 0)
       (effects (font (size 1.27 1.27)) (justify left))
     )
@@
       (effects (font (size 1.27 1.27)) (justify left))
     )
-    (property "Value" "2.2uF/25V" (at 147.32 116.84 0)
+    (property "Value" "2.2uF 25V" (at 147.32 116.84 0)
       (effects (font (size 1.27 1.27)) (justify left))
     )
@@
       (effects (font (size 1.27 1.27)))
     )
-    (property "Value" "270K/1%" (at 193.04 109.22 0)
+    (property "Value" "270K 1%" (at 193.04 109.22 0)
       (effects (font (size 1.27 1.27)))
     )
@@
       (effects (font (size 1.27 1.27)) (justify left))
     )
-    (property "Value" "36K/1%" (at 98.298 106.553 0)
+    (property "Value" "36K 1%" (at 98.298 106.553 0)
       (effects (font (size 1.27 1.27)) (justify left))
     )
@@
       (effects (font (size 1.27 1.27)))
     )
-    (property "Value" "5.1K/1%" (at 247.65 78.74 90)
+    (property "Value" "5.1K 1%" (at 247.65 78.74 90)
       (effects (font (size 1.27 1.27)))
     )
@@
       (effects (font (size 1.27 1.27)) (justify left))
     )
-    (property "Value" "27K/1%" (at 88.138 109.093 0)
+    (property "Value" "27K 1%" (at 88.138 109.093 0)
       (effects (font (size 1.27 1.27)) (justify left))
     )
@@
       (effects (font (size 1.27 1.27)) (justify left))
     )
-    (property "Value" "270K/1%" (at 88.138 48.133 0)
+    (property "Value" "270K 1%" (at 88.138 48.133 0)
       (effects (font (size 1.27 1.27)) (justify left))
     )
@@
       (effects (font (size 1.27 1.27)) (justify left))
     )
-    (property "Value" "49.9K/1%" (at 179.578 124.333 0)
+    (property "Value" "49.9K 1%" (at 179.578 124.333 0)
       (effects (font (size 1.27 1.27)) (justify left))
     )
@@
       (effects (font (size 1.27 1.27)) (justify left))
     )
-    (property "Value" "22uF/25V" (at 109.601 116.713 0)
+    (property "Value" "22uF 25V" (at 109.601 116.713 0)
       (effects (font (size 1.27 1.27)) (justify left))
     )
@@
       (effects (font (size 1.27 1.27)) (justify left))
     )
-    (property "Value" "47uF/16V" (at 246.38 134.62 90)
+    (property "Value" "47uF 16V" (at 246.38 134.62 90)
       (effects (font (size 1.27 1.27)) (justify left))
     )
@@
       (effects (font (size 1.27 1.27)))
     )
-    (property "Value" "5.1K/1%" (at 246.38 33.02 90)
+    (property "Value" "5.1K 1%" (at 246.38 33.02 90)
       (effects (font (size 1.27 1.27)))
     )
@@
       (effects (font (size 1.27 1.27)) (justify left))
     )
-    (property "Value" "47uF/16V" (at 279.4 134.62 90)
+    (property "Value" "47uF 16V" (at 279.4 134.62 90)
       (effects (font (size 1.27 1.27)) (justify left))
     )
@@
       (effects (font (size 1.27 1.27)) (justify left))
     )
-    (property "Value" "270K/1%" (at 193.548 60.833 0)
+    (property "Value" "270K 1%" (at 193.548 60.833 0)
       (effects (font (size 1.27 1.27)) (justify left))
     )
@@
       (effects (font (size 1.27 1.27)))
     )
-    (property "Value" "68K/1%" (at 87.63 167.64 0)
+    (property "Value" "68K 1%" (at 87.63 167.64 0)
       (effects (font (size 1.27 1.27)))
     )
@@
       (effects (font (size 1.27 1.27)) (justify left))
     )
-    (property "Value" "270K/1%" (at 98.298 30.353 0)
+    (property "Value" "270K 1%" (at 98.298 30.353 0)
       (effects (font (size 1.27 1.27)) (justify left))
     )
@@
       (effects (font (size 1.27 1.27)) (justify left))
     )
-    (property "Value" "33uF/25V" (at 246.38 142.24 90)
+    (property "Value" "33uF 25V" (at 246.38 142.24 90)
       (effects (font (size 1.27 1.27)) (justify left))
     )
@@
       (effects (font (size 1.27 1.27)) (justify left))
     )
-    (property "Value" "10uF/25V" (at 210.82 109.22 0)
+    (property "Value" "10uF 25V" (at 210.82 109.22 0)
       (effects (font (size 1.27 1.27)) (justify left))
     )
@@
       (effects (font (size 1.27 1.27)) (justify left))
     )
-    (property "Value" "22uF/25V" (at 109.601 98.933 0)
+    (property "Value" "22uF 25V" (at 109.601 98.933 0)
       (effects (font (size 1.27 1.27)) (justify left))
     )
@@
       (effects (font (size 1.27 1.27)) (justify left))
     )
-    (property "Value" "10uF/25V" (at 210.82 124.46 0)
+    (property "Value" "10uF 25V" (at 210.82 124.46 0)
       (effects (font (size 1.27 1.27)) (justify left))
     )
@@
       (effects (font (size 1.27 1.27)) (justify left))
     )
-    (property "Value" "22uF/25V" (at 109.601 48.133 0)
+    (property "Value" "22uF 25V" (at 109.601 48.133 0)
       (effects (font (size 1.27 1.27)) (justify left))
     )
@@
       (effects (font (size 1.27 1.27)) (justify left))
     )
-    (property "Value" "22uF/25V" (at 109.601 30.353 0)
+    (property "Value" "22uF 25V" (at 109.601 30.353 0)
       (effects (font (size 1.27 1.27)) (justify left))
     )
@@
       (effects (font (size 1.27 1.27)))
     )
-    (property "Value" "36K/1%" (at 87.63 160.02 0)
+    (property "Value" "36K 1%" (at 87.63 160.02 0)
       (effects (font (size 1.27 1.27)))
     )
@@
       (effects (font (size 1.27 1.27)))
     )
-    (property "Value" "24K/1%" (at 193.04 119.38 0)
+    (property "Value" "24K 1%" (at 193.04 119.38 0)
       (effects (font (size 1.27 1.27)))
     )
@@
       (effects (font (size 1.27 1.27)) (justify left))
     )
-    (property "Value" "82K/1%" (at 193.548 53.213 0)
+    (property "Value" "82K 1%" (at 193.548 53.213 0)
       (effects (font (size 1.27 1.27)) (justify left))
     )
@@
       (effects (font (size 1.27 1.27)) (justify left))
     )
-    (property "Value" "22K/1%" (at 88.138 40.513 0)
+    (property "Value" "22K 1%" (at 88.138 40.513 0)
       (effects (font (size 1.27 1.27)) (justify left))
     )
@@
       (effects (font (size 1.27 1.27)) (justify left))
     )
-    (property "Value" "47uF/16V" (at 279.4 142.24 90)
+    (property "Value" "47uF 16V" (at 279.4 142.24 90)
       (effects (font (size 1.27 1.27)) (justify left))
     )

Commit message: Working towards pcb r0.7
Connections:
- net IPSOUT renamed +SYS
Changed lines of the file:
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@@
-    )
-  )
-  (symbol (lib_id "symbols:IPSOUT") (at 30.48 33.02 0) (unit 1)
-    (in_bom yes) (on_board yes) (dnp no)
-    (property "Reference" "#PWR01203" (at 30.48 36.83 0)
-      (effects (font (size 1.27 1.27)) hide)
-    )
-    (property "Value" "IPSOUT" (at 30.9118 28.6258 0)
-      (effects (font (size 1.27 1.27)))
-    )
-    (property "Footprint" "" (at 30.48 33.02 0)
-      (effects (font (size 1.27 1.27)) hide)
-    )
-    (property "Datasheet" "" (at 30.48 33.02 0)
-      (effects (font (size 1.27 1.27)) hide)
-    )
-    (pin "1")
-    (instances
-      (project "pcb"
-        (path "/ba41827b-f176-424d-b6d5-0b0e1ddda097/a00c2049-0a3f-4994-b4b1-e2d67645b8de"
-          (reference "#PWR01203") (unit 1)
-        )
-      )
     )
   )
@@
   (symbol (lib_id "Device:L") (at 184.15 74.93 0) (mirror x) (unit 1)
     (in_bom yes) (on_board yes) (dnp no)
-    (property "Reference" "L1206" (at 186.69 73.66 0)
+    (property "Reference" "L1206" (at 187.96 73.66 0)
       (effects (font (size 1.27 1.27)))
     )
@@
         (path "/ba41827b-f176-424d-b6d5-0b0e1ddda097/a00c2049-0a3f-4994-b4b1-e2d67645b8de"
           (reference "#PWR01248") (unit 1)
+        )
+      )
+    )
+  )
+  (symbol (lib_id "symbols:+SYS") (at 30.48 101.6 0) (unit 1)
+    (in_bom yes) (on_board yes) (dnp no)
+    (property "Reference" "#PWR0508" (at 30.48 105.41 0)
+      (effects (font (size 1.27 1.27)) hide)
+    )
+    (property "Value" "+SYS" (at 30.48 97.79 0)
+      (effects (font (size 1.27 1.27)))
+    )
+    (property "Footprint" "" (at 30.48 101.6 0)
+      (effects (font (size 1.27 1.27)) hide)
+    )
+    (property "Datasheet" "" (at 30.48 101.6 0)
+      (effects (font (size 1.27 1.27)) hide)
+    )
+    (pin "1")
+    (instances
+      (project "pcb"
+        (path "/ba41827b-f176-424d-b6d5-0b0e1ddda097/00000000-0000-0000-0000-00005d4c99f9"
+          (reference "#PWR0508") (unit 1)
+        )
+        (path "/ba41827b-f176-424d-b6d5-0b0e1ddda097/a00c2049-0a3f-4994-b4b1-e2d67645b8de"
+          (reference "#PWR0512") (unit 1)
         )
       )
@@
         (path "/ba41827b-f176-424d-b6d5-0b0e1ddda097/a00c2049-0a3f-4994-b4b1-e2d67645b8de"
           (reference "RV1201") (unit 1)
+        )
+      )
+    )
+  )
+  (symbol (lib_id "symbols:+SYS") (at 135.89 45.72 0) (unit 1)
+    (in_bom yes) (on_board yes) (dnp no)
+    (property "Reference" "#PWR0508" (at 135.89 49.53 0)
+      (effects (font (size 1.27 1.27)) hide)
+    )
+    (property "Value" "+SYS" (at 135.89 41.91 0)
+      (effects (font (size 1.27 1.27)))
+    )
+    (property "Footprint" "" (at 135.89 45.72 0)
+      (effects (font (size 1.27 1.27)) hide)
+    )
+    (property "Datasheet" "" (at 135.89 45.72 0)
+      (effects (font (size 1.27 1.27)) hide)
+    )
+    (pin "1")
+    (instances
+      (project "pcb"
+        (path "/ba41827b-f176-424d-b6d5-0b0e1ddda097/00000000-0000-0000-0000-00005d4c99f9"
+          (reference "#PWR0508") (unit 1)
+        )
+        (path "/ba41827b-f176-424d-b6d5-0b0e1ddda097/a00c2049-0a3f-4994-b4b1-e2d67645b8de"
+          (reference "#PWR0513") (unit 1)
         )
       )
@@
     )
   )
-  (symbol (lib_id "symbols:IPSOUT") (at 135.89 45.72 0) (unit 1)
-    (in_bom yes) (on_board yes) (dnp no)
-    (property "Reference" "#PWR01230" (at 135.89 49.53 0)
-      (effects (font (size 1.27 1.27)) hide)
-    )
-    (property "Value" "IPSOUT" (at 136.3218 41.3258 0)
-      (effects (font (size 1.27 1.27)))
-    )
-    (property "Footprint" "" (at 135.89 45.72 0)
-      (effects (font (size 1.27 1.27)) hide)
-    )
-    (property "Datasheet" "" (at 135.89 45.72 0)
-      (effects (font (size 1.27 1.27)) hide)
-    )
-    (pin "1")
-    (instances
-      (project "pcb"
-        (path "/ba41827b-f176-424d-b6d5-0b0e1ddda097/a00c2049-0a3f-4994-b4b1-e2d67645b8de"
-          (reference "#PWR01230") (unit 1)
-        )
-      )
-    )
-  )
   (symbol (lib_id "Device:C") (at 106.68 97.79 0) (unit 1)
     (in_bom yes) (on_board yes) (dnp no)
@@
         (path "/ba41827b-f176-424d-b6d5-0b0e1ddda097/a00c2049-0a3f-4994-b4b1-e2d67645b8de"
           (reference "D1210") (unit 1)
+        )
+      )
+    )
+  )
+  (symbol (lib_id "symbols:+SYS") (at 30.48 33.02 0) (unit 1)
+    (in_bom yes) (on_board yes) (dnp no)
+    (property "Reference" "#PWR0508" (at 30.48 36.83 0)
+      (effects (font (size 1.27 1.27)) hide)
+    )
+    (property "Value" "+SYS" (at 30.48 29.21 0)
+      (effects (font (size 1.27 1.27)))
+    )
+    (property "Footprint" "" (at 30.48 33.02 0)
+      (effects (font (size 1.27 1.27)) hide)
+    )
+    (property "Datasheet" "" (at 30.48 33.02 0)
+      (effects (font (size 1.27 1.27)) hide)
+    )
+    (pin "1")
+    (instances
+      (project "pcb"
+        (path "/ba41827b-f176-424d-b6d5-0b0e1ddda097/00000000-0000-0000-0000-00005d4c99f9"
+          (reference "#PWR0508") (unit 1)
+        )
+        (path "/ba41827b-f176-424d-b6d5-0b0e1ddda097/a00c2049-0a3f-4994-b4b1-e2d67645b8de"
+          (reference "#PWR0511") (unit 1)
         )
       )
@@
         )
       )
-    )
-  )
-  (symbol (lib_id "symbols:IPSOUT") (at 30.48 101.6 0) (unit 1)
-    (in_bom yes) (on_board yes) (dnp no)
-    (property "Reference" "#PWR01204" (at 30.48 105.41 0)
-      (effects (font (size 1.27 1.27)) hide)
-    )
-    (property "Value" "IPSOUT" (at 30.9118 97.2058 0)
-      (effects (font (size 1.27 1.27)))
-    )
-    (property "Footprint" "" (at 30.48 101.6 0)
-      (effects (font (size 1.27 1.27)) hide)
-    )
-    (property "Datasheet" "" (at 30.48 101.6 0)
-      (effects (font (size 1.27 1.27)) hide)
-    )
-    (pin "1")
-    (instances
-      (project "pcb"
-        (path "/ba41827b-f176-424d-b6d5-0b0e1ddda097/a00c2049-0a3f-4994-b4b1-e2d67645b8de"
-          (reference "#PWR01204") (unit 1)
-        )
-      )
