File: Hardware/mainboard/ccd_driver.kicad_sch (KiCad schematic)
At the start: 61 parts, among them Q801 BC847BPN, U801 74HC4053, U802 74HC2G17, U803 74HC2G17, U804 74HC2G17, U805 74HC2G17, U806 74HC2G17, U807 74HC2G17, U808 CD4053B, U809 UCC27517A, U810 UCC27517A, U811 UCC27517A, U812 UCC27517A

Commit message: New PCB rev
Connections:
- net +15V renamed +16V
- net IPSOUT renamed +5V

Commit message: Update PCB files to rev 0.6 used for production
Parts:
- C808: value 1uF/25V -> 1uF 25V
Other:
- company: Copyright 2022 Wenting Zhang -> Copyright 2023 Wenting Zhang
Changed lines of the file:
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@@
   (title_block
     (title "Sitina 1 Mainboard")
-    (date "2022-04-28")
-    (rev "R0.1")
-    (company "Copyright 2022 Wenting Zhang")
+    (date "2023-03-16")
+    (rev "R0.6")
+    (company "Copyright 2023 Wenting Zhang")
     (comment 2 "MERCHANTABILITY, SATISFACTORY QUALITY AND FITNESS FOR A PARTICULAR PURPOSE.")
     (comment 3 "This source is distributed WITHOUT ANY EXPRESS OR IMPLIED WARRANTY, INCLUDING OF")
@@
       (effects (font (size 1.27 1.27)))
     )
-    (property "Value" "1uF/25V" (at 92.71 158.4706 90)
+    (property "Value" "1uF 25V" (at 92.71 158.4706 90)
       (effects (font (size 1.27 1.27)))
     )

Commit message: Working towards pcb r0.7
Parts:
- removed C819: 10nF, Capacitor_SMD:C_0402_1005Metric, symbol Device:C
- removed R812: 0.1, Resistor_SMD:R_0603_1608Metric, symbol Device:R
- removed U809, U810, U811, U812: UCC27517A, Package_TO_SOT_SMD:SOT-23-5, symbol Sitina:UCC27517A
- added C504, C505, C506, C507, C508, C509, C510, C511: 1nF, Capacitor_SMD:C_0402_1005Metric, symbol Device:C
- added D501, D502, D503, D504: BAT54S, Package_TO_SOT_SMD:SOT-23, symbol Diode:BAT54S
- added Q501, Q503, Q505, Q507: Q_PMOS_DGS, symbol Device:Q_PMOS_DGS
- added Q502, Q504, Q506, Q508: Q_NMOS_DGS, symbol Device:Q_NMOS_DGS
- added R504, R505, R506, R507, R508, R509, R510, R511: 220, Resistor_SMD:R_0402_1005Metric, symbol Device:R
Connections:
- net +5V: now also Q507.3 (S)
- net +8V: now also Q503.3 (S)
- net -9V: now also C822.1, Q502.3 (S), Q506.3 (S), Q508.3 (S); no longer C822.2
- net FDGS: now also D504.3 (COM), R510.2, R511.1
- net FDG_CCD: now also C510.1, C511.2, Q507.1 (D), Q508.1 (D)
- net GND: now also C822.2, Q501.3 (S), Q504.3 (S); no longer C822.1
- net V1S: now also D501.3 (COM), R504.2, R505.1
- net V1_CCD: now also C504.1, C505.2, Q501.1 (D), Q502.1 (D)
- net V23: now also D502.3 (COM), R506.2, R507.1
- net V2S: now also D503.3 (COM), R508.2, R509.1
- net V2_CCD: now also C508.1, C509.2, Q505.1 (D), Q506.1 (D)
- new net: C510.2, D504.2 (K), Q507.2 (G), R510.1
- new net: C508.2, D503.2 (K), Q505.2 (G), R508.1
- new net: C511.1, D504.1 (A), Q508.2 (G), R511.2
- new net: C509.1, D503.1 (A), Q506.2 (G), R509.2
- new net: C505.1, D501.1 (A), Q502.2 (G), R505.2
- new net: C507.1, D502.1 (A), Q504.2 (G), R507.2
- new net: C506.2, D502.2 (K), Q503.2 (G), R506.1
- new net: C504.2, D501.2 (K), Q501.2 (G), R504.1
- new net: C506.1, C507.2, Q503.1 (D), Q504.1 (D), Q505.3 (S)
Other:
- moved on the sheet: C815, C816, C817, C818, C820, C821, C822, R808, R809, R810, R811, U808

Commit message: Fix vclock voltage shifter swing
Connections:
- net +3V3: no longer U808.16 (VDD)
- net +5V: now also U808.13 (X1), U808.16 (VDD)
- net -4V: no longer U808.1 (Y1), U808.13 (X1), U808.3 (Z1)
- net GND: now also U808.1 (Y1), U808.3 (Z1)
Changed lines of the file:
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@@
   (junction (at 223.52 101.6) (diameter 0) (color 0 0 0 0)
   )
-  (junction (at 167.64 124.46) (diameter 0) (color 0 0 0 0)
-  )
   (junction (at 50.8 106.68) (diameter 0) (color 0 0 0 0)
   )
@@
   (junction (at 121.92 50.8) (diameter 0) (color 0 0 0 0)
   )
-  (junction (at 167.64 132.08) (diameter 0) (color 0 0 0 0)
-  )
   (junction (at 48.26 68.58) (diameter 0) (color 0 0 0 0)
   )
@@
   (junction (at 83.82 35.56) (diameter 0) (color 0 0 0 0)
   )
+  (junction (at 167.64 132.08) (diameter 0) (color 0 0 0 0)
+  )
   (junction (at 91.44 124.46) (diameter 0) (color 0 0 0 0)
   )
@@
     (stroke (width 0) (type default))
   )
-  (wire (pts (xy 167.64 119.38) (xy 167.64 124.46))
-    (stroke (width 0) (type default))
-  )
   (wire (pts (xy 60.96 170.18) (xy 63.5 170.18))
     (stroke (width 0) (type solid))
@@
     (stroke (width 0) (type solid))
   )
-  (wire (pts (xy 167.64 124.46) (xy 167.64 132.08))
-    (stroke (width 0) (type default))
-  )
   (wire (pts (xy 243.84 33.02) (xy 246.38 33.02))
     (stroke (width 0) (type default))
@@
     )
   )
-  (symbol (lib_id "power:+3V3") (at 185.42 114.3 0) (unit 1)
-    (in_bom yes) (on_board yes) (dnp no) (fields_autoplaced)
-    (property "Reference" "#PWR0828" (at 185.42 118.11 0)
-      (effects (font (size 1.27 1.27)) hide)
-    )
-    (property "Value" "+3V3" (at 185.42 109.22 0)
-      (effects (font (size 1.27 1.27)))
-    )
-    (property "Footprint" "" (at 185.42 114.3 0)
-      (effects (font (size 1.27 1.27)) hide)
-    )
-    (property "Datasheet" "" (at 185.42 114.3 0)
-      (effects (font (size 1.27 1.27)) hide)
-    )
-    (pin "1")
-    (instances
-      (project "pcb"
-        (path "/ba41827b-f176-424d-b6d5-0b0e1ddda097/45611ff2-2603-4e18-a895-b1c61ddae1cc"
-          (reference "#PWR0828") (unit 1)
-        )
-      )
-    )
-  )
   (symbol (lib_id "Sitina:+2V") (at 121.92 41.91 0) (unit 1)
     (in_bom yes) (on_board yes) (dnp no)
@@
     )
   )
-  (symbol (lib_id "Sitina:-4V") (at 167.64 119.38 0) (unit 1)
-    (in_bom yes) (on_board yes) (dnp no)
-    (property "Reference" "#PWR0823" (at 167.64 123.19 0)
-      (effects (font (size 1.27 1.27)) hide)
-    )
-    (property "Value" "-4V" (at 168.021 114.9858 0)
-      (effects (font (size 1.27 1.27)))
-    )
-    (property "Footprint" "" (at 167.64 119.38 0)
-      (effects (font (size 1.27 1.27)) hide)
-    )
-    (property "Datasheet" "" (at 167.64 119.38 0)
-      (effects (font (size 1.27 1.27)) hide)
-    )
-    (pin "1")
-    (instances
-      (project "pcb"
-        (path "/ba41827b-f176-424d-b6d5-0b0e1ddda097/45611ff2-2603-4e18-a895-b1c61ddae1cc"
-          (reference "#PWR0823") (unit 1)
-        )
-      )
-    )
-  )
   (symbol (lib_id "Device:C") (at 57.15 154.94 270) (unit 1)
     (in_bom yes) (on_board yes) (dnp no)
@@
     )
   )
+  (symbol (lib_id "power:+5V") (at 167.64 124.46 90) (unit 1)
+    (in_bom yes) (on_board yes) (dnp no)
+    (property "Reference" "#PWR0526" (at 171.45 124.46 0)
+      (effects (font (size 1.27 1.27)) hide)
+    )
+    (property "Value" "+5V" (at 165.1 124.46 90)
+      (effects (font (size 1.27 1.27)) (justify left))
+    )
+    (property "Footprint" "" (at 167.64 124.46 0)
+      (effects (font (size 1.27 1.27)) hide)
+    )
+    (property "Datasheet" "" (at 167.64 124.46 0)
+      (effects (font (size 1.27 1.27)) hide)
+    )
+    (pin "1")
+    (instances
+      (project "pcb"
+        (path "/ba41827b-f176-424d-b6d5-0b0e1ddda097/45611ff2-2603-4e18-a895-b1c61ddae1cc"
+          (reference "#PWR0526") (unit 1)
+        )
+      )
+    )
+  )
   (symbol (lib_id "power:-9V") (at 168.91 96.52 180) (unit 1)
     (in_bom yes) (on_board yes) (dnp no)
@@
     )
   )
+  (symbol (lib_id "power:+5V") (at 185.42 114.3 0) (unit 1)
+    (in_bom yes) (on_board yes) (dnp no)
+    (property "Reference" "#PWR0527" (at 185.42 118.11 0)
+      (effects (font (size 1.27 1.27)) hide)
+    )
+    (property "Value" "+5V" (at 182.88 110.49 0)
+      (effects (font (size 1.27 1.27)) (justify left))
+    )
+    (property "Footprint" "" (at 185.42 114.3 0)
+      (effects (font (size 1.27 1.27)) hide)
+    )
+    (property "Datasheet" "" (at 185.42 114.3 0)
+      (effects (font (size 1.27 1.27)) hide)
+    )
+    (pin "1")
+    (instances
+      (project "pcb"
+        (path "/ba41827b-f176-424d-b6d5-0b0e1ddda097/45611ff2-2603-4e18-a895-b1c61ddae1cc"
+          (reference "#PWR0527") (unit 1)
+        )
+      )
+    )
+  )
   (symbol (lib_id "power:GND") (at 48.26 106.68 0) (unit 1)
     (in_bom yes) (on_board yes) (dnp no)
@@
         )
       )
+    )
+  )
+  (symbol (lib_id "power:GND") (at 167.64 132.08 270) (unit 1)
+    (in_bom yes) (on_board yes) (dnp no)
+    (property "Reference" "#PWR0525" (at 161.29 132.08 0)
+      (effects (font (size 1.27 1.27)) hide)
+    )
+    (property "Value" "GND" (at 162.56 132.08 90)
+      (effects (font (size 1.27 1.27)))
+    )
+    (property "Footprint" "" (at 167.64 132.08 0)
+      (effects (font (size 1.27 1.27)) hide)
+    )
+    (property "Datasheet" "" (at 167.64 132.08 0)
+      (effects (font (size 1.27 1.27)) hide)
+    )
+    (pin "1")
+    (instances
+      (project "pcb"
+        (path "/ba41827b-f176-424d-b6d5-0b0e1ddda097/45611ff2-2603-4e18-a895-b1c61ddae1cc"
+          (reference "#PWR0525") (unit 1)
+        )
+      )

Commit message: Update CCD V Driver, New Powertree Documentation Page
Parts:
- removed C818, C820, C821: 100nF, Capacitor_SMD:C_0402_1005Metric, symbol Device:C
- removed Q501, Q503, Q505, Q507: Q_PMOS_DGS, symbol Device:Q_PMOS_DGS
- removed Q502, Q504, Q506, Q508: Q_NMOS_DGS, symbol Device:Q_NMOS_DGS
- added C514, C515, C516, C517: 100nF, Capacitor_SMD:C_0402_1005Metric, symbol Device:C
- added U504, U505, U506, U507: IRF9389/7309, Package_SO:SOIC-8_3.9x4.9mm_P1.27mm, symbol symbols:IRF9389BF
Connections:
- net +5V: now also C515.1, U506.3 (SP)
- net +8V: now also C516.2, U504.3 (SP)
- net -9V: now also C514.2, C517.2, U505.1 (SN), U506.1 (SN), U507.1 (SN)
- net FDG_CCD: now also U506.5 (DP), U506.6 (DP), U506.7 (DN), U506.8 (DN)
- net GND: now also C514.1, C515.2, C516.1, C517.1, U504.1 (SN), U507.3 (SP)
- net V1_CCD: now also U507.5 (DP), U507.6 (DP), U507.7 (DN), U507.8 (DN)
- net V2_CCD: now also U505.5 (DP), U505.6 (DP), U505.7 (DN), U505.8 (DN)
- net at C510.2, D504.2 (K), R510.1: now also U506.4 (GP)
- net at C508.2, D503.2 (K), R508.1: now also U505.4 (GP)
- net at C511.1, D504.1 (A), R511.2: now also U506.2 (GN)
- net at C509.1, D503.1 (A), R509.2: now also U505.2 (GN)
- net at C505.1, D501.1 (A), R505.2: now also U507.2 (GN)
- net at C507.1, D502.1 (A), R507.2: now also U504.2 (GN)
- net at C506.2, D502.2 (K), R506.1: now also U504.4 (GP)
- net at C504.2, D501.2 (K), R504.1: now also U507.4 (GP)
- net at C506.1, C507.2: now also U504.5 (DP), U504.6 (DP), U504.7 (DN), U504.8 (DN), U505.3 (SP)
Other:
- moved on the sheet: C504, C505, C506, C507, C510, C511, C815, C816, C817, C822, D501, D502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
