File: Hardware/mainboard/ddr.kicad_sch (KiCad schematic)
At the start: 35 parts, among them U100 MCIMX6Y2DVM09AB, U202 MT41K256M16HA

Commit message: New PCB rev
Parts:
- removed C201, C202, C203, C204, C207, C208, C210, C212, C213, C216, C217, C221, C222, C225, C226, C229, C230, C235, C236: 220nF, Capacitor_SMD:C_0402_1005Metric, symbol Device:C
- removed C205, C239, C240: 22uF, Capacitor_SMD:C_0603_1608Metric, symbol Device:C
- removed C206, C233, C234: 100nF, Capacitor_SMD:C_0402_1005Metric, symbol Device:C
- removed C220: 4.7uF, Capacitor_SMD:C_0603_1608Metric, symbol Device:C
- removed R201, R204: 240 1%, Resistor_SMD:R_0402_1005Metric, symbol Device:R
- removed R202, R203: 10K, Resistor_SMD:R_0402_1005Metric, symbol Device:R
- removed R205: 470, Resistor_SMD:R_0402_1005Metric, symbol Device:R
- removed R206, R207: 1.5K/0.5%, Resistor_SMD:R_0402_1005Metric, symbol Device:R
- removed U100: MCIMX6Y2DVM09AB, footprints:BGA-289_17x17_14.0x14.0mm, symbol symbols:MCIMX6Y7DVM09AB
- removed U202: MT41K256M16HA, footprints:BGA-96_9.0x14.0mm_P0.8mm, symbol symbols:MT41K256M16HA
- added C404, C405: 4.7uF, Capacitor_SMD:C_0402_1005Metric, symbol Device:C
- added C406, C407: 2.2uF, Capacitor_SMD:C_0402_1005Metric, symbol Device:C
- added C408: 10uF, Capacitor_SMD:C_0402_1005Metric, symbol Device:C
- added C409, C410, C411, C412, C413, C414, C415: 100nF, Capacitor_SMD:C_0402_1005Metric, symbol Device:C
- added TP401, TP402: TestPoint, footprints:TestPoint_Pad_D0.5mm, symbol Connector:TestPoint
- added U301: MIMXRT1176DVMAA, footprints:BGA-289_17x17_14.0x14.0mm, symbol symbols:MIMXRT1176DVMAA
- added U402: MT48H16M32LFB5-6 or IS42VM32160E-6 or W989D2DBJX6, footprints:BGA-90_9x15_8.0x13.0mm, symbol symbols:IS42S32800J-xB
Connections:
- net GND: now also C404.2, C405.2, C406.2, C407.2, C408.2, C409.2, C410.2, C411.2, C412.2, C413.2, C414.2, C415.2, U402.A3 (VSS), U402.B3 (VSSQ), U402.B8 (VSSQ), U402.C1 (VSSQ), U402.D1 (VSSQ), U402.E9 (VSSQ), U402.F1 (VSS), U402.L3 (VSS), U402.L9 (VSSQ), U402.M1 (VSSQ), U402.N1 (VSSQ), U402.P3 (VSSQ), U402.P8 (VSSQ), U402.R3 (VSS)
- new net: TP401.1, U301.J2 (GPIO_EMC_B1_39)
- new net: TP402.1, U301.N3 (GPIO_EMC_B2_18)
- new net +1V8: C404.1, C405.1, C406.1, C407.1, C408.1, C409.1, C410.1, C411.1, C412.1, C413.1, C414.1, C415.1, U301.F6 (NVCC_EMC1), U301.F7 (NVCC_EMC1), U301.G6 (NVCC_EMC1), U301.H6 (NVCC_EMC2), U301.J6 (NVCC_EMC2), U402.A7 (VDD), U402.B2 (VDDQ), U402.B7 (VDDQ), U402.C9 (VDDQ), U402.D9 (VDDQ), U402.E1 (VDDQ), U402.F9 (VDD), U402.L1 (VDDQ), U402.L7 (VDD), U402.M9 (VDDQ), U402.N9 (VDDQ), U402.P2 (VDDQ), U402.P7 (VDDQ), U402.R7 (VDD)
- new net SDRAM_A0: U301.A3 (GPIO_EMC_B1_09), U402.G8 (A0)
- new net SDRAM_A1: U301.A2 (GPIO_EMC_B1_10), U402.G9 (A1)
- new net SDRAM_A10: U301.B2 (GPIO_EMC_B1_23), U402.G7 (A10)
- new net SDRAM_A11: U301.C4 (GPIO_EMC_B1_19), U402.H9 (A11)
- new net SDRAM_A12: U301.C3 (GPIO_EMC_B1_20), U402.H3 (A12)
- new net SDRAM_A2: U301.C2 (GPIO_EMC_B1_11), U402.F7 (A2)
- new net SDRAM_A3: U301.C5 (GPIO_EMC_B1_12), U402.F3 (A3)
- new net SDRAM_A4: U301.D5 (GPIO_EMC_B1_13), U402.G1 (A4)
- new net SDRAM_A5: U301.B1 (GPIO_EMC_B1_14), U402.G2 (A5)
- new net SDRAM_A6: U301.C1 (GPIO_EMC_B1_15), U402.G3 (A6)
- new net SDRAM_A7: U301.D3 (GPIO_EMC_B1_16), U402.H1 (A7)
- new net SDRAM_A8: U301.B3 (GPIO_EMC_B1_17), U402.H2 (A8)
- new net SDRAM_A9: U301.B4 (GPIO_EMC_B1_18), U402.J3 (A9)
- new net SDRAM_BA0: U301.G2 (GPIO_EMC_B1_21), U402.J7 (BA0)
- new net SDRAM_BA1: U301.H2 (GPIO_EMC_B1_22), U402.H8 (BA1)
- new net SDRAM_CAS: U301.J5 (GPIO_EMC_B1_24), U402.K7 (~{CAS})
- new net SDRAM_CKE: U301.G5 (GPIO_EMC_B1_27), U402.J2 (CKE)
- new net SDRAM_CLK: U301.J3 (GPIO_EMC_B1_26), U402.J1 (CLK)
- new net SDRAM_CS0: U301.E6 (GPIO_EMC_B1_29), U402.J8 (~{CS})
- new net SDRAM_D0: U301.F3 (GPIO_EMC_B1_00), U402.R8 (DQ0)
- new net SDRAM_D1: U301.F2 (GPIO_EMC_B1_01), U402.N7 (DQ1)
- new net SDRAM_D10: U301.D1 (GPIO_EMC_B1_32), U402.M2 (DQ10)
- new net SDRAM_D11: U301.E2 (GPIO_EMC_B1_33), U402.P1 (DQ11)
- new net SDRAM_D12: U301.E1 (GPIO_EMC_B1_34), U402.N2 (DQ12)
- new net SDRAM_D13: U301.F1 (GPIO_EMC_B1_35), U402.R1 (DQ13)
- new net SDRAM_D14: U301.G1 (GPIO_EMC_B1_36), U402.N3 (DQ14)
- new net SDRAM_D15: U301.H1 (GPIO_EMC_B1_37), U402.R2 (DQ15)
- new net SDRAM_D16: U301.K2 (GPIO_EMC_B2_00), U402.E8 (DQ16)
- new net SDRAM_D17: U301.K4 (GPIO_EMC_B2_01), U402.D7 (DQ17)
- new net SDRAM_D18: U301.K3 (GPIO_EMC_B2_02), U402.D8 (DQ18)
- new net SDRAM_D19: U301.R1 (GPIO_EMC_B2_03), U402.B9 (DQ19)
- new net SDRAM_D2: U301.G4 (GPIO_EMC_B1_02), U402.R9 (DQ2)
- new net SDRAM_D20: U301.M1 (GPIO_EMC_B2_04), U402.C8 (DQ20)
- new net SDRAM_D21: U301.N1 (GPIO_EMC_B2_05), U402.A9 (DQ21)
- new net SDRAM_D22: U301.T1 (GPIO_EMC_B2_06), U402.C7 (DQ22)
- new net SDRAM_D23: U301.M3 (GPIO_EMC_B2_07), U402.A8 (DQ23)
- new net SDRAM_D24: U301.N2 (GPIO_EMC_B2_09), U402.A2 (DQ24)
- new net SDRAM_D25: U301.R2 (GPIO_EMC_B2_10), U402.C3 (DQ25)
- new net SDRAM_D26: U301.L4 (GPIO_EMC_B2_11), U402.A1 (DQ26)
- new net SDRAM_D27: U301.M2 (GPIO_EMC_B2_12), U402.C2 (DQ27)
- new net SDRAM_D28: U301.K5 (GPIO_EMC_B2_13), U402.B1 (DQ28)
- new net SDRAM_D29: U301.M4 (GPIO_EMC_B2_14), U402.D2 (DQ29)
- new net SDRAM_D3: U301.E4 (GPIO_EMC_B1_03), U402.N8 (DQ3)
- new net SDRAM_D30: U301.L2 (GPIO_EMC_B2_15), U402.D3 (DQ30)
- new net SDRAM_D31: U301.P2 (GPIO_EMC_B2_16), U402.E2 (DQ31)
- new net SDRAM_D4: U301.H5 (GPIO_EMC_B1_04), U402.P9 (DQ4)
- new net SDRAM_D5: U301.F4 (GPIO_EMC_B1_05), U402.M8 (DQ5)
- new net SDRAM_D6: U301.H4 (GPIO_EMC_B1_06), U402.M7 (DQ6)
- new net SDRAM_D7: U301.H3 (GPIO_EMC_B1_07), U402.L8 (DQ7)
- new net SDRAM_D8: U301.E3 (GPIO_EMC_B1_30), U402.L2 (DQ8)
- new net SDRAM_D9: U301.D2 (GPIO_EMC_B1_31), U402.M3 (DQ9)
- new net SDRAM_DM0: U301.F5 (GPIO_EMC_B1_08), U402.K9 (DQM0)
- new net SDRAM_DM1: U301.J1 (GPIO_EMC_B1_38), U402.K1 (DQM1)
- new net SDRAM_DM2: U301.P1 (GPIO_EMC_B2_08), U402.F8 (DQM2)
- new net SDRAM_DM3: U301.T2 (GPIO_EMC_B2_17), U402.F2 (DQM3)
- new net SDRAM_RAS: U301.J4 (GPIO_EMC_B1_25), U402.J9 (~{RAS})
- new net SDRAM_WE: U301.E5 (GPIO_EMC_B1_28), U402.K8 (~{WE})
Other:
- note added: "F7/F6/G6"
- note added: "H6"
- note removed: "CAP for DRAM0"

Commit message: Update PCB files to rev 0.6 used for production
Other:
- company: Copyright 2022 Wenting Zhang -> Copyright 2023 Wenting Zhang
Changed lines of the file:
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@@
   (title_block
     (title "Sitina 1 Mainboard")
-    (date "2022-04-28")
-    (rev "R0.1")
-    (company "Copyright 2022 Wenting Zhang")
+    (date "2023-03-16")
+    (rev "R0.6")
+    (company "Copyright 2023 Wenting Zhang")
     (comment 2 "MERCHANTABILITY, SATISFACTORY QUALITY AND FITNESS FOR A PARTICULAR PURPOSE.")
     (comment 3 "This source is distributed WITHOUT ANY EXPRESS OR IMPLIED WARRANTY, INCLUDING OF")

Commit message: New mainboard rev wip
Parts:
- removed C404, C405: 4.7uF, Capacitor_SMD:C_0402_1005Metric, symbol Device:C
- removed C406, C407: 2.2uF, Capacitor_SMD:C_0402_1005Metric, symbol Device:C
- removed TP401, TP402: TestPoint, footprints:TestPoint_Pad_D0.5mm, symbol Connector:TestPoint
- removed U301: MIMXRT1176DVMAA, footprints:BGA-289_17x17_14.0x14.0mm, symbol symbols:MIMXRT1176DVMAA
- removed U402: MT48H16M32LFB5-6 or IS42VM32160E-6 or W989D2DBJX6, footprints:BGA-90_9x15_8.0x13.0mm, symbol symbols:IS42S32800J-xB
- added C316: 22uF, Capacitor_SMD:C_0603_1608Metric, symbol Device:C
- added U100: IMXRT1050, footprints:BGA-196_14x14_12.0x12.0mm, symbol Sitina:IMXRT1050
- added U3: MT48LC16M16A2BG, footprints:BGA-54_9x9_8.0x8.0mm, symbol symbols:MT48LC32M16A2B4
- C70: renamed from C408; value 10uF -> 4.7uF
- renumbered C409 to C71, C410 to C72, C411 to C73, C412 to C74, C413 to C75, C414 to C76, C415 to C77
Connections:
- net GND: now also C316.2, U3.A1 (GND), U3.A3 (GNDQ), U3.A8 (GND), U3.B7 (GNDQ), U3.C3 (GNDQ), U3.D7 (GNDQ), U3.E3 (GND)
- net SDRAM_A0: now also U100.C2 (GPIO_EMC_09), U3.H7 (A0)
- net SDRAM_A1: now also U100.G1 (GPIO_EMC_10), U3.H8 (A1)
- net SDRAM_A10: now also U100.G2 (GPIO_EMC_23), U3.H9 (A10)
- net SDRAM_A11: now also U100.B4 (GPIO_EMC_19), U3.G2 (A11)
- net SDRAM_A12: now also U100.A3 (GPIO_EMC_20), U3.G1 (A12)
- net SDRAM_A2: now also U100.G3 (GPIO_EMC_11), U3.J8 (A2)
- net SDRAM_A3: now also U100.H1 (GPIO_EMC_12), U3.J7 (A3)
- net SDRAM_A4: now also U100.A6 (GPIO_EMC_13), U3.J3 (A4)
- net SDRAM_A5: now also U100.B6 (GPIO_EMC_14), U3.J2 (A5)
- net SDRAM_A6: now also U100.B1 (GPIO_EMC_15), U3.H3 (A6)
- net SDRAM_A7: now also U100.A5 (GPIO_EMC_16), U3.H2 (A7)
- net SDRAM_A8: now also U100.A4 (GPIO_EMC_17), U3.H1 (A8)
- net SDRAM_A9: now also U100.B2 (GPIO_EMC_18), U3.G3 (A9)
- net SDRAM_BA0: now also U100.C1 (GPIO_EMC_21), U3.G7 (BA0)
- net SDRAM_BA1: now also U100.F1 (GPIO_EMC_22), U3.G8 (BA1)
- net SDRAM_CAS: now also U100.D3 (GPIO_EMC_24), U3.F7 (~{CAS})
- net SDRAM_CKE: now also U100.A2 (GPIO_EMC_27), U3.F3 (CKE)
- net SDRAM_CLK: now also U100.B3 (GPIO_EMC_26), U3.F2 (CLK)
- net SDRAM_CS0: now also U100.E1 (GPIO_EMC_29), U3.G9 (~{CS})
- net SDRAM_D0: now also U100.E3 (GPIO_EMC_00), U3.A8 (GND)
- net SDRAM_D1: now also U100.F3 (GPIO_EMC_01), U3.B9 (DQ1)
- net SDRAM_D10: now also U100.D5 (GPIO_EMC_32), U3.D1 (DQ10)
- net SDRAM_D11: now also U100.C4 (GPIO_EMC_33), U3.C2 (DQ11)
- net SDRAM_D12: now also U100.D4 (GPIO_EMC_34), U3.C1 (DQ12)
- net SDRAM_D13: now also U100.E5 (GPIO_EMC_35), U3.B2 (DQ13)
- net SDRAM_D14: now also U100.C3 (GPIO_EMC_36), U3.B1 (DQ14)
- net SDRAM_D15: now also U100.E4 (GPIO_EMC_37), U3.A2 (DQ15)
- net SDRAM_D2: now also U100.F4 (GPIO_EMC_02), U3.B8 (DQ2)
- net SDRAM_D3: now also U100.G4 (GPIO_EMC_03), U3.C9 (DQ3)
- net SDRAM_D4: now also U100.F2 (GPIO_EMC_04), U3.C8 (DQ4)
- net SDRAM_D5: now also U100.G5 (GPIO_EMC_05), U3.D9 (DQ5)
- net SDRAM_D6: now also U100.H5 (GPIO_EMC_06), U3.D8 (DQ6)
- net SDRAM_D7: now also U100.H4 (GPIO_EMC_07), U3.E9 (DQ7)
- net SDRAM_D8: now also U100.C6 (GPIO_EMC_30), U3.E1 (DQ8)
- net SDRAM_D9: now also U100.C5 (GPIO_EMC_31), U3.D2 (DQ9)
- net SDRAM_DM0: now also U100.H3 (GPIO_EMC_08), U3.E8 (LDQM)
- net SDRAM_DM1: now also U100.D6 (GPIO_EMC_38), U3.F1 (UDQM)
- net SDRAM_RAS: now also U100.D2 (GPIO_EMC_25), U3.F8 (~{RAS})
- net SDRAM_WE: now also U100.D1 (GPIO_EMC_28), U3.F9 (~{WE})
- net +1V8 renamed +3V3
- net +3V3: now also C316.1, U3.A7 (VDDQ), U3.A9 (VDD), U3.B3 (VDDQ), U3.C7 (VDDQ), U3.D3 (VDDQ), U3.E7 (VDD), U3.J9 (VDD)
- new net LCD_EN: U100.C7 (GPIO_EMC_41)
- new net SDRAM_DQS: U100.B7 (GPIO_EMC_39)
- no-connect marks 5 -> 1
Other:
- note removed: "F7/F6/G6"
- note removed: "H6"

Commit message: Mainboard WIP
Connections:
- net +3V3 renamed +1V8
Changed lines of the file:
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@@
   (junction (at 218.44 142.24) (diameter 0.9144) (color 0 0 0 0)
   )
+  (junction (at 231.14 149.86) (diameter 0.9144) (color 0 0 0 0)
+  )
   (junction (at 203.2 50.8) (diameter 0) (color 0 0 0 0)
   )
-  (junction (at 231.14 149.86) (diameter 0.9144) (color 0 0 0 0)
+  (junction (at 218.44 149.86) (diameter 0.9144) (color 0 0 0 0)
+  )
+  (junction (at 154.94 142.24) (diameter 0) (color 0 0 0 0)
   )
   (junction (at 203.2 127) (diameter 0) (color 0 0 0 0)
-  )
-  (junction (at 218.44 149.86) (diameter 0.9144) (color 0 0 0 0)
-  )
-  (junction (at 154.94 142.24) (diameter 0) (color 0 0 0 0)
   )
   (junction (at 205.74 149.86) (diameter 0.9144) (color 0 0 0 0)
@@
     (stroke (width 0) (type solid))
   )
-  (wire (pts (xy 203.2 48.26) (xy 203.2 50.8))
-    (stroke (width 0) (type default))
-  )
   (wire (pts (xy 177.8 88.9) (xy 190.5 88.9))
     (stroke (width 0) (type default))
@@
     (stroke (width 0) (type default))
   )
-  (wire (pts (xy 203.2 127) (xy 203.2 129.54))
-    (stroke (width 0) (type default))
-  )
   (wire (pts (xy 110.49 83.82) (xy 99.06 83.82))
     (stroke (width 0) (type solid))
@@
     (effects (font (size 1.27 1.27)) (justify right bottom))
   )
-  (hierarchical_label "LCD_EN" (shape output) (at 104.14 157.48 0) (fields_autoplaced)
+  (global_label "LCD_EN" (shape output) (at 104.14 157.48 0) (fields_autoplaced)
     (effects (font (size 1.27 1.27)) (justify left))
+    (property "Intersheetrefs" "${INTERSHEET_REFS}" (at 114.1561 157.48 0)
+      (effects (font (size 1.27 1.27)) (justify left) hide)
+    )
   )
   (symbol (lib_id "symbols:MT48LC32M16A2B4") (at 205.74 86.36 0) (unit 1)
@@
     )
   )
+  (symbol (lib_id "power:+1V8") (at 154.94 139.7 0) (unit 1)
+    (in_bom yes) (on_board yes) (dnp no)
+    (property "Reference" "#PWR067" (at 154.94 143.51 0)
+      (effects (font (size 1.27 1.27)) hide)
+    )
+    (property "Value" "+1V8" (at 154.94 135.89 0)
+      (effects (font (size 1.27 1.27)))
+    )
+    (property "Footprint" "" (at 154.94 139.7 0)
+      (effects (font (size 1.27 1.27)) hide)
+    )
+    (property "Datasheet" "" (at 154.94 139.7 0)
+      (effects (font (size 1.27 1.27)) hide)
+    )
+    (pin "1")
+    (instances
+      (project "pcb"
+        (path "/ba41827b-f176-424d-b6d5-0b0e1ddda097/00000000-0000-0000-0000-00005db2122b"
+          (reference "#PWR067") (unit 1)
+        )
+        (path "/ba41827b-f176-424d-b6d5-0b0e1ddda097/00000000-0000-0000-0000-00005d180a01"
+          (reference "#PWR033") (unit 1)
+        )
+        (path "/ba41827b-f176-424d-b6d5-0b0e1ddda097/00000000-0000-0000-0000-00005eff0efc"
+          (reference "#PWR058") (unit 1)
+        )
+      )
+    )
+  )
   (symbol (lib_id "Device:C") (at 180.34 146.05 0) (unit 1)
     (in_bom yes) (on_board yes) (dnp no)
@@
         (path "/ba41827b-f176-424d-b6d5-0b0e1ddda097/00000000-0000-0000-0000-00005eff0efc"
           (reference "C71") (unit 1)
-        )
-      )
-    )
-  )
-  (symbol (lib_id "power:+3V3") (at 154.94 139.7 0) (unit 1)
-    (in_bom yes) (on_board yes) (dnp no)
-    (property "Reference" "#PWR0106" (at 154.94 143.51 0)
-      (effects (font (size 1.27 1.27)) hide)
-    )
-    (property "Value" "+3V3" (at 155.321 135.3058 0)
-      (effects (font (size 1.27 1.27)))
-    )
-    (property "Footprint" "" (at 154.94 139.7 0)
-      (effects (font (size 1.27 1.27)) hide)
-    )
-    (property "Datasheet" "" (at 154.94 139.7 0)
-      (effects (font (size 1.27 1.27)) hide)
-    )
-    (pin "1")
-    (instances
-      (project "Sitina"
-        (path "/46f1d123-bfe2-4f3e-acaa-2114f5fd73de/00000000-0000-0000-0000-00005dc83261"
-          (reference "#PWR0106") (unit 1)
-        )
-      )
-      (project "pcb"
-        (path "/ba41827b-f176-424d-b6d5-0b0e1ddda097/00000000-0000-0000-0000-00005eff0efc"
-          (reference "#PWR058") (unit 1)
-        )
-      )
-    )
-  )
-  (symbol (lib_id "power:+3V3") (at 203.2 48.26 0) (unit 1)
-    (in_bom yes) (on_board yes) (dnp no)
-    (property "Reference" "#PWR0106" (at 203.2 52.07 0)
-      (effects (font (size 1.27 1.27)) hide)
-    )
-    (property "Value" "+3V3" (at 203.581 43.8658 0)
-      (effects (font (size 1.27 1.27)))
-    )
-    (property "Footprint" "" (at 203.2 48.26 0)
-      (effects (font (size 1.27 1.27)) hide)
-    )
-    (property "Datasheet" "" (at 203.2 48.26 0)
-      (effects (font (size 1.27 1.27)) hide)
-    )
-    (pin "1")
-    (instances
-      (project "Sitina"
-        (path "/46f1d123-bfe2-4f3e-acaa-2114f5fd73de/00000000-0000-0000-0000-00005dc83261"
-          (reference "#PWR0106") (unit 1)
-        )
-      )
-      (project "pcb"
-        (path "/ba41827b-f176-424d-b6d5-0b0e1ddda097/00000000-0000-0000-0000-00005eff0efc"
-          (reference "#PWR060") (unit 1)
         )
       )
@@
     )
   )
-  (symbol (lib_id "power:GND") (at 203.2 129.54 0) (unit 1)
-    (in_bom yes) (on_board yes) (dnp no)
-    (property "Reference" "#PWR061" (at 203.2 135.89 0)
-      (effects (font (size 1.27 1.27)) hide)
-    )
-    (property "Value" "GND" (at 203.327 133.9342 0)
+  (symbol (lib_id "power:GND") (at 203.2 127 0) (unit 1)
+    (in_bom yes) (on_board yes) (dnp no)
+    (property "Reference" "#PWR061" (at 203.2 133.35 0)
+      (effects (font (size 1.27 1.27)) hide)
+    )
+    (property "Value" "GND" (at 203.327 131.3942 0)
       (effects (font (size 1.27 1.27)))
     )
-    (property "Footprint" "" (at 203.2 129.54 0)
-      (effects (font (size 1.27 1.27)) hide)
-    )
-    (property "Datasheet" "" (at 203.2 129.54 0)
+    (property "Footprint" "" (at 203.2 127 0)
+      (effects (font (size 1.27 1.27)) hide)
+    )
+    (property "Datasheet" "" (at 203.2 127 0)
       (effects (font (size 1.27 1.27)) hide)
     )
@@
         )
       )
+    )
+  )
+  (symbol (lib_id "power:+1V8") (at 203.2 50.8 0) (unit 1)
+    (in_bom yes) (on_board yes) (dnp no)
+    (property "Reference" "#PWR067" (at 203.2 54.61 0)
+      (effects (font (size 1.27 1.27)) hide)
+    )
+    (property "Value" "+1V8" (at 203.2 46.99 0)
+      (effects (font (size 1.27 1.27)))
+    )
+    (property "Footprint" "" (at 203.2 50.8 0)
+      (effects (font (size 1.27 1.27)) hide)
+    )
+    (property "Datasheet" "" (at 203.2 50.8 0)
+      (effects (font (size 1.27 1.27)) hide)
+    )
+    (pin "1")
+    (instances
+      (project "pcb"
+        (path "/ba41827b-f176-424d-b6d5-0b0e1ddda097/00000000-0000-0000-0000-00005db2122b"
+          (reference "#PWR067") (unit 1)
+        )
+        (path "/ba41827b-f176-424d-b6d5-0b0e1ddda097/00000000-0000-0000-0000-00005d180a01"
+          (reference "#PWR033") (unit 1)
+        )
+        (path "/ba41827b-f176-424d-b6d5-0b0e1ddda097/00000000-0000-0000-0000-00005eff0efc"
+          (reference "#PWR042") (unit 1)
+        )
+      )
