File: Hardware/mainboard/storage.kicad_sch (KiCad schematic)
At the start: 8 parts, among them J502 SD_Card, U501 W25Q128JVP

Commit message: New PCB rev
Parts:
- added C502, C503: 2.2uF, Capacitor_SMD:C_0402_1005Metric, symbol Device:C
- added U301: MIMXRT1176DVMAA, footprints:BGA-289_17x17_14.0x14.0mm, symbol symbols:MIMXRT1176DVMAA
- R501: footprint Capacitor_SMD:C_0402_1005Metric -> Resistor_SMD:R_0402_1005Metric
Connections:
- net +3V3: no longer C501.2, R501.1, U501.8 (VCC)
- net GND: now also C502.2, C503.2
- net QSPI_A_DATA0: now also U301.F15 (GPIO_SD_B2_08)
- net QSPI_A_DATA1: now also U301.H15 (GPIO_SD_B2_09)
- net QSPI_A_DATA2: now also U301.H14 (GPIO_SD_B2_10)
- net QSPI_A_DATA3: now also U301.F16 (GPIO_SD_B2_11)
- net QSPI_A_SCLK: now also U301.G14 (GPIO_SD_B2_07)
- net QSPI_A_SS0: now also U301.F17 (GPIO_SD_B2_06)
- net SD1_CLK: now also U301.D15 (GPIO_SD_B1_01)
- net SD1_CMD: now also U301.B16 (GPIO_SD_B1_00)
- net SD1_DATA0: now also U301.C15 (GPIO_SD_B1_02)
- net SD1_DATA1: now also U301.B17 (GPIO_SD_B1_03)
- net SD1_DATA2: now also U301.B15 (GPIO_SD_B1_04)
- net SD1_DATA3: now also U301.A16 (GPIO_SD_B1_05)
- new net +1V8: C501.2, C503.1, R501.1, U301.G13 (NVCC_SD2), U501.8 (VCC)
- new net +VCCIO_SD: C502.1, U301.D14 (NVCC_SD1)
- no-connect marks 0 -> 6
Other:
- note added: "DQS Leave NC"
- moved on the sheet: C401, C402, C403, C501, J502, R401, R501, U501

Commit message: Update PCB files to rev 0.6 used for production
Other:
- company: Copyright 2022 Wenting Zhang -> Copyright 2023 Wenting Zhang
Changed lines of the file:
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@@
   (title_block
     (title "Sitina 1 Mainboard")
-    (date "2022-04-28")
-    (rev "R0.1")
-    (company "Copyright 2022 Wenting Zhang")
+    (date "2023-03-16")
+    (rev "R0.6")
+    (company "Copyright 2023 Wenting Zhang")
     (comment 2 "MERCHANTABILITY, SATISFACTORY QUALITY AND FITNESS FOR A PARTICULAR PURPOSE.")
     (comment 3 "This source is distributed WITHOUT ANY EXPRESS OR IMPLIED WARRANTY, INCLUDING OF")

Commit message: Working towards pcb r0.7
Parts:
- U501: value W25Q128JVP -> W25Q128JWP
Changed lines of the file:
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@@
       (effects (font (size 1.27 1.27)))
     )
-    (property "Value" "W25Q128JVP" (at 190.5 123.444 0)
+    (property "Value" "W25Q128JWP" (at 190.5 123.444 0)
       (effects (font (size 1.27 1.27)))
     )

Commit message: New mainboard rev wip
Parts:
- removed C502, C503: 2.2uF, Capacitor_SMD:C_0402_1005Metric, symbol Device:C
- removed J502: SD_Card, Connector_Card:SD_Kyocera_145638009511859+, symbol Connector:SD_Card
- removed U301: MIMXRT1176DVMAA, footprints:BGA-289_17x17_14.0x14.0mm, symbol symbols:MIMXRT1176DVMAA
- added MICRO_SD400: MICRO_SD(TFC-WPAPR-08), footprints:TFC-WPAPR-08, symbol Sitina:MICRO_SD(TFC-WPAPR-08)
- U4: renamed from U501; value W25Q128JWP -> W25Q128JV
- renumbered C401 to C78, C402 to C79, C403 to C80, C501 to C81, R401 to R17, R501 to R18
Connections:
- net GND: now also MICRO_SD400.10, MICRO_SD400.11, MICRO_SD400.12, MICRO_SD400.13, MICRO_SD400.6 (VSS)
- net SD1_CD: now also C78.1, R17.1, MICRO_SD400.5 (CLK/SCLK), MICRO_SD400.9
- net SD1_CMD: now also MICRO_SD400.3 (CMD/DI)
- net SD1_DATA0: now also MICRO_SD400.7 (DAT0/DO)
- net SD1_DATA1: now also MICRO_SD400.8 (DAT1/RES)
- net SD1_DATA2: now also MICRO_SD400.1 (DAT2/RES)
- net SD1_DATA3: now also MICRO_SD400.2 (CD/DAT3/CS)
- net +3V3 renamed +VSD
- net +VSD: now also MICRO_SD400.4 (VDD)
- net QSPI_A_DATA0 renamed QSPI_DATA0
- net QSPI_A_DATA1 renamed QSPI_DATA1
- net QSPI_A_DATA2 renamed QSPI_DATA2
- net QSPI_A_DATA3 renamed QSPI_DATA3
- net QSPI_A_SCLK renamed QSPI_SCLK
- net QSPI_A_SS0 renamed QSPI_SS0
- no-connect marks 6 -> 0
Other:
- note removed: "DQS Leave NC"
- moved on the sheet: C78, C79, C80, C81, R17, R18, U4

Commit message: Mainboard WIP
Connections:
- net SD1_CD: no longer C78.1, MICRO_SD400.5 (CLK/SCLK), R17.1
- new net: C78.1, MICRO_SD400.5 (CLK/SCLK), R17.1
Other:
- moved on the sheet: C78
Changed lines of the file:
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@@
   (junction (at 198.12 90.17) (diameter 0) (color 0 0 0 0)
   )
-  (junction (at 91.44 114.3) (diameter 0) (color 0 0 0 0)
-  )
   (junction (at 182.88 90.17) (diameter 0.9144) (color 0 0 0 0)
   )
@@
     (stroke (width 0) (type solid))
   )
-  (wire (pts (xy 91.44 114.3) (xy 104.14 114.3))
+  (wire (pts (xy 68.58 114.3) (xy 104.14 114.3))
     (stroke (width 0) (type default))
   )
@@
     (stroke (width 0) (type solid))
   )
-  (wire (pts (xy 91.44 121.92) (xy 91.44 124.46))
-    (stroke (width 0) (type solid))
-  )
   (wire (pts (xy 210.82 111.76) (xy 215.9 111.76))
     (stroke (width 0) (type solid))
@@
     (stroke (width 0) (type solid))
   )
-  (wire (pts (xy 91.44 104.14) (xy 91.44 114.3))
+  (wire (pts (xy 91.44 104.14) (xy 91.44 116.84))
     (stroke (width 0) (type solid))
   )
@@
     (stroke (width 0) (type solid))
   )
-  (wire (pts (xy 68.58 114.3) (xy 91.44 114.3))
-    (stroke (width 0) (type default))
-  )
   (wire (pts (xy 68.58 93.98) (xy 104.14 93.98))
     (stroke (width 0) (type solid))
@@
     )
   )
-  (symbol (lib_id "Device:C") (at 91.44 118.11 0) (unit 1)
-    (in_bom yes) (on_board yes) (dnp no)
-    (property "Reference" "C78" (at 94.361 116.9416 0)
-      (effects (font (size 1.27 1.27)) (justify left))
-    )
-    (property "Value" "18pF" (at 94.361 119.253 0)
-      (effects (font (size 1.27 1.27)) (justify left))
-    )
-    (property "Footprint" "Capacitor_SMD:C_0402_1005Metric" (at 92.4052 121.92 0)
-      (effects (font (size 1.27 1.27)) hide)
-    )
-    (property "Datasheet" "~" (at 91.44 118.11 0)
-      (effects (font (size 1.27 1.27)) hide)
-    )
+  (symbol (lib_id "Device:C") (at 91.44 120.65 0) (unit 1)
+    (in_bom yes) (on_board yes) (dnp no)
+    (property "Reference" "C78" (at 94.361 119.4816 0)
+      (effects (font (size 1.27 1.27)) (justify left))
+    )
+    (property "Value" "18pF" (at 94.361 121.793 0)
+      (effects (font (size 1.27 1.27)) (justify left))
+    )
+    (property "Footprint" "Capacitor_SMD:C_0402_1005Metric" (at 92.4052 124.46 0)
+      (effects (font (size 1.27 1.27)) hide)
+    )
+    (property "Datasheet" "~" (at 91.44 120.65 0)
+      (effects (font (size 1.27 1.27)) hide)
+    )

Commit message: Update mainboard design
Connections:
- net SD1_CD: no longer MICRO_SD400.9
- no-connect marks 0 -> 2
Other:
- note added: "Can't route CD pin :("
Changed lines of the file:
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@@
   (junction (at 91.44 104.14) (diameter 0.9144) (color 0 0 0 0)
   )
+  (no_connect (at 104.14 114.3))
+  (no_connect (at 68.58 114.3))
   (wire (pts (xy 101.6 116.84) (xy 104.14 116.84))
     (stroke (width 0) (type default))
@@
   (wire (pts (xy 210.82 109.22) (xy 215.9 109.22))
     (stroke (width 0) (type solid))
-  )
-  (wire (pts (xy 68.58 114.3) (xy 104.14 114.3))
-    (stroke (width 0) (type default))
   )
   (wire (pts (xy 200.66 116.84) (xy 198.12 116.84))
@@
     (stroke (width 0) (type default))
   )
+  (text "Can't route CD pin :(" (at 71.12 115.57 0)
+    (effects (font (size 1.27 1.27)) (justify left bottom))
+  )
   (global_label "QSPI_SS0" (shape input) (at 180.34 104.14 180) (fields_autoplaced)

Commit message: MB r0p8/ PB r0p2 routing in progress
Parts:
- U4: value W25Q128JV -> W25Q32JV
Connections:
- net +1V8 renamed +3V3
Other:
- moved on the sheet: C81, R18
Changed lines of the file:
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@@
 	)
 	(junction
-		(at 198.12 90.17)
-		(diameter 0)
-		(color 0 0 0 0)
-	)
-	(junction
-		(at 182.88 90.17)
+		(at 182.88 91.44)
 		(diameter 0.9144)
 		(color 0 0 0 0)
@@
 	)
 	(junction
+		(at 198.12 91.44)
+		(diameter 0)
+		(color 0 0 0 0)
+	)
+	(junction
 		(at 101.6 76.2)
 		(diameter 0)
@@
 	(wire
 		(pts
-			(xy 182.88 90.17) (xy 198.12 90.17)
-		)
-		(stroke
-			(width 0)
-			(type solid)
-		)
-	)
-	(wire
-		(pts
-			(xy 182.88 97.79) (xy 182.88 104.14)
+			(xy 182.88 91.44) (xy 198.12 91.44)
 		)
 		(stroke
@@
 	(wire
 		(pts
+			(xy 198.12 96.52) (xy 198.12 91.44)
+		)
+		(stroke
+			(width 0)
+			(type solid)
+		)
+	)
+	(wire
+		(pts
 			(xy 200.66 116.84) (xy 198.12 116.84)
 		)
@@
 	(wire
 		(pts
-			(xy 172.72 90.17) (xy 182.88 90.17)
+			(xy 172.72 91.44) (xy 182.88 91.44)
 		)
 		(stroke
@@
 	(wire
 		(pts
+			(xy 182.88 99.06) (xy 182.88 104.14)
+		)
+		(stroke
+			(width 0)
+			(type solid)
+		)
+	)
+	(wire
+		(pts
 			(xy 101.6 116.84) (xy 101.6 119.38)
-		)
-		(stroke
-			(width 0)
-			(type solid)
-		)
-	)
-	(wire
-		(pts
-			(xy 198.12 96.52) (xy 198.12 90.17)
 		)
 		(stroke
@@
 	(symbol
 		(lib_id "Device:R")
-		(at 182.88 93.98 0)
+		(at 182.88 95.25 0)
 		(unit 1)
 		(exclude_from_sim no)
@@
 		(dnp no)
 		(property "Reference" "R18"
-			(at 179.07 92.71 0)
+			(at 179.07 93.98 0)
 			(effects
 				(font
@@
 		)
 		(property "Value" "100K"
-			(at 179.07 95.25 0)
+			(at 179.07 96.52 0)
 			(effects
 				(font
@@
 		)
 		(property "Footprint" "Resistor_SMD:R_0402_1005Metric"
-			(at 181.102 93.98 90)
+			(at 181.102 95.25 90)
 			(effects
 				(font
@@
 		)
 		(property "Datasheet" "~"
-			(at 182.88 93.98 0)
+			(at 182.88 95.25 0)
 			(effects
 				(font
@@
 		)
 		(property "Description" ""
-			(at 182.88 93.98 0)
+			(at 182.88 95.25 0)
 			(effects
 				(font
@@
 	)
 	(symbol
-		(lib_id "power:+1V8")
-		(at 198.12 90.17 0)
-		(unit 1)
-		(exclude_from_sim no)
-		(in_bom yes)
-		(on_board yes)
-		(dnp no)
-		(property "Reference" "#PWR067"
-			(at 198.12 93.98 0)
-			(effects
-				(font
-					(size 1.27 1.27)
-				)
-				(hide yes)
-			)
-		)
-		(property "Value" "+1V8"
-			(at 198.12 86.36 0)
-			(effects
-				(font
-					(size 1.27 1.27)
-				)
-			)
-		)
-		(property "Footprint" ""
-			(at 198.12 90.17 0)
-			(effects
-				(font
-					(size 1.27 1.27)
-				)
-				(hide yes)
-			)
-		)
-		(property "Datasheet" ""
-			(at 198.12 90.17 0)
-			(effects
-				(font
-					(size 1.27 1.27)
-				)
-				(hide yes)
-			)
-		)
-		(property "Description" ""
-			(at 198.12 90.17 0)
-			(effects
-				(font
-					(size 1.27 1.27)
-				)
-				(hide yes)
-			)
-		)
-		(pin "1"
-		)
-		(instances
-			(project "pcb"
-				(path "/ba41827b-f176-424d-b6d5-0b0e1ddda097/00000000-0000-0000-0000-00005db2122b"
-					(reference "#PWR067")
-					(unit 1)
-				)
-			)
-		)
-	)
-	(symbol
 		(lib_id "Device:C")
 		(at 111.76 80.01 0)
@@
 	(symbol
 		(lib_id "Device:C")
-		(at 172.72 93.98 180)
+		(at 172.72 95.25 180)
 		(unit 1)
 		(exclude_from_sim no)
@@
 		(dnp no)
 		(property "Reference" "C81"
-			(at 167.64 92.71 0)
+			(at 167.64 93.98 0)
 			(effects
 				(font
@@
 		)
 		(property "Value" "470nF"
-			(at 167.64 95.25 0)
+			(at 167.64 96.52 0)
 			(effects
 				(font
@@
 		)
 		(property "Footprint" "Capacitor_SMD:C_0402_1005Metric"
-			(at 171.7548 90.17 0)
+			(at 171.7548 91.44 0)
 			(effects
 				(font
@@
 		)
 		(property "Datasheet" "~"
-			(at 172.72 93.98 0)
+			(at 172.72 95.25 0)
 			(effects
 				(font
@@
 		)
 		(property "Description" ""
-			(at 172.72 93.98 0)
+			(at 172.72 95.25 0)
 			(effects
 				(font
@@
 	(symbol
 		(lib_id "power:GND")
-		(at 172.72 97.79 0)
+		(at 172.72 99.06 0)
 		(unit 1)
 		(exclude_from_sim no)
@@
 		(dnp no)
 		(property "Reference" "#PWR066"
-			(at 172.72 104.14 0)
+			(at 172.72 105.41 0)
 			(effects
 				(font
@@
 		)
 		(property "Value" "GND"
-			(at 172.847 100.9142 0)
+			(at 172.847 102.1842 0)
 			(effects
 				(font
@@
 		)
 		(property "Footprint" ""
-			(at 172.72 97.79 0)
+			(at 172.72 99.06 0)
 			(effects
 				(font
@@
 		)
 		(property "Datasheet" ""
-			(at 172.72 97.79 0)
+			(at 172.72 99.06 0)
 			(effects
 				(font
@@
 		)
 		(property "Description" ""
-			(at 172.72 97.79 0)
+			(at 172.72 99.06 0)
 			(effects
 				(font
@@
 	)
 	(symbol
+		(lib_id "power:+3V3")
+		(at 198.12 91.44 0)
+		(unit 1)
+		(exclude_from_sim no)
+		(in_bom yes)
+		(on_board yes)
+		(dnp no)
+		(property "Reference" "#PWR067"
+			(at 198.12 95.25 0)
+			(effects
+				(font
+					(size 1.27 1.27)
+				)
+				(hide yes)
+			)
+		)
+		(property "Value" "+3V3"
+			(at 198.12 86.36 0)
+			(effects
+				(font
+					(size 1.27 1.27)
+				)
+			)
+		)
+		(property "Footprint" ""
+			(at 198.12 91.44 0)
+			(effects
+				(font
+					(size 1.27 1.27)
+				)
+				(hide yes)
+			)
+		)
+		(property "Datasheet" ""
+			(at 198.12 91.44 0)
+			(effects
+				(font
+					(size 1.27 1.27)
+				)
+				(hide yes)
+			)
+		)
+		(property "Description" ""
+			(at 198.12 91.44 0)
+			(effects
+				(font
+					(size 1.27 1.27)
+				)
+				(hide yes)
+			)
+		)
+		(pin "1"
+		)
+		(instances
+			(project "pcb"
+				(path "/ba41827b-f176-424d-b6d5-0b0e1ddda097/00000000-0000-0000-0000-00005db2122b"
+					(reference "#PWR067")
+					(unit 1)
+				)
+			)
+		)
+	)
+	(symbol
 		(lib_id "symbols:+VSD")
 		(at 101.6 76.2 0)
@@
 			)
 		)
-		(property "Value" "W25Q128JV"
+		(property "Value" "W25Q32JV"
 			(at 205.74 96.774 0)
 			(effects
