File: Hardware/sensorboard/connector.kicad_sch (KiCad schematic)
At the start: 0 parts

Commit message: Update sensor/power board outline
Parts:
- added H1, H2, H3: MountingHole, MountingHole:MountingHole_2.2mm_M2_DIN965, symbol Mechanical:MountingHole
- added J5: Sensor Board, Connector_FFC-FPC:Hirose_FH12-30S-0.5SH_1x30-1MP_P0.50mm_Horizontal, symbol Connector_Generic_MountingPin:Conn_01x30_MountingPin
Connections:
- net +3V3: now also J5.1 (Pin_1), J5.2 (Pin_2)
- net AFE_RST: now also J5.6 (Pin_6)
- net AFE_SCK: now also J5.7 (Pin_7)
- net AFE_SDATA: now also J5.8 (Pin_8)
- net AFE_SL: now also J5.9 (Pin_9)
- net AFE_SYNC: now also J5.5 (Pin_5)
- net CSI_D10: now also J5.21 (Pin_21)
- net CSI_D11: now also J5.20 (Pin_20)
- net CSI_D12: now also J5.19 (Pin_19)
- net CSI_D13: now also J5.18 (Pin_18)
- net CSI_D14: now also J5.17 (Pin_17)
- net CSI_D15: now also J5.16 (Pin_16)
- net CSI_D2: now also J5.29 (Pin_29)
- net CSI_D3: now also J5.28 (Pin_28)
- net CSI_D4: now also J5.27 (Pin_27)
- net CSI_D5: now also J5.26 (Pin_26)
- net CSI_D6: now also J5.25 (Pin_25)
- net CSI_D7: now also J5.24 (Pin_24)
- net CSI_D8: now also J5.23 (Pin_23)
- net CSI_D9: now also J5.22 (Pin_22)
- net CSI_HSYNC: now also J5.11 (Pin_11)
- net CSI_PIXCLK: now also J5.14 (Pin_14)
- net CSI_VSYNC: now also J5.12 (Pin_12)
- net GND: now also J5.10 (Pin_10), J5.13 (Pin_13), J5.15 (Pin_15), J5.3 (Pin_3), J5.30 (Pin_30), J5.MP (MountPin)

Commit message: Adding PowerBoard Schematic
Parts:
- renumbered H1 to H501, H2 to H502, H3 to H503, J5 to J501
Changed lines of the file:
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@@
   (symbol (lib_id "Mechanical:MountingHole") (at 68.58 160.02 0) (unit 1)
     (in_bom yes) (on_board yes) (dnp no) (fields_autoplaced)
-    (property "Reference" "H1" (at 72.39 159.3849 0)
+    (property "Reference" "H501" (at 72.39 159.3849 0)
       (effects (font (size 1.27 1.27)) (justify left))
     )
@@
   (symbol (lib_id "power:GND") (at 172.72 137.16 0) (unit 1)
     (in_bom yes) (on_board yes) (dnp no)
-    (property "Reference" "#PWR069" (at 172.72 143.51 0)
+    (property "Reference" "#PWR0617" (at 172.72 143.51 0)
       (effects (font (size 1.27 1.27)) hide)
     )
@@
   (symbol (lib_id "Connector_Generic_MountingPin:Conn_01x30_MountingPin") (at 180.34 99.06 0) (mirror x) (unit 1)
     (in_bom yes) (on_board yes) (dnp no) (fields_autoplaced)
-    (property "Reference" "J5" (at 182.88 98.7044 0)
+    (property "Reference" "J501" (at 182.88 98.7044 0)
       (effects (font (size 1.27 1.27)) (justify left))
     )
@@
   (symbol (lib_id "power:+3V3") (at 170.18 132.08 90) (unit 1)
     (in_bom yes) (on_board yes) (dnp no)
-    (property "Reference" "#PWR033" (at 173.99 132.08 0)
+    (property "Reference" "#PWR0502" (at 173.99 132.08 0)
       (effects (font (size 1.27 1.27)) hide)
     )
@@
   (symbol (lib_id "Mechanical:MountingHole") (at 68.58 175.26 0) (unit 1)
     (in_bom yes) (on_board yes) (dnp no) (fields_autoplaced)
-    (property "Reference" "H3" (at 72.39 174.6249 0)
+    (property "Reference" "H503" (at 72.39 174.6249 0)
       (effects (font (size 1.27 1.27)) (justify left))
     )
@@
   (symbol (lib_id "power:GND") (at 180.34 55.88 0) (mirror x) (unit 1)
     (in_bom yes) (on_board yes) (dnp no)
-    (property "Reference" "#PWR07" (at 180.34 49.53 0)
+    (property "Reference" "#PWR0618" (at 180.34 49.53 0)
       (effects (font (size 1.27 1.27)) hide)
     )
@@
   (symbol (lib_id "Mechanical:MountingHole") (at 68.58 167.64 0) (unit 1)
     (in_bom yes) (on_board yes) (dnp no) (fields_autoplaced)
-    (property "Reference" "H2" (at 72.39 167.0049 0)
-      (effects (font (size 1.27 1.27)) (justify left))
-    )
+    (property "Reference" "H502" (at 72.39 167.0049 0)
+      (effects (font (size 1.27 1.27)) (justify left))
+    )

Commit message: Update sensorboard outline and connector
Parts:
- added J502: FPC 0.5mm Bottom Contact, Connector_FFC-FPC:Hirose_FH12-30S-0.5SH_1x30-1MP_P0.50mm_Horizontal, symbol Connector_Generic_MountingPin:Conn_01x30_MountingPin
- J501: value Sensor Board -> FPC 0.5mm Bottom Contact
Connections:
- net AFE_RST: now also J501.7 (Pin_7); no longer J501.6 (Pin_6)
- net AFE_SCK: now also J501.8 (Pin_8); no longer J501.7 (Pin_7)
- net AFE_SDATA: now also J501.9 (Pin_9); no longer J501.8 (Pin_8)
- net AFE_SL: now also J501.10 (Pin_10); no longer J501.9 (Pin_9)
- net AFE_SYNC: now also J501.6 (Pin_6); no longer J501.5 (Pin_5)
- net CSI_HSYNC: now also J501.12 (Pin_12); no longer J501.11 (Pin_11)
- net CSI_VSYNC: now also J501.13 (Pin_13); no longer J501.12 (Pin_12)
- net GND: now also J501.11 (Pin_11), J502.3 (Pin_3), J502.MP (MountPin); no longer J501.10 (Pin_10), J501.13 (Pin_13)
- net I2C_SDA: now reaches J501.4 (Pin_4)
- new net I2C_SCL: J501.5 (Pin_5)
- new net SYNC_CLK1: J502.2 (Pin_2)
- new net SYNC_CLK2: J502.1 (Pin_1)
Other:
- note added: "To Main Board"
- note added: "To Power Board"

Commit message: Update sensorboard to include heatsink
Parts:
- added HS501: Heatsink, footprints:sb_heatsink, symbol Mechanical:Heatsink
Changed lines of the file:
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@@
+    )
+  )
+  (symbol (lib_id "Mechanical:Heatsink") (at 68.58 154.94 0) (unit 1)
+    (in_bom yes) (on_board yes) (dnp no) (fields_autoplaced)
+    (property "Reference" "HS501" (at 72.39 151.765 0)
+      (effects (font (size 1.27 1.27)) (justify left))
+    )
+    (property "Value" "Heatsink" (at 72.39 154.305 0)
+      (effects (font (size 1.27 1.27)) (justify left))
+    )
+    (property "Footprint" "footprints:sb_heatsink" (at 68.8848 154.94 0)
+      (effects (font (size 1.27 1.27)) hide)
+    )
+    (property "Datasheet" "~" (at 68.8848 154.94 0)
+      (effects (font (size 1.27 1.27)) hide)
+    )
+    (instances
+      (project "pcb"
+        (path "/ba41827b-f176-424d-b6d5-0b0e1ddda097/28025b55-6a64-43e1-9d20-34020d299147"
+          (reference "HS501") (unit 1)
+        )
+      )
     )
   )

Commit message: CCD Sensor Board WIP
Connections:
- net +16V: now also J502.13 (Pin_13), J502.14 (Pin_14)
- net +16VD: now also J502.5 (Pin_5)
- net +3V0: now also J502.15 (Pin_15)
- net +8V: now also J502.19 (Pin_19), J502.20 (Pin_20), J502.21 (Pin_21)
- net -4V: now also J502.27 (Pin_27), J502.7 (Pin_7), J502.8 (Pin_8)
- net -9V: now also J502.22 (Pin_22), J502.23 (Pin_23), J502.24 (Pin_24)
- net GND: now also J502.11 (Pin_11), J502.16 (Pin_16), J502.17 (Pin_17), J502.18 (Pin_18), J502.2 (Pin_2), J502.25 (Pin_25), J502.26 (Pin_26), J502.30 (Pin_30), J502.4 (Pin_4), J502.6 (Pin_6); no longer J501.11 (Pin_11), J501.15 (Pin_15), J501.3 (Pin_3), J501.30 (Pin_30), J501.MP (MountPin), J502.3 (Pin_3), J502.MP (MountPin)
- net SYNC_CLK1: now also J502.10 (Pin_10); no longer J502.2 (Pin_2)
- net SYNC_CLK2: now also J502.9 (Pin_9); no longer J502.1 (Pin_1)
- net -9VA: now reaches J502.12 (Pin_12)
- net +5V: now reaches J502.28 (Pin_28)
- net +5V: now also J502.29 (Pin_29)
- new net +2V: J502.3 (Pin_3)
- new net -15V: J502.1 (Pin_1)
- new net DVSS: J501.11 (Pin_11), J501.15 (Pin_15), J501.3 (Pin_3), J501.30 (Pin_30)

Commit message: Sensor Board Routing, First Pass Done, Ground Splitting TBD
Parts:
- removed J501, J502: FPC 0.5mm Bottom Contact, Connector_FFC-FPC:Hirose_FH12-30S-0.5SH_1x30-1MP_P0.50mm_Horizontal, symbol Connector_Generic_MountingPin:Conn_01x30_MountingPin
- added J501, J502: FPC 0.5mm Bottom Contact, Connector_FFC-FPC:Hirose_FH12-30S-0.5SH_1x30-1MP_P0.50mm_Horizontal, symbol Connector_Generic:Conn_01x30
Connections:
- net +16V: now also J502.13 (Pin_13), J502.14 (Pin_14)
- net +16VD: now also J502.5 (Pin_5)
- net +2V: now also J502.3 (Pin_3)
- net +3V0: now also J502.15 (Pin_15)
- net +3V3: now also J501.1 (Pin_1), J501.2 (Pin_2)
- net +5V: now also J502.28 (Pin_28), J502.29 (Pin_29)
- net +8V: now also J502.19 (Pin_19), J502.20 (Pin_20), J502.21 (Pin_21)
- net -15V: now also J502.1 (Pin_1)
- net -4V: now also J502.27 (Pin_27), J502.7 (Pin_7), J502.8 (Pin_8)
- net -9V: now also J502.22 (Pin_22), J502.23 (Pin_23), J502.24 (Pin_24)
- net -9VA: now also J502.12 (Pin_12)
- net AFE_RST: now also J501.7 (Pin_7)
- net AFE_SCK: now also J501.8 (Pin_8)
- net AFE_SDATA: now also J501.9 (Pin_9)
- net AFE_SL: now also J501.10 (Pin_10)
- net AFE_SYNC: now also J501.6 (Pin_6)
- net CSI_D10: now also J501.21 (Pin_21)
- net CSI_D11: now also J501.20 (Pin_20)
- net CSI_D12: now also J501.19 (Pin_19)
- net CSI_D13: now also J501.18 (Pin_18)
- net CSI_D14: now also J501.17 (Pin_17)
- net CSI_D15: now also J501.16 (Pin_16)
- net CSI_D2: now also J501.29 (Pin_29)
- net CSI_D3: now also J501.28 (Pin_28)
- net CSI_D4: now also J501.27 (Pin_27)
- net CSI_D5: now also J501.26 (Pin_26)
- net CSI_D6: now also J501.25 (Pin_25)
- net CSI_D7: now also J501.24 (Pin_24)
- net CSI_D8: now also J501.23 (Pin_23)
- net CSI_D9: now also J501.22 (Pin_22)
- net CSI_HSYNC: now also J501.12 (Pin_12)
- net CSI_PIXCLK: now also J501.14 (Pin_14)
- net CSI_VSYNC: now also J501.13 (Pin_13)
- net DVSS: now also J501.11 (Pin_11), J501.15 (Pin_15), J501.3 (Pin_3), J501.30 (Pin_30)
- net GND: now also J502.11 (Pin_11), J502.16 (Pin_16), J502.17 (Pin_17), J502.18 (Pin_18), J502.2 (Pin_2), J502.25 (Pin_25), J502.26 (Pin_26), J502.30 (Pin_30), J502.4 (Pin_4), J502.6 (Pin_6)
- net I2C_SCL: now also J501.5 (Pin_5)
- net I2C_SDA: now also J501.4 (Pin_4)
- net SYNC_CLK1: now also J502.10 (Pin_10)
- net SYNC_CLK2: now also J502.9 (Pin_9)

Commit message: Sensor Board Routing Done
Connections:
- net DVSS is gone; now on net GND: J501.11 (Pin_11), J501.15 (Pin_15), J501.3 (Pin_3), J501.30 (Pin_30)
Changed lines of the file:
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@@
-    )
-  )
-  (global_label "DVSS" (shape passive) (at 172.72 138.43 270) (fields_autoplaced)
-    (effects (font (size 1.27 1.27)) (justify right))
-    (property "Intersheetrefs" "${INTERSHEET_REFS}" (at 172.72 145.2719 90)
-      (effects (font (size 1.27 1.27)) (justify right) hide)
     )
   )
@@
         )
       )
+    )
+  )
+  (symbol (lib_id "power:GND") (at 172.72 138.43 0) (unit 1)
+    (in_bom yes) (on_board yes) (dnp no)
+    (property "Reference" "#PWR0531" (at 172.72 144.78 0)
+      (effects (font (size 1.27 1.27)) hide)
+    )
+    (property "Value" "GND" (at 172.847 141.6812 90)
+      (effects (font (size 1.27 1.27)) (justify right))
+    )
+    (property "Footprint" "" (at 172.72 138.43 0)
+      (effects (font (size 1.27 1.27)) hide)
+    )
+    (property "Datasheet" "" (at 172.72 138.43 0)
+      (effects (font (size 1.27 1.27)) hide)
+    )
+    (pin "1")
+    (instances
+      (project "pcb"
+        (path "/ba41827b-f176-424d-b6d5-0b0e1ddda097/bbc4a8ed-000d-45bd-b682-5f5fc521899f"
+          (reference "#PWR0531") (unit 1)
+        )
+        (path "/ba41827b-f176-424d-b6d5-0b0e1ddda097/28025b55-6a64-43e1-9d20-34020d299147"
+          (reference "#PWR0653") (unit 1)
+        )
+      )
