File: Hardware/sensorboard/pcb.kicad_pcb (KiCad board)
At the start: 4 copper layers, 221 parts, among them Q501 BC847BPN, U501 XC6206P152MR, U502 LT3045xMSE, U503 LT3045xMSE, U504 ADA4800, U505 ADA4800, U506 AD9990, U507 KAI-1100x, U508 74HC2G17, U509 74HC2G17, U510 74HC2G17, U511 74HC2G17, U512 74HC2G17, U513 74HC2G17, U514 1EDN7550B, U515 1EDN7550B, U516 1EDN7550B, U517 1EDN7550B, U518 IRF9389/7309, U519 IRF9389/7309, U520 IRF9389/7309, Y501 28MHz

Commit message: Update sensor/power board outline
Parts:
- removed REF**: PCB Edge, Connector_FFC-FPC:TE_4-1734839-0_1x40-1MP_P0.5mm_Horizontal
- added H501: MountingHole, MountingHole:MountingHole_2.2mm_M2_DIN965, F.Cu at (131.0, 86.0)
- added H502: MountingHole, MountingHole:MountingHole_2.2mm_M2_DIN965, F.Cu at (169.0, 86.0)
- added H503: MountingHole, MountingHole:MountingHole_2.2mm_M2_DIN965, F.Cu at (169.0, 124.0)
- added J501: Sensor Board, Connector_FFC-FPC:Hirose_FH12-30S-0.5SH_1x30-1MP_P0.50mm_Horizontal, F.Cu at (167.0, 129.8)
- U507: moved to B.Cu
- moved U507 119.9 mm to (150.0, 105.0), turned to 180 degrees
- moved R548 11.9 mm to (110.0, 120.5)
- moved R549 11.9 mm to (112.0, 120.5)
Other:
- board outline added: 56 x 55 mm

Commit message: Update sensorboard outline and connector
Parts:
- added C607: 100nF, Capacitor_SMD:C_0603_1608Metric, F.Cu at (73.3, 48.3)
- added C610: 10uF, Capacitor_SMD:C_0603_1608Metric, F.Cu at (73.3, 50.8)
- added FB511: FerriteBead, Inductor_SMD:L_0603_1608Metric, F.Cu at (73.3, 53.3)
- added J502: FPC 0.5mm Bottom Contact, Connector_FFC-FPC:Hirose_FH12-30S-0.5SH_1x30-1MP_P0.50mm_Horizontal, F.Cu at (82.4, 39.6)
- added U521: Si5351A-B-GT, Package_SO:MSOP-10_3x3mm_P0.5mm, F.Cu at (79.0, 49.4)
- J501: value Sensor Board -> FPC 0.5mm Bottom Contact
- moved J501 42.5 mm to (174.4, 88.0), turned to 90 degrees
Connections:
- C516 pad 2: /afe/CLI -> Net-(U521-XA)
- C517 pad 2: /afe/CLO -> Net-(U521-XB)
- J501 pad 10: GND -> AFE_SL
- J501 pad 11: CSI_HSYNC -> GND
- J501 pad 12: CSI_VSYNC -> CSI_HSYNC
- J501 pad 13: GND -> CSI_VSYNC
- J501 pad 4: unconnected-(J501-Pin_4-Pad4) -> I2C_SDA
- J501 pad 5: AFE_SYNC -> I2C_SCL
- J501 pad 6: AFE_RST -> AFE_SYNC
- J501 pad 7: AFE_SCK -> AFE_RST
- J501 pad 8: AFE_SDATA -> AFE_SCK
- J501 pad 9: AFE_SL -> AFE_SDATA
- U506 pad B6: /afe/CLO -> unconnected-(U506-CLO-PadB6)
- Y501 pad 1: /afe/CLI -> Net-(U521-XA)
- Y501 pad 3: /afe/CLO -> Net-(U521-XB)
Routing:
- net /afe/CLO: track 7.27 -> 0.00 mm
- net /afe/CLI: track 5.34 -> 0.00 mm
- net Net-(U521-XB): track 0.00 -> 1.78 mm
- net Net-(U521-XA): track 0.00 -> 1.76 mm
Other:
- board size 56 x 55 mm -> 58 x 53 mm

Commit message: Update sensorboard to include heatsink
Parts:
- added HS501: Heatsink, footprints:sb_heatsink, B.Cu at (150.0, 105.0)
- C607: footprint Capacitor_SMD:C_0603_1608Metric -> Capacitor_SMD:C_0402_1005Metric
- moved H503 38.0 mm to (131.0, 124.0)
Changed lines of the file:
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@@
   )
   (footprint "MountingHole:MountingHole_2.2mm_M2_DIN965" (layer "F.Cu")
-    (at 169 124)
+    (at 131 124)
     (descr "Mounting Hole 2.2mm, no annular, M2, DIN965")
     (tags "mounting hole 2.2mm no annular m2 din965")
@@
     )
   )
-  (footprint "Capacitor_SMD:C_0603_1608Metric" (layer "F.Cu")
+  (footprint "Capacitor_SMD:C_0402_1005Metric" (layer "F.Cu")
     (at 73.2875 48.28)
-    (descr "Capacitor SMD 0603 (1608 Metric), square (rectangular) end terminal, IPC_7351 nominal, (Body size source: IPC-SM-782 page 76, https://www.pcb-3d.com/wordpress/wp-content/uploads/ipc-sm-782a_amendment_1_and_2.pdf), generated with kicad-footprint-generator")
+    (descr "Capacitor SMD 0402 (1005 Metric), square (rectangular) end terminal, IPC_7351 nominal, (Body size source: IPC-SM-782 page 76, https://www.pcb-3d.com/wordpress/wp-content/uploads/ipc-sm-782a_amendment_1_and_2.pdf), generated with kicad-footprint-generator")
     (tags "capacitor")
     (property "Sheetfile" "afe.kicad_sch")
@@
     (property "ki_keywords" "cap capacitor")
     (attr smd)
-    (fp_text reference "C607" (at 0 -1.43) (layer "F.SilkS")
+    (fp_text reference "C607" (at 0 -1.16) (layer "F.SilkS")
         (effects (font (size 1 1) (thickness 0.15)))
     )
-    (fp_text value "100nF" (at 0 1.43) (layer "F.Fab")
+    (fp_text value "100nF" (at 0 1.16) (layer "F.Fab")
         (effects (font (size 1 1) (thickness 0.15)))
     )
     (fp_text user "${REFERENCE}" (at 0 0) (layer "F.Fab")
-        (effects (font (size 0.4 0.4) (thickness 0.06)))
+        (effects (font (size 0.25 0.25) (thickness 0.04)))
     )
-    (fp_line (start -0.14058 -0.51) (end 0.14058 -0.51)
+    (fp_line (start -0.107836 -0.36) (end 0.107836 -0.36)
       (stroke (width 0.12) (type solid)) (layer "F.SilkS"))
-    (fp_line (start -0.14058 0.51) (end 0.14058 0.51)
+    (fp_line (start -0.107836 0.36) (end 0.107836 0.36)
       (stroke (width 0.12) (type solid)) (layer "F.SilkS"))
-    (fp_line (start -1.48 -0.73) (end 1.48 -0.73)
+    (fp_line (start -0.91 -0.46) (end 0.91 -0.46)
       (stroke (width 0.05) (type solid)) (layer "F.CrtYd"))
-    (fp_line (start -1.48 0.73) (end -1.48 -0.73)
+    (fp_line (start -0.91 0.46) (end -0.91 -0.46)
       (stroke (width 0.05) (type solid)) (layer "F.CrtYd"))
-    (fp_line (start 1.48 -0.73) (end 1.48 0.73)
+    (fp_line (start 0.91 -0.46) (end 0.91 0.46)
       (stroke (width 0.05) (type solid)) (layer "F.CrtYd"))
-    (fp_line (start 1.48 0.73) (end -1.48 0.73)
+    (fp_line (start 0.91 0.46) (end -0.91 0.46)
       (stroke (width 0.05) (type solid)) (layer "F.CrtYd"))
-    (fp_line (start -0.8 -0.4) (end 0.8 -0.4)
+    (fp_line (start -0.5 -0.25) (end 0.5 -0.25)
       (stroke (width 0.1) (type solid)) (layer "F.Fab"))
-    (fp_line (start -0.8 0.4) (end -0.8 -0.4)
+    (fp_line (start -0.5 0.25) (end -0.5 -0.25)
       (stroke (width 0.1) (type solid)) (layer "F.Fab"))
-    (fp_line (start 0.8 -0.4) (end 0.8 0.4)
+    (fp_line (start 0.5 -0.25) (end 0.5 0.25)
       (stroke (width 0.1) (type solid)) (layer "F.Fab"))
-    (fp_line (start 0.8 0.4) (end -0.8 0.4)
+    (fp_line (start 0.5 0.25) (end -0.5 0.25)
       (stroke (width 0.1) (type solid)) (layer "F.Fab"))
-    (pad "1" smd roundrect (at -0.775 0) (size 0.9 0.95) (layers "F.Cu" "F.Paste" "F.Mask") (roundrect_rratio 0.25)
+    (pad "1" smd roundrect (at -0.48 0) (size 0.56 0.62) (layers "F.Cu" "F.Paste" "F.Mask") (roundrect_rratio 0.25)
       (net 196 "Net-(U521-VDD)") (pintype "passive"))
-    (pad "2" smd roundrect (at 0.775 0) (size 0.9 0.95) (layers "F.Cu" "F.Paste" "F.Mask") (roundrect_rratio 0.25)
+    (pad "2" smd roundrect (at 0.48 0) (size 0.56 0.62) (layers "F.Cu" "F.Paste" "F.Mask") (roundrect_rratio 0.25)
       (net 15 "/afe/AVSS") (pintype "passive"))
-    (model "${KICAD6_3DMODEL_DIR}/Capacitor_SMD.3dshapes/C_0603_1608Metric.wrl"
+    (model "${KICAD6_3DMODEL_DIR}/Capacitor_SMD.3dshapes/C_0402_1005Metric.wrl"
       (offset (xyz 0 0 0))
       (scale (xyz 1 1 1))
@@
       (offset (xyz 0 0 0))
       (scale (xyz 1 1 1))
+      (rotate (xyz 0 0 0))
+    )
+  )
+  (footprint "footprints:sb_heatsink" (layer "B.Cu")
+    (at 150 105 180)
+    (property "Sheetfile" "connector.kicad_sch")
+    (property "Sheetname" "connector")
+    (property "ki_description" "Heatsink")
+    (property "ki_keywords" "thermal heat temperature")
+    (attr smd)
+    (fp_text reference "HS501" (at 0 0.5 unlocked) (layer "B.SilkS") hide
+        (effects (font (size 1 1) (thickness 0.1)) (justify mirror))
+    )
+    (fp_text value "Heatsink" (at 0 -1 unlocked) (layer "B.Fab")
+        (effects (font (size 1 1) (thickness 0.15)) (justify mirror))
+    )
+    (fp_text user "${REFERENCE}" (at 0 -2.5 unlocked) (layer "B.Fab")
+        (effects (font (size 1 1) (thickness 0.15)) (justify mirror))
+    )
+    (fp_line (start -33 28.5) (end -33 -21)
+      (stroke (width 0.1) (type default)) (layer "Dwgs.User"))
+    (fp_line (start -18.5 -21) (end -33 -21)
+      (stroke (width 0.1) (type default)) (layer "Dwgs.User"))
+    (fp_line (start -18.5 -15) (end -18.5 -21)
+      (stroke (width 0.1) (type default)) (layer "Dwgs.User"))
+    (fp_line (start -18.5 15) (end -18.5 17)
+      (stroke (width 0.1) (type default)) (layer "Dwgs.User"))
+    (fp_line (start -17 18.5) (end -18.5 17)
+      (stroke (width 0.1) (type default)) (layer "Dwgs.User"))
+    (fp_line (start -17 28.5) (end -33 28.5)
+      (stroke (width 0.1) (type default)) (layer "Dwgs.User"))
+    (fp_line (start -17 28.5) (end -17 18.5)
+      (stroke (width 0.1) (type default)) (layer "Dwgs.User"))
+    (fp_line (start 17 -18.5) (end 17 -21)
+      (stroke (width 0.1) (type default)) (layer "Dwgs.User"))
+    (fp_line (start 17 28.5) (end 17 18.5)
+      (stroke (width 0.1) (type default)) (layer "Dwgs.User"))
+    (fp_line (start 18.5 -17) (end 17 -18.5)
+      (stroke (width 0.1) (type default)) (layer "Dwgs.User"))
+    (fp_line (start 18.5 -17) (end 18.5 -15)
+      (stroke (width 0.1) (type default)) (layer "Dwgs.User"))
+    (fp_line (start 18.5 -15) (end -18.5 -15)
+      (stroke (width 0.1) (type default)) (layer "Dwgs.User"))
+    (fp_line (start 18.5 15) (end -18.5 15)
+      (stroke (width 0.1) (type default)) (layer "Dwgs.User"))
+    (fp_line (start 18.5 15) (end 18.5 17)
+      (stroke (width 0.1) (type default)) (layer "Dwgs.User"))
+    (fp_line (start 18.5 17) (end 17 18.5)
+      (stroke (width 0.1) (type default)) (layer "Dwgs.User"))
+    (fp_line (start 33 -21) (end 17 -21)
+      (stroke (width 0.1) (type default)) (layer "Dwgs.User"))
+    (fp_line (start 33 28.5) (end 17 28.5)
+      (stroke (width 0.1) (type default)) (layer "Dwgs.User"))
+    (fp_line (start 33 28.5) (end 33 -21)
+      (stroke (width 0.1) (type default)) (layer "Dwgs.User"))
+    (fp_rect (start -7.5 -7.5) (end 7.5 7.5)
+      (stroke (width 0.1) (type default)) (fill none) (layer "Dwgs.User"))
+    (fp_circle (center -19 19) (end -17.9 19)
+      (stroke (width 0.1) (type default)) (fill none) (layer "Dwgs.User"))
+    (fp_circle (center 19 -19) (end 20.1 -19)
+      (stroke (width 0.1) (type default)) (fill none) (layer "Dwgs.User"))
+    (fp_circle (center 19 19) (end 20.1 19)
+      (stroke (width 0.1) (type default)) (fill none) (layer "Dwgs.User"))
+    (zone (net 0) (net_name "") (layers "B.Cu" "B.CrtYd") (hatch edge 0.5)
+      (connect_pads (clearance 0))
+      (min_thickness 0.25) (filled_areas_thickness no)
+      (keepout (tracks allowed) (vias allowed) (pads allowed) (copperpour allowed) (footprints not_allowed))
+      (fill (thermal_gap 0.5) (thermal_bridge_width 0.5))
+      (polygon
+        (pts
+          (xy 183 76.5)
+          (xy 183 126)
+          (xy 168.5 126)
+          (xy 168.5 120)
+          (xy 150 120)
+          (xy 150 112.5)
+          (xy 157.5 112.5)
+          (xy 157.5 97.5)
+          (xy 142.5 97.5)
+          (xy 142.5 112.5)
+          (xy 150 112.5)
+          (xy 150 120)
+          (xy 131.5 120)
+          (xy 131.5 122)
+          (xy 133 123.5)
+          (xy 133 126)
+          (xy 117 126)
+          (xy 117 76.5)
+          (xy 133 76.5)
+          (xy 133 86.5)
+          (xy 131.5 88)
+          (xy 131.5 90)
+          (xy 168.5 90)
+          (xy 168.5 88)
+          (xy 167 86.5)
+          (xy 167 76.5)
+        )
+      )
+    )
+    (model "${KIPRJMOD}/../common/footprints.pretty/heatsink.step"
+      (offset (xyz 0 0 0))
+      (scale (xyz 1 1 1))

Commit message: PowerBoard Floorplan
Parts:
- removed JP501, JP502, JP503, JP504: SolderJumper_2_Bridged, Jumper:SolderJumper-2_P1.3mm_Bridged2Bar_Pad1.0x1.5mm
- added R550: 0, Resistor_SMD:R_0402_1005Metric, F.Cu at (30.6, 81.2)
- added R551: 0, Resistor_SMD:R_0402_1005Metric, F.Cu at (19.1, 81.3)
- added R552: 0, Resistor_SMD:R_0402_1005Metric, B.Cu at (25.3, 84.8)
- added R560: 0, Resistor_SMD:R_0402_1005Metric, F.Cu at (16.4, 73.9)
- C503, C504, C508, C509, C607, C610, R506: moved to B.Cu
- moved J502 115.8 mm to (174.3, 110.0), turned to 90 degrees
- moved FB511 85.5 mm to (25.3, 124.0)
- moved U521 64.6 mm to (24.8, 84.6)
- moved C607 61.9 mm to (22.7, 84.1), turned to 90 degrees
- moved C610 59.6 mm to (24.0, 84.3), turned to 90 degrees
- moved C503 32.0 mm to (20.7, 84.7), turned to -90 degrees
- moved C508 31.8 mm to (18.7, 84.7), turned to 90 degrees
- moved R504 31.0 mm to (35.5, 85.2)
- moved R507 31.0 mm to (35.5, 84.0)
- moved U503 31.0 mm to (31.3, 84.0)
- moved C506 31.0 mm to (35.5, 86.2)
- moved R502 31.0 mm to (31.1, 86.9)
- moved R508 31.0 mm to (33.3, 86.9)
- moved U502 29.4 mm to (18.3, 84.1)
- moved C505 29.4 mm to (14.1, 82.0)
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Connections:
- C516 pad 2: Net-(U521-XA) -> Net-(U521-XB)
- C517 pad 2: Net-(U521-XB) -> Net-(U521-XA)
- Y501 pad 1: Net-(U521-XA) -> Net-(U521-XB)
- Y501 pad 3: Net-(U521-XB) -> Net-(U521-XA)
Routing:
- net GND: track 40.8 -> 21.2 mm
- net +16V: track 32.9 -> 13.6 mm
- net Net-(U521-VDD): track 0.00 -> 10.1 mm, vias 0 -> 2
- net /afe/CLI: track 0.00 -> 8.51 mm, vias 0 -> 2
- net Net-(U521-XB): track 1.78 -> 8.29 mm
- net /afe/AVSS: track 20.2 -> 15.1 mm, vias 4 -> 5
- net Net-(U502-ILIM): track 4.46 -> 0.00 mm
- net Net-(U521-XA): track 1.76 -> 6.19 mm
- net SYNC_CLK1: track 0.00 -> 4.29 mm
- net /afe/AVSSA: track 28.3 -> 31.6 mm
- net SYNC_CLK2: track 0.00 -> 2.93 mm
- net /afe/AVSSB: track 28.7 -> 31.3 mm
- net +15VR: track 10.1 -> 7.82 mm
- net Net-(U502-PGFB): track 7.91 -> 10.1 mm, vias 0 -> 3
- net +15VL: track 10.9 -> 8.80 mm
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
Commit message: CCD Sensor Board WIP
Parts:
- removed C538, C539, C570, C571, C572, C573: 100nF, Capacitor_SMD:C_0402_1005Metric
- removed C557, C558, C559: 10uF, Capacitor_SMD:C_0402_1005Metric
- removed JP505, JP506, JP507: Jumper_2_Bridged, Jumper:SolderJumper-2_P1.3mm_Bridged_RoundedPad1.0x1.5mm
- added C611: 100nF, Capacitor_SMD:C_0402_1005Metric, B.Cu at (174.1, 139.3)
- added C612: 100nF, Capacitor_SMD:C_0402_1005Metric, B.Cu at (166.8, 138.3)
- added C613: 100nF, Capacitor_SMD:C_0402_1005Metric, B.Cu at (156.0, 138.4)
- added C614: 100nF, Capacitor_SMD:C_0402_1005Metric, B.Cu at (170.4, 139.5)
- added C615: 100nF, Capacitor_SMD:C_0402_1005Metric, B.Cu at (170.4, 138.3)
- added C616: 100nF, Capacitor_SMD:C_0402_1005Metric, B.Cu at (163.2, 139.6)
- added C617: 100nF, Capacitor_SMD:C_0402_1005Metric, B.Cu at (163.2, 138.4)
- added C618: 100nF, Capacitor_SMD:C_0402_1005Metric, B.Cu at (159.6, 139.6)
- added C619: 100nF, Capacitor_SMD:C_0402_1005Metric, B.Cu at (159.6, 138.4)
- added C620: 100nF, Capacitor_SMD:C_0402_1005Metric, B.Cu at (156.0, 139.6)
- added R561: 50, Resistor_SMD:R_0402_1005Metric, F.Cu at (160.2, 115.2)
- added RN501: 50, Resistor_SMD:R_Array_Convex_4x0402, F.Cu at (171.4, 111.0)
- added RN502: 50, Resistor_SMD:R_Array_Convex_4x0402, F.Cu at (162.3, 109.7)
- added RN503: 50, Resistor_SMD:R_Array_Convex_4x0402, F.Cu at (169.0, 109.7)
- added RN504: 50, Resistor_SMD:R_Array_Convex_4x0402, F.Cu at (164.9, 109.7)
- C501, C528, C529, C534, C535, C536, C537, C542, C568, C569, C596, C597, C600, C603, C606, FB511: moved to B.Cu
- C508, C509, C580, C581, C582, C584, C585, C586, C588, C589, C590, C598, C604, C605, R542, R543, R544, R545, R546, R547: moved to F.Cu
- C541: footprint Capacitor_SMD:C_0603_1608Metric -> Capacitor_SMD:C_0402_1005Metric; moved to B.Cu
- C574, C576: value 1uF -> DNP
- moved C552 177.2 mm to (180.1, 127.5), turned to -90 degrees
- moved C549 172.8 mm to (178.5, 127.4), turned to -90 degrees
- moved FB504 171.3 mm to (177.1, 124.8)
- moved C551 163.7 mm to (177.0, 105.2), turned to 180 degrees
- moved C554 163.5 mm to (180.8, 103.7), turned to 180 degrees
- moved C553 162.8 mm to (180.8, 100.3), turned to 180 degrees
- moved FB505 161.9 mm to (180.2, 104.8)
- moved C546 161.1 mm to (173.1, 103.9), turned to 90 degrees
- moved C550 160.6 mm to (177.0, 101.1), turned to 180 degrees
- moved C545 160.4 mm to (170.7, 104.6), turned to 90 degrees
- moved FB506 159.2 mm to (180.2, 101.6)
- moved C548 158.4 mm to (173.1, 101.9), turned to 90 degrees
- moved C547 157.5 mm to (170.7, 102.6), turned to -90 degrees
- moved RV502 156.6 mm to (183.5, 120.1), turned to 180 degrees
- moved FB507 155.8 mm to (176.4, 103.9)
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Connections:
- C502 pad 1: +3V3 -> +3V0
- C528 pad 1: /afe/DVSS -> DVSS
- C529 pad 1: /afe/DVSS -> DVSS
- C530 pad 1: /afe/DVSS -> DVSS
- C530 pad 2: +3V3 -> +3V0
- C531 pad 1: /afe/DVSS -> DVSS
- C531 pad 2: +3V3 -> +3V0
- C532 pad 1: /afe/DVSS -> DVSS
- C532 pad 2: +3V3 -> +3V0
- C533 pad 1: /afe/DVSS -> DVSS
- C533 pad 2: +3V3 -> +3V0
- C534 pad 1: /afe/DVSS -> DVSS
- C534 pad 2: +3V3 -> +3V0
- C535 pad 1: /afe/DVSS -> DVSS
- C535 pad 2: +3V3 -> +3V0
- C536 pad 1: /afe/DVSS -> DVSS
- C536 pad 2: +3V3 -> +3V0
- C537 pad 1: /afe/DVSS -> DVSS
- C537 pad 2: +3V3 -> +3V0
- C540 pad 1: /afe/DVSS -> DVSS
- C540 pad 2: +3V3 -> +3V0
- C549 pad 1: /ccd/VDDL -> /ccd/VDDR
- C552 pad 1: /ccd/VDDL -> /ccd/VDDR
- C555 pad 1: /ccd/VDDR -> /ccd/VDDL
- C556 pad 1: /ccd/VDDR -> /ccd/VDDL
- C565 pad 2: +16V -> +16VD
- C568 pad 2: -3V5 -> GND
- C569 pad 1: +2V -> GND
- FB502 pad 1: +3V3 -> +3V0
- FB503 pad 1: +3V3 -> +3V0
- FB504 pad 1: +15VL -> +15VR
- FB504 pad 2: /ccd/VDDL -> /ccd/VDDR
- FB509 pad 1: +15VR -> +15VL
- FB509 pad 2: /ccd/VDDR -> /ccd/VDDL
- FB510 pad 1: +3V3 -> +3V0
- FB511 pad 1: +3V3 -> +3V0
- J501 pad 11: GND -> DVSS
- J501 pad 15: GND -> DVSS
- J501 pad 3: GND -> DVSS
- J501 pad 30: GND -> DVSS
- J501 pad MP: GND -> unconnected-(J501-MountPin-PadMP)
- J502 pad 1: SYNC_CLK2 -> -15V
- J502 pad 10: unconnected-(J502-Pin_10-Pad10) -> SYNC_CLK1
- J502 pad 11: unconnected-(J502-Pin_11-Pad11) -> GND
- J502 pad 12: unconnected-(J502-Pin_12-Pad12) -> -9VA
- J502 pad 13: unconnected-(J502-Pin_13-Pad13) -> +16V
- J502 pad 14: unconnected-(J502-Pin_14-Pad14) -> +16V
- J502 pad 15: unconnected-(J502-Pin_15-Pad15) -> +3V0
- J502 pad 16: unconnected-(J502-Pin_16-Pad16) -> GND
- J502 pad 17: unconnected-(J502-Pin_17-Pad17) -> GND
- J502 pad 18: unconnected-(J502-Pin_18-Pad18) -> GND
- J502 pad 19: unconnected-(J502-Pin_19-Pad19) -> +8V
- J502 pad 2: SYNC_CLK1 -> GND
- J502 pad 20: unconnected-(J502-Pin_20-Pad20) -> +8V
- J502 pad 21: unconnected-(J502-Pin_21-Pad21) -> +8V
- J502 pad 22: unconnected-(J502-Pin_22-Pad22) -> -9V
- J502 pad 23: unconnected-(J502-Pin_23-Pad23) -> -9V
- J502 pad 24: unconnected-(J502-Pin_24-Pad24) -> -9V
- J502 pad 25: unconnected-(J502-Pin_25-Pad25) -> GND
- J502 pad 26: unconnected-(J502-Pin_26-Pad26) -> GND
- J502 pad 27: unconnected-(J502-Pin_27-Pad27) -> -4V
- J502 pad 28: unconnected-(J502-Pin_28-Pad28) -> +5V
- J502 pad 29: unconnected-(J502-Pin_29-Pad29) -> +5V
- J502 pad 3: GND -> +2V
- J502 pad 30: unconnected-(J502-Pin_30-Pad30) -> GND
- J502 pad 4: unconnected-(J502-Pin_4-Pad4) -> GND
- J502 pad 5: unconnected-(J502-Pin_5-Pad5) -> +16VD
- J502 pad 6: unconnected-(J502-Pin_6-Pad6) -> GND
- J502 pad 7: unconnected-(J502-Pin_7-Pad7) -> -4V
- J502 pad 8: unconnected-(J502-Pin_8-Pad8) -> -4V
- J502 pad 9: unconnected-(J502-Pin_9-Pad9) -> SYNC_CLK2
- J502 pad MP: GND -> unconnected-(J502-MountPin-PadMP)
- Q501 pad 4: +16V -> +16VD
- R518 pad 1: +16V -> +16VD
- R560 pad 1: /afe/DVSS -> DVSS
- U501 pad 3: +3V3 -> +3V0
- U506 pad C10: +3V3 -> +3V0
- U506 pad C2: +3V3 -> +3V0
- U506 pad C3: /afe/DVSS -> DVSS
- U506 pad C6: /afe/DVSS -> DVSS
- U506 pad C9: /afe/DVSS -> DVSS
- U506 pad D3: +3V3 -> +3V0
- U506 pad D4: /afe/DVSS -> DVSS
- U506 pad D6: /afe/DVSS -> DVSS
- U506 pad D8: /afe/DVSS -> DVSS
- U506 pad D9: +3V3 -> +3V0
- U506 pad E3: /afe/DVSS -> DVSS
- U506 pad E4: +3V3 -> +3V0
- U506 pad H10: CSI_VSYNC -> /afe/CSI_VD_pre
- U506 pad H11: CSI_HSYNC -> /afe/CSI_HD_pre
- U506 pad H6: CSI_D2 -> /afe/CSI_D2_pre
- U506 pad H7: CSI_D9 -> /afe/CSI_D9_pre
- U506 pad J10: +3V3 -> +3V0
- U506 pad J11: +3V3 -> +3V0
- U506 pad J5: /afe/DVSS -> DVSS
- U506 pad J6: CSI_D3 -> /afe/CSI_D3_pre
- U506 pad J7: CSI_D8 -> /afe/CSI_D8_pre
- U506 pad J8: CSI_D12 -> /afe/CSI_D12_pre
- U506 pad J9: /afe/DVSS -> DVSS
- U506 pad K10: CSI_D15 -> /afe/CSI_D15_pre
- U506 pad K11: /afe/DVSS -> DVSS
- U506 pad K6: CSI_D4 -> /afe/CSI_D4_pre
- U506 pad K7: CSI_D7 -> /afe/CSI_D7_pre
- U506 pad K8: CSI_D11 -> /afe/CSI_D11_pre
- U506 pad K9: CSI_D14 -> /afe/CSI_D14_pre
- U506 pad L10: CSI_PIXCLK -> /afe/CSI_DCLK_pre
- U506 pad L6: CSI_D5 -> /afe/CSI_D5_pre
- U506 pad L7: CSI_D6 -> /afe/CSI_D6_pre
- U506 pad L8: CSI_D10 -> /afe/CSI_D10_pre
- U506 pad L9: CSI_D13 -> /afe/CSI_D13_pre
- U507 pad 18: /ccd/VDDR -> /ccd/VDDL
- U507 pad 19: CCDIN_R -> CCDIN_L
- U507 pad 2: CCDIN_L -> CCDIN_R
- U507 pad 3: /ccd/VDDL -> /ccd/VDDR
- U508 pad 4: /ccd_driver/RR -> /ccd_driver/RL
- U508 pad 6: /ccd_driver/RL -> /ccd_driver/RR
- U509 pad 4: /ccd_driver/H1BINR -> /ccd_driver/H1BINL
- U509 pad 6: /ccd_driver/H1BINL -> /ccd_driver/H1BINR
- U510 pad 1: /ccd_driver/H2S -> /ccd_driver/H1S
- U510 pad 4: /ccd_driver/H1SL -> /ccd_driver/H2SL
- U510 pad 6: /ccd_driver/H2SL -> /ccd_driver/H1SL
- U511 pad 1: /ccd_driver/H1S -> /ccd_driver/H2S
- U511 pad 3: /ccd_driver/H2S -> /ccd_driver/H1S
- U511 pad 4: /ccd_driver/H2BL -> /ccd_driver/H1BL
- U511 pad 6: /ccd_driver/H1BL -> /ccd_driver/H2BL
- U512 pad 1: /ccd_driver/H2S -> /ccd_driver/H1S
- U512 pad 3: /ccd_driver/H1S -> /ccd_driver/H2S
- U512 pad 4: /ccd_driver/H1BR -> /ccd_driver/H2BR
- U512 pad 6: /ccd_driver/H2BR -> /ccd_driver/H1BR
- U513 pad 1: /ccd_driver/H1S -> /ccd_driver/H2S
- U513 pad 3: /ccd_driver/H2S -> /ccd_driver/H1S
- U513 pad 4: /ccd_driver/H2SR -> /ccd_driver/H1SR
- U513 pad 6: /ccd_driver/H1SR -> /ccd_driver/H2SR
- U514 pad 5: Net-(JP506-A) -> /ccd_driver_v/V23
- U514 pad 6: Net-(JP506-A) -> /ccd_driver_v/V23
- U515 pad 5: Net-(JP505-A) -> /ccd_driver_v/V2S
- U515 pad 6: Net-(JP505-A) -> /ccd_driver_v/V2S
- U516 pad 5: Net-(JP507-A) -> /ccd_driver_v/V2S
- U516 pad 6: Net-(JP507-A) -> /ccd_driver_v/V2S
Routing:
- net GND: track 21.2 -> 473.2 mm, vias 2 -> 34
- net +5V: track 0.00 -> 121.7 mm, vias 0 -> 8
- net -9V: track 30.6 -> 138.5 mm, vias 0 -> 15
- net +8V: track 0.00 -> 99.9 mm, vias 0 -> 7
- net -4V: track 7.42 -> 100.3 mm, vias 0 -> 9
- net /ccd_driver/H1S: track 0.00 -> 87.3 mm, vias 0 -> 5
- net DVSS: track 0.00 -> 84.4 mm, vias 0 -> 9
- net +3V0: track 0.00 -> 81.0 mm, vias 0 -> 5
- net Net-(U515-IN-): track 0.00 -> 79.1 mm, vias 0 -> 2
- net /ccd_driver/H2S: track 3.93 -> 81.8 mm, vias 0 -> 4
- net +2V: track 7.38 -> 81.5 mm, vias 0 -> 7
- net Net-(U514-IN-): track 1.71 -> 62.4 mm, vias 0 -> 2
- net Net-(D507-K): track 0.00 -> 53.7 mm, vias 0 -> 2
- net Net-(U514-IN+): track 0.00 -> 48.7 mm, vias 0 -> 3
- net AFE_SL: track 1.21 -> 48.9 mm, vias 1 -> 2
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Other:
- board size 58 x 53 mm -> 58.4 x 58.6 mm

Commit message: Sensor Board WIP, minor
Parts:
- added C538: 100nF, Capacitor_SMD:C_0402_1005Metric, F.Cu at (166.8, 104.3)
- added C539: DNP/1nF, Capacitor_SMD:C_0402_1005Metric, F.Cu at (166.8, 105.5)
- added R562: 82K 1%, Resistor_SMD:R_0402_1005Metric, F.Cu at (166.8, 106.6)
- added RV508: 10K, Potentiometer_SMD:Potentiometer_Bourns_3214G_Horizontal, F.Cu at (163.1, 103.7)
- added RV509: 50K, Potentiometer_SMD:Potentiometer_Bourns_3214G_Horizontal, F.Cu at (186.7, 134.6)
- added U522: TLV76701DRVx, Package_SON:WSON-6-1EP_2x2mm_P0.65mm_EP1x1.6mm_ThermalVias, F.Cu at (167.2, 102.0)
- added U523: TPS72301, Package_TO_SOT_SMD:SOT-23-5_HandSoldering, F.Cu at (181.8, 138.7)
- added U524: XC6206P152MR, Package_TO_SOT_SMD:SOT-23-3, F.Cu at (177.7, 138.8)
- C565, C566: moved to F.Cu
- moved C545 33.6 mm to (204.3, 104.0)
- moved C547 33.6 mm to (204.3, 102.0)
- moved R513 33.6 mm to (205.3, 104.0)
- moved R514 33.6 mm to (205.3, 102.0)
- moved C546 33.5 mm to (206.6, 102.6)
- moved C548 33.5 mm to (206.6, 100.6)
- moved R515 33.5 mm to (207.6, 102.6)
- moved R516 33.5 mm to (207.6, 100.6)
- moved C550 25.5 mm to (201.4, 93.8)
- moved C551 25.5 mm to (201.4, 97.9)
- moved C553 25.5 mm to (205.2, 93.0)
- moved FB505 25.5 mm to (204.6, 97.5)
- moved FB506 25.5 mm to (204.6, 94.3)
- moved FB507 25.5 mm to (200.8, 96.6)
- moved FB508 25.5 mm to (200.8, 95.1)
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Connections:
- D510 pad 3: /ccd_driver_v/V2S -> /ccd_driver_v/V1S
- R558 pad 1: /ccd_driver_v/V2S -> /ccd_driver_v/V1S
- R559 pad 2: /ccd_driver_v/V2S -> /ccd_driver_v/V1S
- U516 pad 5: /ccd_driver_v/V2S -> /ccd_driver_v/V1S
- U516 pad 6: /ccd_driver_v/V2S -> /ccd_driver_v/V1S
Routing:
- net I2C_SCL: track 0.00 -> 77.7 mm, vias 0 -> 3
- net I2C_SDA: track 0.00 -> 75.8 mm, vias 0 -> 3
- net -4V: track 100.3 -> 166.0 mm, vias 9 -> 11
- net +16VD: track 0.00 -> 51.9 mm, vias 0 -> 8
- net +3V3: track 12.1 -> 57.3 mm
- net -15V: track 0.00 -> 42.9 mm, vias 0 -> 3
- net +16V: track 54.6 -> 75.4 mm
- net -3V5: track 6.77 -> 23.0 mm, vias 1 -> 2
- net GND: track 473.2 -> 486.4 mm, vias 34 -> 46
- net Net-(U522-FB): track 0.00 -> 12.7 mm, vias 0 -> 1
- net /ccd_driver_v/V1S: track 0.00 -> 10.6 mm
- net /ccd_driver_v/V2S: track 19.8 -> 9.19 mm
- net AFE_STROBE: track 16.7 -> 26.3 mm, vias 2 -> 3
- net Net-(Q501A-C1): track 0.00 -> 8.26 mm, vias 0 -> 4
- net VAB: track 0.00 -> 7.69 mm
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- added copper zone on B.Cu, net GND
- added copper zone on F.Cu, net GND
- added copper zone on In1.Cu, net GND
- added copper zone on In2.Cu, net GND
