File: Hardware/sensorboard/pcb.kicad_pcb (KiCad board)
At the start: 4 copper layers, 58.4 x 58.6 mm, 241 parts, among them J501 FPC 0.5mm Bottom Contact, J502 FPC 0.5mm Bottom Contact, Q501 BC847BPN, U501 XC6206P152MR, U502 LT3045xMSE, U503 LT3045xMSE, U504 ADA4800, U505 ADA4800, U506 AD9990, U507 KAI-1100x, U508 74HC2G17, U509 74HC2G17, U510 74HC2G17, U511 74HC2G17, U512 74HC2G17, U513 74HC2G17, U514 1EDN7550B, U515 1EDN7550B, U516 1EDN7550B, U517 1EDN7550B, U518 IRF9389/7309, U519 IRF9389/7309, U520 IRF9389/7309, U521 Si5351A-B-GT, U522 TLV76701DRVx, U523 TPS72301, U524 XC6206P152MR, Y501 28MHz

Commit message: Sensor Board Routing, First Pass Done, Ground Splitting TBD
Parts:
- removed C530, C532, C540: 10uF, Capacitor_SMD:C_0603_1608Metric
- removed C531, C533: 100nF, Capacitor_SMD:C_0402_1005Metric
- removed C574: DNP, Capacitor_SMD:C_0402_1005Metric
- moved R515 47.7 mm to (160.0, 106.7), turned to 0 degrees
- moved C546 46.7 mm to (160.0, 105.7), turned to 0 degrees
- moved R516 46.0 mm to (162.0, 106.7), turned to 0 degrees
- moved C548 44.9 mm to (162.0, 105.7), turned to 0 degrees
- moved C545 42.7 mm to (161.6, 103.8)
- moved C547 42.7 mm to (161.6, 101.8)
- moved R513 42.7 mm to (162.6, 103.8)
- moved R514 42.7 mm to (162.6, 101.8)
- moved C554 42.3 mm to (163.6, 104.3), turned to -90 degrees
- moved C553 42.1 mm to (164.6, 104.3), turned to -90 degrees
- moved FB506 40.9 mm to (164.6, 102.6)
- moved FB505 40.2 mm to (164.6, 101.1)
- moved C551 35.2 mm to (166.8, 104.3), turned to -90 degrees
- moved C550 35.2 mm to (167.8, 104.3), turned to -90 degrees
- moved FB508 33.9 mm to (167.8, 102.6)
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Connections:
- J501 pad MP: unconnected-(J501-MountPin-PadMP) -> (no net)
- J502 pad MP: unconnected-(J502-MountPin-PadMP) -> (no net)
Routing:
- net -9V: track 142.1 -> 201.6 mm, vias 15 -> 17
- net Net-(D506-K): track 3.49 -> 35.7 mm, vias 1 -> 2
- net -4V: track 166.0 -> 195.5 mm, vias 11 -> 13
- net +2V: track 87.0 -> 115.2 mm, vias 7 -> 9
- net GND: track 486.4 -> 510.8 mm, vias 46 -> 49
- net /ccd/VRDR: track 0.00 -> 23.7 mm, vias 0 -> 1
- net /ccd/VOGR: track 0.00 -> 22.8 mm
- net /ccd/VOGL: track 0.00 -> 21.4 mm
- net +1V5: track 10.6 -> 31.9 mm
- net +15VL: track 21.2 -> 39.8 mm
- net DVSS: track 85.9 -> 102.4 mm
- net -3V5: track 23.0 -> 38.9 mm, vias 2 -> 4
- net /ccd/VRDL: track 0.00 -> 13.9 mm, vias 0 -> 1
- net Net-(R562-Pad2): track 2.16 -> 15.7 mm
- net /afe/AVSS: track 25.0 -> 36.2 mm
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
Commit message: Sensor Board Routing Done
Parts:
- removed RV509: 50K, Potentiometer_SMD:Potentiometer_Bourns_3214G_Horizontal
- added C530: 10uF, Capacitor_SMD:C_0603_1608Metric, F.Cu at (186.1, 114.7)
- added C532: 10uF, Capacitor_SMD:C_0603_1608Metric, F.Cu at (186.1, 116.2)
- added C540: 10uF, Capacitor_SMD:C_0603_1608Metric, F.Cu at (188.5, 118.3)
- added R563: 0, Resistor_SMD:R_0402_1005Metric, F.Cu at (184.6, 140.6)
- added R564: 10K, Resistor_SMD:R_0402_1005Metric, F.Cu at (184.7, 138.1)
- added R565: 10K, Resistor_SMD:R_0402_1005Metric, F.Cu at (184.7, 136.1)
- added R566: 10K, Resistor_SMD:R_0402_1005Metric, F.Cu at (184.7, 137.1)
Connections:
- C528 pad 1: DVSS -> GND
- C529 pad 1: DVSS -> GND
- C534 pad 1: DVSS -> GND
- C535 pad 1: DVSS -> GND
- C536 pad 1: DVSS -> GND
- C537 pad 1: DVSS -> GND
- J501 pad 11: DVSS -> GND
- J501 pad 15: DVSS -> GND
- J501 pad 3: DVSS -> GND
- J501 pad 30: DVSS -> GND
- R546 pad 2: +3V3 -> +3V0
- R548 pad 2: +3V3 -> +3V0
- R560 pad 1: DVSS -> /afe/DVSS
- U506 pad C3: DVSS -> GND
- U506 pad C6: DVSS -> GND
- U506 pad C9: DVSS -> GND
- U506 pad D4: DVSS -> GND
- U506 pad D6: DVSS -> GND
- U506 pad D8: DVSS -> GND
- U506 pad E3: DVSS -> GND
- U506 pad J5: DVSS -> GND
- U506 pad J9: DVSS -> GND
- U506 pad K11: DVSS -> GND
- U523 pad 3: -4V -> Net-(U523-EN)
Routing:
- net GND: track 510.8 -> 618.9 mm, vias 49 -> 62
- net DVSS: track 102.4 -> 0.00 mm, vias 9 -> 0
- net +3V3: track 64.7 -> 5.01 mm, vias 4 -> 2
- net +3V0: track 87.0 -> 141.8 mm, vias 6 -> 8
- net -4V: track 195.5 -> 184.4 mm
- net +2V: track 115.2 -> 112.0 mm
- net Net-(U523-EN): track 0.00 -> 2.20 mm
- net Net-(U517-IN+): track 24.8 -> 26.2 mm, vias 2 -> 3
- net -3V5: track 38.9 -> 40.2 mm
- net Net-(R565-Pad2): track 0.00 -> 1.00 mm
- net (no net): track 0.64 -> 0.00 mm
- net Net-(U514-IN+): track 51.3 -> 50.7 mm
- net Net-(U523-NR/FB): track 3.99 -> 4.52 mm
- net Net-(D507-K): vias 2 -> 3
Other:
- board text added: "FDG"
- board text added: "FDG TIMING"
- board text added: "H1"
- board text added: "H1 Bias"
- board text added: "H2"
- board text added: "H2 Bias"
- board text added: "RG"
- board text added: "RG Bias"
- board text added: "V1"
- board text added: "V1 TIMING"
- board text added: "V2"
- board text added: "V2 TIMING"
- board text added: "V23"
- board text added: "V23 TIMING"
- board text added: "VAB"
- board text added: "VAB Adjust"
