File: Hardware/sensorboard/afe.kicad_sch (KiCad schematic)
At the start: 40 parts, among them U1001 ADA4800, U1002 ADA4800, U1003 AD9990, Y1001 28MHz

Commit message: Power Board WIP
Parts:
- removed C1032: 10uF, Capacitor_SMD:C_0603_1608Metric, symbol Device:C
- removed R1001, R1002: 49.9K 1%, Resistor_SMD:R_0402_1005Metric, symbol Device:R
- removed R1003, R1004: 200K 1%, Resistor_SMD:R_0402_1005Metric, symbol Device:R
- added C541: 100nF, Capacitor_SMD:C_0603_1608Metric, symbol Device:C
- added C542, C544, C609: 10uF, Capacitor_SMD:C_0603_1608Metric, symbol Device:C
- added C543, C608: 100nF, Capacitor_SMD:C_0402_1005Metric, symbol Device:C
- added FB501, FB502, FB503, FB510: FerriteBead, Inductor_SMD:L_0603_1608Metric, symbol Device:FerriteBead
- added JP501, JP502, JP503, JP504: SolderJumper_2_Bridged, Jumper:SolderJumper-2_P1.3mm_Bridged2Bar_Pad1.0x1.5mm, symbol Jumper:SolderJumper_2_Bridged
- added R509, R510: 49.9K 1%, Resistor_SMD:R_0402_1005Metric, symbol Device:R_US
- added R511, R512: 200K 1%, Resistor_SMD:R_0402_1005Metric, symbol Device:R_US
- renumbered C1001 to C510, C1002 to C511, C1003 to C512, C1004 to C513, C1007 to C514, C1008 to C515, C1009 to C516, C1010 to C517, C1011 to C518, C1012 to C519, C1013 to C520, C1014 to C521, C1005 to C522, C1006 to C523, C1015 to C524, C1016 to C525, C1017 to C526, C1018 to C527, C1019 to C528, C1020 to C529, C1021 to C530, C1022 to C531, C1023 to C532, C1024 to C533, C1025 to C534, C1026 to C535, C1027 to C536, C1028 to C537, C1030 to C538, C1031 to C539, C1029 to C540, U1001 to U504, U1002 to U505, U1003 to U506, Y1001 to Y501
Connections:
- net +15VL: now also R510.1, R512.1
- net +15VR: now also R509.1, R511.1
- net +3V3: now also FB502.1, FB503.1, FB510.1; no longer U506.A6 (CLIVDD), U506.B10 (LDOIN_B), U506.B2 (LDOIN_A)
- net AVDDA: no longer C528.2, C529.2, U506.B7 (TCVDD), U506.H5 (DVDD)
- net GND: now also JP501.2 (B), JP502.2 (B), JP503.2 (B), JP504.2 (B); no longer C510.2, C511.2, C512.2, C513.2, C514.2, C515.2, C516.1, C517.1, C518.2, C519.2, C520.2, C521.2, C524.1, C525.1, C526.1, C527.1, C528.1, C529.1, C530.1, C531.1, C532.1, C533.1, C534.1, C535.1, C536.1, C537.1, C538.1, C539.1, C540.1, U504.2 (VEE), U504.7 (EPAD), U505.2 (VEE), U505.7 (EPAD), U506.A3 (AVSS_A), U506.A5 (AVSS_A), U506.A7 (AVSS_B), U506.A9 (AVSS_B), U506.B3 (LDOVSS_A), U506.B9 (LDOVSS_B), U506.C3 (RGVSS_A), U506.C5 (AVSS_A), U506.C6 (TCVSS), U506.C7 (AVSS_B), U506.C9 (RGVSS_B), U506.D4 (HVSS_A), U506.D5 (NC), U506.D6 (TCVSS), U506.D8 (HVSS_B), U506.E3 (XVVSS), U506.J5 (DVSS), U506.J9 (DRVSS), U506.K11 (IOVSS), U506.L1 (NC), U506.L11 (NC), Y501.2, Y501.4
- net at C512.1, U504.4 (IDRV): now also R511.2
- net at C511.1, U505.6 (ISF): now also R510.2
- net at C513.1, U505.4 (IDRV): now also R512.2
- net at C510.1, U504.6 (ISF): now also R509.2
- new net: C608.1, C609.1, FB510.2, U506.B10 (LDOIN_B)
- new net: C529.2, FB501.1, U506.B7 (TCVDD)
- new net: C541.1, C542.1, FB503.2, U506.A6 (CLIVDD)
- new net: C543.1, C544.1, FB502.2, U506.B2 (LDOIN_A)
- new net +1V8: C528.2, FB501.2, U506.H5 (DVDD)
- new net AVSS: C516.1, C517.1, C541.2, C542.2, JP503.1 (A), U506.B3 (LDOVSS_A), U506.B9 (LDOVSS_B), Y501.2, Y501.4
- new net AVSSA: C510.2, C512.2, C514.2, C518.2, C519.2, C524.1, C525.1, C543.2, C544.2, JP501.1 (A), U504.2 (VEE), U504.7 (EPAD), U506.A3 (AVSS_A), U506.A5 (AVSS_A), U506.C5 (AVSS_A)
- new net AVSSB: C511.2, C513.2, C515.2, C520.2, C521.2, C526.1, C527.1, C608.2, C609.2, JP502.1 (A), U505.2 (VEE), U505.7 (EPAD), U506.A7 (AVSS_B), U506.A9 (AVSS_B), U506.C7 (AVSS_B)
- new net DVSS: C528.1, C529.1, C530.1, C531.1, C532.1, C533.1, C534.1, C535.1, C536.1, C537.1, C538.1, C539.1, C540.1, JP504.1 (A), U506.C3 (RGVSS_A), U506.C6 (TCVSS), U506.C9 (RGVSS_B), U506.D4 (HVSS_A), U506.D6 (TCVSS), U506.D8 (HVSS_B), U506.E3 (XVVSS), U506.J5 (DVSS), U506.J9 (DRVSS), U506.K11 (IOVSS)
- no-connect marks 37 -> 40
Other:
- note added: "Analog Timing Core"
- note added: "Digital Core"
- note added: "Digital Data Lines"
- note added: "Digital IO"
- note added: "H Drivers"
- note added: "RG Drivers"
- note added: "Reference Clock Generator"
- note added: "XV Output (V Clocks)"
- moved on the sheet: C518, C520, C522, C523, C524, C525, C526, C527, C528, C529, C530, C531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

Commit message: Update sensorboard outline and connector
Parts:
- added C607: 100nF, Capacitor_SMD:C_0603_1608Metric, symbol Device:C
- added C610: 10uF, Capacitor_SMD:C_0603_1608Metric, symbol Device:C
- added FB511: FerriteBead, Inductor_SMD:L_0603_1608Metric, symbol Device:FerriteBead
- added U521: Si5351A-B-GT, Package_SO:MSOP-10_3x3mm_P0.5mm, symbol Oscillator:Si5351A-B-GT
Connections:
- net +3V3: now also FB511.1
- net AVSS: now also C607.2, C610.2, U521.8 (GND)
- net CLI: now also U521.10 (CLK0); no longer C516.2, Y501.1
- net CLO: no longer names the net of C517.2, Y501.3
- net CLO: now also U521.3 (XB); no longer U506.B6 (CLO)
- new net: C607.1, C610.1, FB511.2, U521.1 (VDD), U521.7 (VDDO)
- new net: C516.2, U521.2 (XA), Y501.1
- new net I2C_SCL: U521.4 (SCL)
- new net I2C_SDA: U521.5 (SDA)
- new net SYNC_CLK1: U521.9 (CLK1)
- new net SYNC_CLK2: U521.6 (CLK2)
Other:
- moved on the sheet: C516, C517, Y501

Commit message: Update sensorboard to include heatsink
Parts:
- C607: footprint Capacitor_SMD:C_0603_1608Metric -> Capacitor_SMD:C_0402_1005Metric
Changed lines of the file:
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@@
       (effects (font (size 1.27 1.27)))
     )
-    (property "Footprint" "Capacitor_SMD:C_0603_1608Metric" (at 86.36 151.4348 0)
+    (property "Footprint" "Capacitor_SMD:C_0402_1005Metric" (at 86.36 151.4348 0)
       (effects (font (size 1.27 1.27)) hide)
     )

Commit message: PowerBoard Floorplan
Parts:
- removed JP501, JP502, JP503, JP504: SolderJumper_2_Bridged, Jumper:SolderJumper-2_P1.3mm_Bridged2Bar_Pad1.0x1.5mm, symbol Jumper:SolderJumper_2_Bridged
- added R550, R551, R552, R560: 0, Resistor_SMD:R_0402_1005Metric, symbol Device:R_US
Connections:
- net AVSS: now also R552.1
- net AVSSA: now also R550.1
- net AVSSB: now also R551.1
- net CLI: no longer U521.10 (CLK0)
- net DVSS: now also R560.1
- net GND: now also R550.2, R551.2, R552.2, R560.2
- net I2C_SCL: now also U521.6 (CLK2); no longer U521.4 (SCL)
- net I2C_SDA: no longer U521.5 (SDA)
- net SYNC_CLK1: no longer U521.9 (CLK1)
- net SYNC_CLK2: now also U521.4 (SCL); no longer U521.6 (CLK2)
- net at C517.2, Y501.3: no longer U521.3 (XB)
- net at C516.2, Y501.1: no longer U521.2 (XA)

Commit message: CCD Sensor Board WIP
Parts:
- removed C538, C539: 100nF, Capacitor_SMD:C_0402_1005Metric, symbol Device:C
- added R561: 50, Resistor_SMD:R_0402_1005Metric, symbol Device:R_US
- added RN501, RN502, RN503, RN504: 50, Resistor_SMD:R_Array_Convex_4x0402, symbol Device:R_Pack04
- C541: footprint Capacitor_SMD:C_0603_1608Metric -> Capacitor_SMD:C_0402_1005Metric
Connections:
- net CLI: now also U521.10 (CLK0)
- net CSI_D10: now also RN504.1 (R1.1); no longer U506.L8 (D8)
- net CSI_D11: now also RN504.2 (R2.1); no longer U506.K8 (D9)
- net CSI_D12: now also RN503.2 (R2.1); no longer U506.J8 (D10)
- net CSI_D13: now also RN504.3 (R3.1); no longer U506.L9 (D11)
- net CSI_D14: now also RN504.4 (R4.1); no longer U506.K9 (D12)
- net CSI_D15: now also RN502.2 (R2.1); no longer U506.K10 (D13)
- net CSI_D2: now also RN501.1 (R1.1); no longer U506.H6 (D0)
- net CSI_D3: now also RN501.2 (R2.1); no longer U506.J6 (D1)
- net CSI_D4: now also RN501.4 (R4.1); no longer U506.K6 (D2)
- net CSI_D5: now also RN503.1 (R1.1); no longer U506.L6 (D3)
- net CSI_D6: now also RN503.3 (R3.1); no longer U506.L7 (D4)
- net CSI_D7: now also RN503.4 (R4.1); no longer U506.K7 (D5)
- net CSI_D8: now also RN501.3 (R3.1); no longer U506.J7 (D6)
- net CSI_D9: now also R561.2; no longer U506.H7 (D7)
- net CSI_HSYNC: now also RN502.4 (R4.1); no longer U506.H11 (HD)
- net CSI_PIXCLK: now also RN502.1 (R1.1); no longer U506.L10 (DCLK)
- net CSI_VSYNC: now also RN502.3 (R3.1); no longer U506.H10 (VD)
- net I2C_SCL: now also U521.4 (SCL); no longer U521.6 (CLK2)
- net I2C_SDA: now also U521.5 (SDA)
- net SYNC_CLK1: now also U521.9 (CLK1)
- net SYNC_CLK2: now also U521.6 (CLK2); no longer U521.4 (SCL)
- net at C517.2, Y501.3: now also U521.2 (XA)
- net at C516.2, Y501.1: now also U521.3 (XB)
- net +3V3 renamed +3V0
- new net CSI_D10_pre: RN504.8 (R1.2), U506.L8 (D8)
- new net CSI_D11_pre: RN504.7 (R2.2), U506.K8 (D9)
- new net CSI_D12_pre: RN503.7 (R2.2), U506.J8 (D10)
- new net CSI_D13_pre: RN504.6 (R3.2), U506.L9 (D11)
- new net CSI_D14_pre: RN504.5 (R4.2), U506.K9 (D12)
- new net CSI_D15_pre: RN502.7 (R2.2), U506.K10 (D13)
- new net CSI_D2_pre: RN501.8 (R1.2), U506.H6 (D0)
- new net CSI_D3_pre: RN501.7 (R2.2), U506.J6 (D1)
- new net CSI_D4_pre: RN501.5 (R4.2), U506.K6 (D2)
- new net CSI_D5_pre: RN503.8 (R1.2), U506.L6 (D3)
- new net CSI_D6_pre: RN503.6 (R3.2), U506.L7 (D4)
- new net CSI_D7_pre: RN503.5 (R4.2), U506.K7 (D5)
- new net CSI_D8_pre: RN501.6 (R3.2), U506.J7 (D6)
- new net CSI_D9_pre: R561.1, U506.H7 (D7)
- new net CSI_DCLK_pre: RN502.8 (R1.2), U506.L10 (DCLK)
- new net CSI_HD_pre: RN502.5 (R4.2), U506.H11 (HD)
- new net CSI_VD_pre: RN502.6 (R3.2), U506.H10 (VD)
Other:
- moved on the sheet: C510, C511, C512, C513, C514, C515, C516, C517, C518, C519, C520, C521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

Commit message: Sensor Board Routing Done
Parts:
- removed C531, C533: 100nF, Capacitor_SMD:C_0402_1005Metric, symbol Device:C
Connections:
- net DVSS: no longer C528.1, C529.1, C530.1, C532.1, C534.1, C535.1, C536.1, C537.1, C540.1, U506.C3 (RGVSS_A), U506.C6 (TCVSS), U506.C9 (RGVSS_B), U506.D4 (HVSS_A), U506.D6 (TCVSS), U506.D8 (HVSS_B), U506.E3 (XVVSS), U506.J5 (DVSS), U506.J9 (DRVSS), U506.K11 (IOVSS)
- net GND: now also C528.1, C529.1, C530.1, C532.1, C534.1, C535.1, C536.1, C537.1, C540.1, U506.C3 (RGVSS_A), U506.C6 (TCVSS), U506.C9 (RGVSS_B), U506.D4 (HVSS_A), U506.D6 (TCVSS), U506.D8 (HVSS_B), U506.E3 (XVVSS), U506.J5 (DVSS), U506.J9 (DRVSS), U506.K11 (IOVSS)
- no-connect marks 40 -> 48

Commit message: Uploading Sensorboard Production Files
Parts:
- removed R560: 0, Resistor_SMD:R_0402_1005Metric, symbol Device:R_US
Changed lines of the file:
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@@
   (junction (at 205.74 115.57) (diameter 0) (color 0 0 0 0)
   )
-  (junction (at 228.6 107.95) (diameter 0) (color 0 0 0 0)
-  )
   (junction (at 44.45 33.02) (diameter 0.9144) (color 0 0 0 0)
   )
@@
   (no_connect (at 218.44 91.44))
   (no_connect (at 210.82 88.9))
-  (bus_entry (at -41.91 114.3) (size 2.54 2.54)
-    (stroke (width 0) (type default))
-  )
-  (bus_entry (at -40.64 111.76) (size 2.54 2.54)
-    (stroke (width 0) (type default))
-  )
   (wire (pts (xy 44.45 68.58) (xy 29.21 68.58))
     (stroke (width 0) (type default))
@@
     (stroke (width 0) (type default))
   )
-  (wire (pts (xy 218.44 107.95) (xy 228.6 107.95))
-    (stroke (width 0) (type default))
-  )
   (wire (pts (xy 76.2 25.4) (xy 82.55 25.4))
     (stroke (width 0) (type default))
@@
     (effects (font (size 1.27 1.27)) (justify right bottom))
   )
-  (label "DVSS" (at 210.82 107.95 180) (fields_autoplaced)
-    (effects (font (size 1.27 1.27)) (justify right bottom))
-  )
   (label "CSI_D8_pre" (at 246.38 121.92 180) (fields_autoplaced)
     (effects (font (size 1.27 1.27)) (justify right bottom))
@@
         )
       )
-    )
-  )
-  (symbol (lib_id "Device:R_US") (at 214.63 107.95 90) (unit 1)
-    (in_bom yes) (on_board yes) (dnp no)
-    (property "Reference" "R560" (at 219.71 106.68 90)
-      (effects (font (size 1.27 1.27)) (justify right))
-    )
-    (property "Value" "0" (at 217.17 106.68 90)
-      (effects (font (size 1.27 1.27)) (justify right))
-    )
-    (property "Footprint" "Resistor_SMD:R_0402_1005Metric" (at 214.884 106.934 90)
-      (effects (font (size 1.27 1.27)) hide)
-    )
-    (property "Datasheet" "~" (at 214.63 107.95 0)
-      (effects (font (size 1.27 1.27)) hide)
-    )
-    (pin "1")
-    (pin "2")
-    (instances
-      (project "pcb"
-        (path "/ba41827b-f176-424d-b6d5-0b0e1ddda097/bbc4a8ed-000d-45bd-b682-5f5fc521899f"
-          (reference "R560") (unit 1)
-        )
-      )

Commit message: Next set of PCB revisions WIP
Parts:
- R561, RN501, RN502, RN503, RN504: value 50 -> 49.9
