File: Hardware/sensorboard/ccd_driver.kicad_sch (KiCad schematic)
At the start: 80 parts, among them Q801 BC847BPN, U504 IRF9389/7309, U505 IRF9389/7309, U506 IRF9389/7309, U507 IRF9389/7309, U801 74HC4053, U802 74HC2G17, U803 74HC2G17, U804 74HC2G17, U805 74HC2G17, U806 74HC2G17, U807 74HC2G17, U808 CD4053B

Commit message: Power Board WIP
Parts:
- removed C504, C505, C506, C507, C508, C509, C510, C511: 1nF, Capacitor_SMD:C_0402_1005Metric, symbol Device:C
- removed C514, C515, C516, C517, C801, C802, C803, C804, C805, C806, C807, C809, C810, C811, C812, C813, C814, C815, C816, C817, C822: 100nF, Capacitor_SMD:C_0402_1005Metric, symbol Device:C
- removed C808: 1uF 25V, Capacitor_SMD:C_0603_1608Metric, symbol Device:C
- removed D501, D502, D503, D504: BAT54S, Package_TO_SOT_SMD:SOT-23, symbol Diode:BAT54S
- removed D801, D802: B0540W, Diode_SMD:D_SOD-323, symbol Device:D_Schottky
- removed Q801: BC847BPN, Package_TO_SOT_SMD:SOT-363_SC-70-6, symbol Transistor_BJT:BC847BPN
- removed R504, R505, R506, R507, R508, R509, R510, R511: 220, Resistor_SMD:R_0402_1005Metric, symbol Device:R
- removed R801, R802, R803, R808, R809, R810, R811: 22, Resistor_SMD:R_0402_1005Metric, symbol Device:R
- removed R804, R805, R807: 10K, Resistor_SMD:R_0402_1005Metric, symbol Device:R
- removed R806: 0, Resistor_SMD:R_0402_1005Metric, symbol Device:R
- removed R813, R814, R815, R816, R817, R818, R819, R820, R821, R822, R823, R824: 0.1, Resistor_SMD:R_0603_1608Metric, symbol Device:R
- removed U504, U505, U506, U507: IRF9389/7309, Package_SO:SOIC-8_3.9x4.9mm_P1.27mm, symbol symbols:IRF9389BF
- removed U801: 74HC4053, Package_SO:SSOP-16_4.4x5.2mm_P0.65mm, symbol 4xxx:4053
- removed U802, U803, U804, U805, U806, U807: 74HC2G17, Package_SO:SC-74-6_1.5x2.9mm_P0.95mm, symbol Sitina:74HC2G17
- removed U808: CD4053B, Package_SO:SSOP-16_4.4x5.2mm_P0.65mm, symbol 4xxx:4053
- added C557, C558, C559: 10uF, Capacitor_SMD:C_0402_1005Metric, symbol Device:C
- added C560, C561, C562, C563, C564, C565, C566, C568, C569, C570, C571, C572, C573: 100nF, Capacitor_SMD:C_0402_1005Metric, symbol Device:C
- added C567: 1uF 25V, Capacitor_SMD:C_0603_1608Metric, symbol Device:C
- added D504, D505: B0540W, Diode_SMD:D_SOD-323, symbol Device:D_Schottky
- added D? (x3): BAT54S, Package_TO_SOT_SMD:SOT-23, symbol Diode:BAT54S
- added Q501: BC847BPN, Package_TO_SOT_SMD:SOT-363_SC-70-6, symbol Transistor_BJT:BC847BPN
- added R518, R519, R521: 10K, Resistor_SMD:R_0402_1005Metric, symbol Device:R
- added R520: 0, Resistor_SMD:R_0402_1005Metric, symbol Device:R
- added R522, R523, R524, R525, R526, R527, R528, R529, R530, R531, R532, R533: 0.1, Resistor_SMD:R_0603_1608Metric, symbol Device:R_Small_US
- added RV501, RV502, RV503: 50K, Potentiometer_SMD:Potentiometer_Bourns_3214G_Horizontal, symbol Device:R_Potentiometer_Trim_US
- added U508, U509, U510, U511, U512, U513: 74HC2G17, Package_SO:SC-74-6_1.5x2.9mm_P0.95mm, symbol Sitina:74HC2G17
Connections:
- net +16V: now also C565.2, Q501.4 (E2), R518.1
- net +1V5: now also C558.2, C568.1, D?.2 (K), RV502.1, U508.5 (VCC)
- net +2V: now also C569.1, C570.1, C571.1, C572.1, C573.1, D?.2 (K), D?.2 (K), RV501.1, RV503.1, U509.5 (VCC), U510.5 (VCC), U511.5 (VCC), U512.5 (VCC), U513.5 (VCC)
- net +3V3: now also C559.2
- net -15V: now also C566.1, D504.2 (A), R520.2
- net -3V5: now also C557.1, C568.2, D?.1 (A), RV502.3, U508.2 (GND)
- net -4V: now also C569.2, C570.2, C571.2, C572.2, C573.2, D?.1 (A), D?.1 (A), RV501.3, RV503.3, U509.2 (GND), U510.2 (GND), U511.2 (GND), U512.2 (GND), U513.2 (GND)
- net AFE_H1: now also C561.1
- net AFE_H2: now also C562.1
- net AFE_RG: now also C560.1
- net AFE_STROBE: now also C563.2, C564.2
- net GND: now also C557.2, C558.1, C559.1, C565.1, C566.2, R519.2, R521.2
- net H1BINL: now also R524.1, U509.6 (1Y)
- net H1BINL_CCD: now also R524.2
- net H1BINR: now also R525.1, U509.4 (2Y)
- net H1BINR_CCD: now also R525.2
- net H1BL: now also R528.1, U511.6 (1Y)
- net H1BL_CCD: now also R528.2
- net H1BR: now also R531.1, U512.4 (2Y)
- net H1BR_CCD: now also R531.2
- net H1S: now also C561.2, D?.3 (COM), RV503.2, U509.1 (1A), U509.3 (2A), U511.1 (1A), U512.3 (2A), U513.1 (1A)
- net H1SL: now also R527.1, U510.4 (2Y)
- net H1SL_CCD: now also R527.2
- net H1SR: now also R532.1, U513.6 (1Y)
- net H1SR_CCD: now also R532.2
- net H2BL: now also R529.1, U511.4 (2Y)
- net H2BL_CCD: now also R529.2
- net H2BR: now also R530.1, U512.6 (1Y)
- net H2BR_CCD: now also R530.2
- net H2S: now also C562.2, D?.3 (COM), RV501.2, U510.1 (1A), U510.3 (2A), U511.3 (2A), U512.1 (1A), U513.3 (2A)
- net H2SL: now also R526.1, U510.6 (1Y)
- net H2SL_CCD: now also R526.2
- net H2SR: now also R533.1, U513.4 (2Y)
- net H2SR_CCD: now also R533.2
- net RGS: now also C560.2, D?.3 (COM), RV502.2, U508.1 (1A), U508.3 (2A)
- net RL: now also R522.1, U508.6 (1Y)
- net RL_CCD: now also R522.2
- net RR: now also R523.1, U508.4 (2Y)
- net RR_CCD: now also R523.2
- net VAB: now also D505.2 (A)
- net VSUB_CCD: now also C567.1, D505.1 (K), R521.1
- new net: C567.2, Q501.3 (C2), Q501.6 (C1)
- new net: C563.1, Q501.5 (B2), R518.2
- new net: C564.1, D504.1 (K), Q501.2 (B1), R519.1
- new net: Q501.1 (E1), R520.1
Other:
- note added: "Keep Length Short"
- company: Copyright 2023 Wenting Zhang -> Copyright 2023 Wenting Zhang, AL
- title: Sitina 1 Mainboard -> Sitina 1 CCD H Drivers

Commit message: Update sensor/power board outline
Other:
- note added: "HC only has 4mA drive. Load capacitance for B/S are ~500pF. LVC has 32mA drive, but only up to 5.5V."
- note removed: "HC only has 4mA drive. Load capacitance for B/S are ~500pF. Consider using LVC with 32mA drive instead?"
Changed lines of the file:
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@@
     (effects (font (size 1.27 1.27)) (justify left bottom))
   )
-  (text "HC only has 4mA drive. Load capacitance for B/S are ~500pF.\nConsider using LVC with 32mA drive instead?"
+  (text "HC only has 4mA drive. Load capacitance for B/S are ~500pF.\nLVC has 32mA drive, but only up to 5.5V."
     (at 71.12 118.11 0)
     (effects (font (size 1.27 1.27)) (justify left bottom))

Commit message: CCD Sensor Board WIP
Parts:
- removed C557, C558, C559: 10uF, Capacitor_SMD:C_0402_1005Metric, symbol Device:C
- removed C570, C571, C572, C573: 100nF, Capacitor_SMD:C_0402_1005Metric, symbol Device:C
- added C611, C612, C613, C614, C615, C616, C617, C618, C619, C620: 100nF, Capacitor_SMD:C_0402_1005Metric, symbol Device:C
Connections:
- net +2V: now also C612.1, C613.1, C615.1, C617.1, C619.1; no longer C569.1
- net -3V5: now also C611.2; no longer C568.2
- net -4V: now also C614.2, C616.2, C618.2, C620.2
- net GND: now also C568.2, C569.1, C611.1, C612.2, C613.2, C614.1, C615.2, C616.1, C617.2, C618.1, C619.2, C620.1
- net H1BINL: now also U509.4 (2Y); no longer U509.6 (1Y)
- net H1BINR: now also U509.6 (1Y); no longer U509.4 (2Y)
- net H1BL: now also U511.4 (2Y); no longer U511.6 (1Y)
- net H1BR: now also U512.6 (1Y); no longer U512.4 (2Y)
- net H1S: now also U510.1 (1A), U511.3 (2A), U512.1 (1A), U513.3 (2A); no longer U511.1 (1A), U512.3 (2A), U513.1 (1A)
- net H1SL: now also U510.6 (1Y); no longer U510.4 (2Y)
- net H1SR: now also U513.4 (2Y); no longer U513.6 (1Y)
- net H2BL: now also U511.6 (1Y); no longer U511.4 (2Y)
- net H2BR: now also U512.4 (2Y); no longer U512.6 (1Y)
- net H2S: now also U511.1 (1A), U512.3 (2A), U513.1 (1A); no longer U510.1 (1A), U511.3 (2A), U512.1 (1A), U513.3 (2A)
- net H2SL: now also U510.4 (2Y); no longer U510.6 (1Y)
- net H2SR: now also U513.6 (1Y); no longer U513.4 (2Y)
- net RL: now also U508.4 (2Y); no longer U508.6 (1Y)
- net RR: now also U508.6 (1Y); no longer U508.4 (2Y)
- net +16V renamed +16VD
- no-connect marks 0 -> 4
Other:
- moved on the sheet: C568, R522, R523, R524, R525, R526, R527, R528, R529, R530, R531, R532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

Commit message: Sensor Board WIP, minor
Parts:
- added C538: 100nF, Capacitor_SMD:C_0402_1005Metric, symbol Device:C
- added C539: DNP/1nF, Capacitor_SMD:C_0402_1005Metric, symbol Device:C
- added R?: 82K 1%, Resistor_SMD:R_0402_1005Metric, symbol Device:R_US
- added RV508: 10K, Potentiometer_SMD:Potentiometer_Bourns_3214G_Horizontal, symbol Device:R_Potentiometer_Trim_US
- added RV509: 50K, Potentiometer_SMD:Potentiometer_Bourns_3214G_Horizontal, symbol Device:R_Potentiometer_Trim_US
- added U522: TLV76701DRVx, Package_SON:WSON-6-1EP_2x2mm_P0.65mm_EP1x1.6mm_ThermalVias, symbol Regulator_Linear:TLV76701DRVx
- added U523: TPS72301, Package_TO_SOT_SMD:SOT-23-5_HandSoldering, symbol symbols:TPS723xx
- added U524: XC6206P152MR, Package_TO_SOT_SMD:SOT-23-3, symbol Regulator_Linear:XC6206PxxxMR
Connections:
- net +16VD: now also U522.4 (EN), U522.6 (IN)
- net +1V5: now also U524.2 (VO)
- net +2V: now also U524.3 (VI)
- net -3V5: now also RV509.1, U523.5 (OUT)
- net -4V: now also U523.2 (IN), U523.3 (EN)
- net GND: now also C538.1, RV508.3, RV509.3, U522.3 (GND), U522.5 (GND), U522.7 (PAD), U523.1 (GND), U524.1 (GND)
- net VAB: now also C538.2, C539.2, R?.1, U522.1 (OUT)
- new net: R?.2, RV508.1
- new net: C539.1, RV508.2, U522.2 (FB)
- new net: RV509.2, U523.4 (NR/FB)

Commit message: Sensor Board Routing Done
Parts:
- removed RV509: 50K, Potentiometer_SMD:Potentiometer_Bourns_3214G_Horizontal, symbol Device:R_Potentiometer_Trim_US
- added R? (x3): 10K, Resistor_SMD:R_0402_1005Metric, symbol Device:R_US
- added R?: 0, Resistor_SMD:R_0402_1005Metric, symbol Device:R_US
Connections:
- net -3V5: now also R?.1
- net -4V: now also R?.1; no longer U523.3 (EN)
- net GND: now also R?.2
- net at U523.4 (NR/FB): now also R?.1, R?.2
- new net: R?.1, R?.2
- new net: R?.2, U523.3 (EN)
Other:
- note added: "FB:-1.186V"

Commit message: Uploading Sensorboard Production Files
Parts:
- added C501, C531: 220uF / 6V, Capacitor_Tantalum_SMD:CP_EIA-3528-15_AVX-H, symbol Device:C_Polarized_US
Connections:
- net +2V: now also C531.1
- net -4V: now also C501.2
- net GND: now also C501.1, C531.2
Changed lines of the file:
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@@
+    )
+  )
+  (symbol (lib_id "Sitina:-4V") (at 45.72 43.18 180) (unit 1)
+    (in_bom yes) (on_board yes) (dnp no)
+    (property "Reference" "#PWR0616" (at 45.72 39.37 0)
+      (effects (font (size 1.27 1.27)) hide)
+    )
+    (property "Value" "-4V" (at 45.339 47.5742 0)
+      (effects (font (size 1.27 1.27)))
+    )
+    (property "Footprint" "" (at 45.72 43.18 0)
+      (effects (font (size 1.27 1.27)) hide)
+    )
+    (property "Datasheet" "" (at 45.72 43.18 0)
+      (effects (font (size 1.27 1.27)) hide)
+    )
+    (pin "1")
+    (instances
+      (project "pcb"
+        (path "/ba41827b-f176-424d-b6d5-0b0e1ddda097/568a197d-3d07-4ce3-9dad-204d21f52839"
+          (reference "#PWR0616") (unit 1)
+        )
+      )
     )
   )
@@
     )
   )
+  (symbol (lib_id "Device:C_Polarized_US") (at 45.72 39.37 0) (unit 1)
+    (in_bom yes) (on_board yes) (dnp no) (fields_autoplaced)
+    (property "Reference" "C501" (at 49.53 37.465 0)
+      (effects (font (size 1.27 1.27)) (justify left))
+    )
+    (property "Value" "220uF / 6V" (at 49.53 40.005 0)
+      (effects (font (size 1.27 1.27)) (justify left))
+    )
+    (property "Footprint" "Capacitor_Tantalum_SMD:CP_EIA-3528-15_AVX-H" (at 45.72 39.37 0)
+      (effects (font (size 1.27 1.27)) hide)
+    )
+    (property "Datasheet" "~" (at 45.72 39.37 0)
+      (effects (font (size 1.27 1.27)) hide)
+    )
+    (pin "1")
+    (pin "2")
+    (instances
+      (project "pcb"
+        (path "/ba41827b-f176-424d-b6d5-0b0e1ddda097/568a197d-3d07-4ce3-9dad-204d21f52839"
+          (reference "C501") (unit 1)
+        )
+      )
+    )
+  )
   (symbol (lib_id "Device:C") (at 237.49 121.92 0) (mirror y) (unit 1)
     (in_bom yes) (on_board yes) (dnp no)
@@
         (path "/ba41827b-f176-424d-b6d5-0b0e1ddda097/568a197d-3d07-4ce3-9dad-204d21f52839"
           (reference "#PWR0634") (unit 1)
+        )
+      )
+    )
+  )
+  (symbol (lib_id "power:GND") (at 45.72 35.56 180) (unit 1)
+    (in_bom yes) (on_board yes) (dnp no)
+    (property "Reference" "#PWR0654" (at 45.72 29.21 0)
+      (effects (font (size 1.27 1.27)) hide)
+    )
+    (property "Value" "GND" (at 45.593 31.1658 0)
+      (effects (font (size 1.27 1.27)))
+    )
+    (property "Footprint" "" (at 45.72 35.56 0)
+      (effects (font (size 1.27 1.27)) hide)
+    )
+    (property "Datasheet" "" (at 45.72 35.56 0)
+      (effects (font (size 1.27 1.27)) hide)
+    )
+    (pin "1")
+    (instances
+      (project "pcb"
+        (path "/ba41827b-f176-424d-b6d5-0b0e1ddda097/568a197d-3d07-4ce3-9dad-204d21f52839"
+          (reference "#PWR0654") (unit 1)
         )
       )
@@
         (path "/ba41827b-f176-424d-b6d5-0b0e1ddda097/568a197d-3d07-4ce3-9dad-204d21f52839"
           (reference "#PWR0643") (unit 1)
+        )
+      )
+    )
+  )
+  (symbol (lib_id "Sitina:+2V") (at 25.4 35.56 0) (unit 1)
+    (in_bom yes) (on_board yes) (dnp no)
+    (property "Reference" "#PWR0656" (at 25.4 39.37 0)
+      (effects (font (size 1.27 1.27)) hide)
+    )
+    (property "Value" "+2V" (at 25.781 31.1658 0)
+      (effects (font (size 1.27 1.27)))
+    )
+    (property "Footprint" "" (at 25.4 35.56 0)
+      (effects (font (size 1.27 1.27)) hide)
+    )
+    (property "Datasheet" "" (at 25.4 35.56 0)
+      (effects (font (size 1.27 1.27)) hide)
+    )
+    (pin "1")
+    (instances
+      (project "pcb"
+        (path "/ba41827b-f176-424d-b6d5-0b0e1ddda097/568a197d-3d07-4ce3-9dad-204d21f52839"
+          (reference "#PWR0656") (unit 1)
         )
       )
@@
     )
   )
+  (symbol (lib_id "power:GND") (at 25.4 43.18 0) (unit 1)
+    (in_bom yes) (on_board yes) (dnp no)
+    (property "Reference" "#PWR0655" (at 25.4 49.53 0)
+      (effects (font (size 1.27 1.27)) hide)
+    )
+    (property "Value" "GND" (at 25.527 47.5742 0)
+      (effects (font (size 1.27 1.27)))
+    )
+    (property "Footprint" "" (at 25.4 43.18 0)
+      (effects (font (size 1.27 1.27)) hide)
+    )
+    (property "Datasheet" "" (at 25.4 43.18 0)
+      (effects (font (size 1.27 1.27)) hide)
+    )
+    (pin "1")
+    (instances
+      (project "pcb"
+        (path "/ba41827b-f176-424d-b6d5-0b0e1ddda097/568a197d-3d07-4ce3-9dad-204d21f52839"
+          (reference "#PWR0655") (unit 1)
+        )
+      )
+    )
+  )
   (symbol (lib_id "power:+1V5") (at 184.15 20.32 0) (unit 1)
     (in_bom yes) (on_board yes) (dnp no) (fields_autoplaced)
@@
         )
       )
+    )
+  )
+  (symbol (lib_id "Device:C_Polarized_US") (at 25.4 39.37 0) (unit 1)
+    (in_bom yes) (on_board yes) (dnp no) (fields_autoplaced)
+    (property "Reference" "C531" (at 29.21 37.465 0)
+      (effects (font (size 1.27 1.27)) (justify left))
+    )
+    (property "Value" "220uF / 6V" (at 29.21 40.005 0)
+      (effects (font (size 1.27 1.27)) (justify left))
+    )
+    (property "Footprint" "Capacitor_Tantalum_SMD:CP_EIA-3528-15_AVX-H" (at 25.4 39.37 0)
+      (effects (font (size 1.27 1.27)) hide)
+    )
+    (property "Datasheet" "~" (at 25.4 39.37 0)
+      (effects (font (size 1.27 1.27)) hide)
+    )
+    (pin "1")
+    (pin "2")
+    (instances
+      (project "pcb"
+        (path "/ba41827b-f176-424d-b6d5-0b0e1ddda097/568a197d-3d07-4ce3-9dad-204d21f52839"
+          (reference "C531") (unit 1)
+        )
+      )

Commit message: Next set of PCB revisions WIP
Parts:
- removed R?: 10K, Resistor_SMD:R_0402_1005Metric, symbol Device:R_US
- R565: renamed from R?; value 10K -> 20K
- RV501, RV502, RV503, RV508: footprint Potentiometer_SMD:Potentiometer_Bourns_3214G_Horizontal -> Potentiometer_SMD:Potentiometer_Bourns_TC33X_Vertical
- gave numbers to parts that had none: 6
Connections:
- net at R564.1, U523.4 (NR/FB): now also R565.2
- net VAB renamed +VAB
Other:
- moved on the sheet: R564

Commit message: Design grip flex, SB/IOB WIP
Parts:
- renumbered C531 to C53, C501 to C54, C539 to C55, C538 to C56, C560 to C57, C561 to C58, C562 to C59, C563 to C60, C564 to C61, C565 to C62, C566 to C63, C567 to C64, C568 to C65, C612 to C66, C613 to C67, C615 to C68, C617 to C69, C619 to C70, C569 to C71, C614 to C72, C616 to C73, C618 to C74, C620 to C75, C611 to C76, D501 to D11, D502 to D12, D503 to D13, D504 to D14, D505 to D15, Q501 to Q1, R563 to R53, R565 to R54, R564 to R55, R562 to R56, R518 to R57, R519 to R58, R520 to R59, R521 to R60, R523 to R61, R522 to R62, R525 to R63, R524 to R64, R527 to R65, R526 to R66, R529 to R67, R528 to R68, R531 to R69, R530 to R70, R533 to R71, R532 to R72, RV508 to RV1, RV501 to RV2, RV502 to RV3, RV503 to RV4, U523 to U11, U524 to U12, U522 to U13, U508 to U14, U509 to U15, U510 to U16, U511 to U17, U512 to U18, U513 to U19
