File: Hardware/sensorboard/fpga_ddr.kicad_sch (KiCad schematic)
At the start: 29 parts, among them U527 XC7Z010-CLG400, U530 MT41K256M16HA

Commit message: Design grip flex, SB/IOB WIP
Parts:
- renumbered C638 to C134, C639 to C135, C640 to C136, C643 to C137, C644 to C138, C646 to C139, C647 to C140, C642 to C141, C648 to C142, C651 to C143, C652 to C144, C653 to C145, C656 to C146, C657 to C147, C658 to C148, C661 to C149, C662 to C150, C663 to C151, C666 to C152, C667 to C153, C668 to C154, R591 to R106, R588 to R107, R587 to R108, R593 to R109, R594 to R110, R589 to R111, U527 to U27, U530 to U29

Commit message: Hardware r0.9
Parts:
- C134, C137, C139, C140, C143, C144, C146, C147, C150: value 220nF -> 470nF
- C148, C152: value 4.7uF -> 10uF
- R107, R108: value 80R -> 82R
Other:
- company: (none) -> Copyright 2024 Wenting Zhang
- title: (none) -> Sitina 1 Sensor Board
Changed lines of the file:
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@@
 	(generator_version "8.0")
 	(paper "A4")
+	(title_block
+		(title "Sitina 1 Sensor Board")
+		(date "2024-03-25")
+		(rev "R0.9")
+		(company "Copyright 2024 Wenting Zhang")
+	)
 	(junction
 		(at 114.3 162.56)
@@
 			)
 		)
-		(property "Value" "220nF"
+		(property "Value" "470nF"
 			(at 74.041 96.393 0)
 			(effects
@@
 			)
 		)
-		(property "Value" "4.7uF"
+		(property "Value" "10uF"
 			(at 107.061 172.593 0)
 			(effects
@@
 			)
 		)
-		(property "Value" "220nF"
+		(property "Value" "470nF"
 			(at 53.721 119.253 0)
 			(effects
@@
 			)
 		)
-		(property "Value" "220nF"
+		(property "Value" "470nF"
 			(at 53.721 96.393 0)
 			(effects
@@
 			)
 		)
-		(property "Value" "80R"
+		(property "Value" "82R"
 			(at 59.69 64.77 90)
 			(effects
@@
 			)
 		)
-		(property "Value" "220nF"
+		(property "Value" "470nF"
 			(at 84.201 119.253 0)
 			(effects
@@
 			)
 		)
-		(property "Value" "220nF"
+		(property "Value" "470nF"
 			(at 63.881 119.253 0)
 			(effects
@@
 			)
 		)
-		(property "Value" "220nF"
+		(property "Value" "470nF"
 			(at 33.401 96.393 0)
 			(effects
@@
 			)
 		)
-		(property "Value" "220nF"
+		(property "Value" "470nF"
 			(at 74.041 119.253 0)
 			(effects
@@
 			)
 		)
-		(property "Value" "220nF"
+		(property "Value" "470nF"
 			(at 43.561 96.393 0)
 			(effects
@@
 			)
 		)
-		(property "Value" "220nF"
+		(property "Value" "470nF"
 			(at 63.881 96.393 0)
 			(effects
@@
 			)
 		)
-		(property "Value" "80R"
+		(property "Value" "82R"
 			(at 62.23 64.77 90)
 			(effects
@@
 			)
 		)
-		(property "Value" "4.7uF"
+		(property "Value" "10uF"
 			(at 74.041 159.893 0)
 			(effects
