File: Hardware/sensorboard/fpga_io.kicad_sch (KiCad schematic)
At the start: 11 parts, among them U527 XC7Z010-CLG400

Commit message: Design grip flex, SB/IOB WIP
Parts:
- renumbered C669 to C155, C670 to C156, C671 to C157, C672 to C158, C673 to C159, C674 to C160, C675 to C161, C676 to C162, C677 to C163, R590 to R112, U527 to U27
Connections:
- net DSI_LP_D1P: now reaches U27.T14 (IO_L5P_T0_34)
- net DSI_LP_D1N: now reaches U27.T15 (IO_L5N_T0_34)
- net DSI_HS_D1N: now reaches U27.V16 (IO_L18P_T2_34)
- net DSI_HS_D1P: now reaches U27.W16 (IO_L18N_T2_34)
- net I2C1_SCL: now reaches U27.C10 (PS_MIO52_501)
- net I2C1_SDA: now reaches U27.C11 (PS_MIO53_501)
- no-connect marks 15 -> 13

Commit message: Sensorboard r0p9 routing done
Parts:
- added D22: LED, LED_SMD:LED_0603_1608Metric, symbol Device:LED
- added R56: 1K, Resistor_SMD:R_0402_1005Metric, symbol Device:R
Connections:
- net AFE_RST: now also U27.Y19 (IO_L17N_T2_34); no longer U27.B20 (IO_L1N_T0_AD0N_35)
- net AFE_SCK: now also U27.W16 (IO_L18N_T2_34); no longer U27.D18 (IO_L3N_T0_DQS_AD1N_35)
- net AFE_SDATA: now also U27.Y17 (IO_L7N_T1_34); no longer U27.C20 (IO_L1P_T0_AD0P_35)
- net AFE_SL: now also U27.Y18 (IO_L17P_T2_34); no longer U27.D19 (IO_L4P_T0_35)
- net AFE_SYNC: now also U27.T11 (IO_L1P_T0_34); no longer U27.B19 (IO_L2P_T0_AD8P_35)
- net CSI_D10: now also U27.V17 (IO_L21P_T3_DQS_34); no longer U27.F20 (IO_L15N_T2_DQS_AD12N_35)
- net CSI_D11: now also U27.W13 (IO_L4N_T0_34); no longer U27.E19 (IO_L5N_T0_AD9N_35)
- net CSI_D12: now also U27.U12 (IO_L2N_T0_34); no longer U27.E18 (IO_L5P_T0_AD9P_35)
- net CSI_D13: now also U27.U18 (IO_L12P_T1_MRCC_34); no longer U27.D20 (IO_L4N_T0_35)
- net CSI_D2: now also U27.V16 (IO_L18P_T2_34); no longer U27.K19 (IO_L10P_T1_AD11P_35)
- net CSI_D3: now also U27.U17 (IO_L9N_T1_DQS_34); no longer U27.J19 (IO_L10N_T1_AD11N_35)
- net CSI_D4: now also U27.V12 (IO_L4P_T0_34); no longer U27.J20 (IO_L17P_T2_AD5P_35)
- net CSI_D5: now also U27.T16 (IO_L9P_T1_DQS_34); no longer U27.H18 (IO_L14N_T2_AD4N_SRCC_35)
- net CSI_D6: now also U27.T12 (IO_L2P_T0_34); no longer U27.H20 (IO_L17N_T2_AD5N_35)
- net CSI_D7: now also U27.T10 (IO_L1N_T0_34); no longer U27.G19 (IO_L18P_T2_AD13P_35)
- net CSI_D8: now also U27.V13 (IO_L3N_T0_DQS_34); no longer U27.G20 (IO_L18N_T2_AD13N_35)
- net CSI_D9: now also U27.W18 (IO_L22P_T3_34); no longer U27.F19 (IO_L15P_T2_DQS_AD12P_35)
- net CSI_HSYNC: now also U27.Y16 (IO_L7P_T1_34); no longer U27.M19 (IO_L7P_T1_AD2P_35)
- net CSI_PIXCLK: now also U27.U14 (IO_L11P_T1_SRCC_34); no longer U27.M18 (IO_L8N_T1_AD10N_35)
- net CSI_VSYNC: now also U27.W15 (IO_L10N_T1_34); no longer U27.M20 (IO_L7N_T1_AD2N_35)
- net DSI_HS_CKN: now also U27.W20 (IO_L16N_T2_34); no longer U27.U20 (IO_L15N_T2_DQS_34)
- net DSI_HS_CKP: now also U27.V20 (IO_L16P_T2_34); no longer U27.T20 (IO_L15P_T2_DQS_34)
- net DSI_HS_D0N: now also U27.U20 (IO_L15N_T2_DQS_34); no longer U27.Y18 (IO_L17P_T2_34)
- net DSI_HS_D0P: now also U27.T20 (IO_L15P_T2_DQS_34); no longer U27.Y19 (IO_L17N_T2_34)
- net DSI_HS_D1N: now also U27.P20 (IO_L14N_T2_SRCC_34); no longer U27.V16 (IO_L18P_T2_34)
- net DSI_HS_D1P: now also U27.N20 (IO_L14P_T2_SRCC_34); no longer U27.W16 (IO_L18N_T2_34)
- net DSI_LP_CKN: now also U27.W19 (IO_L22N_T3_34); no longer U27.V20 (IO_L16P_T2_34)
- net DSI_LP_CKP: now also U27.U19 (IO_L12N_T1_MRCC_34); no longer U27.R18 (IO_L20N_T3_34)
- net DSI_LP_D0N: now also U27.T19 (IO_25_34); no longer U27.Y17 (IO_L7N_T1_34)
- net DSI_LP_D0P: now also U27.R19 (IO_0_34); no longer U27.W19 (IO_L22N_T3_34)
- net DSI_LP_D1N: now also U27.P19 (IO_L13N_T2_MRCC_34); no longer U27.T15 (IO_L5N_T0_34)
- net DSI_LP_D1P: now also U27.N18 (IO_L13P_T2_MRCC_34); no longer U27.T14 (IO_L5P_T0_34)
- net GND: now also D22.1 (K)
- net TCON_RG: now reaches U27.H17 (IO_L13N_T2_MRCC_35)
- net TCON_H2: now reaches U27.L16 (IO_L11P_T1_SRCC_35)
- net TCON_H1: now reaches U27.L17 (IO_L11N_T1_SRCC_35)
- net TCON_STROBE: now reaches U27.M15 (IO_L23N_T3_35)
- net CSI_D14: now reaches U27.V18 (IO_L21N_T3_DQS_34)
- net CSI_D15: now reaches U27.Y14 (IO_L8N_T1_34)
- net LED: now reaches U27.A15 (PS_MIO26_501)
- net LED: now also R56.1
- net CSI_D0 renamed TCON_FDG
- net CSI_D1: no longer names the net of U27.L20 (IO_L9N_T1_DQS_AD3N_35)
- net EXT_SYNC renamed TCON_V23
- net LAN_RESET: no longer names the net of U27.D16 (PS_MIO46_501)
- new net: D22.2 (A), R56.2
- new net TCON_V1: U27.M18 (IO_L8N_T1_AD10N_35)
- new net TCON_V2: U27.C20 (IO_L1P_T0_AD0P_35)
- new net VAB_PWM: U27.B19 (IO_L2P_T0_AD8P_35)

Commit message: Hardware r0.9
Parts:
- C157, C160, C163: value 4.7uF -> 10uF
Other:
- company: (none) -> Copyright 2024 Wenting Zhang
- title: (none) -> Sitina 1 Sensor Board
Changed lines of the file:
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@@
 	(generator_version "8.0")
 	(paper "A4")
+	(title_block
+		(title "Sitina 1 Sensor Board")
+		(date "2024-03-25")
+		(rev "R0.9")
+		(company "Copyright 2024 Wenting Zhang")
+	)
 	(junction
 		(at 175.26 170.18)
@@
 			)
 		)
-		(property "Value" "4.7uF"
+		(property "Value" "10uF"
 			(at 78.74 171.45 90)
 			(effects
@@
 			)
 		)
-		(property "Value" "4.7uF"
+		(property "Value" "10uF"
 			(at 165.1 171.45 90)
 			(effects
@@
 			)
 		)
-		(property "Value" "4.7uF"
+		(property "Value" "10uF"
 			(at 265.43 146.05 90)
 			(effects
