File: Hardware/sensorboard/fpga_power.kicad_sch (KiCad schematic)
At the start: 25 parts, among them U27 XC7Z010-CLG400, U32 SY8120

Commit message: Sensorboard r0p9 routing done
Parts:
- added C115, C116, C117, C119, C125, C126, C127: 470nF, Capacitor_SMD:C_0402_1005Metric, symbol Device:C
- added C121, C122, C128, C129, C130: 4.7uF, Capacitor_SMD:C_0603_1608Metric, symbol Device:C
- added C123, C124, C131, C132, C133: 100uF, Capacitor_SMD:C_0805_2012Metric, symbol Device:C
- C164, C165, C166, C167, C168, C169, C170, C171: footprint Capacitor_SMD:C_0805_2012Metric -> Capacitor_SMD:C_0603_1608Metric
- U30, U31: value ~ -> SYR838
Connections:
- net +1V0_PL: now also C116.1, C119.1, C122.1, C124.1, C125.1, C128.1, C131.1
- net +1V0_PS: now also C115.1, C117.1, C121.1, C123.1
- net +1V8: now also C126.1, C127.1, C129.1, C130.1, C132.1, C133.1
- net GND: now also C115.2, C116.2, C117.2, C119.2, C121.2, C122.2, C123.2, C124.2, C125.2, C126.2, C127.2, C128.2, C129.2, C130.2, C131.2, C132.2, C133.2
- net I2C0_SCL: now also U31.B1 (SCL); no longer U30.B1 (SCL)
- net I2C0_SDA: now also U31.A3 (SDA); no longer U30.A3 (SDA)
- net I2C1_SCL: now also U30.B1 (SCL); no longer U31.B1 (SCL)
- net I2C1_SDA: now also U30.A3 (SDA); no longer U31.A3 (SDA)
Other:
- note added: "VCCAUX"
- note added: "VCCBRAM"
- note added: "VCCINT"
- note added: "VCCPAUX"
- note added: "VCCPINT"
- moved on the sheet: C113, C114, FB11, U27H

Commit message: Revise board design to fit enclosure
Parts:
- added C184, C185: 47uF, Capacitor_SMD:C_0603_1608Metric, symbol Device:C
- C132, C133: value 100uF -> 47uF; footprint Capacitor_SMD:C_0805_2012Metric -> Capacitor_SMD:C_0603_1608Metric
Connections:
- net +1V8: now also C184.1, C185.1
- net GND: now also C184.2, C185.2
Changed lines of the file:
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@@
 	)
 	(junction
+		(at 248.92 124.46)
+		(diameter 0)
+		(color 0 0 0 0)
+	)
+	(junction
 		(at 147.32 96.52)
 		(diameter 0)
@@
 	)
 	(junction
+		(at 248.92 144.78)
+		(diameter 0)
+		(color 0 0 0 0)
+	)
+	(junction
 		(at 220.98 78.74)
 		(diameter 0)
@@
 	)
 	(junction
+		(at 248.92 116.84)
+		(diameter 0)
+		(color 0 0 0 0)
+	)
+	(junction
 		(at 81.28 96.52)
 		(diameter 0)
@@
 	)
 	(junction
+		(at 248.92 137.16)
+		(diameter 0)
+		(color 0 0 0 0)
+	)
+	(junction
 		(at 205.74 137.16)
 		(diameter 0)
@@
 	(wire
 		(pts
+			(xy 248.92 124.46) (xy 259.08 124.46)
+		)
+		(stroke
+			(width 0)
+			(type default)
+		)
+	)
+	(wire
+		(pts
 			(xy 81.28 96.52) (xy 96.52 96.52)
 		)
@@
 	(wire
 		(pts
+			(xy 248.92 144.78) (xy 259.08 144.78)
+		)
+		(stroke
+			(width 0)
+			(type default)
+		)
+	)
+	(wire
+		(pts
 			(xy 137.16 60.96) (xy 147.32 60.96)
 		)
@@
 	(wire
 		(pts
+			(xy 248.92 137.16) (xy 259.08 137.16)
+		)
+		(stroke
+			(width 0)
+			(type default)
+		)
+	)
+	(wire
+		(pts
 			(xy 71.12 96.52) (xy 81.28 96.52)
 		)
@@
 	(wire
 		(pts
+			(xy 248.92 116.84) (xy 259.08 116.84)
+		)
+		(stroke
+			(width 0)
+			(type default)
+		)
+	)
+	(wire
+		(pts
 			(xy 137.16 96.52) (xy 147.32 96.52)
 		)
@@
 	)
 	(symbol
+		(lib_id "Device:C")
+		(at 259.08 120.65 0)
+		(unit 1)
+		(exclude_from_sim no)
+		(in_bom yes)
+		(on_board yes)
+		(dnp no)
+		(property "Reference" "C184"
+			(at 262.001 119.4816 0)
+			(effects
+				(font
+					(size 1.27 1.27)
+				)
+				(justify left)
+			)
+		)
+		(property "Value" "47uF"
+			(at 262.001 121.793 0)
+			(effects
+				(font
+					(size 1.27 1.27)
+				)
+				(justify left)
+			)
+		)
+		(property "Footprint" "Capacitor_SMD:C_0603_1608Metric"
+			(at 260.0452 124.46 0)
+			(effects
+				(font
+					(size 1.27 1.27)
+				)
+				(hide yes)
+			)
+		)
+		(property "Datasheet" "~"
+			(at 259.08 120.65 0)
+			(effects
+				(font
+					(size 1.27 1.27)
+				)
+				(hide yes)
+			)
+		)
+		(property "Description" ""
+			(at 259.08 120.65 0)
+			(effects
+				(font
+					(size 1.27 1.27)
+				)
+				(hide yes)
+			)
+		)
+		(pin "1"
+		)
+		(pin "2"
+		)
+		(instances
+			(project "pcb"
+				(path "/ba41827b-f176-424d-b6d5-0b0e1ddda097/6bd93fa5-b04c-403a-8268-88485f724a4c"
+					(reference "C184")
+					(unit 1)
+				)
+			)
+		)
+	)
+	(symbol
 		(lib_id "power:+1V0")
 		(at 228.6 96.52 0)
@@
 			)
 		)
-		(property "Value" "100uF"
+		(property "Value" "47uF"
 			(at 251.841 142.113 0)
 			(effects
@@
 			)
 		)
-		(property "Footprint" "Capacitor_SMD:C_0805_2012Metric"
+		(property "Footprint" "Capacitor_SMD:C_0603_1608Metric"
 			(at 249.8852 144.78 0)
 			(effects
@@
 	)
 	(symbol
+		(lib_id "Device:C")
+		(at 248.92 120.65 0)
+		(unit 1)
+		(exclude_from_sim no)
+		(in_bom yes)
+		(on_board yes)
+		(dnp no)
+		(property "Reference" "C132"
+			(at 251.841 119.4816 0)
+			(effects
+				(font
+					(size 1.27 1.27)
+				)
+				(justify left)
+			)
+		)
+		(property "Value" "47uF"
+			(at 251.841 121.793 0)
+			(effects
+				(font
+					(size 1.27 1.27)
+				)
+				(justify left)
+			)
+		)
+		(property "Footprint" "Capacitor_SMD:C_0603_1608Metric"
+			(at 249.8852 124.46 0)
+			(effects
+				(font
+					(size 1.27 1.27)
+				)
+				(hide yes)
+			)
+		)
+		(property "Datasheet" "~"
+			(at 248.92 120.65 0)
+			(effects
+				(font
+					(size 1.27 1.27)
+				)
+				(hide yes)
+			)
+		)
+		(property "Description" ""
+			(at 248.92 120.65 0)
+			(effects
+				(font
+					(size 1.27 1.27)
+				)
+				(hide yes)
+			)
+		)
+		(pin "1"
+		)
+		(pin "2"
+		)
+		(instances
+			(project "pcb"
+				(path "/ba41827b-f176-424d-b6d5-0b0e1ddda097/6bd93fa5-b04c-403a-8268-88485f724a4c"
+					(reference "C132")
+					(unit 1)
+				)
+			)
+		)
+	)
+	(symbol
 		(lib_id "power:GND")
 		(at 223.52 60.96 90)
@@
 	(symbol
 		(lib_id "Device:C")
-		(at 248.92 120.65 0)
+		(at 259.08 140.97 0)
 		(unit 1)
 		(exclude_from_sim no)
@@
 		(on_board yes)
 		(dnp no)
-		(property "Reference" "C132"
-			(at 251.841 119.4816 0)
+		(property "Reference" "C185"
+			(at 262.001 139.8016 0)
 			(effects
 				(font
@@
 			)
 		)
-		(property "Value" "100uF"
-			(at 251.841 121.793 0)
+		(property "Value" "47uF"
+			(at 262.001 142.113 0)
 			(effects
 				(font
@@
 			)
 		)
-		(property "Footprint" "Capacitor_SMD:C_0805_2012Metric"
-			(at 249.8852 124.46 0)
+		(property "Footprint" "Capacitor_SMD:C_0603_1608Metric"
+			(at 260.0452 144.78 0)
 			(effects
 				(font
@@
 		)
 		(property "Datasheet" "~"
-			(at 248.92 120.65 0)
+			(at 259.08 140.97 0)
 			(effects
 				(font
@@
 		)
 		(property "Description" ""
-			(at 248.92 120.65 0)
+			(at 259.08 140.97 0)
 			(effects
 				(font
@@
 			(project "pcb"
 				(path "/ba41827b-f176-424d-b6d5-0b0e1ddda097/6bd93fa5-b04c-403a-8268-88485f724a4c"
-					(reference "C132")
+					(reference "C185")
 					(unit 1)
 				)

Commit message: Hardware r0.9
Parts:
- C121, C122, C128, C129, C130: value 4.7uF -> 10uF
- FB11: footprint Resistor_SMD:R_0402_1005Metric -> Inductor_SMD:L_0402_1005Metric
Other:
- company: Copyright 2023 Wenting Zhang -> Copyright 2024 Wenting Zhang
- title: Sitina 1 Mainboard -> Sitina 1 Sensor Board
Changed lines of the file:
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@@
 	(paper "A4")
 	(title_block
-		(title "Sitina 1 Mainboard")
-		(date "2023-03-16")
-		(rev "R0.6")
-		(company "Copyright 2023 Wenting Zhang")
+		(title "Sitina 1 Sensor Board")
+		(date "2024-03-25")
+		(rev "R0.9")
+		(company "Copyright 2024 Wenting Zhang")
 	)
 	(junction
@@
 			)
 		)
-		(property "Value" "4.7uF"
+		(property "Value" "10uF"
 			(at 241.681 101.473 0)
 			(effects
@@
 			)
 		)
-		(property "Footprint" "Resistor_SMD:R_0402_1005Metric"
+		(property "Footprint" "Inductor_SMD:L_0402_1005Metric"
 			(at 238.76 77.978 90)
 			(effects
@@
 			)
 		)
-		(property "Value" "4.7uF"
+		(property "Value" "10uF"
 			(at 208.661 142.113 0)
 			(effects
@@
 			)
 		)
-		(property "Value" "4.7uF"
+		(property "Value" "10uF"
 			(at 241.681 121.793 0)
 			(effects
@@
 			)
 		)
-		(property "Value" "4.7uF"
+		(property "Value" "10uF"
 			(at 241.681 142.113 0)
 			(effects
@@
 			)
 		)
-		(property "Value" "4.7uF"
+		(property "Value" "10uF"
 			(at 208.661 101.473 0)
 			(effects
