File: Hardware/sensorboard/pcb.kicad_sch (KiCad schematic)
At the start: 0 parts

Commit message: Power Board WIP
Other:
- added sheet ccd_driver_v (ccd_driver_v.kicad_sch)
- note added: "CCD Driver - V Clocks"
Changed lines of the file:
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@@
+    (effects (font (size 2.54 2.54)) (justify left bottom))
+  )
+  (text "CCD Driver - V Clocks" (at 43.18 96.52 0)
     (effects (font (size 2.54 2.54)) (justify left bottom))
   )
@@
   (text "Rev  Date      Description " (at 199.39 41.91 0)
     (effects (font (size 2 2)) (justify left bottom))
+  )
+  (text "3" (at 33.02 96.52 0)
+    (effects (font (size 2.54 2.54)) (justify left bottom))
   )
   (text "CCD Driver" (at 43.18 66.04 0)
@@
       )
     )
+  )
+  (sheet (at 40.64 91.44) (size 73.66 5.08) (fields_autoplaced)
+    (stroke (width 0.1524) (type solid))
+    (fill (color 0 0 0 0.0000))
+    (property "Sheetname" "ccd_driver_v" (at 40.64 90.7284 0)
+      (effects (font (size 1.27 1.27)) (justify left bottom))
+    )
+    (property "Sheetfile" "ccd_driver_v.kicad_sch" (at 40.64 97.1046 0)
+      (effects (font (size 1.27 1.27)) (justify left top))
+    )
+    (instances
+      (project "pcb"
+        (path "/ba41827b-f176-424d-b6d5-0b0e1ddda097" (page "7"))
+      )
+    )

Commit message: Merge mainboard and powerboard
Other:
- added sheet fpga_config (fpga_config.kicad_sch)
- added sheet fpga_ddr (fpga_ddr.kicad_sch)
- added sheet fpga_io (fpga_io.kicad_sch)
- note added: "10"
- note added: "6"
- note added: "7"
- note added: "8"
- note added: "9"
- note added: "FPGA Config"
- note added: "FPGA DDR"
- note added: "FPGA IO"
Changed lines of the file:
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@@
+		)
+	)
+	(text "8"
+		(exclude_from_sim no)
+		(at 33.02 106.68 0)
+		(effects
+			(font
+				(size 2.54 2.54)
+			)
+			(justify left bottom)
 		)
 	)
@@
 		)
 	)
-	(text "3"
-		(exclude_from_sim no)
-		(at 33.02 66.04 0)
+	(text "6"
+		(exclude_from_sim no)
+		(at 33.02 86.36 0)
 		(effects
 			(font
@@
 	(text "CCD"
 		(exclude_from_sim no)
-		(at 43.18 76.2 0)
+		(at 43.18 66.04 0)
 		(effects
 			(font
@@
 	(text "Connector"
 		(exclude_from_sim no)
+		(at 43.18 76.2 0)
+		(effects
+			(font
+				(size 2.54 2.54)
+			)
+			(justify left bottom)
+		)
+	)
+	(text "FPGA Config"
+		(exclude_from_sim no)
+		(at 43.18 106.68 0)
+		(effects
+			(font
+				(size 2.54 2.54)
+			)
+			(justify left bottom)
+		)
+	)
+	(text "5"
+		(exclude_from_sim no)
+		(at 33.02 76.2 0)
+		(effects
+			(font
+				(size 2.54 2.54)
+			)
+			(justify left bottom)
+		)
+	)
+	(text "1"
+		(exclude_from_sim no)
+		(at 33.02 35.56 0)
+		(effects
+			(font
+				(size 2.54 2.54)
+			)
+			(justify left bottom)
+		)
+	)
+	(text "Rev  Date      Description "
+		(exclude_from_sim no)
+		(at 199.39 41.91 0)
+		(effects
+			(font
+				(size 2 2)
+			)
+			(justify left bottom)
+		)
+	)
+	(text "7"
+		(exclude_from_sim no)
+		(at 33.02 96.52 0)
+		(effects
+			(font
+				(size 2.54 2.54)
+			)
+			(justify left bottom)
+		)
+	)
+	(text "CCD Driver"
+		(exclude_from_sim no)
 		(at 43.18 86.36 0)
 		(effects
@@
 		)
 	)
-	(text "5"
-		(exclude_from_sim no)
-		(at 33.02 86.36 0)
-		(effects
-			(font
-				(size 2.54 2.54)
-			)
-			(justify left bottom)
-		)
-	)
-	(text "1"
-		(exclude_from_sim no)
-		(at 33.02 35.56 0)
-		(effects
-			(font
-				(size 2.54 2.54)
-			)
-			(justify left bottom)
-		)
-	)
-	(text "Rev  Date      Description "
-		(exclude_from_sim no)
-		(at 199.39 41.91 0)
-		(effects
-			(font
-				(size 2 2)
-			)
-			(justify left bottom)
-		)
-	)
-	(text "3"
-		(exclude_from_sim no)
-		(at 33.02 96.52 0)
-		(effects
-			(font
-				(size 2.54 2.54)
-			)
-			(justify left bottom)
-		)
-	)
-	(text "CCD Driver"
-		(exclude_from_sim no)
-		(at 43.18 66.04 0)
+	(text "9"
+		(exclude_from_sim no)
+		(at 33.02 116.84 0)
 		(effects
 			(font
@@
 		(exclude_from_sim no)
 		(at 43.18 45.72 0)
+		(effects
+			(font
+				(size 2.54 2.54)
+			)
+			(justify left bottom)
+		)
+	)
+	(text "FPGA DDR"
+		(exclude_from_sim no)
+		(at 43.18 116.84 0)
+		(effects
+			(font
+				(size 2.54 2.54)
+			)
+			(justify left bottom)
+		)
+	)
+	(text "10"
+		(exclude_from_sim no)
+		(at 33.02 127 0)
 		(effects
 			(font
@@
 		)
 	)
+	(text "FPGA IO"
+		(exclude_from_sim no)
+		(at 43.18 127 0)
+		(effects
+			(font
+				(size 2.54 2.54)
+			)
+			(justify left bottom)
+		)
+	)
 	(text "4"
 		(exclude_from_sim no)
-		(at 33.02 76.2 0)
+		(at 33.02 66.04 0)
 		(effects
 			(font
@@
 	)
 	(sheet
+		(at 40.64 71.12)
+		(size 73.66 5.08)
+		(fields_autoplaced yes)
+		(stroke
+			(width 0.1524)
+			(type solid)
+		)
+		(fill
+			(color 0 0 0 0.0000)
+		)
+		(property "Sheetname" "connector"
+			(at 40.64 70.4084 0)
+			(effects
+				(font
+					(size 1.27 1.27)
+				)
+				(justify left bottom)
+			)
+		)
+		(property "Sheetfile" "connector.kicad_sch"
+			(at 40.64 76.7846 0)
+			(effects
+				(font
+					(size 1.27 1.27)
+				)
+				(justify left top)
+			)
+		)
+		(instances
+			(project "pcb"
+				(path "/ba41827b-f176-424d-b6d5-0b0e1ddda097"
+					(page "5")
+				)
+			)
+		)
+	)
+	(sheet
 		(at 40.64 81.28)
 		(size 73.66 5.08)
@@
 			(color 0 0 0 0.0000)
 		)
-		(property "Sheetname" "connector"
+		(property "Sheetname" "ccd_driver"
 			(at 40.64 80.5684 0)
 			(effects
@@
 			)
 		)
-		(property "Sheetfile" "connector.kicad_sch"
+		(property "Sheetfile" "ccd_driver.kicad_sch"
 			(at 40.64 86.9446 0)
-			(effects
-				(font
-					(size 1.27 1.27)
-				)
-				(justify left top)
-			)
-		)
-		(instances
-			(project "pcb"
-				(path "/ba41827b-f176-424d-b6d5-0b0e1ddda097"
-					(page "5")
-				)
-			)
-		)
-	)
-	(sheet
-		(at 40.64 60.96)
-		(size 73.66 5.08)
-		(fields_autoplaced yes)
-		(stroke
-			(width 0.1524)
-			(type solid)
-		)
-		(fill
-			(color 0 0 0 0.0000)
-		)
-		(property "Sheetname" "ccd_driver"
-			(at 40.64 60.2484 0)
-			(effects
-				(font
-					(size 1.27 1.27)
-				)
-				(justify left bottom)
-			)
-		)
-		(property "Sheetfile" "ccd_driver.kicad_sch"
-			(at 40.64 66.6246 0)
 			(effects
 				(font
@@
 	)
 	(sheet
+		(at 40.64 101.6)
+		(size 73.66 5.08)
+		(fields_autoplaced yes)
+		(stroke
+			(width 0.1524)
+			(type solid)
+		)
+		(fill
+			(color 0 0 0 0.0000)
+		)
+		(property "Sheetname" "fpga_config"
+			(at 40.64 100.8884 0)
+			(effects
+				(font
+					(size 1.27 1.27)
+				)
+				(justify left bottom)
+			)
+		)
+		(property "Sheetfile" "fpga_config.kicad_sch"
+			(at 40.64 107.2646 0)
+			(effects
+				(font
+					(size 1.27 1.27)
+				)
+				(justify left top)
+			)
+		)
+		(instances
+			(project "pcb"
+				(path "/ba41827b-f176-424d-b6d5-0b0e1ddda097"
+					(page "8")
+				)
+			)
+		)
+	)
+	(sheet
 		(at 40.64 50.8)
 		(size 73.66 5.08)
@@
 	)
 	(sheet
-		(at 40.64 71.12)
+		(at 40.64 121.92)
+		(size 73.66 5.08)
+		(fields_autoplaced yes)
+		(stroke
+			(width 0.1524)
+			(type solid)
+		)
+		(fill
+			(color 0 0 0 0.0000)
+		)
+		(property "Sheetname" "fpga_io"
+			(at 40.64 121.2084 0)
+			(effects
+				(font
+					(size 1.27 1.27)
+				)
+				(justify left bottom)
+			)
+		)
+		(property "Sheetfile" "fpga_io.kicad_sch"
+			(at 40.64 127.5846 0)
+			(effects
+				(font
+					(size 1.27 1.27)
+				)
+				(justify left top)
+			)
+		)
+		(instances
+			(project "pcb"
+				(path "/ba41827b-f176-424d-b6d5-0b0e1ddda097"
+					(page "10")
+				)
+			)
+		)
+	)
+	(sheet
+		(at 40.64 111.76)
+		(size 73.66 5.08)
+		(fields_autoplaced yes)
+		(stroke
+			(width 0.1524)
+			(type solid)
+		)
+		(fill
+			(color 0 0 0 0.0000)
+		)
+		(property "Sheetname" "fpga_ddr"
+			(at 40.64 111.0484 0)
+			(effects
+				(font
+					(size 1.27 1.27)
+				)
+				(justify left bottom)
+			)
+		)
+		(property "Sheetfile" "fpga_ddr.kicad_sch"
+			(at 40.64 117.4246 0)
+			(effects
+				(font
+					(size 1.27 1.27)
+				)
+				(justify left top)
+			)
+		)
+		(instances
+			(project "pcb"
+				(path "/ba41827b-f176-424d-b6d5-0b0e1ddda097"
+					(page "9")
+				)
+			)
+		)
+	)
+	(sheet
+		(at 40.64 60.96)
 		(size 73.66 5.08)
 		(fields_autoplaced yes)
@@
 		)
 		(property "Sheetname" "ccd"
-			(at 40.64 70.4084 0)
+			(at 40.64 60.2484 0)
 			(effects
 				(font
@@
 		)
 		(property "Sheetfile" "ccd.kicad_sch"
-			(at 40.64 76.7846 0)
-			(effects
-				(font
+			(at 40.64 66.6246 0)
+			(effects
+				(font

Commit message: Design grip flex, SB/IOB WIP
Other:
- added sheet fpga_power (fpga_power.kicad_sch)
- note added: "11"
- note added: "FPGA Power"
Changed lines of the file:
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@@
+		)
+	)
+	(text "FPGA Power"
+		(exclude_from_sim no)
+		(at 43.18 137.16 0)
+		(effects
+			(font
+				(size 2.54 2.54)
+			)
+			(justify left bottom)
 		)
 	)
@@
 		(exclude_from_sim no)
 		(at 43.18 86.36 0)
+		(effects
+			(font
+				(size 2.54 2.54)
+			)
+			(justify left bottom)
+		)
+	)
+	(text "11"
+		(exclude_from_sim no)
+		(at 33.02 137.16 0)
 		(effects
 			(font
@@
 				)
 			)
+		)
+	)
+	(sheet
+		(at 40.64 132.08)
+		(size 73.66 5.08)
+		(fields_autoplaced yes)
+		(stroke
+			(width 0.1524)
+			(type solid)
+		)
+		(fill
+			(color 0 0 0 0.0000)
+		)
+		(property "Sheetname" "fpga_power"
+			(at 40.64 131.3684 0)
+			(effects
+				(font
+					(size 1.27 1.27)
+				)
+				(justify left bottom)
+			)
+		)
+		(property "Sheetfile" "fpga_power.kicad_sch"
+			(at 40.64 137.7446 0)
+			(effects
+				(font
+					(size 1.27 1.27)
+				)
+				(justify left top)
+			)
+		)
+		(instances
+			(project "pcb"
+				(path "/ba41827b-f176-424d-b6d5-0b0e1ddda097"
+					(page "11")
+				)
+			)

Commit message: Hardware r0.9
Other:
- company: Copyright 2023 Wenting Zhang -> Copyright 2024 Wenting Zhang
- title: Sitina 1 Mainboard -> Sitina 1 Sensor Board
Changed lines of the file:
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@@
 	(paper "A4")
 	(title_block
-		(title "Sitina 1 Mainboard")
-		(date "2023-03-16")
-		(rev "R0.6")
-		(company "Copyright 2023 Wenting Zhang")
+		(title "Sitina 1 Sensor Board")
+		(date "2024-03-25")
+		(rev "R0.9")
+		(company "Copyright 2024 Wenting Zhang")
 		(comment 2 "MERCHANTABILITY, SATISFACTORY QUALITY AND FITNESS FOR A PARTICULAR PURPOSE.")
 		(comment 3 "This source is distributed WITHOUT ANY EXPRESS OR IMPLIED WARRANTY, INCLUDING OF")
