File: Hardware/powerboard/power_plan.kicad_sch (KiCad schematic)
At the start: 0 parts

Commit message: PowerBoard Schematic, adding part values
Other:
- note added: "+3.2~4.2"
- note added: "VSUB"
Changed lines of the file:
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@@
+    (stroke (width 0) (type default))
+  )
+  (polyline (pts (xy 157.48 64.77) (xy 158.75 66.04))
     (stroke (width 0) (type default))
   )
@@
     (stroke (width 0) (type default))
   )
+  (polyline (pts (xy 208.28 66.04) (xy 207.01 64.77))
+    (stroke (width 0) (type default))
+  )
   (polyline (pts (xy 207.01 153.67) (xy 208.28 152.4))
     (stroke (width 0) (type default))
@@
     (stroke (width 0) (type default))
   )
+  (polyline (pts (xy 180.34 66.04) (xy 208.28 66.04))
+    (stroke (width 0) (type default))
+  )
   (polyline (pts (xy 181.61 110.49) (xy 182.88 109.22))
     (stroke (width 0) (type default))
@@
     (stroke (width 0) (type default))
   )
-  (polyline (pts (xy 157.48 52.07) (xy 157.48 55.88))
+  (polyline (pts (xy 207.01 67.31) (xy 208.28 66.04))
+    (stroke (width 0) (type default))
+  )
+  (polyline (pts (xy 156.21 52.07) (xy 156.21 55.88))
     (stroke (width 0) (type default))
   )
@@
     (stroke (width 0) (type default))
   )
-  (polyline (pts (xy 91.44 21.59) (xy 105.41 21.59))
+  (polyline (pts (xy 101.6 21.59) (xy 105.41 21.59))
     (stroke (width 0) (type default))
   )
@@
     (stroke (width 0) (type default))
   )
+  (polyline (pts (xy 156.21 66.04) (xy 156.21 81.28))
+    (stroke (width 0) (type default))
+  )
   (polyline (pts (xy 207.01 102.87) (xy 208.28 101.6))
     (stroke (width 0) (type default))
@@
     (stroke (width 0) (type default))
   )
-  (polyline (pts (xy 157.48 52.07) (xy 160.02 52.07))
+  (polyline (pts (xy 156.21 52.07) (xy 158.75 52.07))
     (stroke (width 0) (type default))
   )
@@
     (stroke (width 0) (type default))
   )
+  (polyline (pts (xy 157.48 67.31) (xy 158.75 66.04))
+    (stroke (width 0) (type default))
+  )
   (polyline (pts (xy 128.27 66.04) (xy 147.32 55.88))
     (stroke (width 0) (type default))
@@
     (stroke (width 0) (type default))
   )
+  (polyline (pts (xy 156.21 66.04) (xy 158.75 66.04))
+    (stroke (width 0) (type default))
+  )
   (polyline (pts (xy 172.72 39.37) (xy 173.99 40.64))
     (stroke (width 0) (type default))
@@
     (stroke (width 0) (type default))
   )
-  (polyline (pts (xy 158.75 50.8) (xy 160.02 52.07))
+  (polyline (pts (xy 157.48 50.8) (xy 158.75 52.07))
     (stroke (width 0) (type default))
   )
@@
     (stroke (width 0) (type default))
   )
+  (polyline (pts (xy 101.6 21.59) (xy 101.6 59.69))
+    (stroke (width 0) (type default))
+  )
   (polyline (pts (xy 147.32 99.06) (xy 208.28 99.06))
     (stroke (width 0) (type default))
@@
     (stroke (width 0) (type default))
   )
-  (polyline (pts (xy 158.75 53.34) (xy 160.02 52.07))
+  (polyline (pts (xy 157.48 53.34) (xy 158.75 52.07))
     (stroke (width 0) (type default))
   )
@@
     (fill (type none))
   )
-  (circle (center 157.48 55.88) (radius 1.27)
+  (circle (center 156.21 55.88) (radius 1.27)
     (stroke (width 0) (type default))
     (fill (type none))
@@
     (fill (type none))
   )
+  (rectangle (start 158.75 63.5) (end 180.34 68.58)
+    (stroke (width 0.3) (type default))
+    (fill (type none))
+  )
   (circle (center 101.6 85.09) (radius 1.27)
     (stroke (width 0) (type default))
@@
     (fill (type none))
   )
+  (circle (center 156.21 81.28) (radius 1.27)
+    (stroke (width 0) (type default))
+    (fill (type none))
+  )
   (rectangle (start 208.28 118.11) (end 243.84 124.46)
     (stroke (width 0.3) (type default) (color 0 132 132 1))
@@
     (fill (type none))
   )
-  (rectangle (start 160.02 49.53) (end 180.34 54.61)
+  (rectangle (start 158.75 49.53) (end 180.34 54.61)
     (stroke (width 0.3) (type default))
     (fill (type none))
@@
     (fill (type none))
   )
+  (rectangle (start 208.28 64.77) (end 220.98 67.31)
+    (stroke (width 0) (type default) (color 0 132 132 1))
+    (fill (type none))
+  )
   (rectangle (start 190.5 50.8) (end 198.12 53.34)
     (stroke (width 0.3) (type default))
@@
     (effects (font (size 2.54 2.54) (thickness 0.508) bold) (justify left bottom))
   )
+  (text "+3.2~4.2" (at 92.71 57.15 0)
+    (effects (font (size 0.635 0.635) (color 0 194 0 1)) (justify left bottom))
+  )
   (text "SENSITIVE" (at 151.13 33.02 0)
     (effects (font (size 0.635 0.635) (color 255 0 0 1)) (justify left bottom))
@@
     (effects (font (size 1.27 1.27)) (justify left bottom))
   )
-  (text "+3V3" (at 92.71 21.59 0)
-    (effects (font (size 1.27 1.27)) (justify left bottom))
-  )
   (text "PULSE" (at 148.59 129.54 0)
     (effects (font (size 0.635 0.635) (color 0 0 255 1)) (justify left bottom))
@@
     (effects (font (face "KiCad Font") (size 2.54 2.54)) (justify left bottom))
   )
-  (text "KAI-1100x" (at 209.55 68.58 0)
+  (text "KAI-1100x" (at 220.98 68.58 0)
     (effects (font (size 2.54 2.54)) (justify left bottom))
   )
@@
     (effects (font (size 1.27 1.27)) (justify left bottom))
   )
+  (text "TPS72301" (at 160.02 67.31 0)
+    (effects (font (size 2.54 2.54)) (justify left bottom))
+  )
   (text "SENSITIVE" (at 208.28 20.32 0)
     (effects (font (size 0.635 0.635) (color 255 0 0 1)) (justify left bottom))
@@
     (effects (font (size 1.27 1.27)) (justify left bottom))
   )
+  (text "VSUB" (at 209.55 67.31 0)
+    (effects (font (size 1.27 1.27)) (justify left bottom))
+  )
   (text "TPS62175" (at 106.68 86.36 0)
     (effects (font (size 2.54 2.54)) (justify left bottom))
@@
     (effects (font (size 1.27 1.27)) (justify left bottom))
   )
-  (text "TPS72301" (at 161.29 53.34 0)
-    (effects (font (size 2.54 2.54)) (justify left bottom))
-  )
+  (text "TPS72301" (at 160.02 53.34 0)
+    (effects (font (size 2.54 2.54)) (justify left bottom))
+  )

Commit message: Power Board Routing WI{
Changed lines of the file:
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@@
     (fill (type none))
   )
-  (rectangle (start 34.29 166.37) (end 45.72 168.91)
+  (rectangle (start 91.44 135.89) (end 102.87 138.43)
     (stroke (width 0.3) (type default))
     (fill (type none))
@@
     (fill (type none))
   )
-  (rectangle (start 34.29 170.18) (end 45.72 172.72)
+  (rectangle (start 91.44 139.7) (end 102.87 142.24)
     (stroke (width 0.3) (type default) (color 0 132 132 1))
     (fill (type none))
@@
     (effects (font (size 1.27 1.27)) (justify left bottom))
   )
-  (text "Legends" (at 34.29 165.1 0)
+  (text "Legends" (at 91.44 134.62 0)
     (effects (font (size 1.27 1.27)) (justify left bottom))
   )
@@
     (effects (font (size 1.27 1.27)) (justify left bottom))
   )
-  (text "Power Conversion / Switch" (at 48.26 168.91 0)
+  (text "Power Conversion / Switch" (at 105.41 138.43 0)
     (effects (font (size 1.27 1.27)) (justify left bottom))
   )
@@
     (effects (font (size 1.27 1.27)) (justify left bottom))
   )
-  (text "Consumers" (at 48.26 172.72 0)
+  (text "Consumers" (at 105.41 142.24 0)
     (effects (font (size 1.27 1.27)) (justify left bottom))
   )
@@
     (effects (font (size 1.27 1.27)) (justify left bottom))
   )
-  (text "Capability" (at 48.26 176.53 0)
+  (text "Capability" (at 105.41 146.05 0)
     (effects (font (size 1.27 1.27)) (justify left bottom))
   )
@@
     (effects (font (size 0.635 0.635) (color 255 0 0 1)) (justify left bottom))
   )
-  (text "abcd" (at 34.29 176.53 0)
+  (text "abcd" (at 91.44 146.05 0)
     (effects (font (size 1.27 1.27) (thickness 0.254) bold (color 194 0 0 1)) (justify left bottom))
   )

Commit message: Next set of PCB revisions WIP
Other:
- note added: "+1.0~3.0"
- note added: "+1V0"
- note added: "+3.3VA"
- note added: "+3V3_LENS"
- note added: "+5VP"
- note added: "+5V_LENS"
- note added: "+BATT"
- note added: "+CCDPWR"
- note added: "+FAN"
- note added: "+RTC"
- note added: "+VCCIO_SD"
- note added: "+VSD"
- note added: "19.2V 40mA"
- note added: "2.5A"
- note added: "ADP5071"
- note added: "BL"
- note added: "Backlight"
- note added: "Battery"
- note added: "CAT4139"
- note added: "Charge LM 1.8A"
- note added: "DCDC"
- note added: "DCDC2"
- note added: "DCDC3"
- note added: "Display"
- note added: "FAN"
- note added: "GPIO"
- note added: "ILM0.5A"
- note added: "ILM0.7A"
- note added: "ILM1.7A"
- note added: "IMXRT1052"
- note added: "IO"
- note added: "IPSOUT Internal Supply"
- note added: "LDO1"
- note added: "LDO2"
- note added: "LDO3"
- note added: "LDO4"
- note added: "LENS"
- note added: "MT9700"
- note added: "Mainboard"
- note added: "OLM0.03A"
- note added: "OLM0.2A"
- note added: "OLM<0.5A"
- note added: "OLM<1A"
- note added: "PMIC AXP209"
- note added: "QSPI"
- note added: "SD"
- note added: "SD0"
- note added: "SD1, EMC"
- note added: "SDRAM"
- note added: "SNVS"
- note added: "STM32G0"
- note added: "SWLM1.4A"
- note added: "SWLM2.3A"
- note added: "SY7208"
- note added: "SY8120"
- note added: "SoC"
- note added: "TLV76701"
- note added: "USBC-1"
- note added: "USBC-2"
- note added: "VBUS"
- note added: "VCI"
- note added: "XC6206"
- note removed: "LT8471"
- note removed: "TLV74315"
- note removed: "TLV74318"
- note removed: "TLV74330"
- note removed: "TPS62175"

Commit message: MB r0p8/ PB r0p2 routing in progress
Other:
- note removed: "-3.3V"
- company: Copyright 2023 Anhang Li -> Copyright 2024 Wenting Z, Anhang Li
Changed lines of the file:
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@@
 		(date "2023-11-24")
 		(rev "R0.1")
-		(company "Copyright 2023 Anhang Li")
+		(company "Copyright 2024 Wenting Z, Anhang Li")
 		(comment 2 "MERCHANTABILITY, SATISFACTORY QUALITY AND FITNESS FOR A PARTICULAR PURPOSE.")
 		(comment 3 "This source is distributed WITHOUT ANY EXPRESS OR IMPLIED WARRANTY, INCLUDING OF")
@@
 	(polyline
 		(pts
-			(xy 200.66 54.61) (xy 210.82 54.61)
+			(xy 182.88 54.61) (xy 210.82 54.61)
 		)
 		(stroke
@@
 	(polyline
 		(pts
-			(xy 191.77 53.34) (xy 193.04 54.61)
-		)
-		(stroke
-			(width 0)
-			(type default)
-		)
-	)
-	(polyline
-		(pts
 			(xy 200.66 146.05) (xy 200.66 154.94)
 		)
@@
 	(polyline
 		(pts
-			(xy 191.77 55.88) (xy 193.04 54.61)
-		)
-		(stroke
-			(width 0)
-			(type default)
-		)
-	)
-	(polyline
-		(pts
 			(xy 29.21 140.97) (xy 29.21 144.78)
 		)
@@
 	(polyline
 		(pts
-			(xy 182.88 54.61) (xy 193.04 54.61)
-		)
-		(stroke
-			(width 0)
-			(type default)
-		)
-	)
-	(polyline
-		(pts
-			(xy 20.32 85.09) (xy 26.67 85.09)
-		)
-		(stroke
-			(width 0)
-			(type default)
-		)
-	)
-	(polyline
-		(pts
 			(xy 184.15 110.49) (xy 185.42 111.76)
 		)
@@
 	(polyline
 		(pts
+			(xy 19.05 85.09) (xy 26.67 85.09)
+		)
+		(stroke
+			(width 0)
+			(type default)
+		)
+	)
+	(polyline
+		(pts
 			(xy 149.86 115.57) (xy 148.59 114.3)
 		)
@@
 	(polyline
 		(pts
-			(xy 20.32 63.5) (xy 20.32 85.09)
+			(xy 20.32 63.5) (xy 20.32 77.47)
 		)
 		(stroke
@@
 		)
 	)
-	(circle
-		(center 20.32 85.09)
-		(radius 1.27)
-		(stroke
-			(width 0)
-			(type default)
-		)
-		(fill
-			(type none)
-		)
-	)
-	(rectangle
-		(start 193.04 53.34)
-		(end 200.66 55.88)
-		(stroke
-			(width 0.3)
-			(type default)
-		)
-		(fill
-			(type none)
-		)
-	)
 	(rectangle
 		(start 26.67 82.55)
@@
 		)
 	)
-	(circle
-		(center 20.32 77.47)
-		(radius 1.27)
-		(stroke
-			(width 0)
-			(type default)
-		)
-		(fill
-			(type none)
-		)
-	)
 	(rectangle
 		(start 210.82 151.13)
@@
 		)
 	)
-	(text "-3.3V"
-		(exclude_from_sim no)
-		(at 185.42 54.61 0)
-		(effects
-			(font
-				(size 1.27 1.27)
-			)
-			(justify left bottom)
-		)
-	)
 	(text "1EDN7550B"
 		(exclude_from_sim no)
@@
 		)
 	)
-	(text "RDIV"
-		(exclude_from_sim no)
-		(at 194.31 55.88 0)
-		(effects
-			(font
-				(size 1.27 1.27)
-			)
-			(justify left bottom)
-		)
-	)
 	(text "IO"
 		(exclude_from_sim no)
@@
 			)
 			(justify left bottom)
+		)
+	)
+	(text "+3V3"
+		(exclude_from_sim no)
+		(at 19.05 85.09 0)
+		(effects
+			(font
+				(size 1.27 1.27)
+			)
+			(justify left bottom)
