File: Hardware/powerboard/PowerBoard.kicad_pcb (KiCad board)
At the start: 2 copper layers, 70 x 70 mm, 91 parts, among them J1 FPC 0.5mm Bottom Contact, J2 DF12NC(3.0)-20DS-0.5V, U1 TPS65130RGE, U2 ADP5071ACPZ, U3 TPS62175DQC, U4 ADP5071ACPZ, U5 TLV74330, U6 TPS65130RGE

Commit message: Power Board Routing WI{
Parts:
- removed C21: 10uF 25V, Capacitor_SMD:C_0805_2012Metric
- added C31: 10uF 25V, Capacitor_SMD:C_0805_2012Metric, F.Cu at (182.8, 97.5)
- added CT1: 330uF 6.3V, Capacitor_Tantalum_SMD:CP_EIA-7343-43_Kemet-X, F.Cu at (183.0, 136.9)
- added CT2: 330uF 6.3V, Capacitor_Tantalum_SMD:CP_EIA-7343-43_Kemet-X, F.Cu at (151.5, 133.5)
- added CT3: 330uF 6.3V, Capacitor_Tantalum_SMD:CP_EIA-7343-43_Kemet-X, F.Cu at (146.5, 133.5)
- added CT4: 330uF 6.3V, Capacitor_Tantalum_SMD:CP_EIA-7343-43_Kemet-X, F.Cu at (174.2, 79.8)
- moved C1 60.3 mm to (176.2, 83.2)
- moved C10 23.7 mm to (167.5, 127.0), turned to -90 degrees
- moved D4 22.8 mm to (180.2, 122.5), turned to -90 degrees
- moved C16 22.5 mm to (183.0, 122.0)
- moved C15 22.5 mm to (186.8, 122.0)
- moved L3 22.5 mm to (179.8, 126.8), turned to -90 degrees
- moved L4 22.5 mm to (184.0, 125.0)
- moved C12 22.5 mm to (182.2, 133.5)
- moved C13 22.5 mm to (185.2, 133.5)
- moved R10 22.5 mm to (180.8, 129.8)
- moved R11 22.5 mm to (180.8, 131.8)
- moved R14 22.5 mm to (180.8, 132.8)
- moved R6 22.5 mm to (183.2, 133.5)
- moved R7 22.5 mm to (186.2, 133.5)
- moved R8 22.5 mm to (184.2, 133.5)
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Connections:
- J1 pad 17: /-4VD -> GND
- J1 pad 18: /-4VD -> GND
- J1 pad 19: /+5VD -> /+8VD
- J1 pad 20: /+5VD -> /+8VD
- J1 pad 21: GND -> /+8VD
- J1 pad 22: GND -> /-9VD
- J1 pad 25: /-9VD -> GND
- J1 pad 27: GND -> /-4VD
- J1 pad 28: /+8VD -> /+5VD
- J1 pad 29: /+8VD -> /+5VD
- J1 pad 30: /+8VD -> GND
Routing:
- net GND: track 7.75 -> 370.3 mm, vias 0 -> 62
- net +SYS: track 0.00 -> 135.1 mm, vias 0 -> 40
- net CCD_POWEREN: track 0.00 -> 111.4 mm, vias 0 -> 7
- net /+16VD: track 0.00 -> 52.1 mm, vias 0 -> 5
- net /-9VA: track 10.4 -> 51.9 mm, vias 0 -> 2
- net /+8VD: track 4.36 -> 42.8 mm, vias 0 -> 2
- net /-9VD: track 1.77 -> 37.7 mm
- net /-15VD: track 0.00 -> 33.4 mm
- net /+16VA: track 4.34 -> 34.6 mm, vias 0 -> 2
- net /-4VD: track 0.00 -> 20.5 mm, vias 0 -> 4
- net /+2VD: track 5.97 -> 19.7 mm
- net /+3VA: track 0.00 -> 12.8 mm
- net Net-(U6-PSN): track 0.00 -> 11.5 mm, vias 0 -> 2
- net Net-(D17-A): track 0.00 -> 8.42 mm
- net Net-(D5-A): track 0.00 -> 7.82 mm
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Other:
- board size 70 x 70 mm -> 67 x 66 mm
- copper layers 2 -> 4

Commit message: PowerBoard Alpha ver. Release
Parts:
- moved C9 1.65 mm to (181.2, 84.6), turned to 0 degrees
- moved R3 1.01 mm to (179.2, 86.3), turned to -90 degrees
- moved C7 0.99 mm to (180.2, 86.3), turned to -90 degrees
- moved L1 0.29 mm to (180.7, 94.9)
- moved C31 0.16 mm to (182.8, 97.7)
- moved C8 0.09 mm to (178.9, 97.7)
- moved L2 0.06 mm to (183.1, 89.8)
Connections:
- J1 pad 1: GND -> /-15VD
- J1 pad 10: SYNC_CLK1 -> CCD_PULSE_SYNC
- J1 pad 4: /-15VD -> GND
- J1 pad 6: /-4VD -> GND
- J1 pad 8: GND -> /-4VD
- J1 pad 9: SYNC_CLK2 -> CCD_AFE_SYNC
- J1 pad MP: GND -> unconnected-(J1-MountPin-PadMP)
- J2 pad 12: CCD_AFE_SYNC -> unconnected-(J2-Pin_12-Pad12)
- J2 pad 13: CCD_PULSE_SYNC -> unconnected-(J2-Pin_13-Pad13)
Routing:
- net GND: track 370.3 -> 584.4 mm, vias 62 -> 95
- net CCD_POWEREN: track 111.4 -> 256.2 mm, vias 7 -> 12
- net +SYS: track 135.1 -> 239.9 mm, vias 40 -> 57
- net /-4VD: track 20.5 -> 67.9 mm, vias 4 -> 11
- net CCD_AFE_SYNC: track 0.68 -> 34.3 mm, vias 1 -> 2
- net CCD_PULSE_SYNC: track 1.04 -> 24.6 mm, vias 1 -> 2
- net /+5VD: track 2.58 -> 21.0 mm, vias 0 -> 2
- net Net-(U1-PSN): track 0.00 -> 16.5 mm, vias 0 -> 4
- net /+16VA: track 34.6 -> 45.2 mm, vias 2 -> 4
- net Net-(D2-K): track 0.00 -> 7.81 mm
- net Net-(D1-A): track 0.00 -> 7.28 mm
- net Net-(U1-FBN): track 0.00 -> 3.73 mm
- net Net-(U1-FBP): track 0.00 -> 3.40 mm
- net Net-(U1-VREF): track 0.00 -> 2.86 mm
- net /-15VD: track 33.4 -> 30.8 mm
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- added copper zone on F.Cu, net +SYS
- added copper zone on B.Cu, net GND
Other:
- copper layers 4 -> 2
- board text added: "(c) 2023 Anhang Li, Wenting Zhang"
- board text added: "+15"
- board text added: "+16"
- board text added: "+16VA"
- board text added: "+2"
- board text added: "+3VA"
- board text added: "+5"
- board text added: "+8"
- board text added: "+9VA"
- board text added: "-4"
- board text added: "-9"
- board text added: "1"
- board text added: "GND"
- board text added: "Sitina 1 - Power Board"
- board text added: "VSYS"
- board text added: "Ver.alpha"

Commit message: PowerBoard DRC Clean
Parts:
- moved L2 0.07 mm to (183.1, 89.8)
Routing:
- net GND: track 584.4 -> 607.7 mm, vias 95 -> 90
- net CCD_POWEREN: track 256.2 -> 259.3 mm
- net +SYS: track 239.9 -> 242.7 mm
- net /+2VD: track 19.0 -> 21.2 mm
- net /+5VD: track 21.0 -> 22.2 mm, vias 2 -> 0
- net /+16VD: track 52.4 -> 51.7 mm
- net Net-(D1-A): track 7.28 -> 6.74 mm

Commit message: CCD Sensor Board WIP
Parts:
- moved C17 14.9 mm to (184.4, 131.8)
- moved C18 14.9 mm to (186.8, 129.8)
- moved C1 14.9 mm to (187.2, 93.2)
- moved C10 14.9 mm to (178.5, 137.0)
- moved C11 14.9 mm to (199.0, 138.0)
- moved C12 14.9 mm to (193.2, 143.5)
- moved C13 14.9 mm to (196.2, 143.5)
- moved C14 14.9 mm to (199.0, 141.0)
- moved C15 14.9 mm to (197.8, 132.0)
- moved C16 14.9 mm to (194.0, 132.0)
- moved C19 14.9 mm to (180.5, 136.5)
- moved C2 14.9 mm to (194.7, 103.1)
- moved C20 14.9 mm to (166.2, 140.5)
- moved C22 14.9 mm to (188.2, 145.2)
- moved C23 14.9 mm to (181.8, 139.4)
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
Commit message: Next set of PCB revisions WIP
Parts:
- removed C18: 22uF 25V, Capacitor_SMD:C_0805_2012Metric
- removed J2: DF12NC(3.0)-20DS-0.5V, Connector_Hirose:Hirose_DF12_DF12C3.0-20DS-0.5V_2x10_P0.50mm_Vertical
- removed U3: TPS62175DQC, Package_SON:WSON-10-1EP_2x3mm_P0.5mm_EP0.84x2.4mm_ThermalVias
- removed U5: TLV74330, Package_SON:Texas_X2SON-4_1x1mm_P0.65mm
- added C21: 100nF, Capacitor_SMD:C_0402_1005Metric, F.Cu at (180.9, 134.1)
- added C32: 100nF, Capacitor_SMD:C_0402_1005Metric, F.Cu at (182.9, 132.3)
- added J3: Conn_02x04_Odd_Even, Connector_PinSocket_2.00mm:PinSocket_2x04_P2.00mm_Vertical_SMD, F.Cu at (149.1, 141.0)
- added R16: 27K 1%, Resistor_SMD:R_0402_1005Metric, F.Cu at (187.4, 135.0)
- added R21: 12K 1%, Resistor_SMD:R_0402_1005Metric, F.Cu at (187.4, 136.2)
- added U7: SY8120, Package_TO_SOT_SMD:TSOT-23-6, F.Cu at (184.1, 135.1)
- C1: value 10uF 25V -> 22pF; footprint Capacitor_SMD:C_0805_2012Metric -> Capacitor_SMD:C_0402_1005Metric
- C17: value 22uF 25V -> 22uF
- moved C1 40.7 mm to (187.4, 133.9), turned to 180 degrees
- moved C17 4.05 mm to (186.8, 128.5), turned to 0 degrees
- moved L9 3.91 mm to (185.8, 131.4), turned to 180 degrees
Connections:
- C1 pad 1: +SYS -> /+2VD
- C1 pad 2: GND -> Net-(U7-FB)
- J1 pad 15: /+3VA -> GND
Routing:
- net GND: track 607.7 -> 509.3 mm, vias 90 -> 84
- net +SYS: track 242.7 -> 179.1 mm, vias 57 -> 48
- net CCD_POWEREN: track 259.3 -> 245.5 mm, vias 12 -> 10
- net /+3VA: track 13.6 -> 0.00 mm
- net /+2VD: track 21.2 -> 7.99 mm, vias 2 -> 0
- net Net-(U7-SW): track 2.85 -> 0.00 mm
- added copper zone on F.Cu, net CCD_POWEREN
- removed copper zone on F.Cu, net +SYS
Other:
- outline, holes or cut-outs redrawn
- board text removed: "+3VA"

Commit message: MB r0p8/ PB r0p2 routing in progress
Parts:
- J3: moved to B.Cu
- moved CT4 70.8 mm to (138.8, 143.2), turned to 180 degrees
- moved CT1 59.8 mm to (182.1, 88.3), turned to -90 degrees
- moved CT2 50.0 mm to (194.3, 104.9)
- moved L9 30.8 mm to (157.3, 143.0)
- moved C17 29.6 mm to (160.9, 143.0), turned to 90 degrees
- moved U7 27.4 mm to (157.0, 139.2), turned to 180 degrees
- moved C21 27.2 mm to (154.3, 139.7), turned to 90 degrees
- moved C1 26.4 mm to (161.3, 137.9)
- moved R16 26.4 mm to (161.3, 139.0)
- moved R21 26.4 mm to (161.3, 140.1)
- moved C32 24.5 mm to (159.6, 140.0), turned to 90 degrees
- moved CT3 19.7 mm to (138.8, 137.3), turned to 180 degrees
- moved C10 12.4 mm to (188.3, 144.6), turned to 0 degrees
- moved C19 9.89 mm to (188.3, 142.6), turned to 0 degrees
- moved C31 9.25 mm to (195.6, 98.6), turned to 90 degrees
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Connections:
- J3 pad 1: GND -> CCD_POWEREN
- J3 pad 2: +SYS -> GND
- J3 pad 3: GND -> +SYS
- J3 pad 4: +SYS -> GND
- J3 pad 5: GND -> +SYS
- J3 pad 6: +SYS -> GND
- J3 pad 7: GND -> +SYS
- J3 pad 8: CCD_POWEREN -> GND
Routing:
- net GND: track 509.3 -> 585.7 mm, vias 84 -> 65
- net /+2VD: track 7.99 -> 51.2 mm, vias 0 -> 3
- net CCD_AFE_SYNC: track 34.3 -> 60.4 mm, vias 2 -> 4
- net +SYS: track 179.1 -> 200.5 mm, vias 48 -> 21
- net /+5VD: track 22.2 -> 36.3 mm, vias 0 -> 2
- net /-15VD: track 30.8 -> 19.5 mm
- net /-4VD: track 67.7 -> 59.1 mm, vias 11 -> 3
- net Net-(U7-SW): track 0.00 -> 6.66 mm
- net Net-(U7-FB): track 0.00 -> 5.05 mm
- net /-9VA: track 52.6 -> 57.5 mm
- net CCD_POWEREN: track 245.5 -> 249.2 mm, vias 10 -> 12
- net Net-(U1-PSN): track 17.0 -> 13.4 mm
- net Net-(D1-A): track 6.74 -> 10.3 mm
- net /+16VA: track 45.2 -> 48.6 mm, vias 4 -> 3
- net Net-(U1-CN): track 1.78 -> 4.25 mm
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- added copper zone on F.Cu, net +SYS
- removed copper zone on F.Cu, net CCD_POWEREN
Other:
- board size 67 x 66 mm -> 67 x 66.6 mm
- board text added: "2"
- board text added: "3"
- board text added: "4"
- board text added: "A"
- board text added: "A4"
- board text added: "B"
- board text added: "C"
- board text added: "D"
- board text added: "E"
- board text added: "F"
- board text added: "filterholder"
- board text added: "ǩ\U+540D"
- board text added: "ͼֽ 1 (\U+51711)"

Commit message: Use IPSOUT for lens 5V supply
Parts:
- J3: value Conn_02x04_Odd_Even -> FH-00176
Routing:
- net +SYS: track 200.5 -> 192.9 mm, vias 21 -> 17
- net GND: track 585.7 -> 588.9 mm, vias 65 -> 64
Other:
- outline, holes or cut-outs redrawn
