File: Hardware/ioboard/storage.kicad_sch (KiCad schematic)
At the start: 8 parts, among them U4 W25Q32JV

Commit message: Merge mainboard and powerboard
Connections:
- net SD1_CLK renamed SD_CLK
- net SD1_CMD renamed SD_CMD
- net SD1_DATA0 renamed SD_DATA0
- net SD1_DATA1 renamed SD_DATA1
- net SD1_DATA2 renamed SD_DATA2
- net SD1_DATA3 renamed SD_DATA3
- no-connect marks 2 -> 1
Other:
- note removed: "Can't route CD pin :("
- company: Copyright 2023 Wenting Zhang -> Copyright 2024 Wenting Zhang, Anhang Li
- title: Sitina 1 Mainboard -> Sitina 1 IO Board
Changed lines of the file:
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@@
 	(paper "A4")
 	(title_block
-		(title "Sitina 1 Mainboard")
-		(date "2023-03-16")
-		(rev "R0.6")
-		(company "Copyright 2023 Wenting Zhang")
+		(title "Sitina 1 IO Board")
+		(date "2024-03-08")
+		(rev "R0.9")
+		(company "Copyright 2024 Wenting Zhang, Anhang Li")
 		(comment 2 "MERCHANTABILITY, SATISFACTORY QUALITY AND FITNESS FOR A PARTICULAR PURPOSE.")
 		(comment 3 "This source is distributed WITHOUT ANY EXPRESS OR IMPLIED WARRANTY, INCLUDING OF")
@@
 		(at 104.14 114.3)
 	)
-	(no_connect
-		(at 68.58 114.3)
-	)
 	(wire
 		(pts
@@
 			(width 0)
 			(type default)
-		)
-	)
-	(text "Can't route CD pin :("
-		(exclude_from_sim no)
-		(at 71.12 115.57 0)
-		(effects
-			(font
-				(size 1.27 1.27)
-			)
-			(justify left bottom)
 		)
 	)
@@
 		)
 	)
-	(global_label "SD1_DATA2"
+	(global_label "SD_DATA2"
 		(shape bidirectional)
 		(at 68.58 111.76 180)
@@
 		)
 		(property "Intersheetrefs" "${INTERSHEET_REFS}"
-			(at 55.8859 111.6806 0)
+			(at 55.4123 111.76 0)
 			(effects
 				(font
@@
 		)
 	)
-	(global_label "SD1_DATA0"
+	(global_label "SD_DATA0"
 		(shape bidirectional)
 		(at 68.58 106.68 180)
@@
 		)
 		(property "Intersheetrefs" "${INTERSHEET_REFS}"
-			(at 55.8859 106.6006 0)
-			(effects
-				(font
-					(size 1.27 1.27)
-				)
-				(justify right)
-				(hide yes)
-			)
-		)
-	)
-	(global_label "SD1_CD"
-		(shape output)
-		(at 68.58 114.3 180)
-		(fields_autoplaced yes)
-		(effects
-			(font
-				(size 1.27 1.27)
-			)
-			(justify right)
-		)
-		(property "Intersheetrefs" "${INTERSHEET_REFS}"
-			(at 58.3031 114.3 0)
+			(at 55.4123 106.68 0)
 			(effects
 				(font
@@
 		)
 	)
-	(global_label "SD1_DATA3"
+	(global_label "SD_DATA3"
 		(shape bidirectional)
 		(at 68.58 93.98 180)
@@
 		)
 		(property "Intersheetrefs" "${INTERSHEET_REFS}"
-			(at 55.8859 93.9006 0)
-			(effects
-				(font
-					(size 1.27 1.27)
-				)
-				(justify right)
-				(hide yes)
-			)
-		)
-	)
-	(global_label "SD1_DATA1"
+			(at 55.4123 93.98 0)
+			(effects
+				(font
+					(size 1.27 1.27)
+				)
+				(justify right)
+				(hide yes)
+			)
+		)
+	)
+	(global_label "SD_DATA1"
 		(shape bidirectional)
 		(at 68.58 109.22 180)
@@
 		)
 		(property "Intersheetrefs" "${INTERSHEET_REFS}"
-			(at 55.8859 109.1406 0)
-			(effects
-				(font
-					(size 1.27 1.27)
-				)
-				(justify right)
-				(hide yes)
-			)
-		)
-	)
-	(global_label "SD1_CLK"
+			(at 55.4123 109.22 0)
+			(effects
+				(font
+					(size 1.27 1.27)
+				)
+				(justify right)
+				(hide yes)
+			)
+		)
+	)
+	(global_label "SD_CLK"
 		(shape input)
 		(at 68.58 104.14 180)
@@
 		)
 		(property "Intersheetrefs" "${INTERSHEET_REFS}"
-			(at 57.9421 104.0606 0)
-			(effects
-				(font
-					(size 1.27 1.27)
-				)
-				(justify right)
-				(hide yes)
-			)
-		)
-	)
-	(global_label "SD1_CMD"
+			(at 58.4845 104.14 0)
+			(effects
+				(font
+					(size 1.27 1.27)
+				)
+				(justify right)
+				(hide yes)
+			)
+		)
+	)
+	(global_label "SD_CMD"
 		(shape input)
 		(at 68.58 96.52 180)
@@
 		)
 		(property "Intersheetrefs" "${INTERSHEET_REFS}"
-			(at 57.5188 96.4406 0)
-			(effects
-				(font
+			(at 58.0612 96.52 0)
+			(effects
+				(font

Commit message: Design grip flex, SB/IOB WIP
Parts:
- removed C81: 470nF, Capacitor_SMD:C_0402_1005Metric, symbol Device:C
- removed R18: 100K, Resistor_SMD:R_0402_1005Metric, symbol Device:R
- removed U4: W25Q32JV, Package_SON:WSON-8-1EP_6x5mm_P1.27mm_EP3.4x4.3mm, symbol Memory_Flash:W25Q32JVZP
Connections:
- net SD_CLK renamed SDIO_CLK
- net SD_CMD renamed SDIO_CMD
- net SD_DATA0 renamed SDIO_DAT0
- net SD_DATA1 renamed SDIO_DAT1
- net SD_DATA2 renamed SDIO_DAT2
- net SD_DATA3 renamed SDIO_DAT3
Other:
- moved on the sheet: C78, C79, C80, MICRO_SD400, R17
