File: Hardware/ioboard/connectors.kicad_sch (KiCad schematic)
At the start: 18 parts, among them J10 2.54mm pitch, J11 2.54mm pitch, J12 LensMount, J13 LensMount, J14 LensMount, J15 LensMount, J16 LensMount, J17 LensMount, J18 LensMount, J19 LensMount, J2 02x04_P2.0, J20 LensMount, J21 LensMount, J5 FPC 0.5mm Bottom Contact, J7 FFC 0.5mm Bottom Contact, J8 AudioJack2

Commit message: Merge mainboard and powerboard
Parts:
- added R8: 200R, Resistor_SMD:R_0402_1005Metric, symbol Device:R
- added U5: FODM3023, Package_DIP:SMDIP-4_W7.62mm, symbol Relay_SolidState:FODM3023
Connections:
- net FLASH_SYNC_S: now also U5.4
- net FLASH_SYNC_T: now also U5.3
- net GND: now also U5.2
- new net: R8.2, U5.1
- new net FLASH_SYNC: R8.1
Other:
- company: (none) -> Copyright 2024 Wenting Zhang, Anhang Li
- title: (none) -> Sitina 1 IO Board

Commit message: Design grip flex, SB/IOB WIP
Parts:
- removed J2: 02x04_P2.0, Connector_PinHeader_2.00mm:PinHeader_2x04_P2.00mm_Vertical_SMD, symbol Connector_Generic:Conn_02x04_Odd_Even
- added J2: 0.5mm Bottom Contact, Connector_FFC-FPC:Hirose_FH12-30S-0.5SH_1x30-1MP_P0.50mm_Horizontal, symbol Connector_Generic_MountingPin:Conn_01x30_MountingPin
- J5: value FPC 0.5mm Bottom Contact -> 0.5mm Bottom Contact
- J7: value FFC 0.5mm Bottom Contact -> 0.5mm Bottom Contact
Connections:
- net AFE_RST is gone; now on net +3V3: J5.24 (Pin_24)
- net AFE_SCK is gone; now on net +3V3: J5.23 (Pin_23)
- net AFE_SDATA is gone; now on net GND: J5.22 (Pin_22)
- net AFE_SYNC is gone; now on net GND: J5.25 (Pin_25)
- net CSI_D10 is gone; now on net I2C_SCL: J5.10 (Pin_10)
- net CSI_D8 is gone; now on net GND: J5.8 (Pin_8)
- net GND: now also J5.29 (Pin_29), J2.11 (Pin_11), J2.15 (Pin_15), J2.16 (Pin_16), J2.17 (Pin_17), J2.18 (Pin_18), J2.2 (Pin_2), J2.25 (Pin_25), J2.26 (Pin_26), J2.30 (Pin_30), J2.4 (Pin_4), J2.6 (Pin_6), J2.MP (MountPin); no longer J5.16 (Pin_16), J5.20 (Pin_20), J5.28 (Pin_28)
- net I2C_SCL: no longer J5.26 (Pin_26)
- net +3.3VA renamed +1V8
- net +1V8: no longer J5.29 (Pin_29)
- net AFE_SL renamed SDIO_CLK
- net CSI_D11 renamed PS_POR_B
- net CSI_D12 renamed FPGA_TMS
- net CSI_D13 renamed FPGA_TDO
- net CSI_D14 renamed FPGA_TDI
- net CSI_D15 renamed FPGA_TCK
- net CSI_D2 renamed MIPI_D1N
- net CSI_D3 renamed MIPI_D1P
- net CSI_D4 renamed MIPI_D0N
- net CSI_D5 renamed MIPI_D0P
- net CSI_D6 renamed MIPI_CKN
- net CSI_D7 renamed MIPI_CKP
- net CSI_D9 renamed I2C0_SDA
- net CSI_HSYNC renamed SDIO_DAT0
- net CSI_PIXCLK renamed SDIO_DAT2
- net CSI_VSYNC renamed SDIO_DAT1
- net GRIP_IO0 renamed GRIP_SCK
- net GRIP_IO1 renamed GRIP_MOSI
- net GRIP_IO2 renamed GRIP_CS
- net GRIP_IO3 renamed GRIP_MISO
- net I2C_SDA renamed IPSOUT
- net IPSOUT: now also J5.28 (Pin_28)
- new net +16VA: J2.13 (Pin_13), J2.14 (Pin_14)
- new net +16VD: J2.5 (Pin_5)
- new net +2VD: J2.3 (Pin_3)
- new net +5VD: J2.28 (Pin_28), J2.29 (Pin_29)
- new net +8VD: J2.19 (Pin_19), J2.20 (Pin_20), J2.21 (Pin_21)
- new net -15VD: J2.1 (Pin_1)
- new net -4VD: J2.27 (Pin_27), J2.7 (Pin_7), J2.8 (Pin_8)
- new net -9VA: J2.12 (Pin_12)
- new net -9VD: J2.22 (Pin_22), J2.23 (Pin_23), J2.24 (Pin_24)
- new net CCD_AFE_SYNC: J2.9 (Pin_9)
- new net CCD_PULSE_SYNC: J2.10 (Pin_10)
- new net EXTEN: J5.26 (Pin_26)
- new net SDIO_CMD: J5.20 (Pin_20)
- new net SDIO_DAT3: J5.16 (Pin_16)
Other:
- note added: "HIGH POWER PULSE"
- note added: "PULSE"
- note added: "SENSITIVE"
- note added: "To Sensor Board J1"
- note added: "To Sensor Board J2"
- note removed: "To Power Board"
- note removed: "To Sensor Board"
- moved on the sheet: J12, J13, J14, J15, J16, J17, J18, J19, J20, J21, J5, J8

Commit message: IOB r0p9 RC
Parts:
- added C108, C81: 22uF, Capacitor_SMD:C_0603_1608Metric, symbol Device:C
- added J4, J6: 2.54mm pitch, Connector_PinSocket_2.54mm:PinSocket_1x02_P2.54mm_Vertical, symbol Connector_Generic:Conn_01x02
Connections:
- net +FAN: now also C108.2, C81.2, J4.1 (Pin_1), J6.1 (Pin_1)
- net GND: now also C108.1, C81.1, J4.2 (Pin_2), J6.2 (Pin_2); no longer J2.15 (Pin_15)
- net MIPI_CKN: now also J5.7 (Pin_7); no longer J5.6 (Pin_6)
- net MIPI_CKP: now also J5.6 (Pin_6); no longer J5.7 (Pin_7)
- net MIPI_D0N: now also J5.5 (Pin_5); no longer J5.4 (Pin_4)
- net MIPI_D0P: now also J5.4 (Pin_4); no longer J5.5 (Pin_5)
- net MIPI_D1N: now also J5.3 (Pin_3); no longer J5.2 (Pin_2)
- net MIPI_D1P: now also J5.2 (Pin_2); no longer J5.3 (Pin_3)
- net I2C0_SDA renamed I2C_SDA
- new net +3.3VA: J2.15 (Pin_15)
