File: Hardware/ioboard/usb.kicad_sch (KiCad schematic)
At the start: 5 parts, among them J3 USB_C_Receptacle_USB2.0, U7 USBLC6-2P6

Commit message: IOB r0p9 RC
Parts:
- R19, R20: value 5.1K 1% -> 5.1K
Changed lines of the file:
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@@
 			)
 		)
-		(property "Value" "5.1K 1%"
+		(property "Value" "5.1K"
 			(at 124.46 111.76 0)
 			(effects
@@
 			)
 		)
-		(property "Value" "5.1K 1%"
+		(property "Value" "5.1K"
 			(at 111.76 111.76 0)
 			(effects
