File: Hardware/ioboard/pcb.kicad_pcb (KiCad board)
At the start: 4 copper layers, 71.6 x 73.2 mm, 198 parts, among them J1 2.54mm pitch, J10 2.54mm pitch, J11 2.54mm pitch, J12 LensMount, J13 LensMount, J14 LensMount, J15 LensMount, J16 LensMount, J17 LensMount, J18 LensMount, J19 LensMount, J2 02x04_P2.0, J20 LensMount, J21 LensMount, J3 USB_C_Receptacle_USB2.0, J4 USB_C_Receptacle_USB2.0, J5 FPC 0.5mm Bottom Contact, J7 FFC 0.5mm Bottom Contact, J8 AudioJack2, J9 2.54mm pitch, SW1 SW_Push_LED, U1 AXP209, U10 SY8120, U11 MT9700, U12 SY7208, U2 IMXRT1050, U3 MT48LC16M16A2BG, U4 W25Q32JV, U5 STM32G030F6Px, U6 CAT4139, U7 FODM3023, U8 USBLC6-2P6, U9 MT9700, Y1 24MHz, Y2 32.768K

Commit message: Merge mainboard and powerboard
Parts:
- removed C8, C98: 22uF, Capacitor_SMD:C_0603_1608Metric
- removed J1, J9: 2.54mm pitch, Connector_PinSocket_2.54mm:PinSocket_1x02_P2.54mm_Vertical
- added BZ1: Buzzer, Connector_PinHeader_2.54mm:PinHeader_1x02_P2.54mm_Vertical, F.Cu at (155.8, 149.0)
- added R37: 1K, Resistor_SMD:R_0402_1005Metric, F.Cu at (158.5, 148.5)
Connections:
- U5 pad 14: unconnected-(U5-PA7-Pad14) -> Net-(U5-PA7)
Routing:
- net +FAN: track 168.9 -> 67.6 mm
- net Net-(U5-PA7): track 0.00 -> 19.4 mm
- net Net-(BZ1-+): track 0.00 -> 2.73 mm

Commit message: IOB r0p9 RC
Parts:
- removed C94: 100nF, Capacitor_SMD:C_0402_1005Metric
- removed C95: 22uF, Capacitor_SMD:C_0603_1608Metric
- removed C96: 47pF, Capacitor_SMD:C_0402_1005Metric
- removed C97: 220nF, Capacitor_SMD:C_0402_1005Metric
- removed L8: FTC201610S4R7MBCA, Inductor_SMD:L_Murata_DFE201610P
- added C108: 22uF, Capacitor_SMD:C_0603_1608Metric, B.Cu at (172.1, 149.7)
- added C8: 2.2uF, Capacitor_SMD:C_0402_1005Metric, B.Cu at (173.7, 137.3)
- added D10: B0540W, Diode_SMD:D_SOD-323, F.Cu at (196.4, 145.6)
- added D11: B0540W, Diode_SMD:D_SOD-323, F.Cu at (178.6, 139.2)
- added D3: B0540W, Diode_SMD:D_SOD-323, F.Cu at (168.8, 137.4)
- added D5: B0540W, Diode_SMD:D_SOD-323, F.Cu at (183.0, 130.4)
- added D6: B0540W, Diode_SMD:D_SOD-323, F.Cu at (171.4, 145.4)
- added D7: B0540W, Diode_SMD:D_SOD-323, F.Cu at (179.6, 133.8)
- added D8: B0540W, Diode_SMD:D_SOD-323, F.Cu at (198.4, 134.4)
- added D9: B0540W, Diode_SMD:D_SOD-323, F.Cu at (188.8, 146.2)
- added J1: ~, footprints:Hirose_FH12-20S-0.5SH_1x20-1MP_P0.50mm_Horizontal_Reversed, F.Cu at (165.0, 88.4)
- added L10: 4.7uH, footprints:L_1212, F.Cu at (182.6, 134.0)
- added L11: 4.7uH, footprints:L_1212, F.Cu at (168.6, 141.0)
- added L12: 4.7uH, footprints:L_1212, F.Cu at (187.4, 131.0)
- added L13: 4.7uH, footprints:L_1212, F.Cu at (194.6, 133.0)
- added L14: 4.7uH, footprints:L_1212, F.Cu at (188.8, 142.6)
- added L15: 4.7uH, footprints:L_1212, F.Cu at (193.4, 142.6)
- added L16: 4.7uH, footprints:L_1212, F.Cu at (179.2, 142.8)
- added R38: DNP, Resistor_SMD:R_0402_1005Metric, B.Cu at (174.0, 144.8)
- added R39: DNP, Resistor_SMD:R_0402_1005Metric, B.Cu at (183.2, 136.2)
- added R40: DNP, Resistor_SMD:R_0402_1005Metric, B.Cu at (173.0, 144.8)
- added R41: DNP, Resistor_SMD:R_0402_1005Metric, B.Cu at (183.2, 135.2)
- added R42: 27K, Resistor_SMD:R_0402_1005Metric, B.Cu at (175.0, 144.8)
- added R43: 22K, Resistor_SMD:R_0402_1005Metric, B.Cu at (176.0, 137.5)
- added R44: 30K, Resistor_SMD:R_0402_1005Metric, B.Cu at (183.2, 138.2)
- added R45: 22K, Resistor_SMD:R_0402_1005Metric, B.Cu at (189.4, 136.8)
- added R46: 510K, Resistor_SMD:R_0402_1005Metric, B.Cu at (176.0, 144.8)
- added R47: 270K, Resistor_SMD:R_0402_1005Metric, B.Cu at (177.0, 137.5)
- added R48: 270K, Resistor_SMD:R_0402_1005Metric, B.Cu at (183.2, 137.2)
- added R49: 270K, Resistor_SMD:R_0402_1005Metric, B.Cu at (189.4, 138.8)
- added R50: 100, Resistor_SMD:R_0402_1005Metric, F.Cu at (191.0, 137.2)
- added R51: 100, Resistor_SMD:R_0402_1005Metric, F.Cu at (181.4, 139.6)
- added R52: 82K, Resistor_SMD:R_0402_1005Metric, B.Cu at (196.4, 142.4)
- added R53: 270K, Resistor_SMD:R_0402_1005Metric, B.Cu at (194.4, 142.4)
- added R54: 22K, Resistor_SMD:R_0402_1005Metric, B.Cu at (180.2, 143.0)
- added R55: 270K, Resistor_SMD:R_0402_1005Metric, B.Cu at (180.2, 141.0)
- added R56: 680K, Resistor_SMD:R_0402_1005Metric, B.Cu at (198.6, 137.2)
- added R57: 220K, Resistor_SMD:R_0402_1005Metric, B.Cu at (198.6, 139.2)
- added R58: 270K, Resistor_SMD:R_0402_1005Metric, B.Cu at (185.4, 145.8)
- added R59: 22K, Resistor_SMD:R_0402_1005Metric, B.Cu at (183.6, 145.8)
- added R60: 510K, Resistor_SMD:R_0402_1005Metric, F.Cu at (160.1, 134.3)
- added R61: 220K, Resistor_SMD:R_0402_1005Metric, F.Cu at (158.1, 134.3)
- added R62: 30K, Resistor_SMD:R_0402_1005Metric, F.Cu at (156.4, 86.5)
- added R63: 36K, Resistor_SMD:R_0402_1005Metric, F.Cu at (153.8, 86.5)
- added R64: 10K, Resistor_SMD:R_0402_1005Metric, F.Cu at (152.8, 86.5)
- added R65: 10K, Resistor_SMD:R_0402_1005Metric, B.Cu at (157.1, 143.9)
- added U13: TPS65130RGE, footprints:VQFN-24-1EP_4x4mm_P0.5mm_EP2.45x2.45mm_0.3ThermalVias, F.Cu at (194.4, 137.8)
- added U14: TPS65130RGE, footprints:VQFN-24-1EP_4x4mm_P0.5mm_EP2.45x2.45mm_0.3ThermalVias, F.Cu at (184.0, 143.2)
- added U15: SY8120, Package_TO_SOT_SMD:TSOT-23-6, F.Cu at (164.0, 135.8)
- BZ1: footprint Connector_PinHeader_2.54mm:PinHeader_1x02_P2.54mm_Vertical -> Buzzer_Beeper:Buzzer_12x9.5RM7.6
- C2: value 10uF -> 47uF; footprint Capacitor_SMD:C_0603_1608Metric -> Capacitor_SMD:C_0805_2012Metric; moved to B.Cu
- C21: value 4.7uF -> 100nF
- C25: value 1uF -> 4.7uF
- C26: value 18pF -> 2.2uF
- C27: value 18pF -> 47nF; moved to B.Cu
- C28: value 18pF -> 47nF; moved to F.Cu
- C29: value 18pF -> 47nF
- C30: value 1uF -> 47nF
- C31, C33, C99, R4: moved to B.Cu
- C32, C34: value 4.7uF -> 47uF; footprint Capacitor_SMD:C_0603_1608Metric -> Capacitor_SMD:C_0805_2012Metric
- C35, C36: value 4.7uF -> 47uF; footprint Capacitor_SMD:C_0603_1608Metric -> Capacitor_SMD:C_0805_2012Metric; moved to F.Cu
- C37: value 220nF -> 2.2uF; moved to F.Cu
- C38: value 470nF -> 2.2uF
- C39, C41: value 220nF -> 10uF 25V; footprint Capacitor_SMD:C_0402_1005Metric -> Capacitor_SMD:C_0805_2012Metric; moved to F.Cu
- C4, C6: value 2.2uF -> 4.7uF
- C40, C55: value 100nF -> 10uF 25V; footprint Capacitor_SMD:C_0402_1005Metric -> Capacitor_SMD:C_0805_2012Metric; moved to F.Cu
- C42: value 47uF -> 10uF 25V; footprint Capacitor_SMD:C_0603_1608Metric -> Capacitor_SMD:C_0805_2012Metric
- C43, C44, C76: value 100nF -> 220nF; moved to F.Cu
- C45: value 4.7uF -> 220nF; footprint Capacitor_SMD:C_0603_1608Metric -> Capacitor_SMD:C_0402_1005Metric; moved to F.Cu
- C46, C49: value 220nF -> 4.7nF; moved to F.Cu
- C47: value 4.7uF -> 10nF; footprint Capacitor_SMD:C_0603_1608Metric -> Capacitor_SMD:C_0402_1005Metric; moved to F.Cu
- C48: value 4.7uF -> 220nF; footprint Capacitor_SMD:C_0603_1608Metric -> Capacitor_SMD:C_0402_1005Metric
- C50: value 220nF -> 10nF; moved to F.Cu
- C51, C52: value 100nF -> 22pF
- C53, C54: value 220nF -> DNP
- C56: value 220nF -> 10uF; footprint Capacitor_SMD:C_0402_1005Metric -> Capacitor_SMD:C_0603_1608Metric; moved to F.Cu
- C57: value 220nF -> 10uF 25V; footprint Capacitor_SMD:C_0402_1005Metric -> Capacitor_SMD:C_0805_2012Metric
- C58, C73: value 100nF -> 10uF; footprint Capacitor_SMD:C_0402_1005Metric -> Capacitor_SMD:C_0603_1608Metric; moved to F.Cu
- C59, C60: value 220nF -> 100nF; moved to F.Cu
- C61: value 4.7uF -> 22pF; footprint Capacitor_SMD:C_0603_1608Metric -> Capacitor_SMD:C_0402_1005Metric
- C62: value 220nF -> 47uF; footprint Capacitor_SMD:C_0402_1005Metric -> Capacitor_SMD:C_0805_2012Metric; moved to F.Cu
- C63: value 1uF -> 18pF
- C64: value 220nF -> 18pF; moved to F.Cu
- C65: value 470nF -> 18pF; moved to F.Cu
- C66: value 4.7uF -> 18pF; footprint Capacitor_SMD:C_0603_1608Metric -> Capacitor_SMD:C_0402_1005Metric
- C67, C75: moved to F.Cu
- C68: value 10uF -> 100nF; footprint Capacitor_SMD:C_0603_1608Metric -> Capacitor_SMD:C_0402_1005Metric; moved to F.Cu
- C69: value 22uF -> 47uF; footprint Capacitor_SMD:C_0603_1608Metric -> Capacitor_SMD:C_0805_2012Metric
- C70: value 4.7uF -> 47uF; footprint Capacitor_SMD:C_0402_1005Metric -> Capacitor_SMD:C_0805_2012Metric
- C71, C72: value 100nF -> 47uF; footprint Capacitor_SMD:C_0402_1005Metric -> Capacitor_SMD:C_0805_2012Metric
- C77: value 100nF -> 18pF; moved to F.Cu
- C81: value 470nF -> 22uF; footprint Capacitor_SMD:C_0402_1005Metric -> Capacitor_SMD:C_0603_1608Metric
- C89: value 1uF 25V -> 10uF 25V; footprint Capacitor_SMD:C_0603_1608Metric -> Capacitor_SMD:C_0805_2012Metric
- C91: value 10uF -> 22uF
- C92: value 10uF -> 100nF; footprint Capacitor_SMD:C_0603_1608Metric -> Capacitor_SMD:C_0402_1005Metric; moved to B.Cu
- C93: value 100nF -> 22uF; footprint Capacitor_SMD:C_0402_1005Metric -> Capacitor_SMD:C_0603_1608Metric; moved to B.Cu
- J2: value 02x04_P2.0 -> 0.5mm Bottom Contact; footprint Connector_PinHeader_2.00mm:PinHeader_2x04_P2.00mm_Vertical_SMD -> Connector_FFC-FPC:Hirose_FH12-30S-0.5SH_1x30-1MP_P0.50mm_Horizontal
- J4: value USB_C_Receptacle_USB2.0 -> 2.54mm pitch; footprint Connector_USB:USB_C_Receptacle_HRO_TYPE-C-31-M-12 -> Connector_PinSocket_2.54mm:PinSocket_1x02_P2.54mm_Vertical
- J5: value FPC 0.5mm Bottom Contact -> 0.5mm Bottom Contact
- J6: value ~ -> 2.54mm pitch; footprint footprints:Hirose_FH12-45S-0.5SH_1x45-1MP_P0.50mm_Horizontal_Reversed -> Connector_PinSocket_2.54mm:PinSocket_1x02_P2.54mm_Vertical
- J7: value FFC 0.5mm Bottom Contact -> 0.5mm Bottom Contact
- L4: value FTC201610S4R7MBCA -> 4.7uH; footprint Inductor_SMD:L_Murata_DFE201610P -> footprints:L_1212
- L6: value EXC14CE900U -> FTC201610S4R7MBCA; footprint footprints:L_CommonModeChoke_Panasonic_EXC14CE -> Inductor_SMD:L_Murata_DFE201610P
- L7: value 120R -> FTC201610S4R7MBCA; footprint Inductor_SMD:L_0603_1608Metric -> Inductor_SMD:L_Murata_DFE201610P
- R11: value 36K -> 10K
- R12, R13, R7: value 10K -> 12K
- R14: value 10K -> 22R; moved to B.Cu
- R15: value 10K -> DNP; moved to B.Cu
- R16: value 36K -> DNP
- R18: value 100K -> 10K
- R19, R20: value 5.1K 1% -> 5.1K
- R22: value 49.9K 1% -> 30K
- R26: value 5.1K 1% -> 22R; moved to B.Cu
- R27: value 5.1K 1% -> 10K; moved to B.Cu
- R29: value 49.9K/1% -> 1.5K; moved to B.Cu
- R30: value 49.9K/1% -> 10K
- R33: value 200K/1% -> 220K
- R34: value 27K/1% -> 30K
- R36: value 10K -> 30K
- R9: value 10K -> 12K; moved to F.Cu
- U10: value SY8120 -> MT9700; footprint Package_TO_SOT_SMD:TSOT-23-6 -> Package_TO_SOT_SMD:SOT-23-5; moved to B.Cu
- U2: value IMXRT1050 -> ADP5071ACPZ; footprint footprints:BGA-196_14x14_12.0x12.0mm -> Package_CSP:LFCSP-20-1EP_4x4mm_P0.5mm_EP2.6x2.6mm_ThermalVias
- U3: value MT48LC16M16A2BG -> ADP5071ACPZ; footprint footprints:BGA-54_9x9_8.0x8.0mm -> Package_CSP:LFCSP-20-1EP_4x4mm_P0.5mm_EP2.6x2.6mm_ThermalVias
- U4: value W25Q32JV -> STM32F103C8Tx; footprint Package_SON:WSON-8-1EP_6x5mm_P1.27mm_EP3.4x4.3mm -> Package_QFP:LQFP-48_7x7mm_P0.5mm
- U5: value STM32G030F6Px -> FODM3023; footprint Package_SO:TSSOP-20_4.4x6.5mm_P0.65mm -> Package_DIP:SMDIP-4_W7.62mm
- U7: value FODM3023 -> USBLC6-2P6; footprint Package_DIP:SMDIP-4_W7.62mm -> Package_TO_SOT_SMD:SOT-666; moved to B.Cu
- U8: value USBLC6-2P6 -> SY8120; footprint Package_TO_SOT_SMD:SOT-666 -> Package_TO_SOT_SMD:TSOT-23-6
- Y1: value 24MHz -> 8MHz
- moved R18 75.3 mm to (130.0, 101.3), turned to 0 degrees
- moved Y2 73.5 mm to (130.0, 104.7), turned to 90 degrees
- moved U4 73.5 mm to (136.2, 100.7), turned to 90 degrees
- moved C66 70.9 mm to (130.0, 102.3), turned to 0 degrees
- moved C63 70.9 mm to (131.4, 108.5)
- moved Y1 69.9 mm to (134.0, 107.7), turned to 0 degrees
- moved C65 69.7 mm to (130.0, 107.1), turned to 0 degrees
- moved R13 67.8 mm to (187.4, 139.4), turned to 180 degrees
- moved C64 65.1 mm to (136.6, 107.3), turned to -90 degrees
- moved J6 62.2 mm to (174.9, 149.6), turned to 90 degrees
- moved C77 61.7 mm to (154.8, 86.5), turned to -90 degrees
- moved C67 61.4 mm to (137.6, 107.3), turned to -90 degrees
- moved R15 61.4 mm to (177.6, 141.2)
- moved C68 60.7 mm to (141.9, 99.4), turned to -90 degrees
- moved C2 58.5 mm to (189.9, 133.9)
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Connections:
- C104 pad 2: IPSOUT -> Net-(U10-VOUT)
- C2 pad 1: VBUS -> +CCDPWR
- C26 pad 1: Net-(U2E-XTALI) -> GND
- C26 pad 2: GND -> Net-(U3-VREG)
- C27 pad 1: Net-(U2E-XTALO) -> GND
- C27 pad 2: GND -> Net-(C27-Pad2)
- C28 pad 2: Net-(U2E-RTC_XTALI) -> Net-(C28-Pad2)
- C29 pad 2: Net-(U2E-RTC_XTALO) -> Net-(C29-Pad2)
- C30 pad 1: +1V0 -> GND
- C30 pad 2: GND -> Net-(C30-Pad2)
- C32 pad 1: /cpu/VDDA_2P5_CAP -> +CCDPWR
- C34 pad 1: +3V3 -> +CCDPWR
- C35 pad 1: +1V8 -> +CCDPWR
- C36 pad 1: +3V3 -> +CCDPWR
- C37 pad 1: /cpu/VDDA_2P5_CAP -> GND
- C37 pad 2: GND -> Net-(U2-VREF)
- C38 pad 1: +1V0 -> GND
- C38 pad 2: GND -> Net-(U3-VREF)
- C39 pad 1: /cpu/VDDA_1P1_CAP -> -9VD
- C40 pad 1: +3V3 -> +16VA
- C41 pad 1: +3V3 -> -9VA
- C42 pad 1: +1V0 -> +8VD
- C43 pad 1: +1V8 -> Net-(U13-PSN)
- C44 pad 1: +3V3 -> Net-(U14-PSN)
- C45 pad 1: +3V3 -> Net-(U13-VREF)
- C46 pad 1: +1V0 -> Net-(U13-CN)
- C47 pad 1: /cpu/VDDA_1P1_CAP -> Net-(U13-CP)
- C48 pad 1: +3V3 -> Net-(U14-VREF)
- C49 pad 1: +3V3 -> Net-(U14-CN)
- C50 pad 1: +1V0 -> Net-(U14-CP)
- C51 pad 1: +1V8 -> +5VD
- C51 pad 2: GND -> Net-(U13-FBP)
- C52 pad 1: +3V3 -> +16VD
- C52 pad 2: GND -> Net-(U14-FBP)
- C53 pad 1: +3V3 -> Net-(U13-FBN)
- C53 pad 2: GND -> -4VD
- C54 pad 1: +1V0 -> Net-(U14-FBN)
- C54 pad 2: GND -> -15VD
- C55 pad 1: +VCCIO_SD -> +5VD
- C56 pad 1: Net-(U2F-VDDA_ADC_3P3) -> -4VD
- C57 pad 1: +3V3 -> +16VD
- C58 pad 1: +3V3 -> -15VD
- C59 pad 1: Net-(U2F-VDD_SNVS_CAP) -> GND
- C59 pad 2: GND -> +CCDPWR
- C60 pad 1: +1V0 -> Net-(U15-SW)
- C60 pad 2: GND -> Net-(U15-BS)
- C61 pad 1: +VCCIO_SD -> +2VD
- C61 pad 2: GND -> Net-(U15-FB)
- C62 pad 1: Net-(U2F-DCDC_PSWITCH) -> +2VD
- C63 pad 1: Net-(U2F-VDDA_ADC_3P3) -> Net-(U4-PD0)
- C64 pad 1: +RTC -> Net-(U4-PD1)
- C65 pad 1: +1V0 -> GND
- C65 pad 2: GND -> Net-(U4-PC14)
- C66 pad 1: +1V0 -> GND
- C66 pad 2: GND -> Net-(U4-PC15)
- C67 pad 1: Net-(U2F-VDD_USB_CAP) -> +3V3
- C68 pad 1: Net-(U2F-VDD_USB_CAP) -> +3V3
- C69 pad 1: +1V8 -> +CCDPWR
- C70 pad 1: +1V8 -> +CCDPWR
- C71 pad 1: +1V8 -> +CCDPWR
- C72 pad 1: +1V8 -> +CCDPWR
- C73 pad 1: +1V8 -> +3V3
- C74 pad 1: +1V8 -> GND
- C74 pad 2: GND -> +3V3
- C75 pad 1: +1V8 -> Net-(U8-SW)
- C75 pad 2: GND -> Net-(U8-BS)
- C76 pad 1: +1V8 -> GND
- C76 pad 2: GND -> Net-(C76-Pad2)
- C77 pad 1: +1V8 -> Net-(U8-FB)
- C77 pad 2: GND -> +FAN
- C81 pad 2: +3V3 -> +FAN
- C91 pad 1: +3V3 -> +FAN
- C92 pad 1: VBUS -> +RTC
- C93 pad 1: GND -> Net-(U10-VOUT)
- C93 pad 2: +3V3 -> GND
- J2 pad 1: +CCDPWR -> -15VD
- J2 pad 3: +CCDPWR -> +2VD
- J2 pad 5: +CCDPWR -> +16VD
- J2 pad 7: +CCDPWR -> -4VD
- J2 pad 8: GND -> -4VD
- J3 pad A6: unconnected-(J3-D+-PadA6) -> USB_DP
- J3 pad A7: unconnected-(J3-D--PadA7) -> USB_DN
- J3 pad A8: CPU_SWDIO -> MCU_SWDIO
- J3 pad B6: unconnected-(J3-D+-PadB6) -> USB_DP
- J3 pad B7: unconnected-(J3-D--PadB7) -> USB_DN
- J3 pad B8: CPU_SWCLK -> MCU_SWCLK
- J5 pad 10: CSI_D10 -> I2C_SCL
- J5 pad 11: CSI_D11 -> PS_POR_B
- J5 pad 12: CSI_D12 -> FPGA_TMS
- J5 pad 13: CSI_D13 -> FPGA_TDO
- J5 pad 14: CSI_D14 -> FPGA_TDI
- J5 pad 15: CSI_D15 -> FPGA_TCK
- J5 pad 16: GND -> SDIO_DAT3
- J5 pad 17: CSI_PIXCLK -> SDIO_DAT2
- J5 pad 18: CSI_VSYNC -> SDIO_DAT1
- J5 pad 19: CSI_HSYNC -> SDIO_DAT0
- J5 pad 2: CSI_D2 -> MIPI_D1P
- J5 pad 20: GND -> SDIO_CMD
- J5 pad 21: AFE_SL -> SDIO_CLK
- J5 pad 22: AFE_SDATA -> GND
- J5 pad 23: AFE_SCK -> +3V3
- J5 pad 24: AFE_RST -> +3V3
- J5 pad 25: AFE_SYNC -> GND
- J5 pad 26: I2C_SCL -> EXTEN
- J5 pad 27: I2C_SDA -> IPSOUT
- J5 pad 28: GND -> IPSOUT
- J5 pad 29: +3.3VA -> GND
- J5 pad 3: CSI_D3 -> MIPI_D1N
- J5 pad 30: +3.3VA -> +1V8
- J5 pad 4: CSI_D4 -> MIPI_D0P
- J5 pad 5: CSI_D5 -> MIPI_D0N
- J5 pad 6: CSI_D6 -> MIPI_CKP
- J5 pad 7: CSI_D7 -> MIPI_CKN
- J5 pad 8: CSI_D8 -> GND
- J5 pad 9: CSI_D9 -> I2C_SDA
- J6 pad 1: unconnected-(J6-XR-Pad1) -> +FAN
- J6 pad 2: unconnected-(J6-YD-Pad2) -> GND
- J7 pad 1: GRIP_IO0 -> GRIP_SCK
- J7 pad 2: GRIP_IO1 -> GRIP_MOSI
- J7 pad 3: GRIP_IO2 -> GRIP_CS
- J7 pad 4: GRIP_IO3 -> GRIP_MISO
- L4 pad 1: +1V0 -> Net-(D6-A)
- L4 pad 2: Net-(L4-Pad2) -> Net-(U2-INBK)
- L6 pad 1: /usb/USB1_DN -> Net-(U8-SW)
- L6 pad 2: /usb/USB1_DP -> +FAN
- L7 pad 1: VBUS -> Net-(U15-SW)
- L7 pad 2: Net-(U8-VBUS) -> +2VD
- L9 pad 1: IPSOUT -> Net-(U10-VOUT)
- MICRO_SD1 pad 1: SD1_DATA2 -> SDIO_DAT2
- MICRO_SD1 pad 2: SD1_DATA3 -> SDIO_DAT3
- MICRO_SD1 pad 3: SD1_CMD -> SDIO_CMD
- MICRO_SD1 pad 7: SD1_DATA0 -> SDIO_DAT0
- MICRO_SD1 pad 8: SD1_DATA1 -> SDIO_DAT1
- R11 pad 1: Net-(U10-FB) -> +CCDPWR
- R11 pad 2: +FAN -> CCD_POWEREN
- R12 pad 1: GND -> Net-(U2-COMP2)
- R12 pad 2: /cpu/BOOTMODE0 -> Net-(C29-Pad2)
- R13 pad 1: +3V3 -> Net-(U3-COMP2)
- R13 pad 2: I2C_SDA -> Net-(C30-Pad2)
- R14 pad 1: GND -> USB_DN
- R14 pad 2: Net-(U10-FB) -> Net-(U4-PA11)
- R15 pad 1: +3V3 -> Net-(U2-SS)
- R15 pad 2: I2C_SCL -> GND
- R16 pad 1: +3V3 -> Net-(U3-SS)
- R16 pad 2: Net-(U2F-DCDC_PSWITCH) -> GND
- R17 pad 2: SD1_CLK -> SDIO_CLK
- R18 pad 1: +3V3 -> GND
- R18 pad 2: QSPI_SS0 -> /mcu/BOOT0
- R26 pad 1: Net-(J4-CC1) -> USB_DP
- R26 pad 2: GND -> Net-(U4-PA12)
- R27 pad 1: Net-(J4-CC2) -> GND
- R27 pad 2: GND -> LENS_PWR_EN
- R29 pad 1: Net-(C97-Pad2) -> +3V3
- R29 pad 2: FAN_PWM -> USB_DP
- R30 pad 1: Net-(U10-FB) -> GND
- R30 pad 2: Net-(C97-Pad2) -> FAN_EN
- R35 pad 1: /mcu/LED -> /mcu/LED_R
- R36 pad 1: GND -> Net-(C76-Pad2)
- R36 pad 2: FAN_EN -> FAN_PWM
- R37 pad 2: Net-(U5-PA7) -> /mcu/BEEPER
- R7 pad 1: /cpu/JTAG_MOD -> Net-(U2-COMP1)
- R7 pad 2: GND -> Net-(C27-Pad2)
- R8 pad 1: /mcu/FLASH_SYNC -> FLASH_SYNC
- R9 pad 1: GND -> Net-(U3-COMP1)
- R9 pad 2: /cpu/BOOTMODE1 -> Net-(C28-Pad2)
- U1 pad 31: VBUS -> unconnected-(U1-VBUS-Pad31)
- U10 pad 1: Net-(U10-BS) -> Net-(U10-VOUT)
- U10 pad 3: Net-(U10-FB) -> Net-(U10-SET)
- U10 pad 4: FAN_EN -> LENS_PWR_EN
- U10 pad 5: +3V3 -> IPSOUT
- U12 pad 4: IPSOUT -> Net-(U10-VOUT)
- U12 pad 5: IPSOUT -> Net-(U10-VOUT)
- U4 pad 1: QSPI_SS0 -> +RTC
- U4 pad 2: QSPI_DATA1 -> FLASH_SYNC
- U4 pad 3: QSPI_DATA2 -> Net-(U4-PC14)
- U4 pad 4: GND -> Net-(U4-PC15)
- U4 pad 5: QSPI_DATA0 -> Net-(U4-PD0)
- U4 pad 6: QSPI_SCLK -> Net-(U4-PD1)
- U4 pad 7: QSPI_DATA3 -> PWROK
- U4 pad 8: +3V3 -> GND
- U4 pad 9: GND -> +3V3
- U5 pad 1: DCDC_EN -> Net-(R8-Pad2)
- U5 pad 2: FAN_EN -> GND
- U5 pad 3: /mcu/LED -> FLASH_SYNC_T
- U5 pad 4: +3V3 -> FLASH_SYNC_S
- U7 pad 1: Net-(R8-Pad2) -> USB_DP
- U7 pad 3: FLASH_SYNC_T -> USB_DN
- U7 pad 4: FLASH_SYNC_S -> USB_DN
- U8 pad 1: /usb/USB1_DN -> Net-(U8-BS)
- U8 pad 3: /usb/USB1_DP -> Net-(U8-FB)
- U8 pad 4: /usb/USB1_DP -> FAN_EN
- U8 pad 5: Net-(U8-VBUS) -> +3V3
- U8 pad 6: /usb/USB1_DN -> Net-(U8-SW)
- Y1 pad 1: Net-(U2E-XTALI) -> Net-(U4-PD0)
- Y1 pad 3: Net-(U2E-XTALO) -> Net-(U4-PD1)
- Y2 pad 1: Net-(U2E-RTC_XTALI) -> Net-(U4-PC14)
- Y2 pad 2: Net-(U2E-RTC_XTALO) -> Net-(U4-PC15)
Routing:
- net VBUS: track 148.3 -> 0.00 mm, vias 3 -> 0
- net I2C_SDA: track 211.8 -> 77.0 mm, vias 4 -> 3
- net I2C_SCL: track 210.7 -> 78.1 mm, vias 4 -> 3
- net +RTC: track 156.2 -> 34.5 mm, vias 3 -> 2
- net CPU_SWCLK: track 121.4 -> 0.00 mm, vias 2 -> 0
- net PWROK: track 151.3 -> 32.9 mm, vias 3 -> 2
- net CPU_SWDIO: track 115.5 -> 0.00 mm, vias 2 -> 0
- net +VCCIO_SD: track 116.5 -> 1.61 mm, vias 6 -> 1
- net +FAN: track 67.6 -> 181.7 mm, vias 4 -> 2
- net SDIO_DAT2: track 0.00 -> 104.8 mm, vias 0 -> 2
- net SDIO_DAT3: track 0.00 -> 103.9 mm, vias 0 -> 2
- net SDIO_CMD: track 0.00 -> 102.6 mm, vias 0 -> 2
- net SDIO_DAT0: track 0.00 -> 97.7 mm, vias 0 -> 2
- net SDIO_DAT1: track 0.00 -> 95.7 mm, vias 0 -> 2
- net USB_DN: track 111.1 -> 16.3 mm, vias 4 -> 2
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- added copper zone on In1.Cu, net +CCDPWR
- removed copper zone on In1.Cu, net +1V0
- removed copper zone on In1.Cu, net +1V8
Other:
- board text added: "IOB R0.9"
- board text removed: "2024 Wenting"
- board text removed: "MB R0.8"

Commit message: Revise board design to fit enclosure
Parts:
- BZ1: footprint Buzzer_Beeper:Buzzer_12x9.5RM7.6 -> Buzzer_Beeper:Buzzer_Murata_PKMCS0909E
- moved BZ1 4.50 mm to (154.0, 140.7), turned to -90 degrees
- moved J7 0.35 mm to (185.8, 90.2)
- moved D5 0.20 mm to (183.0, 130.6)
- moved U11 0.10 mm to (173.8, 134.3)
- moved C39 0.10 mm to (179.4, 130.5)
Routing:
- net Net-(BZ1-+): track 9.36 -> 2.71 mm
- net GND: track 231.3 -> 232.9 mm
- net GRIP_MISO: track 56.6 -> 57.2 mm
- net GRIP_SCK: track 57.7 -> 58.2 mm
