File: Hardware/gripflex/gripflex.kicad_sch (KiCad schematic)
At the start: 21 parts, among them J1 Conn_01x10_MountingPin, J2 Conn_01x12, J3 Conn_01x02_MountingPin, U2 74HC165, U3 74HC165

Commit message: Hardware r0.9
Other:
- company: (none) -> Copyright 2024 Wenting Zhang
- title: (none) -> Sitina 1 Grip Flex
Changed lines of the file:
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@@
 	(generator_version "8.0")
 	(paper "A4")
+	(title_block
+		(title "Sitina 1 Grip Flex")
+		(date "2024-03-25")
+		(rev "R0.9")
+		(company "Copyright 2024 Wenting Zhang")
+	)
 	(junction
 		(at 60.96 162.56)
