File: hardware/ioboard/lcd.kicad_sch (KiCad schematic)
At the start: 16 parts, among them U6 CAT4139

Commit message: PCB changes for r0p10
Parts:
- L5: footprint footprints:L_1212 -> Inductor_SMD:L_Changjiang_FNR3015S
- R23: value 10K -> 5.1K
Changed lines of the file:
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@@
 			)
 		)
-		(property "Footprint" "footprints:L_1212"
+		(property "Footprint" "Inductor_SMD:L_Changjiang_FNR3015S"
 			(at 116.84 88.9 0)
 			(effects
@@
 			)
 		)
-		(property "Value" "10K"
+		(property "Value" "5.1K"
 			(at 131.318 114.173 0)
 			(effects

Commit message: PCB r0p10 release
Other:
- company: Copyright 2024 Wenting Zhang, Anhang Li -> Copyright 2024 Anhang Li, Wenting Zhang
- title: Sitina 1 IO Board -> LCD Power Supply and Connector
Changed lines of the file:
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@@
 	(paper "A4")
 	(title_block
-		(title "Sitina 1 IO Board")
-		(date "2024-03-08")
-		(rev "R0.9")
-		(company "Copyright 2024 Wenting Zhang, Anhang Li")
+		(title "LCD Power Supply and Connector")
+		(date "2024-06-09")
+		(rev "R0.10")
+		(company "Copyright 2024 Anhang Li, Wenting Zhang")
 		(comment 2 "MERCHANTABILITY, SATISFACTORY QUALITY AND FITNESS FOR A PARTICULAR PURPOSE.")
 		(comment 3 "This source is distributed WITHOUT ANY EXPRESS OR IMPLIED WARRANTY, INCLUDING OF")
