File: hardware/ioboard/storage.kicad_sch (KiCad schematic)
At the start: 5 parts

Commit message: PCB r0p10 release
Other:
- company: Copyright 2024 Wenting Zhang, Anhang Li -> Copyright 2024 Anhang Li, Wenting Zhang
- title: Sitina 1 IO Board -> Storage
Changed lines of the file:
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@@
 	(paper "A4")
 	(title_block
-		(title "Sitina 1 IO Board")
-		(date "2024-03-08")
-		(rev "R0.9")
-		(company "Copyright 2024 Wenting Zhang, Anhang Li")
+		(title "Storage")
+		(date "2024-06-09")
+		(rev "R0.10")
+		(company "Copyright 2024 Anhang Li, Wenting Zhang")
 		(comment 2 "MERCHANTABILITY, SATISFACTORY QUALITY AND FITNESS FOR A PARTICULAR PURPOSE.")
 		(comment 3 "This source is distributed WITHOUT ANY EXPRESS OR IMPLIED WARRANTY, INCLUDING OF")
