File: hardware/ioboard/pcb.kicad_pcb (KiCad board)
At the start: 4 copper layers, 71.6 x 73.2 mm, 240 parts, among them J10 2.54mm pitch, J11 2.54mm pitch, J12 LensMount, J13 LensMount, J14 LensMount, J15 LensMount, J16 LensMount, J17 LensMount, J18 LensMount, J19 LensMount, J2 0.5mm Bottom Contact, J20 LensMount, J21 LensMount, J3 USB_C_Receptacle_USB2.0, J4 2.54mm pitch, J5 0.5mm Bottom Contact, J6 2.54mm pitch, J7 0.5mm Bottom Contact, J8 AudioJack2, SW1 SW_Push_LED, U1 AXP209, U10 MT9700, U11 MT9700, U12 SY7208, U13 TPS65130RGE, U14 TPS65130RGE, U15 SY8120, U2 ADP5071ACPZ, U3 ADP5071ACPZ, U4 STM32F103C8Tx, U5 FODM3023, U6 CAT4139, U7 USBLC6-2P6, U8 SY8120, U9 MT9700, Y1 8MHz, Y2 32.768K

Commit message: PCB changes for r0p10
Parts:
- removed C100, C101, C108, C81, C91: 22uF, Capacitor_SMD:C_0603_1608Metric
- removed C31, C67, C68, C74, C75: 100nF, Capacitor_SMD:C_0402_1005Metric
- removed C63, C64, C77: 18pF, Capacitor_SMD:C_0402_1005Metric
- removed C73: 10uF, Capacitor_SMD:C_0603_1608Metric
- removed C76: 220nF, Capacitor_SMD:C_0402_1005Metric
- removed J10, J11, J4, J6: 2.54mm pitch, Connector_PinSocket_2.54mm:PinSocket_1x02_P2.54mm_Vertical
- removed L6: FTC201610S4R7MBCA, Inductor_SMD:L_Murata_DFE201610P
- removed R14, R26: 22R, Resistor_SMD:R_0402_1005Metric
- removed R29: 1.5K, Resistor_SMD:R_0402_1005Metric
- removed R30, R64: 10K, Resistor_SMD:R_0402_1005Metric
- removed R36, R62: 30K, Resistor_SMD:R_0402_1005Metric
- removed R63: 36K, Resistor_SMD:R_0402_1005Metric
- removed U8: SY8120, Package_TO_SOT_SMD:TSOT-23-6
- removed Y1: 8MHz, Oscillator:Oscillator_SMD_Abracon_ASE-4Pin_3.2x2.5mm
- added J9: Conn_02x06_Odd_Even, Connector_PinHeader_1.27mm:PinHeader_2x06_P1.27mm_Horizontal, F.Cu at (133.0, 108.2)
- C33, C92, R4: moved to F.Cu
- C43, C44, C45, C48, C5, C88: value 220nF -> 470nF
- C51, C52, C61: value 22pF -> 18pF
- D1: value B0530WS -> B0540WS
- D10, D11, D3, D4, D5, D6, D7, D8, D9: value B0540W -> B0540WS
- L10, L11, L12, L13, L14, L15, L16, L4: value 4.7uH -> YHNR3015-4R7M; footprint footprints:L_1212 -> Inductor_SMD:L_Changjiang_FNR3015S
- L5: value 22uH -> YHNR3015-220M; footprint footprints:L_1212 -> Inductor_SMD:L_Changjiang_FNR3015S
- R23: value 10K -> 5.1K
- R35: value 200R -> 10K
- U4: value STM32F103C8Tx -> STM32G030K6Tx; footprint Package_QFP:LQFP-48_7x7mm_P0.5mm -> Package_QFP:LQFP-32_7x7mm_P0.8mm
- U5: footprint Package_DIP:SMDIP-4_W7.62mm -> footprints:MFP4_3.85x4.4
- moved D2 16.4 mm to (135.0, 81.6)
- moved R35 15.3 mm to (136.4, 82.2), turned to 90 degrees
- moved R18 14.5 mm to (142.2, 93.4), turned to -90 degrees
- moved C65 9.97 mm to (130.8, 97.2)
- moved C15 9.02 mm to (150.2, 91.0)
- moved C14 9.02 mm to (148.9, 90.5)
- moved Y2 7.86 mm to (132.8, 97.4), turned to -90 degrees
- moved C92 6.63 mm to (132.8, 100.0), turned to 180 degrees
- moved L2 5.32 mm to (146.5, 90.2)
- moved C10 5.32 mm to (143.0, 84.5)
- moved C18 5.32 mm to (154.0, 89.0)
- moved C23 5.32 mm to (150.8, 80.4)
- moved C24 5.32 mm to (143.0, 85.5)
- moved C3 5.32 mm to (144.4, 80.1)
- moved C4 5.32 mm to (153.2, 80.2)
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Connections:
- C33 pad 1: +3V3 -> +RTC
- J2 pad 1: -15VD -> GND
- J2 pad 10: CCD_PULSE_SYNC -> +8VD
- J2 pad 11: GND -> +8VD
- J2 pad 12: -9VA -> +8VD
- J2 pad 13: +16VA -> GND
- J2 pad 14: +16VA -> GND
- J2 pad 15: +3.3VA -> GND
- J2 pad 16: GND -> +3.3VA
- J2 pad 17: GND -> +16VA
- J2 pad 18: GND -> +16VA
- J2 pad 19: +8VD -> -9VA
- J2 pad 2: GND -> +5VD
- J2 pad 20: +8VD -> GND
- J2 pad 21: +8VD -> CCD_PULSE_SYNC
- J2 pad 22: -9VD -> CCD_AFE_SYNC
- J2 pad 23: -9VD -> -4VD
- J2 pad 24: -9VD -> -4VD
- J2 pad 26: GND -> +16VD
- J2 pad 27: -4VD -> GND
- J2 pad 28: +5VD -> +2VD
- J2 pad 29: +5VD -> GND
- J2 pad 3: +2VD -> +5VD
- J2 pad 30: GND -> -15VD
- J2 pad 4: GND -> -4VD
- J2 pad 5: +16VD -> GND
- J2 pad 7: -4VD -> -9VD
- J2 pad 8: -4VD -> -9VD
- J2 pad 9: CCD_AFE_SYNC -> -9VD
- J3 pad A8: MCU_SWDIO -> unconnected-(J3-SBU1-PadA8)
- J3 pad B8: MCU_SWCLK -> unconnected-(J3-SBU2-PadB8)
- J5 pad 1: GND -> +1V8
- J5 pad 10: I2C_SCL -> SDIO_CLK
- J5 pad 11: PS_POR_B -> SDIO_CMD
- J5 pad 12: FPGA_TMS -> SDIO_DAT0
- J5 pad 13: FPGA_TDO -> SDIO_DAT1
- J5 pad 14: FPGA_TDI -> SDIO_DAT2
- J5 pad 15: FPGA_TCK -> SDIO_DAT3
- J5 pad 16: SDIO_DAT3 -> FPGA_TCK
- J5 pad 17: SDIO_DAT2 -> FPGA_TDI
- J5 pad 18: SDIO_DAT1 -> FPGA_TDO
- J5 pad 19: SDIO_DAT0 -> FPGA_TMS
- J5 pad 2: MIPI_D1P -> GND
- J5 pad 20: SDIO_CMD -> PS_POR_B
- J5 pad 21: SDIO_CLK -> I2C_SCL
- J5 pad 22: GND -> I2C_SDA
- J5 pad 23: +3V3 -> GND
- J5 pad 24: +3V3 -> MIPI_CKN
- J5 pad 25: GND -> MIPI_CKP
- J5 pad 26: EXTEN -> MIPI_D0N
- J5 pad 27: IPSOUT -> MIPI_D0P
- J5 pad 28: IPSOUT -> MIPI_D1N
- J5 pad 29: GND -> MIPI_D1P
- J5 pad 3: MIPI_D1N -> IPSOUT
- J5 pad 30: +1V8 -> GND
- J5 pad 4: MIPI_D0P -> IPSOUT
- J5 pad 5: MIPI_D0N -> EXTEN
- J5 pad 6: MIPI_CKP -> GND
- J5 pad 7: MIPI_CKN -> +3V3
- J5 pad 8: GND -> +3V3
- J5 pad 9: I2C_SDA -> GND
- R18 pad 2: /mcu/BOOT0 -> MCU_SWCLK
- U4 pad 1: +RTC -> FLASH_SYNC
- U4 pad 10: PS_POR_B -> LENS_RXD
- U4 pad 11: FAN_PWM -> GRIP_CS
- U4 pad 12: FAN_EN -> GRIP_SCK
- U4 pad 13: DCDC_EN -> GRIP_MISO
- U4 pad 14: /mcu/BEEPER -> GRIP_MOSI
- U4 pad 15: /mcu/LED_R -> BODY_VD_LENS
- U4 pad 16: /mcu/LED_G -> unconnected-(U4-PB1-Pad16)
- U4 pad 18: unconnected-(U4-PB0-Pad18) -> LENS_CS_BODY
- U4 pad 19: BODY_VD_LENS -> BODY_CS_LENS
- U4 pad 2: FLASH_SYNC -> Net-(U4-PC14)
- U4 pad 20: LENS_CS_BODY -> unconnected-(U4-PC6-Pad20)
- U4 pad 21: I2C_SCL -> unconnected-(U4-PA10/NC-Pad21)
- U4 pad 22: I2C_SDA -> I2C_SCL
- U4 pad 23: GND -> I2C_SDA
- U4 pad 24: +3V3 -> MCU_SWDIO
- U4 pad 25: GRIP_CS -> MCU_SWCLK
- U4 pad 26: GRIP_SCK -> unconnected-(U4-PA15-Pad26)
- U4 pad 27: GRIP_MISO -> /mcu/BEEPER
- U4 pad 28: GRIP_MOSI -> LCD_PWM
- U4 pad 29: LCD_PWM -> unconnected-(U4-PB5-Pad29)
- U4 pad 3: Net-(U4-PC14) -> Net-(U4-PC15)
- U4 pad 30: LENS_TXD -> PS_POR_B
- U4 pad 31: LENS_RXD -> DCDC_EN
- U4 pad 32: Net-(U4-PA11) -> /mcu/LED_R
- U4 pad 4: Net-(U4-PC15) -> +RTC
- U4 pad 5: Net-(U4-PD0) -> GND
- U4 pad 6: Net-(U4-PD1) -> PWROK
- U4 pad 7: PWROK -> LENS_DET
- U4 pad 8: GND -> LENS_PWR_EN
- U4 pad 9: +3V3 -> LENS_TXD
Routing:
- net +FAN: track 181.7 -> 0.00 mm, vias 2 -> 0
- net LENS_PWR_EN: track 99.8 -> 1.45 mm, vias 2 -> 0
- net LENS_DET: track 90.3 -> 0.00 mm, vias 1 -> 0
- net BODY_CS_LENS: track 87.9 -> 0.00 mm, vias 1 -> 0
- net LENS_TXD: track 84.7 -> 0.00 mm, vias 1 -> 0
- net LENS_RXD: track 80.8 -> 0.00 mm, vias 1 -> 0
- net IPSOUT: track 171.9 -> 91.8 mm, vias 16 -> 9
- net I2C_SCL: track 78.1 -> 0.00 mm, vias 3 -> 0
- net I2C_SDA: track 77.0 -> 0.00 mm, vias 3 -> 0
- net +1V8: track 74.9 -> 0.00 mm, vias 2 -> 0
- net FPGA_TMS: track 74.8 -> 0.00 mm, vias 2 -> 0
- net FPGA_TDO: track 73.4 -> 0.00 mm, vias 2 -> 0
- net FPGA_TDI: track 73.0 -> 0.00 mm, vias 2 -> 0
- net PS_POR_B: track 72.9 -> 0.00 mm, vias 2 -> 0
- net FPGA_TCK: track 72.0 -> 0.00 mm, vias 2 -> 0
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Other:
- outline, holes or cut-outs redrawn

Commit message: PCB r0.10
Parts:
- removed L11, L12: YHNR3015-4R7M, Inductor_SMD:L_Changjiang_FNR3015S
- removed R38, R39, R40, R41: DNP, Resistor_SMD:R_0402_1005Metric
- removed R42: 27K, Resistor_SMD:R_0402_1005Metric
- removed R43, R45: 22K, Resistor_SMD:R_0402_1005Metric
- removed R44: 30K, Resistor_SMD:R_0402_1005Metric
- removed R46: 510K, Resistor_SMD:R_0402_1005Metric
- removed R47, R48, R49: 270K, Resistor_SMD:R_0402_1005Metric
- added C31: 4.7nF, Capacitor_SMD:C_0402_1005Metric, F.Cu at (177.2, 145.2)
- added C63: 10uF 25V, Capacitor_SMD:C_0805_2012Metric, F.Cu at (180.0, 150.0)
- added C64: 10uF 25V, Capacitor_SMD:C_0805_2012Metric, F.Cu at (175.4, 134.5)
- added C67: 10uF 25V, Capacitor_SMD:C_0805_2012Metric, F.Cu at (172.6, 150.0)
- added C68: 47uF, Capacitor_SMD:C_0805_2012Metric, F.Cu at (153.6, 133.2)
- added C73: 47uF, Capacitor_SMD:C_0805_2012Metric, F.Cu at (150.1, 133.2)
- added C74: 47uF, Capacitor_SMD:C_0805_2012Metric, F.Cu at (150.1, 130.8)
- added C75: 47uF, Capacitor_SMD:C_0805_2012Metric, F.Cu at (150.4, 136.4)
- added C76: 47uF, Capacitor_SMD:C_0805_2012Metric, F.Cu at (139.6, 149.2)
- added C77: 47uF, Capacitor_SMD:C_0805_2012Metric, F.Cu at (137.4, 149.2)
- added C81: 47uF, Capacitor_SMD:C_0805_2012Metric, F.Cu at (135.2, 149.2)
- added C91: 47uF, Capacitor_SMD:C_0805_2012Metric, F.Cu at (197.2, 86.8)
- added L6: YHNR3015-4R7M, Inductor_SMD:L_Changjiang_FNR3015S, F.Cu at (173.0, 137.6)
- added L8: YHNR3015-4R7M, Inductor_SMD:L_Changjiang_FNR3015S, F.Cu at (182.2, 147.0)
- added R14: 30K, Resistor_SMD:R_0402_1005Metric, B.Cu at (174.8, 146.2)
- added R26: 22K, Resistor_SMD:R_0402_1005Metric, B.Cu at (185.4, 142.6)
- added R29: 200K, Resistor_SMD:R_0402_1005Metric, B.Cu at (178.0, 140.6)
- added R30: 36K, Resistor_SMD:R_0402_1005Metric, B.Cu at (178.0, 142.6)
- C2, C32, C34, C48, C69, C70, C71, C90, C93, C99, R27, R65, U10: moved to F.Cu
- C26: value 2.2uF -> 470nF
- C27: value 47nF -> 470nF; moved to F.Cu
- C28: value 47nF -> 4.7nF
- C29: value 47nF -> 10nF; moved to F.Cu
- C30: value 47nF -> 470nF
- C37: value 2.2uF -> 10nF
- C38: value 2.2uF -> 18pF
- C39: value 10uF 25V -> 18pF; footprint Capacitor_SMD:C_0805_2012Metric -> Capacitor_SMD:C_0402_1005Metric; moved to B.Cu
- C40, C41: value 10uF 25V -> DNP; footprint Capacitor_SMD:C_0805_2012Metric -> Capacitor_SMD:C_0402_1005Metric; moved to B.Cu
- C56, C58: value 10uF -> 10uF 25V; footprint Capacitor_SMD:C_0603_1608Metric -> Capacitor_SMD:C_0805_2012Metric
- C72: value 47uF -> 100nF; footprint Capacitor_SMD:C_0805_2012Metric -> Capacitor_SMD:C_0402_1005Metric; moved to F.Cu
- C8: value 2.2uF -> 470nF; moved to F.Cu
- J12, J13, J14, J15, J16, J17, J18, J19, J20, J21: footprint footprints:YTC1P-4520 -> footprints:YZP0652-15072-01
- R12: value 12K -> 30K
- R13: value 12K -> 200K; moved to B.Cu
- R15: value DNP -> 220K
- R16: value DNP -> 270K
- R7: value 12K -> 100; moved to F.Cu
- R9: value 12K -> 100
- U13, U14: value TPS65130RGE -> TPS65131RGE
- U2, U3: value ADP5071ACPZ -> TPS65131RGE; footprint Package_CSP:LFCSP-20-1EP_4x4mm_P0.5mm_EP2.6x2.6mm_ThermalVias -> footprints:VQFN-24-1EP_4x4mm_P0.5mm_EP2.45x2.45mm_0.3ThermalVias
- moved C72 68.5 mm to (138.9, 93.4)
- moved R11 60.4 mm to (137.8, 93.4), turned to -90 degrees
- moved C32 30.7 mm to (158.4, 137.0)
- moved C26 22.5 mm to (169.8, 141.8), turned to 180 degrees
- moved C49 18.4 mm to (198.3, 144.4), turned to -90 degrees
- moved D11 18.2 mm to (193.8, 149.2), turned to -90 degrees
- moved C48 17.0 mm to (197.2, 144.4), turned to -90 degrees
- moved C50 16.8 mm to (199.0, 140.8), turned to -90 degrees
- moved R54 15.9 mm to (196.1, 144.7), turned to 90 degrees
- moved R59 15.8 mm to (198.5, 140.4), turned to 0 degrees
- moved R9 15.7 mm to (169.8, 140.8)
- moved D7 15.3 mm to (171.8, 147.0), turned to -90 degrees
- moved L16 15.3 mm to (194.4, 144.6), turned to 180 degrees
- moved L10 15.2 mm to (174.8, 147.0), turned to 180 degrees
- moved U3 15.1 mm to (173.8, 142.4), turned to -90 degrees
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Connections:
- C26 pad 1: GND -> Net-(U3-PSN)
- C26 pad 2: Net-(U3-VREG) -> GND
- C27 pad 1: GND -> Net-(U2-VREF)
- C27 pad 2: Net-(C27-Pad2) -> GND
- C28 pad 1: GND -> Net-(U2-CN)
- C28 pad 2: Net-(C28-Pad2) -> GND
- C29 pad 1: GND -> Net-(U2-CP)
- C29 pad 2: Net-(C29-Pad2) -> GND
- C30 pad 1: GND -> Net-(U3-VREF)
- C30 pad 2: Net-(C30-Pad2) -> GND
- C37 pad 1: GND -> Net-(U3-CP)
- C37 pad 2: Net-(U2-VREF) -> GND
- C38 pad 1: GND -> +16VA
- C38 pad 2: Net-(U3-VREF) -> Net-(U2-FBP)
- C39 pad 1: -9VD -> +8VD
- C39 pad 2: GND -> Net-(U3-FBP)
- C40 pad 1: +16VA -> Net-(U2-FBN)
- C40 pad 2: GND -> -8VA
- C41 pad 1: -9VA -> Net-(U3-FBN)
- C41 pad 2: GND -> -9VD
- C42 pad 1: +8VD -> +16VA
- C55 pad 1: +5VD -> -15VD
- C56 pad 1: -4VD -> +5VD
- C58 pad 1: -15VD -> -4VD
- C72 pad 1: +CCDPWR -> GND
- C72 pad 2: GND -> Net-(U4-NRST)
- C8 pad 1: GND -> Net-(U2-PSN)
- C8 pad 2: Net-(U2-VREG) -> GND
- D3 pad 1: Net-(D3-K) -> +16VA
- D3 pad 2: -9VA -> Net-(D3-A)
- D5 pad 1: Net-(D5-K) -> +8VD
- D5 pad 2: -9VD -> Net-(D5-A)
- D6 pad 1: +16VA -> Net-(D6-K)
- D6 pad 2: Net-(D6-A) -> -8VA
- D7 pad 1: +8VD -> Net-(D7-K)
- D7 pad 2: Net-(D7-A) -> -9VD
- J2 pad 19: -9VA -> -8VA
- J9 pad 1: +3V3 -> MCU_SWDIO
- J9 pad 10: FPGA_TDO -> GND
- J9 pad 11: GND -> FPGA_TCK
- J9 pad 12: FPGA_TMS -> GND
- J9 pad 2: MCU_SWDIO -> +3V3
- J9 pad 3: GND -> MCU_SWCLK
- J9 pad 4: MCU_SWCLK -> GND
- J9 pad 5: GND -> FPGA_TMS
- J9 pad 6: FPGA_TCK -> GND
- J9 pad 7: GND -> FPGA_TDO
- J9 pad 8: FPGA_TDI -> GND
- J9 pad 9: GND -> FPGA_TDI
- L10 pad 1: Net-(D7-A) -> GND
- L10 pad 2: Net-(U3-INBK) -> Net-(D7-K)
- L4 pad 1: Net-(D6-A) -> Net-(D3-A)
- L4 pad 2: Net-(U2-INBK) -> +CCDPWR
- R11 pad 1: +CCDPWR -> +RTC
- R11 pad 2: CCD_POWEREN -> Net-(U4-NRST)
- R12 pad 1: Net-(U2-COMP2) -> Net-(U2-VREF)
- R12 pad 2: Net-(C29-Pad2) -> Net-(U2-FBN)
- R13 pad 1: Net-(U3-COMP2) -> Net-(U2-FBN)
- R13 pad 2: Net-(C30-Pad2) -> -8VA
- R15 pad 1: Net-(U2-SS) -> Net-(U3-FBN)
- R15 pad 2: GND -> -9VD
- R16 pad 1: Net-(U3-SS) -> +16VA
- R16 pad 2: GND -> Net-(U2-FBP)
- R7 pad 1: Net-(U2-COMP1) -> Net-(U2-PSN)
- R7 pad 2: Net-(C27-Pad2) -> +CCDPWR
- R9 pad 1: Net-(U3-COMP1) -> Net-(U3-PSN)
- R9 pad 2: Net-(C28-Pad2) -> +CCDPWR
- U2 pad 1: Net-(U2-INBK) -> Net-(D3-A)
- U2 pad 10: Net-(U2-COMP2) -> CCD_POWEREN
- U2 pad 11: Net-(U2-FB2) -> Net-(U2-PSN)
- U2 pad 12: Net-(U2-VREF) -> unconnected-(U2-NC-Pad12)
- U2 pad 13: GND -> Net-(D6-K)
- U2 pad 14: Net-(U2-VREG) -> Net-(D6-K)
- U2 pad 15: +CCDPWR -> -8VA
- U2 pad 16: +CCDPWR -> Net-(U2-FBN)
- U2 pad 17: +CCDPWR -> Net-(U2-VREF)
- U2 pad 18: Net-(D3-K) -> Net-(U2-CN)
- U2 pad 2: CCD_AFE_SYNC -> GND
- U2 pad 20: Net-(D6-A) -> unconnected-(U2-NC-Pad20)
- U2 pad 21: GND -> Net-(U2-CP)
- U2 pad 3: Net-(U2-SEQ) -> GND
- U2 pad 4: Net-(U2-SLEW) -> Net-(U2-PSN)
- U2 pad 5: Net-(U2-FB1) -> +CCDPWR
- U2 pad 6: Net-(U2-COMP1) -> +CCDPWR
- U2 pad 7: CCD_POWEREN -> unconnected-(U2-BSW-Pad7)
- U2 pad 8: Net-(U2-SS) -> CCD_POWEREN
- U2 pad 9: CCD_POWEREN -> Net-(U2-PSN)
- U3 pad 1: Net-(U3-INBK) -> Net-(D5-A)
- U3 pad 10: Net-(U3-COMP2) -> CCD_POWEREN
- U3 pad 11: Net-(U3-FB2) -> Net-(U3-PSN)
- U3 pad 12: Net-(U3-VREF) -> unconnected-(U3-NC-Pad12)
- U3 pad 13: GND -> Net-(D7-K)
- U3 pad 14: Net-(U3-VREG) -> Net-(D7-K)
- U3 pad 15: +CCDPWR -> -9VD
- U3 pad 16: +CCDPWR -> Net-(U3-FBN)
- U3 pad 17: +CCDPWR -> Net-(U3-VREF)
- U3 pad 18: Net-(D5-K) -> Net-(U3-CN)
- U3 pad 2: CCD_PULSE_SYNC -> GND
- U3 pad 20: Net-(D7-A) -> unconnected-(U3-NC-Pad20)
- U3 pad 21: GND -> Net-(U3-CP)
- U3 pad 3: Net-(U3-SEQ) -> GND
- U3 pad 4: Net-(U3-SLEW) -> Net-(U3-PSN)
- U3 pad 5: Net-(U3-FB1) -> +CCDPWR
- U3 pad 6: Net-(U3-COMP1) -> +CCDPWR
- U3 pad 7: CCD_POWEREN -> unconnected-(U3-BSW-Pad7)
- U3 pad 8: Net-(U3-SS) -> CCD_POWEREN
- U3 pad 9: CCD_POWEREN -> Net-(U3-PSN)
- U4 pad 16: unconnected-(U4-PB1-Pad16) -> DCDC_EN
- U4 pad 17: unconnected-(U4-PB2-Pad17) -> CCD_POWEREN
- U4 pad 26: unconnected-(U4-PA15-Pad26) -> PWROK
- U4 pad 31: DCDC_EN -> LCD_EN
- U4 pad 6: PWROK -> Net-(U4-NRST)
Routing:
- net I2C_SCL: track 0.00 -> 84.5 mm, vias 0 -> 2
- net LENS_TXD: track 0.00 -> 84.0 mm, vias 0 -> 1
- net I2C_SDA: track 0.00 -> 81.9 mm, vias 0 -> 2
- net LENS_PWR_EN: track 1.45 -> 82.6 mm, vias 0 -> 3
- net LENS_DET: track 0.00 -> 76.7 mm, vias 0 -> 1
- net PS_POR_B: track 0.00 -> 76.0 mm, vias 0 -> 2
- net BODY_CS_LENS: track 0.00 -> 72.7 mm, vias 0 -> 1
- net FPGA_TMS: track 0.00 -> 72.2 mm, vias 0 -> 1
- net FPGA_TDO: track 0.00 -> 71.6 mm, vias 0 -> 1
- net FPGA_TDI: track 0.00 -> 71.1 mm, vias 0 -> 1
- net FPGA_TCK: track 0.00 -> 70.6 mm, vias 0 -> 1
- net +1V8: track 0.00 -> 68.5 mm, vias 0 -> 2
- net LENS_RXD: track 0.00 -> 62.5 mm, vias 0 -> 1
- net +3V3: track 35.1 -> 96.9 mm, vias 6 -> 11
- net GRIP_CS: track 0.00 -> 61.0 mm, vias 0 -> 2
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- added copper zone on F.Cu, net +CCDPWR
- added copper zone on In1.Cu, net IPSOUT
- added copper zone on F.Cu, net Net-(D10-K)
- added copper zone on F.Cu, net Net-(D11-K)
- added copper zone on F.Cu, net Net-(D3-A)
- added copper zone on F.Cu, net Net-(D5-A)
- added copper zone on F.Cu, net Net-(D6-K)
- added copper zone on F.Cu, net Net-(D7-K)
- added copper zone on F.Cu, net Net-(D8-A)
- added copper zone on F.Cu, net Net-(D9-A)
- removed copper zone on F.Cu, net +1V8
- removed copper zone on B.Cu, net GND
- removed copper zone on F.Cu, net GND
Other:
- outline, holes or cut-outs redrawn
- board text added: "IOB R0.10"
- board text removed: "IOB R0.9"

Commit message: PCB r0p10 release
Parts:
- removed C60: 100nF, Capacitor_SMD:C_0402_1005Metric
- removed U15: SY8120, Package_TO_SOT_SMD:TSOT-23-6
- added U8: SY8008, Package_TO_SOT_SMD:TSOT-23-5, F.Cu at (164.2, 142.8)
- moved C59 5.90 mm to (162.8, 139.9), turned to -90 degrees
Connections:
- net +VCCIO_SD renamed Net-(U1-LDO3)
- J7 pad 11: +3V3 -> +RTC
Routing:
- net +RTC: track 47.1 -> 87.4 mm, vias 3 -> 4
- net Net-(U8-SW): track 4.14 -> 2.70 mm
- net Net-(U15-BS): track 1.40 -> 0.00 mm
- net +3V3: track 96.9 -> 96.0 mm, vias 11 -> 10
- net +CCDPWR: track 41.1 -> 40.3 mm
- net GND: vias 153 -> 154

Commit message: Add backport version board
Parts:
- added C60: 47uF, Capacitor_SMD:C_0805_2012Metric, F.Cu at (150.0, 135.6)
- added C94: 47uF, Capacitor_SMD:C_0805_2012Metric, F.Cu at (137.1, 80.6)
- added C95: 47uF, Capacitor_SMD:C_0805_2012Metric, F.Cu at (139.2, 84.2)
- added C96: 47uF, Capacitor_SMD:C_0805_2012Metric, F.Cu at (137.1, 84.2)
- added R36: 10K, Resistor_SMD:R_0402_1005Metric, F.Cu at (146.5, 98.0)
- added R38: 10K, Resistor_SMD:R_0402_1005Metric, F.Cu at (146.5, 99.0)
- added R39: 2.2K, Resistor_SMD:R_0402_1005Metric, B.Cu at (191.1, 102.9)
- added R40: 2.2K, Resistor_SMD:R_0402_1005Metric, B.Cu at (191.1, 101.8)
- R10: value 4.3K -> 10K
- SW1: value SW_Push_LED -> C725874
- moved C71 64.7 mm to (139.2, 80.6), turned to 90 degrees
- moved C70 53.4 mm to (153.1, 97.9)
- moved C2 46.7 mm to (198.8, 86.8), turned to 90 degrees
- moved C69 45.6 mm to (153.1, 95.7)
- moved R35 2.16 mm to (135.0, 83.8), turned to 180 degrees
- moved C75 1.36 mm to (150.0, 137.7), turned to 180 degrees
- moved C91 0.50 mm to (196.7, 86.8)
Connections:
- C2 pad 1: +CCDPWR -> IPSOUT
- C69 pad 1: +CCDPWR -> IPSOUT
- C70 pad 1: +CCDPWR -> IPSOUT
- C71 pad 1: +CCDPWR -> IPSOUT
- J5 pad 21: I2C_SCL -> I2C1_SCL
- J5 pad 22: I2C_SDA -> I2C1_SDA
- U1 pad 1: I2C_SDA -> I2C2_SDA
- U1 pad 2: I2C_SCL -> I2C2_SCL
- U4 pad 19: BODY_CS_LENS -> I2C1_SCL
- U4 pad 21: unconnected-(U4-PA10/NC-Pad21) -> I2C1_SDA
- U4 pad 22: I2C_SCL -> I2C2_SCL
- U4 pad 23: I2C_SDA -> I2C2_SDA
- U4 pad 29: unconnected-(U4-PB5-Pad29) -> BODY_CS_LENS
Routing:
- net I2C_SCL: track 84.5 -> 0.00 mm, vias 2 -> 0
- net I2C_SDA: track 81.9 -> 0.00 mm, vias 2 -> 0
- net I2C1_SDA: track 0.00 -> 76.5 mm, vias 0 -> 2
- net I2C1_SCL: track 0.00 -> 76.0 mm, vias 0 -> 2
- net I2C2_SCL: track 0.00 -> 20.4 mm
- net IPSOUT: track 127.5 -> 145.5 mm, vias 16 -> 23
- net I2C2_SDA: track 0.00 -> 17.2 mm
- net +3V3: track 96.0 -> 110.0 mm, vias 10 -> 12
- net GND: track 260.5 -> 265.9 mm, vias 154 -> 159
- net BODY_CS_LENS: track 72.7 -> 77.3 mm
- net +CCDPWR: track 40.3 -> 37.4 mm
- net LENS_DET: track 76.7 -> 76.2 mm
Other:
- board text added: "IOB R0.11"
- board text removed: "IOB R0.10"

Commit message: Use header instead of pin for JTAG port on IOB
Parts:
- J9: footprint Connector_PinHeader_1.27mm:PinHeader_2x06_P1.27mm_Horizontal -> Connector_PinSocket_1.27mm:PinSocket_2x06_P1.27mm_Horizontal
- moved J9 6.35 mm to (133.0, 101.8), turned to 0 degrees
Connections:
- J9 pad 1: MCU_SWDIO -> FPGA_TCK
- J9 pad 11: FPGA_TCK -> MCU_SWDIO
- J9 pad 12: GND -> +3V3
- J9 pad 2: +3V3 -> GND
- J9 pad 3: MCU_SWCLK -> FPGA_TDI
- J9 pad 5: FPGA_TMS -> FPGA_TDO
- J9 pad 7: FPGA_TDO -> FPGA_TMS
- J9 pad 9: FPGA_TDI -> MCU_SWCLK
