File: hardware/sensorboard/ccd_driver_v_adiabatic.kicad_sch (KiCad schematic)
At the start: 71 parts, among them U40 IRLHS6376PBF, U41 IRLHS6376PBF, U42 IRLHS6376PBF, U43 IRLHS6376PBF, U44 IRLHS6376PBF, U45 DG412xY, U46 IRLHS6376PBF, U47 DG412xY, U48 DG412xY, U49 DG412xY, U50 DG412xY

Commit message: r0p11 sb pcb layout wip
Parts:
- L4, L5, L6: footprint AL_common:Coilcraft_0807SQ-11N -> footprints:Coilcraft_0807SQ-11N
- U40, U41, U42, U43, U44, U46: symbol AL_common:IRLHS6376PBF -> symbols:IRLHS6376PBF
- U45, U47, U48, U49, U50: value DG412xY -> DG412DQ; footprint Package_SO:SOIC-16_3.9x9.9mm_P1.27mm -> Package_SO:TSSOP-16_4.4x5mm_P0.65mm
