File: hardware/sensorboard/fpga_config.kicad_sch (KiCad schematic)
At the start: 19 parts, among them U27 XC7Z010-CLG400, U28 W25Q128JVP, X1 33.33MHz

Commit message: PCB r0p10 release
Other:
- company: Copyright 2024 Wenting Zhang -> Copyright 2024 Anhang Li, Wenting Zhang
- title: Sitina 1 Sensor Board -> FPGA Configuration
Changed lines of the file:
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@@
 	(paper "A4")
 	(title_block
-		(title "Sitina 1 Sensor Board")
-		(date "2024-03-25")
-		(rev "R0.9")
-		(company "Copyright 2024 Wenting Zhang")
+		(title "FPGA Configuration")
+		(date "2024-06-09")
+		(rev "R0.10")
+		(company "Copyright 2024 Anhang Li, Wenting Zhang")
+		(comment 2 "MERCHANTABILITY, SATISFACTORY QUALITY AND FITNESS FOR A PARTICULAR PURPOSE.")
+		(comment 3 "This source is distributed WITHOUT ANY EXPRESS OR IMPLIED WARRANTY, INCLUDING OF")
+		(comment 4 "This source describes Open Hardware and is licensed under the CERN-OHL-P v2.")
 	)
 	(junction
