File: hardware/sensorboard/fpga_io.kicad_sch (KiCad schematic)
At the start: 13 parts, among them U27 XC7Z010-CLG400

Commit message: PCB r0p10 release
Other:
- company: Copyright 2024 Wenting Zhang -> Copyright 2024 Anhang Li, Wenting Zhang
- title: Sitina 1 Sensor Board -> FPGA IO
Changed lines of the file:
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@@
 	(paper "A4")
 	(title_block
-		(title "Sitina 1 Sensor Board")
-		(date "2024-03-25")
-		(rev "R0.9")
-		(company "Copyright 2024 Wenting Zhang")
+		(title "FPGA IO")
+		(date "2024-06-09")
+		(rev "R0.10")
+		(company "Copyright 2024 Anhang Li, Wenting Zhang")
+		(comment 2 "MERCHANTABILITY, SATISFACTORY QUALITY AND FITNESS FOR A PARTICULAR PURPOSE.")
+		(comment 3 "This source is distributed WITHOUT ANY EXPRESS OR IMPLIED WARRANTY, INCLUDING OF")
+		(comment 4 "This source describes Open Hardware and is licensed under the CERN-OHL-P v2.")
 	)
 	(junction

Commit message: r0p11 sb pcb layout wip
Parts:
- added TP1, TP2: TestPoint, TestPoint:TestPoint_Pad_D1.5mm, symbol Connector:TestPoint
Connections:
- net PS_UART_RX: now also TP2.1
- net PS_UART_TX: now also TP1.1
- net DRV_V2_PDN_LO: now reaches U27.D19 (IO_L4P_T0_35)
- net DRV_V2_PDN_HI: now reaches U27.E17 (IO_L3P_T0_DQS_AD1P_35)
- net XADC_V2_P: now reaches U27.E18 (IO_L5P_T0_AD9P_35)
- net XADC_V2_N: now reaches U27.E19 (IO_L5N_T0_AD9N_35)
- net DRV_V2_PLO_HI: now reaches U27.F16 (IO_L6P_T0_35)
- net DRV_V2_SELH_PHI_LO: now reaches U27.F17 (IO_L6N_T0_VREF_35)
- net DRV_V2_SELL_HI: now reaches U27.G15 (IO_L19N_T3_VREF_35)
- net DRV_V1_PLO_LO: now reaches U27.G17 (IO_L16P_T2_35)
- net DRV_V1_PLO_HI: now reaches U27.G18 (IO_L16N_T2_35)
- net DRV_V1_PDN_LO: now reaches U27.G19 (IO_L18P_T2_AD13P_35)
- net DRV_V1_SELL_LO: now reaches U27.J18 (IO_L14P_T2_AD4P_SRCC_35)
- net DRV_V2_PHI_MID: now reaches U27.J19 (IO_L10N_T1_AD11N_35)
- net DRV_V1_PDN_HI: now reaches U27.J20 (IO_L17P_T2_AD5P_35)
- net DRV_V1_SELL_HI: now reaches U27.K19 (IO_L10P_T1_AD11P_35)
- net DRV_V2_SELL_LO: now reaches U27.L15 (IO_L22N_T3_AD7N_35)
- net XADC_V1_P: now reaches U27.M17 (IO_L8P_T1_AD10P_35)
- net DRV_FDG_LO: now reaches U27.M20 (IO_L7N_T1_AD2N_35)
- net DRV_FDG_HI: now reaches U27.N15 (IO_L21P_T3_DQS_AD14P_35)
- net DRV_V2_PLO_LO: now reaches U27.N16 (IO_L21N_T3_DQS_AD14N_35)
- net TCON_FDG renamed DRV_V2_PHI_HI
- net TCON_V1 renamed XADC_V1_N
- net TCON_V2 renamed DRV_V2_SELH_HI
- net TCON_V23 renamed DRV_V2_SELH_MID

Commit message: Sensorboard r0p11 freeze
Connections:
- net AFE_RST: now also U27.U14 (IO_L11P_T1_SRCC_34); no longer U27.Y19 (IO_L17N_T2_34)
- net AFE_SCK: now also U27.T10 (IO_L1N_T0_34); no longer U27.W16 (IO_L18N_T2_34)
- net AFE_SDATA: now also U27.T12 (IO_L2P_T0_34); no longer U27.Y17 (IO_L7N_T1_34)
- net AFE_SL: now also U27.U12 (IO_L2N_T0_34); no longer U27.Y18 (IO_L17P_T2_34)
- net CSI_D10: now also U27.Y14 (IO_L8N_T1_34); no longer U27.V17 (IO_L21P_T3_DQS_34)
- net CSI_D11: now also U27.V12 (IO_L4P_T0_34); no longer U27.W13 (IO_L4N_T0_34)
- net CSI_D12: now also U27.V18 (IO_L21N_T3_DQS_34); no longer U27.U12 (IO_L2N_T0_34)
- net CSI_D13: now also U27.V13 (IO_L3N_T0_DQS_34); no longer U27.U18 (IO_L12P_T1_MRCC_34)
- net CSI_D14: now also U27.V16 (IO_L18P_T2_34); no longer U27.V18 (IO_L21N_T3_DQS_34)
- net CSI_D15: now also U27.V17 (IO_L21P_T3_DQS_34); no longer U27.Y14 (IO_L8N_T1_34)
- net CSI_D2: now also U27.Y19 (IO_L17N_T2_34); no longer U27.V16 (IO_L18P_T2_34)
- net CSI_D3: now also U27.W18 (IO_L22P_T3_34); no longer U27.U17 (IO_L9N_T1_DQS_34)
- net CSI_D4: now also U27.Y17 (IO_L7N_T1_34); no longer U27.V12 (IO_L4P_T0_34)
- net CSI_D5: now also U27.W16 (IO_L18N_T2_34); no longer U27.T16 (IO_L9P_T1_DQS_34)
- net CSI_D6: now also U27.Y16 (IO_L7P_T1_34); no longer U27.T12 (IO_L2P_T0_34)
- net CSI_D7: now also U27.W15 (IO_L10N_T1_34); no longer U27.T10 (IO_L1N_T0_34)
- net CSI_D8: now also U27.Y18 (IO_L17P_T2_34); no longer U27.V13 (IO_L3N_T0_DQS_34)
- net CSI_D9: now also U27.T16 (IO_L9P_T1_DQS_34); no longer U27.W18 (IO_L22P_T3_34)
- net CSI_HSYNC: now also U27.U17 (IO_L9N_T1_DQS_34); no longer U27.Y16 (IO_L7P_T1_34)
- net CSI_PIXCLK: now also U27.U18 (IO_L12P_T1_MRCC_34); no longer U27.U14 (IO_L11P_T1_SRCC_34)
- net CSI_VSYNC: now also U27.W13 (IO_L4N_T0_34); no longer U27.W15 (IO_L10N_T1_34)
- net DRV_FDG_HI: now also U27.K19 (IO_L10P_T1_AD11P_35); no longer U27.N15 (IO_L21P_T3_DQS_AD14P_35)
- net DRV_FDG_LO: now also U27.E18 (IO_L5P_T0_AD9P_35); no longer U27.M20 (IO_L7N_T1_AD2N_35)
- net DRV_V1_PDN_LO: now also U27.G18 (IO_L16N_T2_35); no longer U27.G19 (IO_L18P_T2_AD13P_35)
- net DRV_V1_PLO_HI: now also U27.G19 (IO_L18P_T2_AD13P_35); no longer U27.G18 (IO_L16N_T2_35)
- net DRV_V1_PLO_LO: now also U27.J19 (IO_L10N_T1_AD11N_35); no longer U27.G17 (IO_L16P_T2_35)
- net DRV_V1_SELL_HI: now also U27.D19 (IO_L4P_T0_35); no longer U27.K19 (IO_L10P_T1_AD11P_35)
- net DRV_V1_SELL_LO: now also U27.E17 (IO_L3P_T0_DQS_AD1P_35); no longer U27.J18 (IO_L14P_T2_AD4P_SRCC_35)
- net DRV_V2_PDN_HI: now also U27.H17 (IO_L13N_T2_MRCC_35); no longer U27.E17 (IO_L3P_T0_DQS_AD1P_35)
- net DRV_V2_PDN_LO: now also U27.D20 (IO_L4N_T0_35); no longer U27.D19 (IO_L4P_T0_35)
- net DRV_V2_PHI_HI: now also U27.F17 (IO_L6N_T0_VREF_35); no longer U27.L19 (IO_L9P_T1_DQS_AD3P_35)
- net DRV_V2_PHI_MID: now also U27.G17 (IO_L16P_T2_35); no longer U27.J19 (IO_L10N_T1_AD11N_35)
- net DRV_V2_PLO_LO: now also U27.F20 (IO_L15N_T2_DQS_AD12N_35); no longer U27.N16 (IO_L21N_T3_DQS_AD14N_35)
- net DRV_V2_SELH_HI: now also U27.G15 (IO_L19N_T3_VREF_35); no longer U27.C20 (IO_L1P_T0_AD0P_35)
- net DRV_V2_SELH_MID: now also U27.M20 (IO_L7N_T1_AD2N_35); no longer U27.A20 (IO_L2N_T0_AD8N_35)
- net DRV_V2_SELH_PHI_LO: now also U27.L19 (IO_L9P_T1_DQS_AD3P_35); no longer U27.F17 (IO_L6N_T0_VREF_35)
- net DRV_V2_SELL_HI: now also U27.E19 (IO_L5N_T0_AD9N_35); no longer U27.G15 (IO_L19N_T3_VREF_35)
- net DRV_V2_SELL_LO: now also U27.J18 (IO_L14P_T2_AD4P_SRCC_35); no longer U27.L15 (IO_L22N_T3_AD7N_35)
- net TCON_H1: now also U27.L16 (IO_L11P_T1_SRCC_35); no longer U27.L17 (IO_L11N_T1_SRCC_35)
- net TCON_H2: now also U27.L15 (IO_L22N_T3_AD7N_35); no longer U27.L16 (IO_L11P_T1_SRCC_35)
- net TCON_RG: now also U27.L17 (IO_L11N_T1_SRCC_35); no longer U27.H17 (IO_L13N_T2_MRCC_35)
- net XADC_V1_N: now also U27.N16 (IO_L21N_T3_DQS_AD14N_35); no longer U27.M18 (IO_L8N_T1_AD10N_35)
- net XADC_V1_P: now also U27.N15 (IO_L21P_T3_DQS_AD14P_35); no longer U27.M17 (IO_L8P_T1_AD10P_35)
- net XADC_V2_N: now also U27.M18 (IO_L8N_T1_AD10N_35); no longer U27.E19 (IO_L5N_T0_AD9N_35)
- net XADC_V2_P: now also U27.M17 (IO_L8P_T1_AD10P_35); no longer U27.E18 (IO_L5P_T0_AD9P_35)
