File: hardware/gripflex/gripflex.kicad_pcb (KiCad board)
At the start: 2 copper layers, 68.3 x 78.8 mm, 21 parts, among them J1 Conn_01x10_MountingPin, J2 Conn_01x12, J3 Conn_01x02_MountingPin, U2 74HC165, U3 74HC165

Commit message: USBC breakout board for JTAG, bug fix for grip flex cable
Parts:
- added RN4: 10K, Resistor_SMD:R_Array_Convex_4x0402, F.Cu at (159.4, 96.1)
- added SW10: ~, footprints:HX-TS5208A, F.Cu at (158.1, 144.1)
- added SW11: ~, footprints:HX-TS5208A, F.Cu at (167.1, 144.1)
- J3: footprint Connector_JST:JST_PH_B2B-PH-SM4-TB_1x02-1MP_P2.00mm_Vertical -> Connector_JST:JST_PH_S2B-PH-SM4-TB_1x02-1MP_P2.00mm_Horizontal
- U1: footprint footprints:SIQ-02FVS3 -> footprints:SIQ-02FVS3_L
- moved J3 1.98 mm to (157.0, 101.3), turned to -90 degrees
Connections:
- U3 pad 3: unconnected-(U3-D4-Pad3) -> /KEYMENU
- U3 pad 4: unconnected-(U3-D5-Pad4) -> /KEYPB
Routing:
- net /KEYMENU: track 0.00 -> 77.1 mm, vias 0 -> 2
- net /KEYPB: track 0.00 -> 67.8 mm, vias 0 -> 2
- net +3V3: track 143.0 -> 152.6 mm, vias 6 -> 7
- net SPI_MOSI: track 138.2 -> 144.9 mm
- net SPI_SCLK: track 137.9 -> 143.6 mm
- net +BATT: track 103.5 -> 108.8 mm
- net /KEYRIGHT: track 45.4 -> 47.2 mm
- net GND: track 259.9 -> 258.5 mm, vias 45 -> 57
- net SPI_CS: track 136.9 -> 138.1 mm
- net /ENCA: track 11.6 -> 10.7 mm
- net SPI_MISO: track 101.5 -> 102.3 mm
- net /ENCS: track 11.7 -> 11.0 mm
- net /ENCB: track 5.80 -> 6.40 mm
Other:
- board size 68.3 x 78.8 mm -> 68.3 x 86.7 mm

Commit message: PCB changes for r0p10
Connections:
- RN4 pad 1: unconnected-(RN4-R1.1-Pad1) -> Net-(RN4-R1.1)
- RN4 pad 2: unconnected-(RN4-R2.1-Pad2) -> Net-(RN4-R2.1)
- U2 pad 1: KEY_LOAD -> SPI_CS
- U3 pad 5: unconnected-(U3-D6-Pad5) -> Net-(RN4-R2.1)
- U3 pad 6: unconnected-(U3-D7-Pad6) -> Net-(RN4-R1.1)
Routing:
- net SPI_CS: track 138.1 -> 147.6 mm, vias 4 -> 6
- net Net-(RN4-R1.1): track 0.00 -> 1.94 mm
- net Net-(RN4-R2.1): track 0.00 -> 1.89 mm
- net /KEYPB: track 67.8 -> 68.3 mm
- net /KEYMENU: track 77.1 -> 77.7 mm
Other:
- outline, holes or cut-outs redrawn
- board text added: "Sitina1"
- board text added: "Wenting 2024"

Commit message: PCB r0p10 release
Routing:
- net GND: track 258.5 -> 232.0 mm
Other:
- board size 68.3 x 86.7 mm -> 68.3 x 86.2 mm

Commit message: Add 2 more buttons on the grip flex
Parts:
- added SW12: ~, footprints:HX-TS5208A, F.Cu at (158.1, 125.1)
- added SW13: ~, footprints:HX-TS5208A, F.Cu at (167.1, 125.1)
- moved SW4 6.80 mm to (162.6, 143.4)
- moved SW1 6.80 mm to (162.6, 132.1)
- moved SW2 6.80 mm to (156.9, 137.7)
- moved SW3 6.80 mm to (168.2, 137.7)
- moved SW10 6.00 mm to (158.1, 150.1)
- moved SW11 6.00 mm to (167.1, 150.1)
Connections:
- net Net-(RN4-R1.1) renamed /KEYFN6
- net Net-(RN4-R2.1) renamed /KEYFN5
Routing:
- net /KEYFN5: track 1.89 -> 62.0 mm, vias 0 -> 2
- net /KEYFN6: track 1.94 -> 47.1 mm, vias 0 -> 2
- net GND: track 232.0 -> 191.3 mm, vias 57 -> 61
- net /KEYMENU: track 77.7 -> 88.1 mm
- net /KEYPB: track 68.3 -> 78.8 mm
- net /KEYLEFT: track 44.1 -> 53.1 mm, vias 0 -> 2
- net /KEYDOWN: track 52.7 -> 59.9 mm
- net /KEYUP: track 40.6 -> 46.9 mm
- net /KEYRIGHT: track 47.2 -> 52.6 mm
- net SPI_CS: track 147.6 -> 145.1 mm
- net SPI_MOSI: track 145.2 -> 143.0 mm
- net SPI_MISO: track 102.3 -> 104.0 mm
- net +3V3: track 152.6 -> 154.0 mm
Other:
- board size 68.3 x 86.2 mm -> 68.3 x 92.2 mm
