File: hardware/sensorboard-backport/ccd_driver_v.kicad_sch (KiCad schematic)
At the start: 73 parts, among them U20 1EDN7550B, U21 1EDN7550B, U22 1EDN7550B, U23 1EDN7550B, U24 IRF9389/7309, U25 IRF9389/7309, U26 IRF9389/7309

Commit message: SB r0p12b WIP
Parts:
- removed RV5, RV6, RV7, RV8: 10K, footprints:Potentiometer_Bourns_TC33X_Vertical, symbol Device:R_Potentiometer_Trim_US
- R81, R82, R83, R84, R85, R86, R87, R88: value 5.1K -> 10K
Connections:
- net at C84.2, U22.1 (IN-): now also R83.1, R84.2
- net at C85.2, U20.1 (IN-): now also R85.1, R86.2
- net at C83.2, U21.1 (IN-): now also R81.1, R82.2
- net at C86.2, U23.1 (IN-): now also R87.1, R88.2
