File: hardware/sensorboard-backport/ccd_driver.kicad_sch (KiCad schematic)
At the start: 66 parts, among them Q1 BC847BPN, U11 TPS72301, U12 XC6206P152MR, U13 TLV76701DRVx, U14 74HC2G17GW, U15 74HC2G17GW, U16 74HC2G17GW, U17 74HC2G17GW, U18 74HC2G17GW, U19 74HC2G17GW

Commit message: Fix wrong part number for H driver
Parts:
- U14, U15, U16, U17, U18, U19: value 74HC2G17GW -> 74HC2G17GV
Changed lines of the file:
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@@
 			)
 		)
-		(property "Value" "74HC2G17GW"
+		(property "Value" "74HC2G17GV"
 			(at 176.53 93.98 0)
 			(effects
@@
 			)
 		)
-		(property "Value" "74HC2G17GW"
+		(property "Value" "74HC2G17GV"
 			(at 176.53 113.03 0)
 			(effects
@@
 			)
 		)
-		(property "Value" "74HC2G17GW"
+		(property "Value" "74HC2G17GV"
 			(at 176.53 39.37 0)
 			(effects
@@
 			)
 		)
-		(property "Value" "74HC2G17GW"
+		(property "Value" "74HC2G17GV"
 			(at 176.53 21.59 0)
 			(effects
@@
 			)
 		)
-		(property "Value" "74HC2G17GW"
+		(property "Value" "74HC2G17GV"
 			(at 176.53 57.15 0)
 			(effects
@@
 			)
 		)
-		(property "Value" "74HC2G17GW"
+		(property "Value" "74HC2G17GV"
 			(at 176.53 74.93 0)
 			(effects

Commit message: SB r0p12b WIP
Parts:
- removed C58, C59, C68, C69, C70, C73, C74, C75: 100nF, Capacitor_SMD:C_0402_1005Metric, symbol Device:C
- removed D11, D12, D13: BAT54S, Package_TO_SOT_SMD:SOT-23, symbol Diode:BAT54S
- removed RV2, RV3, RV4: 50K, footprints:Potentiometer_Bourns_TC33X_Vertical, symbol Device:R_Potentiometer_Trim_US
- removed U14, U15, U16, U17, U18, U19: 74HC2G17GV, Package_SO:SC-74-6_1.5x2.9mm_P0.95mm, symbol Sitina:74HC2G17
- added U32, U34: 4053, Package_SO:TSSOP-16_4.4x5mm_P0.65mm, symbol 4xxx:4053
- added U35, U36, U37: 74AC04, Package_SO:TSSOP-14_4.4x5mm_P0.65mm, symbol 74xx:74HC04
- C55: value DNP/1nF -> 100nF
Connections:
- net +1V5: now also U32.12 (X0), U37.14 (VCC)
- net +2V: now also U32.2 (Y0), U32.5 (Z0), U34.2 (Y0), U34.5 (Z0), U35.14 (VCC), U36.14 (VCC)
- net +VAB: no longer C55.2
- net -3V5: now also U32.13 (X1), U37.1, U37.7 (GND), U37.9
- net -4V: now also U32.1 (Y1), U32.3 (Z1), U32.7 (VEE), U34.1 (Y1), U34.3 (Z1), U34.7 (VEE), U35.7 (GND), U35.9, U36.13, U36.7 (GND)
- net GND: now also C55.2, C57.2, U32.6 (Inh), U32.8 (VSS), U34.11 (A), U34.12 (X0), U34.13 (X1), U34.6 (Inh), U34.8 (VSS)
- net H1BINL: now also U35.2
- net H1BINR: now also U36.2
- net H1BL: now also U35.4
- net H1BR: now also U36.8
- net H1S: now also U32.15 (Y), U35.1, U35.11, U35.3, U36.1, U36.5
- net H1SL: now also U35.10
- net H1SR: now also U36.6
- net H2BL: now also U35.6
- net H2BR: now also U36.10
- net H2S: now also U32.4 (Z), U35.13, U35.5, U36.3
- net H2SL: now also U35.12
- net H2SR: now also U36.4
- net RGS: now also U32.14 (X), U37.11, U37.13, U37.3, U37.5; no longer C57.2
- net RL: now also U37.10, U37.12
- net RR: now also U37.4, U37.6
- net TCON_H1: now also U32.10 (B)
- net TCON_H2: now also U32.9 (C)
- net TCON_RG: now also U32.11 (A); no longer C57.1
- net at R113.1, R114.1, R115.2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: no longer C55.1
- new net +3V3: C55.1, C57.1, U32.16 (VDD), U34.16 (VDD)
- new net H1BRS: U34.4 (Z), U36.9
- new net H2BRS: U34.15 (Y), U36.11
- new net TCON_H1BR: U34.9 (C)
- new net TCON_H2BR: U34.10 (B)
- no-connect marks 4 -> 5
Other:
- note added: "H1BR = H2, H2BR = H1: Single output H1BR = H1, H2BR = H2: Dual output"
- note removed: "HC only has 4mA drive. Load capacitance for B/S are ~500pF. LVC has 32mA drive, but only up to 5.5V."
- moved on the sheet: C179, C53, C54, C56, C60, C61, C62, C63, C64, C65, C66, C67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

Commit message: Reworking on power tree for SB
Parts:
- removed U13: TLV76701DRVx, Package_SON:WSON-6-1EP_2x2mm_P0.65mm_EP1x1.6mm_ThermalVias, symbol Regulator_Linear:TLV76701DRVx
- added C58, C59, C68, C69: 1uF, Capacitor_SMD:C_0402_1005Metric, symbol Device:C
- added C70, C73: 1uF 25V, Capacitor_SMD:C_0603_1608Metric, symbol Device:C
- added U14: AP2205-W5-7, Package_TO_SOT_SMD:SOT-23-5, symbol Regulator_Linear:AP2204K-ADJ
- R114: value 180K -> 150K
Connections:
- net +1V5: now also C59.1
- net +2V: now also C58.1
- net +VAB: now also C73.1, U14.5 (VOUT)
- net -3V5: now also C68.1
- net -4V: now also C69.1
- net GND: now also C58.2, C59.2, C68.2, C69.2, C70.2, C73.2, U14.2 (GND)
- net at R113.1, R114.1, R115.2: now also U14.4 (ADJ)
- net +16VD renamed +22V
- net +22V: now also C70.1, U14.1 (VIN), U14.3 (EN)
- net -15V renamed -9V
Other:
- note added: "FB:1.24V"
- moved on the sheet: C179, C53, C54, C56, R113, R114, R115, R23, R53, R54, R55, U11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
