File: hardware/sensorboard-backport/fpga_power.kicad_sch (KiCad schematic)
At the start: 50 parts, among them U27 XC7Z010-CLG400, U30 SYR838, U31 SYR838, U33 SY8008

Commit message: Reworking on power tree for SB
Connections:
- net +SYS is gone; now on net +3V3: C164.1, C165.1, C168.1, C169.1, C174.1, U30.D1 (VIN), U30.D2 (VIN), U30.E1 (VIN), U30.E2 (VIN), U31.D1 (VIN), U31.D2 (VIN), U31.E1 (VIN), U31.E2 (VIN)
- net PWREN is gone; now on net +3V3: U30.A2 (EN), U31.A2 (EN)
